File: BPS-PeripheralSOM.kicad_sch (KiCad schematic)
At the start: 21 parts, among them J2 Can_In, J5 Can_Out, J7 SWD, SW2 Reset, U1 STM32L431CBTx, Y1 8M

Commit message: Fixed can schematic and added can connector on main sheet
Parts:
- removed J5: Can_Out, symbol Connector_Generic:Conn_01x04
Connections:
- net CAN_H: now reaches J2.2 (Pin_2)
- net CAN_L: now reaches J2.3 (Pin_3)
Other:
- sheet CAN ports: added CAN_H, CAN_L; removed none
Changed lines of the file:
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@@
     (stroke (width 0) (type default))
   )
-  (wire (pts (xy 209.55 29.21) (xy 209.55 30.48))
-    (stroke (width 0) (type default))
-  )
-  (wire (pts (xy 68.58 86.36) (xy 81.28 86.36))
+  (wire (pts (xy 68.58 92.075) (xy 81.28 92.075))
     (stroke (width 0) (type default))
   )
@@
     (stroke (width 0) (type default))
   )
-  (wire (pts (xy 68.58 57.15) (xy 82.55 57.15))
+  (wire (pts (xy 68.58 60.325) (xy 79.375 60.325))
     (stroke (width 0) (type default))
   )
@@
     (stroke (width 0) (type default))
   )
-  (wire (pts (xy 209.55 40.64) (xy 209.55 38.1))
-    (stroke (width 0) (type default))
-  )
   (wire (pts (xy 223.52 140.97) (xy 224.79 140.97))
     (stroke (width 0) (type default))
@@
     (stroke (width 0) (type default))
   )
-  (wire (pts (xy 209.55 38.1) (xy 210.82 38.1))
-    (stroke (width 0) (type default))
-  )
   (wire (pts (xy 140.97 57.15) (xy 130.81 57.15))
     (stroke (width 0) (type default))
   )
+  (wire (pts (xy 172.72 31.75) (xy 181.61 31.75))
+    (stroke (width 0) (type default))
+  )
   (wire (pts (xy 132.08 25.4) (xy 144.78 25.4))
     (stroke (width 0) (type default))
@@
     (stroke (width 0) (type default))
   )
-  (wire (pts (xy 68.58 81.28) (xy 81.28 81.28))
+  (wire (pts (xy 68.58 86.995) (xy 81.28 86.995))
+    (stroke (width 0) (type default))
+  )
+  (wire (pts (xy 172.72 34.29) (xy 181.61 34.29))
     (stroke (width 0) (type default))
   )
@@
     (stroke (width 0) (type default))
   )
-  (wire (pts (xy 209.55 30.48) (xy 210.82 30.48))
-    (stroke (width 0) (type default))
-  )
   (wire (pts (xy 71.755 21.59) (xy 71.755 22.86))
     (stroke (width 0) (type default))
@@
     (stroke (width 0) (type default))
   )
-  (wire (pts (xy 68.58 62.23) (xy 82.55 62.23))
+  (wire (pts (xy 68.58 65.405) (xy 79.375 65.405))
     (stroke (width 0) (type default))
   )
@@
     (stroke (width 0) (type default))
   )
+  (wire (pts (xy 68.58 55.245) (xy 71.12 55.245))
+    (stroke (width 0) (type default))
+  )
   (wire (pts (xy 109.22 34.29) (xy 109.22 33.02))
+    (stroke (width 0) (type default))
+  )
+  (wire (pts (xy 68.58 52.705) (xy 71.12 52.705))
     (stroke (width 0) (type default))
   )
@@
     (effects (font (size 1.27 1.27) (thickness 0.254) bold) (justify left bottom))
   )
-  (label "USART1_RX" (at 81.28 81.28 180) (fields_autoplaced)
+  (label "CAN_L" (at 172.72 34.29 0) (fields_autoplaced)
+    (effects (font (size 1.27 1.27)) (justify left bottom))
+  )
+  (label "USART1_RX" (at 81.28 86.995 180) (fields_autoplaced)
     (effects (font (size 1.27 1.27)) (justify right bottom))
   )
@@
     (effects (font (size 1.27 1.27)) (justify left bottom))
   )
-  (label "CAN_TX" (at 82.55 62.23 180) (fields_autoplaced)
+  (label "CAN_TX" (at 79.375 65.405 180) (fields_autoplaced)
     (effects (font (size 1.27 1.27)) (justify right bottom))
   )
@@
     (effects (font (size 1.27 1.27)) (justify left bottom))
   )
+  (label "CAN_L" (at 71.12 55.245 0) (fields_autoplaced)
+    (effects (font (size 1.27 1.27)) (justify left bottom))
+  )
   (label "SWCLK" (at 130.81 57.15 0) (fields_autoplaced)
     (effects (font (size 1.27 1.27)) (justify left bottom))
   )
-  (label "USART1_TX" (at 81.28 86.36 180) (fields_autoplaced)
+  (label "USART1_TX" (at 81.28 92.075 180) (fields_autoplaced)
     (effects (font (size 1.27 1.27)) (justify right bottom))
   )
-  (label "CAN_RX" (at 82.55 57.15 180) (fields_autoplaced)
+  (label "CAN_H" (at 71.12 52.705 0) (fields_autoplaced)
+    (effects (font (size 1.27 1.27)) (justify left bottom))
+  )
+  (label "CAN_RX" (at 79.375 60.325 180) (fields_autoplaced)
     (effects (font (size 1.27 1.27)) (justify right bottom))
+  )
+  (label "CAN_H" (at 172.72 31.75 0) (fields_autoplaced)
+    (effects (font (size 1.27 1.27)) (justify left bottom))
   )
   (symbol (lib_id "power:GND") (at 168.91 96.52 0) (unit 1)
@@
     )
   )
-  (symbol (lib_id "power:GNDPWR") (at 209.55 40.64 0) (unit 1)
-    (in_bom yes) (on_board yes) (dnp no) (fields_autoplaced)
-    (property "Reference" "#PWR038" (at 209.55 45.72 0)
-      (effects (font (size 1.27 1.27)) hide)
-    )
-    (property "Value" "GNDPWR" (at 209.423 45.72 0)
-      (effects (font (size 1.27 1.27)))
-    )
-    (property "Footprint" "" (at 209.55 41.91 0)
-      (effects (font (size 1.27 1.27)) hide)
-    )
-    (property "Datasheet" "" (at 209.55 41.91 0)
-      (effects (font (size 1.27 1.27)) hide)
-    )
-    (pin "1")
-    (instances
-      (project "BPS-PeripheralSOM"
-        (path "/d5ebd247-5a7c-47c2-8aee-beabaef72d6d"
-          (reference "#PWR038") (unit 1)
-        )
-      )
-    )
-  )
   (symbol (lib_id "Switch:SW_Push") (at 119.38 55.88 270) (unit 1)
     (in_bom yes) (on_board yes) (dnp no)
@@
         (path "/d5ebd247-5a7c-47c2-8aee-beabaef72d6d"
           (reference "C16") (unit 1)
-        )
-      )
-    )
-  )
-  (symbol (lib_id "Connector_Generic:Conn_01x04") (at 215.9 33.02 0) (unit 1)
-    (in_bom yes) (on_board yes) (dnp no) (fields_autoplaced)
-    (property "Reference" "J5" (at 218.44 33.655 0)
-      (effects (font (size 1.27 1.27)) (justify left))
-    )
-    (property "Value" "Can_Out" (at 218.44 36.195 0)
-      (effects (font (size 1.27 1.27)) (justify left))
-    )
-    (property "Footprint" "" (at 215.9 33.02 0)
-      (effects (font (size 1.27 1.27)) hide)
-    )
-    (property "Datasheet" "~" (at 215.9 33.02 0)
-      (effects (font (size 1.27 1.27)) hide)
-    )
-    (pin "1")
-    (pin "2")
-    (pin "3")
-    (pin "4")
-    (instances
-      (project "BPS-PeripheralSOM"
-        (path "/d5ebd247-5a7c-47c2-8aee-beabaef72d6d"
-          (reference "J5") (unit 1)
         )
       )
@@
     )
   )
-  (symbol (lib_id "power:+12V") (at 209.55 29.21 0) (unit 1)
-    (in_bom yes) (on_board yes) (dnp no) (fields_autoplaced)
-    (property "Reference" "#PWR037" (at 209.55 33.02 0)
-      (effects (font (size 1.27 1.27)) hide)
-    )
-    (property "Value" "+12V" (at 209.55 25.4 0)
-      (effects (font (size 1.27 1.27)))
-    )
-    (property "Footprint" "" (at 209.55 29.21 0)
-      (effects (font (size 1.27 1.27)) hide)
-    )
-    (property "Datasheet" "" (at 209.55 29.21 0)
-      (effects (font (size 1.27 1.27)) hide)
-    )
-    (pin "1")
-    (instances
-      (project "BPS-PeripheralSOM"
-        (path "/d5ebd247-5a7c-47c2-8aee-beabaef72d6d"
-          (reference "#PWR037") (unit 1)
-        )
-      )
-    )
-  )
   (symbol (lib_id "Mechanical:MountingHole") (at 166.37 182.88 0) (unit 1)
     (in_bom yes) (on_board yes) (dnp no)
@@
       (effects (font (size 1.27 1.27)) hide)
     )
-    (pin "CAN_RX" output (at 68.58 57.15 0)
+    (pin "CAN_RX" output (at 68.58 60.325 0)
       (effects (font (size 1.27 1.27)) (justify right))
     )
-    (pin "CAN_TX" input (at 68.58 62.23 0)
+    (pin "CAN_TX" input (at 68.58 65.405 0)
+      (effects (font (size 1.27 1.27)) (justify right))
+    )
+    (pin "CAN_L" input (at 68.58 55.245 0)
+      (effects (font (size 1.27 1.27)) (justify right))
+    )
+    (pin "CAN_H" input (at 68.58 52.705 0)
       (effects (font (size 1.27 1.27)) (justify right))
     )
@@
     )
   )
-  (sheet (at 29.21 76.2) (size 39.37 15.24) (fields_autoplaced)
+  (sheet (at 29.21 81.915) (size 39.37 15.24) (fields_autoplaced)
     (stroke (width 0.1524) (type solid))
     (fill (color 0 0 0 0.0000))
-    (property "Sheetname" "USB" (at 29.21 75.4884 0)
+    (property "Sheetname" "USB" (at 29.21 81.2034 0)
       (effects (font (size 1.27 1.27)) (justify left bottom))
     )
-    (property "Sheetfile" "USB.kicad_sch" (at 29.21 92.0246 0)
+    (property "Sheetfile" "USB.kicad_sch" (at 29.21 97.7396 0)
       (effects (font (size 1.27 1.27)) (justify left top))
     )
-    (property "Field2" "" (at 29.21 76.2 0)
-      (effects (font (size 1.27 1.27)) hide)
-    )
-    (pin "UART_RX" input (at 68.58 81.28 0)
+    (property "Field2" "" (at 29.21 81.915 0)
+      (effects (font (size 1.27 1.27)) hide)
+    )
+    (pin "UART_RX" input (at 68.58 86.995 0)
       (effects (font (size 1.27 1.27)) (justify right))
     )
-    (pin "UART_TX" output (at 68.58 86.36 0)
+    (pin "UART_TX" output (at 68.58 92.075 0)
       (effects (font (size 1.27 1.27)) (justify right))
     )

Commit message: you kiss your mom with that face?
Parts:
- added D4, D5: SP0504BAHT, Package_TO_SOT_SMD:SOT-23-5, symbol Power_Protection:SP0504BAHT
- added J5: Conn_02x10_Counter_Clockwise, symbol Connector_Generic:Conn_02x10_Counter_Clockwise
Connections:
- net +3.3V: now also J5.19 (Pin_19), J5.2 (Pin_2)
- net +5V: now also J5.1 (Pin_1), J5.20 (Pin_20)
- net CAN_RX: now also U1.45 (PB8)
- net CAN_TX: now also U1.46 (PB9)
- net GND: now also D4.2 (A), D5.2 (A), J5.10 (Pin_10), J5.11 (Pin_11), J5.18 (Pin_18), J5.3 (Pin_3)
- net USART1_RX: now also U1.31 (PA10); no longer U1.30 (PA9)
- net USART1_TX: now also U1.30 (PA9); no longer U1.31 (PA10)
- net SPI1_NSS: now reaches U1.14 (PA4)
- net SPI1_NSS: now also D4.5 (K), J5.7 (Pin_7)
- net SPI1_SCK: now reaches U1.15 (PA5)
- net SPI1_SCK: now also D4.4 (K), J5.6 (Pin_6)
- net SPI1_MISO: now reaches U1.16 (PA6)
- net SPI1_MISO: now also D4.3 (K), J5.5 (Pin_5)
- net SPI1_MOSI: now reaches U1.17 (PA7)
- net SPI1_MOSI: now also D4.1 (K), J5.4 (Pin_4)
- net I2C2_SCL: now reaches U1.21 (PB10)
- net I2C2_SCL: now also J5.12 (Pin_12)
- net I2C2_SDA: now reaches U1.22 (PB11)
- net I2C2_SDA: now also J5.13 (Pin_13)
- net SPI2_NSS: now reaches U1.25 (PB12)
- net SPI2_NSS: now also D5.1 (K), J5.14 (Pin_14)
- net SPI2_SCK: now reaches U1.26 (PB13)
- net SPI2_SCK: now also D5.3 (K), J5.15 (Pin_15)
- net SPI2_MISO: now reaches U1.27 (PB14)
- net SPI2_MISO: now also D5.4 (K), J5.16 (Pin_16)
- net SPI2_MOSI: now reaches U1.28 (PB15)
- net SPI2_MOSI: now also D5.5 (K), J5.17 (Pin_17)
- net I2C1_SCL: now reaches U1.42 (PB6)
- net I2C1_SCL: now also J5.8 (Pin_8)
- net I2C1_SDA: now reaches U1.43 (PB7)
- net I2C1_SDA: now also J5.9 (Pin_9)
Other:
- moved on the sheet: C21, C22, U1, Y1

Commit message: Added I2C pull up resistors and questions
Parts:
- added R10, R2, R8, R9: 4.7K, symbol Device:R
Connections:
- net +3.3V: now also R10.1, R2.1, R8.1, R9.1
- net CAN_H: now also J2.3 (Pin_3); no longer J2.2 (Pin_2)
- net CAN_L: now also J2.4 (Pin_4); no longer J2.3 (Pin_3)
- net GNDPWR: now also J2.2 (Pin_2); no longer J2.4 (Pin_4)
- net I2C1_SCL: now also R8.2
- net I2C1_SDA: now also R2.2
- net I2C2_SCL: now also R10.2
- net I2C2_SDA: now also R9.2
- no-connect marks 0 -> 18
Other:
- note added: "Questions: I2C pull up resistor values right? TI said make em big bois Can circuit Switching between GPIO and I2C or SPI since they require different protection circuitry Check crystal oscillator Do we need NSS since we don't have multiple slaves?"
- note added: "V1.0: USing STM32L4CBT1 with 2 I2C, 2 SPI, 1 CAN, 1 UART (USB)"
- note added: "Version History"

Commit message: Added TVS diodes for Vin protection
Parts:
- added D6: SD12_SOD323, Diode_SMD:D_SOD-323, symbol Diode:SD12_SOD323
Connections:
- net +12V: now also D6.2 (A2)
- net GNDPWR: now also D6.1 (A1)
- no-connect marks 18 -> 19
Other:
- note added: "Questions: I2C pull up resistor values right? TI said make em big bois Can circuit Switching between GPIO and I2C or SPI since they require different protection circuitry Check crystal oscillator Do we need NSS since we don't have multiple slaves? Correct use of GNDPWR Is a 5V TVS diode needed at the LDO needed since the 12V is isolated?"
- note added: "Reset Button"
- note added: "Vin protection"
- note removed: "Questions: I2C pull up resistor values right? TI said make em big bois Can circuit Switching between GPIO and I2C or SPI since they require different protection circuitry Check crystal oscillator Do we need NSS since we don't have multiple slaves?"
- note removed: "USART1 on pins PA9/PA10, USART2 on pins PA2/PA3, USART3 on pins PC10/PC11 I2C1 on pins PB6/PB7, I2C2 on pins PB10/PB11, I2C3 on pins PC0/PC1 SPI1 on pins PA4/PA5/PA6/PA7, SPI2 on pins PB12/PB13/PB14/PB15 USB DFU interface on pins PA11/PA12 CAN1 on pins PB8/PB9"
- moved on the sheet: C27, C28

Commit message: removed 5V TVS diode :cry:
Other:
- note added: "Questions: I2C pull up resistor values right? TI said make em big bois Can circuit (changed up the connectors) Switching between GPIO and I2C or SPI since they require different protection circuitry Check crystal oscillator Do we need NSS since we don't have multiple slaves? Correct use of GNDPWR for the input connector? Is a 5V TVS diode needed at the LDO needed? (no cuz the 12V is isolated and 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"
- note removed: "Questions: I2C pull up resistor values right? TI said make em big bois Can circuit Switching between GPIO and I2C or SPI since they require different protection circuitry Check crystal oscillator Do we need NSS since we don't have multiple slaves? Correct use of GNDPWR Is a 5V TVS diode needed at the LDO needed since the 12V is isolated?"
Changed lines of the file:
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@@
     (fill (type none))
   )
-  (text "Questions:\nI2C pull up resistor values right? TI said make em big bois\nCan circuit\nSwitching between GPIO and I2C or SPI since they require different protection circuitry\nCheck crystal oscillator\nDo we need NSS since we don't have multiple slaves?\nCorrect use of GNDPWR\nIs a 5V TVS diode needed at the LDO needed since the 12V is isolated?"
+  (text "Questions:\nI2C pull up resistor values right? TI said make em big bois\nCan circuit (changed up the connectors)\nSwitching between GPIO and I2C or SPI since they require different protection circuitry\nCheck crystal oscillator\nDo we need NSS since we don't have multiple slaves?\nCorrect use of GNDPWR for the input connector?\nIs a 5V TVS diode needed at the LDO needed? (no cuz the 12V is isolated and coming from board?)"
     (at 30.48 147.955 0)
     (effects (font (size 1.27 1.27)) (justify left bottom))

Commit message: Added some footprints
Parts:
- C24, C25, C26, C27: footprint (none) -> Capacitor_SMD:C_0805_2012Metric
- J2: footprint (none) -> UTSVT_Connectors:Molex_MicroFit3.0_1x4xP3.00mm_PolarizingPeg_Vertical
Changed lines of the file:
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@@
       (effects (font (size 1.27 1.27)) (justify left))
     )
-    (property "Footprint" "" (at 145.7452 33.02 0)
+    (property "Footprint" "Capacitor_SMD:C_0805_2012Metric" (at 145.7452 33.02 0)
       (effects (font (size 1.27 1.27)) hide)
     )
@@
       (effects (font (size 1.27 1.27)) (justify left))
     )
-    (property "Footprint" "" (at 108.2802 97.79 0)
+    (property "Footprint" "Capacitor_SMD:C_0805_2012Metric" (at 108.2802 97.79 0)
       (effects (font (size 1.27 1.27)) hide)
     )
@@
       (effects (font (size 1.27 1.27)) (justify left))
     )
-    (property "Footprint" "" (at 121.6152 33.02 0)
+    (property "Footprint" "Capacitor_SMD:C_0805_2012Metric" (at 121.6152 33.02 0)
       (effects (font (size 1.27 1.27)) hide)
     )
@@
       (effects (font (size 1.27 1.27)) (justify left))
     )
-    (property "Footprint" "" (at 133.0452 33.02 0)
+    (property "Footprint" "Capacitor_SMD:C_0805_2012Metric" (at 133.0452 33.02 0)
       (effects (font (size 1.27 1.27)) hide)
     )
@@
       (effects (font (size 1.27 1.27)) (justify left))
     )
-    (property "Footprint" "" (at 186.69 31.75 0)
-      (effects (font (size 1.27 1.27)) hide)
-    )
+    (property "Footprint" "UTSVT_Connectors:Molex_MicroFit3.0_1x4xP3.00mm_PolarizingPeg_Vertical" (at 186.69 31.75 0)
+      (effects (font (size 1.27 1.27)) hide)
+    )

Commit message: Added ferrite beads to power input
Parts:
- added FB1: 12VFB, Inductor_SMD:L_0805_2012Metric, symbol Device:FerriteBead_Small
- added FB2: GPWRFB, Inductor_SMD:L_0805_2012Metric, symbol Device:FerriteBead_Small
Connections:
- net +12V: now also FB1.2; no longer J2.1 (Pin_1)
- net +3.3V: no longer J5.19 (Pin_19)
- net +5V: no longer J5.20 (Pin_20)
- net GND: no longer J5.11 (Pin_11), J5.18 (Pin_18)
- net GNDPWR: now also FB2.1; no longer J2.2 (Pin_2)
- new net: FB2.2, J2.2 (Pin_2)
- new net: FB1.1, J2.1 (Pin_1)
- no-connect marks 19 -> 23
Other:
- moved on the sheet: D6, J2

Commit message: started to add changes from PCB camp
Parts:
- removed D6: SD12_SOD323, Diode_SMD:D_SOD-323, symbol Diode:SD12_SOD323
- removed FB2: GPWRFB, Inductor_SMD:L_0805_2012Metric, symbol Device:FerriteBead_Small
- R10, R2, R8, R9: value 4.7K -> 10K
Connections:
- net CAN_H: now also J2.2 (Pin_2); no longer J2.3 (Pin_3)
- net CAN_L: now also J2.3 (Pin_3); no longer J2.4 (Pin_4)
- net GND: no longer J5.10 (Pin_10)
- net GNDPWR: now also J2.4 (Pin_4)
- net USART1_RX: now also U1.30 (PA9); no longer U1.31 (PA10)
- net USART1_TX: now also U1.31 (PA10); no longer U1.30 (PA9)
- no-connect marks 23 -> 24
Other:
- note added: "Things to change: Change SPI protectiont to 4 seperate diodes instead (put speed into consideration) Heartbeat LED Check RX and TX on mcu Use mosfets to switch between SPI/I2C to GPIO Add extra LEDs and switches When we add anything analog, seperate analog and digital domains Discuss with Tianda optimal connector layout Things to add if extra time: Make power LEDs oscillate with analog circuitry"
- note removed: "Questions: I2C pull up resistor values right? TI said make em big bois Can circuit (changed up the connectors) Switching between GPIO and I2C or SPI since they require different protection circuitry Check crystal oscillator Do we need NSS since we don't have multiple slaves? Correct use of GNDPWR for the input connector? Is a 5V TVS diode needed at the LDO needed? (no cuz the 12V is isolated and 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"
- note removed: "Vin protection"
- moved on the sheet: C29, SW2
