File: BPS-PeripheralSOM.kicad_sch (KiCad schematic)
At the start: 30 parts, among them J2 Can_In, J5 Conn_02x10_Counter_Clockwise, J7 SWD, SW2 Reset, U1 STM32L431CBTx, Y1 8M

Commit message: switched order or ESD and SPI
Parts:
- added R21: 4.7K, symbol Device:R
- added U7: ADG824BCP, Package_CSP:Analog_LFCSP-UQ-10_1.3x1.6mm_P0.4mm, symbol Analog_Switch:ADG824BCP
Connections:
- net +3.3V: now also R21.1, U7.6 (VDD)
- net GND: now also U7.10 (GND)
- net SPI1_MISO: now also D4.4 (K); no longer D4.3 (K)
- net SPI1_MOSI: now also D4.5 (K); no longer D4.1 (K)
- net SPI1_NSS: now also D4.1 (K); no longer D4.5 (K)
- net SPI1_SCK: now also D4.3 (K); no longer D4.4 (K)
- net SPI2_MISO: now also D5.3 (K); no longer D5.4 (K)
- net SPI2_MOSI: now also D5.1 (K); no longer D5.5 (K)
- net SPI2_NSS: now also D5.5 (K); no longer D5.1 (K)
- net SPI2_SCK: now also D5.4 (K); no longer D5.3 (K)
- new net: R21.2, U7.3 (S1B), U7.7 (S2B)
- new net: U7.1 (S1A), U7.9 (S2A)
- new net Conn1: U7.2 (D1)
- new net EN: U7.4 (IN1), U7.5 (IN2)
- new net GPIO: U7.8 (D2)
Other:
- moved on the sheet: D4, D5

Commit message: removed side reference circuits
Parts:
- removed R21: 4.7K, symbol Device:R
- removed U7: ADG824BCP, Package_CSP:Analog_LFCSP-UQ-10_1.3x1.6mm_P0.4mm, symbol Analog_Switch:ADG824BCP
Changed lines of the file:
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@@
   (junction (at 166.37 123.825) (diameter 0) (color 0 0 0 0)
   )
-  (junction (at 130.81 233.68) (diameter 0) (color 0 0 0 0)
-  )
   (junction (at 182.88 86.995) (diameter 0) (color 0 0 0 0)
   )
@@
   )
   (junction (at 269.24 90.805) (diameter 0) (color 0 0 0 0)
-  )
-  (junction (at 144.78 239.395) (diameter 0) (color 0 0 0 0)
   )
   (junction (at 107.95 63.5) (diameter 0) (color 0 0 0 0)
@@
   (no_connect (at 207.01 83.185))
   (no_connect (at 237.49 78.105))
-  (wire (pts (xy 144.78 239.395) (xy 144.78 241.3))
-    (stroke (width 0) (type default))
-  )
   (wire (pts (xy 186.055 36.83) (xy 187.325 36.83))
     (stroke (width 0) (type default))
   )
-  (wire (pts (xy 140.335 228.6) (xy 140.335 243.84))
-    (stroke (width 0) (type default))
-  )
-  (wire (pts (xy 167.64 246.38) (xy 171.45 246.38))
-    (stroke (width 0) (type default))
-  )
   (wire (pts (xy 196.85 118.745) (xy 207.01 118.745))
     (stroke (width 0) (type default))
@@
     (stroke (width 0) (type default))
   )
-  (wire (pts (xy 167.64 231.14) (xy 170.18 231.14))
-    (stroke (width 0) (type default))
-  )
   (wire (pts (xy 266.7 88.265) (xy 237.49 88.265))
     (stroke (width 0) (type default))
@@
     (stroke (width 0) (type default))
   )
-  (wire (pts (xy 144.78 241.3) (xy 147.32 241.3))
-    (stroke (width 0) (type default))
-  )
   (wire (pts (xy 77.47 26.035) (xy 77.47 27.305))
     (stroke (width 0) (type default))
@@
     (stroke (width 0) (type default))
   )
-  (wire (pts (xy 140.335 243.84) (xy 147.32 243.84))
-    (stroke (width 0) (type default))
-  )
   (wire (pts (xy 224.79 67.945) (xy 227.33 67.945))
     (stroke (width 0) (type default))
@@
     (stroke (width 0) (type default))
   )
-  (wire (pts (xy 130.81 233.68) (xy 147.32 233.68))
-    (stroke (width 0) (type default))
-  )
   (wire (pts (xy 66.675 31.115) (xy 83.185 31.115))
     (stroke (width 0) (type default))
@@
     (stroke (width 0) (type default))
   )
-  (wire (pts (xy 147.32 228.6) (xy 140.335 228.6))
-    (stroke (width 0) (type default))
-  )
   (wire (pts (xy 257.175 45.72) (xy 258.445 45.72))
     (stroke (width 0) (type default))
@@
     (stroke (width 0) (type default))
   )
-  (wire (pts (xy 140.97 239.395) (xy 144.78 239.395))
-    (stroke (width 0) (type default))
-  )
   (wire (pts (xy 69.85 40.64) (xy 69.85 39.37))
     (stroke (width 0) (type default))
@@
     (stroke (width 0) (type default))
   )
-  (wire (pts (xy 157.48 256.54) (xy 157.48 258.445))
-    (stroke (width 0) (type default))
-  )
   (wire (pts (xy 187.96 93.345) (xy 207.01 93.345))
     (stroke (width 0) (type default))
@@
     (stroke (width 0) (type default))
   )
-  (wire (pts (xy 130.81 248.92) (xy 147.32 248.92))
-    (stroke (width 0) (type default))
-  )
   (wire (pts (xy 132.08 25.4) (xy 144.78 25.4))
     (stroke (width 0) (type default))
@@
     (stroke (width 0) (type default))
   )
-  (wire (pts (xy 157.48 219.71) (xy 157.48 220.98))
-    (stroke (width 0) (type default))
-  )
   (wire (pts (xy 71.755 21.59) (xy 71.755 22.86))
     (stroke (width 0) (type default))
@@
     (stroke (width 0) (type default))
   )
-  (wire (pts (xy 144.78 236.22) (xy 144.78 239.395))
-    (stroke (width 0) (type default))
-  )
   (wire (pts (xy 83.185 31.115) (xy 83.185 29.21))
     (stroke (width 0) (type default))
@@
     (stroke (width 0) (type default))
   )
-  (wire (pts (xy 147.32 236.22) (xy 144.78 236.22))
-    (stroke (width 0) (type default))
-  )
-  (wire (pts (xy 130.81 233.68) (xy 130.81 248.92))
-    (stroke (width 0) (type default))
-  )
   (wire (pts (xy 196.85 133.985) (xy 207.01 133.985))
-    (stroke (width 0) (type default))
-  )
-  (wire (pts (xy 130.81 233.045) (xy 130.81 233.68))
     (stroke (width 0) (type default))
   )
@@
     (effects (font (size 1.27 1.27)) (justify right bottom))
   )
-  (label "GPIO" (at 171.45 246.38 0) (fields_autoplaced)
-    (effects (font (size 1.27 1.27)) (justify left bottom))
-  )
   (label "SPI2_MISO" (at 258.445 45.72 0) (fields_autoplaced)
     (effects (font (size 1.27 1.27)) (justify left bottom))
@@
     (effects (font (size 1.27 1.27)) (justify left bottom))
   )
-  (label "EN" (at 140.97 239.395 0) (fields_autoplaced)
-    (effects (font (size 1.27 1.27)) (justify left bottom))
-  )
   (label "PB3" (at 202.565 106.045 0) (fields_autoplaced)
     (effects (font (size 1.27 1.27)) (justify left bottom))
@@
   (label "USART1_RX" (at 81.28 92.075 180) (fields_autoplaced)
     (effects (font (size 1.27 1.27)) (justify right bottom))
-  )
-  (label "Conn1" (at 170.18 231.14 0) (fields_autoplaced)
-    (effects (font (size 1.27 1.27)) (justify left bottom))
   )
   (label "I2C1_SDA" (at 184.15 116.205 180) (fields_autoplaced)
@@
     )
   )
-  (symbol (lib_id "power:GND") (at 157.48 258.445 0) (unit 1)
-    (in_bom yes) (on_board yes) (dnp no) (fields_autoplaced)
-    (property "Reference" "#PWR048" (at 157.48 264.795 0)
-      (effects (font (size 1.27 1.27)) hide)
-    )
-    (property "Value" "GND" (at 157.48 262.89 0)
-      (effects (font (size 1.27 1.27)))
-    )
-    (property "Footprint" "" (at 157.48 258.445 0)
-      (effects (font (size 1.27 1.27)) hide)
-    )
-    (property "Datasheet" "" (at 157.48 258.445 0)
-      (effects (font (size 1.27 1.27)) hide)
-    )
-    (pin "1")
-    (instances
-      (project "BPS-PeripheralSOM"
-        (path "/d5ebd247-5a7c-47c2-8aee-beabaef72d6d"
-          (reference "#PWR048") (unit 1)
-        )
-      )
-    )
-  )
   (symbol (lib_id "power:GND") (at 264.16 104.775 0) (unit 1)
     (in_bom yes) (on_board yes) (dnp no) (fields_autoplaced)
@@
     )
   )
-  (symbol (lib_id "Device:R") (at 130.81 229.235 0) (unit 1)
-    (in_bom yes) (on_board yes) (dnp no) (fields_autoplaced)
-    (property "Reference" "R21" (at 133.35 228.6 0)
-      (effects (font (size 1.27 1.27)) (justify left))
-    )
-    (property "Value" "4.7K" (at 133.35 231.14 0)
-      (effects (font (size 1.27 1.27)) (justify left))
-    )
-    (property "Footprint" "" (at 129.032 229.235 90)
-      (effects (font (size 1.27 1.27)) hide)
-    )
-    (property "Datasheet" "~" (at 130.81 229.235 0)
-      (effects (font (size 1.27 1.27)) hide)
-    )
-    (pin "1")
-    (pin "2")
-    (instances
-      (project "BPS-PeripheralSOM"
-        (path "/d5ebd247-5a7c-47c2-8aee-beabaef72d6d"
-          (reference "R21") (unit 1)
-        )
-      )
-    )
-  )
-  (symbol (lib_id "power:+3.3V") (at 130.81 225.425 0) (unit 1)
-    (in_bom yes) (on_board yes) (dnp no) (fields_autoplaced)
-    (property "Reference" "#PWR052" (at 130.81 229.235 0)
-      (effects (font (size 1.27 1.27)) hide)
-    )
-    (property "Value" "+3.3V" (at 130.81 221.615 0)
-      (effects (font (size 1.27 1.27)))
-    )
-    (property "Footprint" "" (at 130.81 225.425 0)
-      (effects (font (size 1.27 1.27)) hide)
-    )
-    (property "Datasheet" "" (at 130.81 225.425 0)
-      (effects (font (size 1.27 1.27)) hide)
-    )
-    (pin "1")
-    (instances
-      (project "BPS-PeripheralSOM"
-        (path "/d5ebd247-5a7c-47c2-8aee-beabaef72d6d"
-          (reference "#PWR052") (unit 1)
-        )
-      )
-    )
-  )
   (symbol (lib_id "power:+3.3V") (at 161.925 113.665 0) (unit 1)
     (in_bom yes) (on_board yes) (dnp no) (fields_autoplaced)
@@
         (path "/d5ebd247-5a7c-47c2-8aee-beabaef72d6d"
           (reference "#PWR017") (unit 1)
-        )
-      )
-    )
-  )
-  (symbol (lib_id "power:+3.3V") (at 157.48 219.71 0) (unit 1)
-    (in_bom yes) (on_board yes) (dnp no) (fields_autoplaced)
-    (property "Reference" "#PWR053" (at 157.48 223.52 0)
-      (effects (font (size 1.27 1.27)) hide)
-    )
-    (property "Value" "+3.3V" (at 157.48 215.9 0)
-      (effects (font (size 1.27 1.27)))
-    )
-    (property "Footprint" "" (at 157.48 219.71 0)
-      (effects (font (size 1.27 1.27)) hide)
-    )
-    (property "Datasheet" "" (at 157.48 219.71 0)
-      (effects (font (size 1.27 1.27)) hide)
-    )
-    (pin "1")
-    (instances
-      (project "BPS-PeripheralSOM"
-        (path "/d5ebd247-5a7c-47c2-8aee-beabaef72d6d"
-          (reference "#PWR053") (unit 1)
         )
       )
@@
         )
       )
-    )
-  )
-  (symbol (lib_id "Analog_Switch:ADG824BCP") (at 157.48 238.76 0) (unit 1)
-    (in_bom yes) (on_board yes) (dnp no) (fields_autoplaced)
-    (property "Reference" "U7" (at 159.4359 219.71 0)
-      (effects (font (size 1.27 1.27)) (justify left))
-    )
-    (property "Value" "ADG824BCP" (at 159.4359 222.25 0)
-      (effects (font (size 1.27 1.27)) (justify left))
-    )
-    (property "Footprint" "Package_CSP:Analog_LFCSP-UQ-10_1.3x1.6mm_P0.4mm" (at 157.48 238.76 0)
-      (effects (font (size 1.27 1.27)) hide)
-    )
-    (property "Datasheet" "https://www.analog.com/media/en/technical-documentation/data-sheets/ADG884.pdf" (at 157.48 238.76 0)
-      (effects (font (size 1.27 1.27)) hide)
-    )
-    (pin "1")
-    (pin "10")
-    (pin "2")
-    (pin "3")
-    (pin "4")
-    (pin "5")
-    (pin "6")
-    (pin "7")
-    (pin "8")
-    (pin "9")
-    (instances
-      (project "BPS-PeripheralSOM"
-        (path "/d5ebd247-5a7c-47c2-8aee-beabaef72d6d"
-          (reference "U7") (unit 1)
-        )
-      )

Commit message: add 3.3v tvs diode
Parts:
- removed D4, D5: SP0504BAHT, Package_TO_SOT_SMD:SOT-23-5, symbol Power_Protection:SP0504BAHT
- added CR1, CR2: D5V0P4UR6SO-7, UTSVT_ICs:SOT26_DIO, symbol utsvt-chips:D5V0P4UR6SO-7
Connections:
- net +3.3V: now also J5.16 (Pin_16), J5.5 (Pin_5); no longer J5.18 (Pin_18), J5.6 (Pin_6), R10.1, R9.1
- net +5V: now also J5.6 (Pin_6); no longer J5.5 (Pin_5)
- net GND: now also J5.20 (Pin_20), CR1.2, CR2.2; no longer J5.16 (Pin_16)
- net I2C1_SCL: now also J5.8 (Pin_8); no longer J5.20 (Pin_20)
- net I2C1_SDA: now also J5.9 (Pin_9); no longer J5.19 (Pin_19)
- net I2C2_SCL: now also J5.19 (Pin_19); no longer J5.8 (Pin_8)
- net I2C2_SDA: now also J5.18 (Pin_18); no longer J5.9 (Pin_9)
- net SPI1_MISO: now also CR2.6
- net SPI1_MOSI: now also CR2.4
- net SPI1_NSS: now also CR2.3
- net SPI1_SCK: now also CR2.1
- net SPI2_MISO: now also CR1.6
- net SPI2_MOSI: now also CR1.1
- net SPI2_NSS: now also CR1.3
- net SPI2_SCK: now also CR1.4
- new net: R10.1, R9.1
- no-connect marks 13 -> 14
Other:
- moved on the sheet: C21, C22, J5, R10, R14, R15, R2, R20, R8, R9, U1, Y1

Commit message: Cleaned up schematic and updated to do
Connections:
- no-connect marks 14 -> 15
Other:
- note added: "To do: Software enabled I2C pull down resistors Things to add if extra time: Make power LEDs oscillate with analog circuitry"
- note removed: "Change SPI protection IC by account for speed and clamping voltage One SPI with GPIO protection + SPI protection Add one i2c with GPIO protection + I2C protection Software enabled I2C pull down resistors Things to add if extra time: Make power LEDs oscillate with analog circuitry"
Changed lines of the file:
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@@
   (no_connect (at 222.25 85.09))
   (no_connect (at 222.25 105.41))
+  (no_connect (at 276.86 133.35))
   (no_connect (at 222.25 115.57))
   (no_connect (at 222.25 107.95))
@@
     (effects (font (size 1.27 1.27)) (justify left bottom))
   )
-  (text "Change SPI protection IC by account for speed and clamping voltage\nOne SPI with GPIO protection + SPI protection\nAdd one i2c with GPIO protection + I2C protection\nSoftware enabled I2C pull down resistors\n\nThings to add if extra time:\nMake power LEDs oscillate with analog circuitry"
-    (at 29.21 188.595 0)
+  (text "To do:\nSoftware enabled I2C pull down resistors\n\nThings to add if extra time:\nMake power LEDs oscillate with analog circuitry"
+    (at 29.845 181.61 0)
     (effects (font (size 1.27 1.27)) (justify left bottom))
   )

Commit message: moved the 3.3V label
Connections:
- net +3.3V: now also R10.1, R9.1
Changed lines of the file:
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@@
     (stroke (width 0) (type default))
   )
-  (wire (pts (xy 146.685 118.11) (xy 146.685 119.38))
+  (wire (pts (xy 146.685 117.475) (xy 146.685 119.38))
     (stroke (width 0) (type default))
   )
@@
     )
   )
-  (symbol (lib_id "power:+3.3V") (at 161.925 113.665 0) (unit 1)
+  (symbol (lib_id "power:+3.3V") (at 146.685 117.475 0) (unit 1)
     (in_bom yes) (on_board yes) (dnp no)
-    (property "Reference" "#PWR050" (at 161.925 117.475 0)
-      (effects (font (size 1.27 1.27)) hide)
-    )
-    (property "Value" "+3.3V" (at 146.685 114.935 0)
+    (property "Reference" "#PWR050" (at 146.685 121.285 0)
+      (effects (font (size 1.27 1.27)) hide)
+    )
+    (property "Value" "+3.3V" (at 141.605 114.935 0)
       (effects (font (size 1.27 1.27)))
     )
-    (property "Footprint" "" (at 161.925 113.665 0)
-      (effects (font (size 1.27 1.27)) hide)
-    )
-    (property "Datasheet" "" (at 161.925 113.665 0)
-      (effects (font (size 1.27 1.27)) hide)
-    )
+    (property "Footprint" "" (at 146.685 117.475 0)
+      (effects (font (size 1.27 1.27)) hide)
+    )
+    (property "Datasheet" "" (at 146.685 117.475 0)
+      (effects (font (size 1.27 1.27)) hide)
+    )

Commit message: Added extra todo stuff from PCB camp
Parts:
- removed R14: 50, symbol Device:R
Connections:
- net SPI1_NSS: now also U1.14 (PA4)
Other:
- note added: "To do: Software enabled I2C pull down resistors Move 12V and PWRGND together on connector Things to add if extra time: Make power LEDs oscillate with analog circuitry"
- note removed: "To do: Software enabled I2C pull down resistors Things to add if extra time: Make power LEDs oscillate with analog circuitry"
Changed lines of the file:
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@@
-    (stroke (width 0) (type default))
-  )
-  (wire (pts (xy 244.475 87.63) (xy 246.38 87.63))
     (stroke (width 0) (type default))
   )
@@
     (stroke (width 0) (type default))
   )
-  (wire (pts (xy 222.25 87.63) (xy 236.855 87.63))
+  (wire (pts (xy 222.25 87.63) (xy 246.38 87.63))
     (stroke (width 0) (type default))
   )
@@
     (effects (font (size 1.27 1.27)) (justify left bottom))
   )
-  (text "To do:\nSoftware enabled I2C pull down resistors\n\nThings to add if extra time:\nMake power LEDs oscillate with analog circuitry"
-    (at 29.845 181.61 0)
+  (text "To do:\nSoftware enabled I2C pull down resistors\nMove 12V and PWRGND together on connector\n\nThings to add if extra time:\nMake power LEDs oscillate with analog circuitry"
+    (at 29.845 183.515 0)
     (effects (font (size 1.27 1.27)) (justify left bottom))
   )
   (text "SPI1 is main SPI\nI2C1 is main I2C\nSPI2 and I2C can be swapped out for GPIO"
-    (at 209.55 18.415 0)
+    (at 209.55 20.955 0)
     (effects (font (size 1.27 1.27)) (justify left bottom))
   )
@@
         )
       )
-    )
-  )
-  (symbol (lib_id "Device:R") (at 240.665 87.63 90) (unit 1)
-    (in_bom yes) (on_board yes) (dnp no) (fields_autoplaced)
-    (property "Reference" "R14" (at 240.665 83.185 90)
-      (effects (font (size 1.27 1.27)))
-    )
-    (property "Value" "50" (at 240.665 85.725 90)
-      (effects (font (size 1.27 1.27)))
-    )
-    (property "Footprint" "" (at 240.665 89.408 90)
-      (effects (font (size 1.27 1.27)) hide)
-    )
-    (property "Datasheet" "~" (at 240.665 87.63 0)
-      (effects (font (size 1.27 1.27)) hide)
-    )
-    (pin "1")
-    (pin "2")
-    (instances
-      (project "BPS-PeripheralSOM"
-        (path "/d5ebd247-5a7c-47c2-8aee-beabaef72d6d"
-          (reference "R14") (unit 1)
-        )
-      )
