File: BPS-PeripheralSOM.kicad_sch (KiCad schematic)
At the start: 29 parts, among them J2 Can_In, J5 Conn_02x10_Counter_Clockwise, J7 SWD, SW2 Reset, U1 STM32L431CBTx, Y1 8M

Commit message: changed connector layout (moved 12V and pwrgnd next to eachother)
Connections:
- net +12V: now also J5.12 (Pin_12); no longer J5.17 (Pin_17)
- net +3.3V: now also J5.20 (Pin_20); no longer J5.16 (Pin_16)
- net GND: now also J5.17 (Pin_17); no longer J5.20 (Pin_20)
- net SPI2_MISO: now also J5.14 (Pin_14); no longer J5.13 (Pin_13)
- net SPI2_MOSI: now also J5.13 (Pin_13); no longer J5.12 (Pin_12)
- net SPI2_NSS: now also J5.16 (Pin_16); no longer J5.15 (Pin_15)
- net SPI2_SCK: now also J5.15 (Pin_15); no longer J5.14 (Pin_14)
Other:
- note added: "To do: Software enabled I2C pull down resistors Move 12V and PWRGND together on connector Pick new molex connector Things to add if extra time: Make power LEDs oscillate with analog circuitry"
- note removed: "To do: Software enabled I2C pull down resistors Move 12V and PWRGND together on connector Things to add if extra time: Make power LEDs oscillate with analog circuitry"
Changed lines of the file:
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@@
     (stroke (width 0) (type default))
   )
-  (wire (pts (xy 267.97 33.02) (xy 267.97 36.83))
+  (wire (pts (xy 260.35 48.26) (xy 260.35 49.53))
     (stroke (width 0) (type default))
   )
@@
     (stroke (width 0) (type default))
   )
+  (wire (pts (xy 258.445 26.67) (xy 258.445 29.21))
+    (stroke (width 0) (type default))
+  )
   (wire (pts (xy 120.65 33.02) (xy 132.08 33.02))
     (stroke (width 0) (type default))
   )
-  (wire (pts (xy 246.38 49.53) (xy 247.65 49.53))
+  (wire (pts (xy 246.38 41.91) (xy 247.65 41.91))
     (stroke (width 0) (type default))
   )
@@
     (stroke (width 0) (type default))
   )
-  (wire (pts (xy 267.97 36.83) (xy 246.38 36.83))
-    (stroke (width 0) (type default))
-  )
   (wire (pts (xy 276.86 130.81) (xy 276.86 105.41))
     (stroke (width 0) (type default))
@@
     (stroke (width 0) (type default))
   )
+  (wire (pts (xy 260.985 36.83) (xy 246.38 36.83))
+    (stroke (width 0) (type default))
+  )
   (wire (pts (xy 140.97 54.61) (xy 130.81 54.61))
     (stroke (width 0) (type default))
@@
     (stroke (width 0) (type default))
   )
+  (wire (pts (xy 246.38 46.99) (xy 247.65 46.99))
+    (stroke (width 0) (type default))
+  )
   (wire (pts (xy 66.675 31.115) (xy 83.185 31.115))
     (stroke (width 0) (type default))
@@
     (stroke (width 0) (type default))
   )
-  (wire (pts (xy 246.38 46.99) (xy 247.65 46.99))
-    (stroke (width 0) (type default))
-  )
   (wire (pts (xy 172.72 153.035) (xy 181.61 153.035))
     (stroke (width 0) (type default))
@@
     (stroke (width 0) (type default))
   )
+  (wire (pts (xy 246.38 44.45) (xy 247.65 44.45))
+    (stroke (width 0) (type default))
+  )
   (wire (pts (xy 186.69 133.35) (xy 191.77 133.35))
     (stroke (width 0) (type default))
@@
     (stroke (width 0) (type default))
   )
+  (wire (pts (xy 258.445 29.21) (xy 246.38 29.21))
+    (stroke (width 0) (type default))
+  )
   (wire (pts (xy 231.775 95.25) (xy 254 95.25))
     (stroke (width 0) (type default))
@@
     (stroke (width 0) (type default))
   )
-  (wire (pts (xy 246.38 41.91) (xy 247.65 41.91))
-    (stroke (width 0) (type default))
-  )
   (wire (pts (xy 140.97 57.15) (xy 130.81 57.15))
     (stroke (width 0) (type default))
@@
     (stroke (width 0) (type default))
   )
-  (wire (pts (xy 246.38 44.45) (xy 247.65 44.45))
-    (stroke (width 0) (type default))
-  )
   (wire (pts (xy 130.81 54.61) (xy 130.81 53.34))
     (stroke (width 0) (type default))
@@
     (stroke (width 0) (type default))
   )
-  (wire (pts (xy 271.78 36.83) (xy 271.78 39.37))
-    (stroke (width 0) (type default))
-  )
   (wire (pts (xy 140.97 59.69) (xy 130.81 59.69))
     (stroke (width 0) (type default))
@@
     (stroke (width 0) (type default))
   )
-  (wire (pts (xy 271.78 39.37) (xy 246.38 39.37))
+  (wire (pts (xy 260.35 49.53) (xy 246.38 49.53))
+    (stroke (width 0) (type default))
+  )
+  (wire (pts (xy 246.38 39.37) (xy 247.65 39.37))
     (stroke (width 0) (type default))
   )
@@
   )
   (wire (pts (xy 73.66 35.56) (xy 73.66 34.925))
-    (stroke (width 0) (type default))
-  )
-  (wire (pts (xy 261.62 29.21) (xy 246.38 29.21))
     (stroke (width 0) (type default))
   )
@@
     (effects (font (size 1.27 1.27)) (justify left bottom))
   )
-  (text "To do:\nSoftware enabled I2C pull down resistors\nMove 12V and PWRGND together on connector\n\nThings to add if extra time:\nMake power LEDs oscillate with analog circuitry"
-    (at 29.845 183.515 0)
+  (text "To do:\nSoftware enabled I2C pull down resistors\nMove 12V and PWRGND together on connector\nPick new molex connector\n\nThings to add if extra time:\nMake power LEDs oscillate with analog circuitry"
+    (at 29.845 185.42 0)
     (effects (font (size 1.27 1.27)) (justify left bottom))
   )
@@
     (effects (font (size 1.27 1.27)) (justify left bottom))
   )
-  (label "SPI2_MOSI" (at 247.65 49.53 0) (fields_autoplaced)
+  (label "SPI2_MOSI" (at 247.65 46.99 0) (fields_autoplaced)
     (effects (font (size 1.27 1.27)) (justify left bottom))
   )
@@
     (effects (font (size 1.27 1.27)) (justify left bottom))
   )
-  (label "SPI2_SCK" (at 247.65 44.45 0) (fields_autoplaced)
+  (label "SPI2_SCK" (at 247.65 41.91 0) (fields_autoplaced)
     (effects (font (size 1.27 1.27)) (justify left bottom))
   )
@@
     (effects (font (size 1.27 1.27)) (justify right bottom))
   )
-  (label "SPI2_MISO" (at 247.65 46.99 0) (fields_autoplaced)
+  (label "SPI2_MISO" (at 247.65 44.45 0) (fields_autoplaced)
     (effects (font (size 1.27 1.27)) (justify left bottom))
   )
@@
     (effects (font (size 1.27 1.27)) (justify left bottom))
   )
-  (label "SPI2_NSS" (at 247.65 41.91 0) (fields_autoplaced)
+  (label "SPI2_NSS" (at 247.65 39.37 0) (fields_autoplaced)
     (effects (font (size 1.27 1.27)) (justify left bottom))
   )
@@
     )
   )
-  (symbol (lib_id "power:GND") (at 261.62 29.21 0) (unit 1)
+  (symbol (lib_id "power:GND") (at 260.985 36.83 0) (unit 1)
     (in_bom yes) (on_board yes) (dnp no)
-    (property "Reference" "#PWR033" (at 261.62 35.56 0)
-      (effects (font (size 1.27 1.27)) hide)
-    )
-    (property "Value" "GND" (at 261.747 33.6042 0)
-      (effects (font (size 1.27 1.27)))
-    )
-    (property "Footprint" "" (at 261.62 29.21 0)
-      (effects (font (size 1.27 1.27)) hide)
-    )
-    (property "Datasheet" "" (at 261.62 29.21 0)
+    (property "Reference" "#PWR033" (at 260.985 43.18 0)
+      (effects (font (size 1.27 1.27)) hide)
+    )
+    (property "Value" "GND" (at 261.112 41.2242 0)
+      (effects (font (size 1.27 1.27)))
+    )
+    (property "Footprint" "" (at 260.985 36.83 0)
+      (effects (font (size 1.27 1.27)) hide)
+    )
+    (property "Datasheet" "" (at 260.985 36.83 0)
       (effects (font (size 1.27 1.27)) hide)
     )
@@
     )
   )
-  (symbol (lib_id "power:+3.3V") (at 271.78 36.83 0) (unit 1)
-    (in_bom yes) (on_board yes) (dnp no) (fields_autoplaced)
-    (property "Reference" "#PWR024" (at 271.78 40.64 0)
-      (effects (font (size 1.27 1.27)) hide)
-    )
-    (property "Value" "+3.3V" (at 271.78 33.02 0)
-      (effects (font (size 1.27 1.27)))
-    )
-    (property "Footprint" "" (at 271.78 36.83 0)
-      (effects (font (size 1.27 1.27)) hide)
-    )
-    (property "Datasheet" "" (at 271.78 36.83 0)
+  (symbol (lib_id "power:+3.3V") (at 258.445 26.67 0) (unit 1)
+    (in_bom yes) (on_board yes) (dnp no) (fields_autoplaced)
+    (property "Reference" "#PWR024" (at 258.445 30.48 0)
+      (effects (font (size 1.27 1.27)) hide)
+    )
+    (property "Value" "+3.3V" (at 258.445 22.86 0)
+      (effects (font (size 1.27 1.27)))
+    )
+    (property "Footprint" "" (at 258.445 26.67 0)
+      (effects (font (size 1.27 1.27)) hide)
+    )
+    (property "Datasheet" "" (at 258.445 26.67 0)
       (effects (font (size 1.27 1.27)) hide)
     )
@@
     )
   )
-  (symbol (lib_id "power:+12V") (at 267.97 33.02 0) (unit 1)
+  (symbol (lib_id "power:+12V") (at 260.35 48.26 0) (unit 1)
     (in_bom yes) (on_board yes) (dnp no)
-    (property "Reference" "#PWR043" (at 267.97 36.83 0)
-      (effects (font (size 1.27 1.27)) hide)
-    )
-    (property "Value" "+12V" (at 267.97 29.845 0)
-      (effects (font (size 1.27 1.27)))
-    )
-    (property "Footprint" "" (at 267.97 33.02 0)
-      (effects (font (size 1.27 1.27)) hide)
-    )
-    (property "Datasheet" "" (at 267.97 33.02 0)
-      (effects (font (size 1.27 1.27)) hide)
-    )
+    (property "Reference" "#PWR043" (at 260.35 52.07 0)
+      (effects (font (size 1.27 1.27)) hide)
+    )
+    (property "Value" "+12V" (at 260.35 44.45 0)
+      (effects (font (size 1.27 1.27)))
+    )
+    (property "Footprint" "" (at 260.35 48.26 0)
+      (effects (font (size 1.27 1.27)) hide)
+    )
+    (property "Datasheet" "" (at 260.35 48.26 0)
+      (effects (font (size 1.27 1.27)) hide)
+    )

Commit message: made schematic look nicer
Connections:
- net SPI2_NSS: no longer J5.16 (Pin_16)
Other:
- moved on the sheet: C21, C22, C29, CR1, CR2, J2, J7, R10, R15, R2, R20, R8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
