File: BPS-PeripheralSOM.kicad_sch (KiCad schematic)
At the start: 34 parts, among them IC1 TPS1120DR, J1 SWD, J2 Conn_01x04, J4 Conn_01x04, J6 SOMConnector, SW2 Reset, U1 STM32L431CBTx, Y1 8M

Commit message: dumbass
Other:
- note added: "Todo: Inductor footprints SHDN on pp UVLO and OVLO divider Change connector out Switch heartbeat pin (do when layout)"
- note removed: "Todo: UART TX and RX switch on USB chip? Inductor footprints SHDN on pp UVLO and OVLO divider Change connector out Switch heartbeat pin (do when layout)"
Changed lines of the file:
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@@
 		)
 	)
-	(text "Todo:\nUART TX and RX switch on USB chip?\nInductor footprints\nSHDN on pp\nUVLO and OVLO divider\nChange connector out\nSwitch heartbeat pin (do when layout)"
+	(text "Todo:\nInductor footprints\nSHDN on pp\nUVLO and OVLO divider\nChange connector out\nSwitch heartbeat pin (do when layout)"
 		(exclude_from_sim no)
 		(at 14.732 101.6 0)

Commit message: SHDN pin
Other:
- note added: "Todo: Inductor footprints SHDN on pp UVLO and OVLO divider on pp Change connector out Switch heartbeat pin (do when layout) Fault pin on pp"
- note removed: "Todo: Inductor footprints SHDN on pp UVLO and OVLO divider Change connector out Switch heartbeat pin (do when layout)"
Changed lines of the file:
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@@
 		)
 	)
-	(text "Todo:\nInductor footprints\nSHDN on pp\nUVLO and OVLO divider\nChange connector out\nSwitch heartbeat pin (do when layout)"
+	(text "Todo:\nInductor footprints\nSHDN on pp\nUVLO and OVLO divider on pp\nChange connector out\nSwitch heartbeat pin (do when layout)\nFault pin on pp"
 		(exclude_from_sim no)
 		(at 14.732 101.6 0)
@@
 		)
 		(instances
-			(project ""
+			(project "BPS-PeripheralSOM"
 				(path "/d5ebd247-5a7c-47c2-8aee-beabaef72d6d"
 					(reference "#PWR041")
@@
 		)
 		(instances
-			(project ""
+			(project "BPS-PeripheralSOM"
 				(path "/d5ebd247-5a7c-47c2-8aee-beabaef72d6d"
 					(reference "#PWR013")
@@
 		)
 		(instances
-			(project ""
+			(project "BPS-PeripheralSOM"
 				(path "/d5ebd247-5a7c-47c2-8aee-beabaef72d6d"
 					(reference "#PWR038")
@@
 		)
 		(instances
-			(project ""
+			(project "BPS-PeripheralSOM"
 				(path "/d5ebd247-5a7c-47c2-8aee-beabaef72d6d"
 					(reference "#PWR035")
@@
 		)
 		(instances
-			(project ""
+			(project "BPS-PeripheralSOM"
 				(path "/d5ebd247-5a7c-47c2-8aee-beabaef72d6d"
 					(reference "J2")

Commit message: changed pullup
Other:
- note added: "Todo: Inductor footprints UVLO and OVLO divider on pp Change connector out Switch heartbeat pin (do when layout) Fault pin on pp"
- note removed: "Todo: Inductor footprints SHDN on pp UVLO and OVLO divider on pp Change connector out Switch heartbeat pin (do when layout) Fault pin on pp"
Changed lines of the file:
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@@
 		)
 	)
-	(text "Todo:\nInductor footprints\nSHDN on pp\nUVLO and OVLO divider on pp\nChange connector out\nSwitch heartbeat pin (do when layout)\nFault pin on pp"
+	(text "Todo:\nInductor footprints\nUVLO and OVLO divider on pp\nChange connector out\nSwitch heartbeat pin (do when layout)\nFault pin on pp"
 		(exclude_from_sim no)
 		(at 14.732 101.6 0)

Commit message: fault pp
Other:
- note added: "Todo: Inductor footprints UVLO and OVLO divider on pp Change connector out Switch heartbeat pin (do when layout)"
- note removed: "Todo: Inductor footprints UVLO and OVLO divider on pp Change connector out Switch heartbeat pin (do when layout) Fault pin on pp"
Changed lines of the file:
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@@
 		)
 	)
-	(text "Todo:\nInductor footprints\nUVLO and OVLO divider on pp\nChange connector out\nSwitch heartbeat pin (do when layout)\nFault pin on pp"
+	(text "Todo:\nInductor footprints\nUVLO and OVLO divider on pp\nChange connector out\nSwitch heartbeat pin (do when layout)"
 		(exclude_from_sim no)
 		(at 14.732 101.6 0)

Commit message: wahoooooooooooooooooooooooooooooooooooo
Other:
- note added: "Todo: UVLO and OVLO divider on pp Change out pp footprint Change connector out Switch heartbeat pin (do when layout)"
- note removed: "Todo: Inductor footprints UVLO and OVLO divider on pp Change connector out Switch heartbeat pin (do when layout)"
Changed lines of the file:
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@@
 		)
 	)
-	(text "Todo:\nInductor footprints\nUVLO and OVLO divider on pp\nChange connector out\nSwitch heartbeat pin (do when layout)"
+	(text "Todo:\nUVLO and OVLO divider on pp\nChange out pp footprint\nChange connector out\nSwitch heartbeat pin (do when layout)"
 		(exclude_from_sim no)
 		(at 14.732 101.6 0)

Commit message: pp foot
Other:
- note added: "Todo: UVLO and OVLO divider on pp Change connector out Switch heartbeat pin (do when layout)"
- note removed: "Todo: UVLO and OVLO divider on pp Change out pp footprint Change connector out Switch heartbeat pin (do when layout)"
Changed lines of the file:
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@@
 	)
 	(rectangle
-		(start 12.065 12.7)
-		(end 69.85 198.12)
+		(start 12.065 11.938)
+		(end 69.85 197.358)
 		(stroke
 			(width 0)
@@
 		)
 	)
-	(text "Todo:\nUVLO and OVLO divider on pp\nChange out pp footprint\nChange connector out\nSwitch heartbeat pin (do when layout)"
+	(text "Todo:\nUVLO and OVLO divider on pp\nChange connector out\nSwitch heartbeat pin (do when layout)"
 		(exclude_from_sim no)
 		(at 14.732 101.6 0)

Commit message: update todo
Other:
- note added: "Todo: Change connector out Switch heartbeat pin (do when layout)"
- note removed: "Todo: UVLO and OVLO divider on pp Change connector out Switch heartbeat pin (do when layout)"
Changed lines of the file:
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@@
 		)
 	)
-	(text "Todo:\nUVLO and OVLO divider on pp\nChange connector out\nSwitch heartbeat pin (do when layout)"
+	(text "Todo:\nChange connector out\nSwitch heartbeat pin (do when layout)"
 		(exclude_from_sim no)
 		(at 14.732 101.6 0)

Commit message: fix SPI prot
Connections:
- net +3.3V: now also CR1.5, CR2.5
- no-connect marks 11 -> 9
Other:
- moved on the sheet: CR1
