File: Leds.kicad_sch (KiCad schematic)
At the start: 8 parts

Commit message: Made things look nicer
Changed lines of the file:
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@@
     (stroke (width 0) (type default))
   )
-  (text "Heartbeat LED Green!!" (at 102.235 115.57 0)
+  (text "Heartbeat LED Green!!" (at 60.325 97.79 0)
     (effects (font (size 1.27 1.27)) (justify left bottom))
   )

Commit message: Added LEDs and Switches
Parts:
- added C55 (x2): 10nF, symbol Device:C
- added D1: PowerLED, LED_SMD:LED_0805_2012Metric, symbol Device:LED
- added R13, R6: 220, Resistor_SMD:R_0805_2012Metric, symbol Device:R
- added R5: 1.5k, Resistor_SMD:R_0805_2012Metric, symbol Device:R
- added SW2: SW_SPST, symbol Switch:SW_SPST
- added SW7: SW_Push, UTSVT_Special:SW_SPST_B3SL-1002P, symbol Switch:SW_Push
Connections:
- net GND: now reaches R16.2, R17.2, R18.2, R19.2
- net GND: now also D1.1 (K), SW2.1 (A), SW7.1
- new net: C55.2, R6.2, SW7.2
- new net: D1.2 (A), R5.2
- new net: C55.2, R13.2, SW2.2 (B)
- new net +5V: R5.1
- new net PB4: C55.1, R6.1
- new net PB5: C55.1, R13.1
Other:
- note removed: "Heartbeat LED Green!!"

Commit message: added more footprints
Parts:
- C55: footprint (none) -> Capacitor_SMD:C_0805_2012Metric
- D6, D7, D9: footprint (none) -> LED_SMD:LED_0805_2012Metric
Other:
- moved on the sheet: D6
Changed lines of the file:
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@@
     (stroke (width 0) (type default))
   )
-  (wire (pts (xy 105.41 83.185) (xy 105.41 90.805))
+  (wire (pts (xy 105.41 83.185) (xy 105.41 92.075))
     (stroke (width 0) (type default))
   )
@@
     (stroke (width 0) (type default))
   )
-  (wire (pts (xy 105.41 98.425) (xy 105.41 100.965))
+  (wire (pts (xy 105.41 99.695) (xy 105.41 100.965))
     (stroke (width 0) (type default))
   )
@@
       (effects (font (size 1.27 1.27)) (justify right))
     )
-    (property "Footprint" "" (at 118.11 95.885 0)
-      (effects (font (size 1.27 1.27)) hide)
-    )
-    (property "Datasheet" "~" (at 118.11 95.885 0)
+    (property "Footprint" "LED_SMD:LED_0805_2012Metric" (at 118.11 95.885 0)
+      (effects (font (size 1.27 1.27)) hide)
+    )
+    (property "Datasheet" "https://www.mouser.com/datasheet/2/216/APT2012LSECK_J3_PRV-535674.pdf" (at 118.11 95.885 0)
       (effects (font (size 1.27 1.27)) hide)
     )
@@
       (effects (font (size 1.27 1.27)) (justify right))
     )
-    (property "Footprint" "" (at 130.81 95.885 0)
-      (effects (font (size 1.27 1.27)) hide)
-    )
-    (property "Datasheet" "~" (at 130.81 95.885 0)
+    (property "Footprint" "LED_SMD:LED_0805_2012Metric" (at 130.81 95.885 0)
+      (effects (font (size 1.27 1.27)) hide)
+    )
+    (property "Datasheet" "https://www.mouser.com/datasheet/2/216/APT2012LSECK_J3_PRV-535674.pdf" (at 130.81 95.885 0)
       (effects (font (size 1.27 1.27)) hide)
     )
@@
     )
   )
-  (symbol (lib_id "Device:LED") (at 105.41 94.615 90) (unit 1)
+  (symbol (lib_id "Device:LED") (at 105.41 95.885 90) (unit 1)
     (in_bom yes) (on_board yes) (dnp no) (fields_autoplaced)
-    (property "Reference" "D6" (at 109.22 95.5675 90)
-      (effects (font (size 1.27 1.27)) (justify right))
-    )
-    (property "Value" "LED" (at 109.22 98.1075 90)
-      (effects (font (size 1.27 1.27)) (justify right))
-    )
-    (property "Footprint" "" (at 105.41 94.615 0)
-      (effects (font (size 1.27 1.27)) hide)
-    )
-    (property "Datasheet" "~" (at 105.41 94.615 0)
+    (property "Reference" "D6" (at 109.22 96.8375 90)
+      (effects (font (size 1.27 1.27)) (justify right))
+    )
+    (property "Value" "LED" (at 109.22 99.3775 90)
+      (effects (font (size 1.27 1.27)) (justify right))
+    )
+    (property "Footprint" "LED_SMD:LED_0805_2012Metric" (at 105.41 95.885 0)
+      (effects (font (size 1.27 1.27)) hide)
+    )
+    (property "Datasheet" "https://www.mouser.com/datasheet/2/216/APT2012LSECK_J3_PRV-535674.pdf" (at 105.41 95.885 0)
       (effects (font (size 1.27 1.27)) hide)
     )
@@
       (effects (font (size 1.27 1.27)) (justify left))
     )
-    (property "Footprint" "" (at 64.4652 98.425 0)
+    (property "Footprint" "Capacitor_SMD:C_0805_2012Metric" (at 64.4652 98.425 0)
       (effects (font (size 1.27 1.27)) hide)
     )
@@
       (effects (font (size 1.27 1.27)) (justify left))
     )
-    (property "Footprint" "" (at 45.4152 98.425 0)
-      (effects (font (size 1.27 1.27)) hide)
-    )
+    (property "Footprint" "Capacitor_SMD:C_0805_2012Metric" (at 45.4152 98.425 0)
+      (effects (font (size 1.27 1.27)) hide)
+    )

Commit message: added SPI terminating resistors
Other:
- moved on the sheet: D1, R5
Changed lines of the file:
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@@
 (kicad_sch (version 20230121) (generator eeschema)
   (paper "A4")
-  (junction (at 184.15 88.9) (diameter 0) (color 0 0 0 0)
+  (junction (at 166.37 86.995) (diameter 0) (color 0 0 0 0)
   )
   (junction (at 53.975 98.425) (diameter 0) (color 0 0 0 0)
@@
     (stroke (width 0) (type default))
   )
-  (wire (pts (xy 186.69 88.9) (xy 184.15 88.9))
-    (stroke (width 0) (type default))
-  )
-  (wire (pts (xy 184.15 86.36) (xy 184.15 88.9))
+  (wire (pts (xy 168.91 86.995) (xy 166.37 86.995))
+    (stroke (width 0) (type default))
+  )
+  (wire (pts (xy 166.37 84.455) (xy 166.37 86.995))
     (stroke (width 0) (type default))
   )
@@
     (stroke (width 0) (type default))
   )
-  (wire (pts (xy 184.15 88.9) (xy 184.15 91.44))
+  (wire (pts (xy 166.37 86.995) (xy 166.37 89.535))
     (stroke (width 0) (type default))
   )
@@
     (stroke (width 0) (type default))
   )
-  (wire (pts (xy 184.15 100.33) (xy 184.15 99.06))
-    (stroke (width 0) (type default))
-  )
-  (wire (pts (xy 184.15 109.22) (xy 184.15 107.95))
+  (wire (pts (xy 166.37 98.425) (xy 166.37 97.155))
+    (stroke (width 0) (type default))
+  )
+  (wire (pts (xy 166.37 107.315) (xy 166.37 106.045))
     (stroke (width 0) (type default))
   )
@@
     )
   )
-  (symbol (lib_id "power:+5V") (at 184.15 86.36 0) (unit 1)
-    (in_bom yes) (on_board yes) (dnp no)
-    (property "Reference" "#PWR0126" (at 184.15 90.17 0)
-      (effects (font (size 1.27 1.27)) hide)
-    )
-    (property "Value" "+5V" (at 184.531 81.9658 0)
+  (symbol (lib_id "power:+5V") (at 166.37 84.455 0) (unit 1)
+    (in_bom yes) (on_board yes) (dnp no)
+    (property "Reference" "#PWR0126" (at 166.37 88.265 0)
+      (effects (font (size 1.27 1.27)) hide)
+    )
+    (property "Value" "+5V" (at 166.751 80.0608 0)
       (effects (font (size 1.27 1.27)))
     )
-    (property "Footprint" "" (at 184.15 86.36 0)
-      (effects (font (size 1.27 1.27)) hide)
-    )
-    (property "Datasheet" "" (at 184.15 86.36 0)
+    (property "Footprint" "" (at 166.37 84.455 0)
+      (effects (font (size 1.27 1.27)) hide)
+    )
+    (property "Datasheet" "" (at 166.37 84.455 0)
       (effects (font (size 1.27 1.27)) hide)
     )
@@
     )
   )
-  (symbol (lib_id "Device:R") (at 184.15 95.25 0) (unit 1)
-    (in_bom yes) (on_board yes) (dnp no)
-    (property "Reference" "R5" (at 185.928 94.0816 0)
-      (effects (font (size 1.27 1.27)) (justify left))
-    )
-    (property "Value" "1.5k" (at 185.928 96.393 0)
-      (effects (font (size 1.27 1.27)) (justify left))
-    )
-    (property "Footprint" "Resistor_SMD:R_0805_2012Metric" (at 182.372 95.25 90)
-      (effects (font (size 1.27 1.27)) hide)
-    )
-    (property "Datasheet" "https://www.mouser.com/datasheet/2/427/dcrcwe3-1762152.pdf" (at 184.15 95.25 0)
-      (effects (font (size 1.27 1.27)) hide)
-    )
-    (property "P/N" "CRCW080521K5FKEA" (at 184.15 95.25 0)
+  (symbol (lib_id "Device:R") (at 166.37 93.345 0) (unit 1)
+    (in_bom yes) (on_board yes) (dnp no)
+    (property "Reference" "R5" (at 168.148 92.1766 0)
+      (effects (font (size 1.27 1.27)) (justify left))
+    )
+    (property "Value" "1.5k" (at 168.148 94.488 0)
+      (effects (font (size 1.27 1.27)) (justify left))
+    )
+    (property "Footprint" "Resistor_SMD:R_0805_2012Metric" (at 164.592 93.345 90)
+      (effects (font (size 1.27 1.27)) hide)
+    )
+    (property "Datasheet" "https://www.mouser.com/datasheet/2/427/dcrcwe3-1762152.pdf" (at 166.37 93.345 0)
+      (effects (font (size 1.27 1.27)) hide)
+    )
+    (property "P/N" "CRCW080521K5FKEA" (at 166.37 93.345 0)
       (effects (font (size 1.27 1.27)) hide)
     )
@@
     )
   )
-  (symbol (lib_id "power:GND") (at 184.15 109.22 0) (unit 1)
-    (in_bom yes) (on_board yes) (dnp no)
-    (property "Reference" "#PWR0125" (at 184.15 115.57 0)
-      (effects (font (size 1.27 1.27)) hide)
-    )
-    (property "Value" "GND" (at 184.277 113.6142 0)
+  (symbol (lib_id "power:GND") (at 166.37 107.315 0) (unit 1)
+    (in_bom yes) (on_board yes) (dnp no)
+    (property "Reference" "#PWR0125" (at 166.37 113.665 0)
+      (effects (font (size 1.27 1.27)) hide)
+    )
+    (property "Value" "GND" (at 166.497 111.7092 0)
       (effects (font (size 1.27 1.27)))
     )
-    (property "Footprint" "" (at 184.15 109.22 0)
-      (effects (font (size 1.27 1.27)) hide)
-    )
-    (property "Datasheet" "" (at 184.15 109.22 0)
+    (property "Footprint" "" (at 166.37 107.315 0)
+      (effects (font (size 1.27 1.27)) hide)
+    )
+    (property "Datasheet" "" (at 166.37 107.315 0)
       (effects (font (size 1.27 1.27)) hide)
     )
@@
     )
   )
-  (symbol (lib_id "Device:LED") (at 184.15 104.14 90) (unit 1)
-    (in_bom yes) (on_board yes) (dnp no)
-    (property "Reference" "D1" (at 187.1472 103.1748 90)
-      (effects (font (size 1.27 1.27)) (justify right))
-    )
-    (property "Value" "PowerLED" (at 187.1472 105.4862 90)
-      (effects (font (size 1.27 1.27)) (justify right))
-    )
-    (property "Footprint" "LED_SMD:LED_0805_2012Metric" (at 184.15 104.14 0)
-      (effects (font (size 1.27 1.27)) hide)
-    )
-    (property "Datasheet" "https://www.mouser.com/datasheet/2/216/APTD2012LCGCK-1102037.pdf" (at 184.15 104.14 0)
-      (effects (font (size 1.27 1.27)) hide)
-    )
-    (property "Color" "Green" (at 184.15 104.14 90)
-      (effects (font (size 1.27 1.27)) hide)
-    )
-    (property "P/N" "APTD2012LCGCK" (at 184.15 104.14 90)
-      (effects (font (size 1.27 1.27)) hide)
-    )
-    (property "Vf" "1.9V" (at 184.15 104.14 90)
-      (effects (font (size 1.27 1.27)) hide)
-    )
-    (property "If" "2mA" (at 184.15 104.14 90)
+  (symbol (lib_id "Device:LED") (at 166.37 102.235 90) (unit 1)
+    (in_bom yes) (on_board yes) (dnp no)
+    (property "Reference" "D1" (at 169.3672 101.2698 90)
+      (effects (font (size 1.27 1.27)) (justify right))
+    )
+    (property "Value" "PowerLED" (at 169.3672 103.5812 90)
+      (effects (font (size 1.27 1.27)) (justify right))
+    )
+    (property "Footprint" "LED_SMD:LED_0805_2012Metric" (at 166.37 102.235 0)
+      (effects (font (size 1.27 1.27)) hide)
+    )
+    (property "Datasheet" "https://www.mouser.com/datasheet/2/216/APTD2012LCGCK-1102037.pdf" (at 166.37 102.235 0)
+      (effects (font (size 1.27 1.27)) hide)
+    )
+    (property "Color" "Green" (at 166.37 102.235 90)
+      (effects (font (size 1.27 1.27)) hide)
+    )
+    (property "P/N" "APTD2012LCGCK" (at 166.37 102.235 90)
+      (effects (font (size 1.27 1.27)) hide)
+    )
+    (property "Vf" "1.9V" (at 166.37 102.235 90)
+      (effects (font (size 1.27 1.27)) hide)
+    )
+    (property "If" "2mA" (at 166.37 102.235 90)
       (effects (font (size 1.27 1.27)) hide)
     )
@@
     )
   )
-  (symbol (lib_id "power:PWR_FLAG") (at 186.69 88.9 270) (unit 1)
-    (in_bom yes) (on_board yes) (dnp no)
-    (property "Reference" "#FLG0103" (at 188.595 88.9 0)
-      (effects (font (size 1.27 1.27)) hide)
-    )
-    (property "Value" "PWR_FLAG" (at 189.9412 88.9 90)
-      (effects (font (size 1.27 1.27)) (justify left))
-    )
-    (property "Footprint" "" (at 186.69 88.9 0)
-      (effects (font (size 1.27 1.27)) hide)
-    )
-    (property "Datasheet" "~" (at 186.69 88.9 0)
-      (effects (font (size 1.27 1.27)) hide)
-    )
+  (symbol (lib_id "power:PWR_FLAG") (at 168.91 86.995 270) (unit 1)
+    (in_bom yes) (on_board yes) (dnp no)
+    (property "Reference" "#FLG0103" (at 170.815 86.995 0)
+      (effects (font (size 1.27 1.27)) hide)
+    )
+    (property "Value" "PWR_FLAG" (at 172.1612 86.995 90)
+      (effects (font (size 1.27 1.27)) (justify left))
+    )
+    (property "Footprint" "" (at 168.91 86.995 0)
+      (effects (font (size 1.27 1.27)) hide)
+    )
+    (property "Datasheet" "~" (at 168.91 86.995 0)
+      (effects (font (size 1.27 1.27)) hide)
+    )

Commit message: add 3.3v tvs diode
Parts:
- R16: value 680 -> 1k
- R17, R18, R19: value 750 -> 1k
Changed lines of the file:
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@@
       (effects (font (size 1.27 1.27)) (justify left))
     )
-    (property "Value" "750" (at 107.188 105.918 0)
+    (property "Value" "1k" (at 107.188 105.918 0)
       (effects (font (size 1.27 1.27)) (justify left))
     )
@@
       (effects (font (size 1.27 1.27)) (justify left))
     )
-    (property "Value" "680" (at 86.868 105.918 0)
+    (property "Value" "1k" (at 86.868 105.918 0)
       (effects (font (size 1.27 1.27)) (justify left))
     )
@@
       (effects (font (size 1.27 1.27)) (justify left))
     )
-    (property "Value" "750" (at 119.888 105.918 0)
+    (property "Value" "1k" (at 119.888 105.918 0)
       (effects (font (size 1.27 1.27)) (justify left))
     )
@@
       (effects (font (size 1.27 1.27)) (justify left))
     )
-    (property "Value" "750" (at 132.588 105.918 0)
-      (effects (font (size 1.27 1.27)) (justify left))
-    )
+    (property "Value" "1k" (at 132.588 105.918 0)
+      (effects (font (size 1.27 1.27)) (justify left))
+    )

Commit message: Updated PCB from schematic + assigned push button footprint
Parts:
- SW7: footprint UTSVT_Special:SW_SPST_B3SL-1002P -> Button_Switch_SMD:SW_SPST_B3SL-1002P
Changed lines of the file:
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@@
       (effects (font (size 1.27 1.27)) (justify right))
     )
-    (property "Footprint" "UTSVT_Special:SW_SPST_B3SL-1002P" (at 67.945 105.41 0)
+    (property "Footprint" "Button_Switch_SMD:SW_SPST_B3SL-1002P" (at 67.945 105.41 0)
       (effects (font (size 1.27 1.27)) hide)
     )

Commit message: switch datasheet
Parts:
- removed SW2: SW_SPST, symbol Switch:SW_SPST
- added SW4: SW_SPDT, symbol Switch:SW_SPDT
Connections:
- net GND: now also SW4.3 (C)
- net at C55.2, R13.2: now also SW4.2 (B)
Other:
- moved on the sheet: C55, D1, D11, D6, D7, D9, R13, R16, R17, R18, R19, R5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
