File: Leds.kicad_sch (KiCad schematic)
At the start: 16 parts, among them SW4 SW_SPDT, SW7 SW_Push

Commit message: ready for PCB layout
Parts:
- R5: value 1.5k -> 1k
- SW4: footprint (none) -> UTSVT_Mechanical:CJS-1200B_NDC
Connections:
- no-connect marks 0 -> 1
Changed lines of the file:
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@@
   (junction (at 121.285 111.76) (diameter 0) (color 0 0 0 0)
   )
+  (no_connect (at 80.01 106.68))
   (bus_entry (at 88.9 83.82) (size 2.54 -2.54)
     (stroke (width 0) (type default))
@@
       (effects (font (size 1.27 1.27)))
     )
-    (property "Footprint" "" (at 74.93 109.22 0)
+    (property "Footprint" "UTSVT_Mechanical:CJS-1200B_NDC" (at 74.93 109.22 0)
       (effects (font (size 1.27 1.27)) hide)
     )
@@
       (effects (font (size 1.27 1.27)) (justify left))
     )
-    (property "Value" "1.5k" (at 184.023 95.123 0)
-      (effects (font (size 1.27 1.27)) (justify left))
-    )
+    (property "Value" "1k" (at 184.023 95.123 0)
+      (effects (font (size 1.27 1.27)) (justify left))
+    )

Commit message: 40mm layout
Connections:
- net GND: now also D11.1 (K), D6.1 (K), D7.1 (K), D9.1 (K); no longer R16.2, R17.2, R18.2, R19.2
- net PB0: now also R19.1; no longer D9.2 (A)
- net PB1: now also R18.1; no longer D7.2 (A)
- net PB2: now also R17.1; no longer D6.2 (A)
- net PB3: now also R16.1; no longer D11.2 (A)
- new net: D7.2 (A), R18.2
- new net: D9.2 (A), R19.2
- new net: D11.2 (A), R16.2
- new net: D6.2 (A), R17.2
Other:
- moved on the sheet: D11, D6, D7, D9, R16, R17, R18, R19

Commit message: Added Matthew's suggested changes
Parts:
- removed D1: PowerLED, LED_SMD:LED_0805_2012Metric, symbol Device:LED
- removed R5: 1k, Resistor_SMD:R_0805_2012Metric, symbol Device:R
Changed lines of the file:
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@@
   (junction (at 121.92 111.76) (diameter 0) (color 0 0 0 0)
-  )
-  (junction (at 182.245 87.63) (diameter 0) (color 0 0 0 0)
   )
   (junction (at 69.85 91.44) (diameter 0) (color 0 0 0 0)
@@
     (stroke (width 0) (type default))
   )
-  (wire (pts (xy 184.785 87.63) (xy 182.245 87.63))
-    (stroke (width 0) (type default))
-  )
-  (wire (pts (xy 182.245 85.09) (xy 182.245 87.63))
-    (stroke (width 0) (type default))
-  )
   (wire (pts (xy 88.9 111.76) (xy 95.25 111.76))
     (stroke (width 0) (type default))
   )
-  (wire (pts (xy 182.245 87.63) (xy 182.245 90.17))
-    (stroke (width 0) (type default))
-  )
   (wire (pts (xy 88.9 111.125) (xy 88.9 111.76))
     (stroke (width 0) (type default))
@@
   )
   (wire (pts (xy 121.92 100.33) (xy 121.92 101.6))
-    (stroke (width 0) (type default))
-  )
-  (wire (pts (xy 182.245 99.06) (xy 182.245 97.79))
-    (stroke (width 0) (type default))
-  )
-  (wire (pts (xy 182.245 107.95) (xy 182.245 106.68))
     (stroke (width 0) (type default))
   )
@@
         (path "/d5ebd247-5a7c-47c2-8aee-beabaef72d6d/40e00f49-8295-4a27-8e00-c31cad3b7d6c"
           (reference "D9") (unit 1)
-        )
-      )
-    )
-  )
-  (symbol (lib_id "power:+5V") (at 182.245 85.09 0) (unit 1)
-    (in_bom yes) (on_board yes) (dnp no)
-    (property "Reference" "#PWR0126" (at 182.245 88.9 0)
-      (effects (font (size 1.27 1.27)) hide)
-    )
-    (property "Value" "+5V" (at 182.626 80.6958 0)
-      (effects (font (size 1.27 1.27)))
-    )
-    (property "Footprint" "" (at 182.245 85.09 0)
-      (effects (font (size 1.27 1.27)) hide)
-    )
-    (property "Datasheet" "" (at 182.245 85.09 0)
-      (effects (font (size 1.27 1.27)) hide)
-    )
-    (pin "1")
-    (instances
-      (project "Telemetry-Primary"
-        (path "/7f2a449b-14af-42b3-8d38-5f0f8a5ee7ce/00000000-0000-0000-0000-00005f6cdfd6"
-          (reference "#PWR0126") (unit 1)
-        )
-      )
-      (project "BPS-PeripheralSOM"
-        (path "/d5ebd247-5a7c-47c2-8aee-beabaef72d6d/40e00f49-8295-4a27-8e00-c31cad3b7d6c"
-          (reference "#PWR030") (unit 1)
         )
       )
@@
     )
   )
-  (symbol (lib_id "Device:R") (at 182.245 93.98 0) (unit 1)
-    (in_bom yes) (on_board yes) (dnp no)
-    (property "Reference" "R5" (at 184.023 92.8116 0)
-      (effects (font (size 1.27 1.27)) (justify left))
-    )
-    (property "Value" "1k" (at 184.023 95.123 0)
-      (effects (font (size 1.27 1.27)) (justify left))
-    )
-    (property "Footprint" "Resistor_SMD:R_0805_2012Metric" (at 180.467 93.98 90)
-      (effects (font (size 1.27 1.27)) hide)
-    )
-    (property "Datasheet" "~" (at 182.245 93.98 0)
-      (effects (font (size 1.27 1.27)) hide)
-    )
-    (property "P/N" "CRCW080521K5FKEA" (at 182.245 93.98 0)
-      (effects (font (size 1.27 1.27)) hide)
-    )
-    (pin "1")
-    (pin "2")
-    (instances
-      (project "Telemetry-Primary"
-        (path "/7f2a449b-14af-42b3-8d38-5f0f8a5ee7ce/00000000-0000-0000-0000-00005f6cdfd6"
-          (reference "R5") (unit 1)
-        )
-      )
-      (project "BPS-PeripheralSOM"
-        (path "/d5ebd247-5a7c-47c2-8aee-beabaef72d6d/40e00f49-8295-4a27-8e00-c31cad3b7d6c"
-          (reference "R12") (unit 1)
-        )
-      )
-    )
-  )
   (symbol (lib_id "Device:R") (at 101.6 96.52 0) (unit 1)
     (in_bom yes) (on_board yes) (dnp no)
@@
     )
   )
-  (symbol (lib_id "power:GND") (at 182.245 107.95 0) (unit 1)
-    (in_bom yes) (on_board yes) (dnp no)
-    (property "Reference" "#PWR0125" (at 182.245 114.3 0)
-      (effects (font (size 1.27 1.27)) hide)
-    )
-    (property "Value" "GND" (at 182.372 112.3442 0)
-      (effects (font (size 1.27 1.27)))
-    )
-    (property "Footprint" "" (at 182.245 107.95 0)
-      (effects (font (size 1.27 1.27)) hide)
-    )
-    (property "Datasheet" "" (at 182.245 107.95 0)
-      (effects (font (size 1.27 1.27)) hide)
-    )
-    (pin "1")
-    (instances
-      (project "Telemetry-Primary"
-        (path "/7f2a449b-14af-42b3-8d38-5f0f8a5ee7ce/00000000-0000-0000-0000-00005f6cdfd6"
-          (reference "#PWR0125") (unit 1)
-        )
-      )
-      (project "BPS-PeripheralSOM"
-        (path "/d5ebd247-5a7c-47c2-8aee-beabaef72d6d/40e00f49-8295-4a27-8e00-c31cad3b7d6c"
-          (reference "#PWR040") (unit 1)
-        )
-      )
-    )
-  )
   (symbol (lib_id "Device:R") (at 134.62 96.52 0) (unit 1)
     (in_bom yes) (on_board yes) (dnp no)
@@
         (path "/f7d7e637-f98b-407c-b73b-57d398ad2f71/00000000-0000-0000-0000-00005c392c6a"
           (reference "R10") (unit 1)
-        )
-      )
-    )
-  )
-  (symbol (lib_id "Device:LED") (at 182.245 102.87 90) (unit 1)
-    (in_bom yes) (on_board yes) (dnp no)
-    (property "Reference" "D1" (at 185.2422 101.9048 90)
-      (effects (font (size 1.27 1.27)) (justify right))
-    )
-    (property "Value" "PowerLED" (at 185.2422 104.2162 90)
-      (effects (font (size 1.27 1.27)) (justify right))
-    )
-    (property "Footprint" "LED_SMD:LED_0805_2012Metric" (at 182.245 102.87 0)
-      (effects (font (size 1.27 1.27)) hide)
-    )
-    (property "Datasheet" "~" (at 182.245 102.87 0)
-      (effects (font (size 1.27 1.27)) hide)
-    )
-    (property "Color" "Green" (at 182.245 102.87 90)
-      (effects (font (size 1.27 1.27)) hide)
-    )
-    (property "P/N" "APTD2012LCGCK" (at 182.245 102.87 90)
-      (effects (font (size 1.27 1.27)) hide)
-    )
-    (property "Vf" "1.9V" (at 182.245 102.87 90)
-      (effects (font (size 1.27 1.27)) hide)
-    )
-    (property "If" "2mA" (at 182.245 102.87 90)
-      (effects (font (size 1.27 1.27)) hide)
-    )
-    (pin "1")
-    (pin "2")
-    (instances
-      (project "Telemetry-Primary"
-        (path "/7f2a449b-14af-42b3-8d38-5f0f8a5ee7ce/00000000-0000-0000-0000-00005f6cdfd6"
-          (reference "D1") (unit 1)
-        )
-      )
-      (project "BPS-PeripheralSOM"
-        (path "/d5ebd247-5a7c-47c2-8aee-beabaef72d6d/40e00f49-8295-4a27-8e00-c31cad3b7d6c"
-          (reference "D10") (unit 1)
         )
       )
@@
         )
       )
-    )
-  )
-  (symbol (lib_id "power:PWR_FLAG") (at 184.785 87.63 270) (unit 1)
-    (in_bom yes) (on_board yes) (dnp no)
-    (property "Reference" "#FLG0103" (at 186.69 87.63 0)
-      (effects (font (size 1.27 1.27)) hide)
-    )
-    (property "Value" "PWR_FLAG" (at 188.0362 87.63 90)
-      (effects (font (size 1.27 1.27)) (justify left))
-    )
-    (property "Footprint" "" (at 184.785 87.63 0)
-      (effects (font (size 1.27 1.27)) hide)
-    )
-    (property "Datasheet" "~" (at 184.785 87.63 0)
-      (effects (font (size 1.27 1.27)) hide)
-    )
-    (pin "1")
-    (instances
-      (project "Telemetry-Primary"
-        (path "/7f2a449b-14af-42b3-8d38-5f0f8a5ee7ce/00000000-0000-0000-0000-00005f6cdfd6"
-          (reference "#FLG0103") (unit 1)
-        )
-      )
-      (project "BPS-PeripheralSOM"
-        (path "/d5ebd247-5a7c-47c2-8aee-beabaef72d6d/40e00f49-8295-4a27-8e00-c31cad3b7d6c"
-          (reference "#FLG06") (unit 1)
-        )
-      )

Commit message: changed pins around to make routing easier
Parts:
- removed C55 (x2): 10nF, Capacitor_SMD:C_0805_2012Metric, symbol Device:C
- removed D11: Heartbeat, LED_SMD:LED_0805_2012Metric, symbol Device:LED
- removed D6, D7, D9: LED, LED_SMD:LED_0805_2012Metric, symbol Device:LED
- removed R13, R6: 220, Resistor_SMD:R_0805_2012Metric, symbol Device:R
- removed R16, R17, R18, R19: 1k, Resistor_SMD:R_0805_2012Metric, symbol Device:R
- removed SW4: SW_SPDT, UTSVT_Mechanical:CJS-1200B_NDC, symbol Switch:SW_SPDT
- added C55 (x2): 10nF, Capacitor_SMD:C_0805_2012Metric, symbol Device:C
- added D12, D13, D14: LED, LED_SMD:LED_0805_2012Metric, symbol Device:LED
- added D4: Heartbeat, LED_SMD:LED_0805_2012Metric, symbol Device:LED
- added R11, R23, R24, R25: 1k, Resistor_SMD:R_0805_2012Metric, symbol Device:R
- added R12, R22: 220, Resistor_SMD:R_0805_2012Metric, symbol Device:R
- added SW2: SW_SPDT, UTSVT_Mechanical:CJS-1200B_NDC, symbol Switch:SW_SPDT
Connections:
- net GND: now also D12.1 (K), D13.1 (K), D14.1 (K), D4.1 (K), SW2.3 (C)
- net PB3: now also R25.1
- net PB4: now also R24.1
- net PB5: now also R23.1
- net at SW7.2: now also C55.2, R22.2
- new net: D4.2 (A), R11.2
- new net: D13.2 (A), R24.2
- new net: D12.2 (A), R23.2
- new net: C55.2, R12.2, SW2.2 (B)
- new net: D14.2 (A), R25.2
- new net PA1: C55.1, R22.1
- new net PA15: R11.1
- new net PA2: C55.1, R12.1
Other:
- note added: "Generic LED Pins: PB3-5 Heartbeat LED: PA15"

Commit message: Prelim layout v2 final draft (ahhhhhhhhh), also connected GPIO to STDBY and SILENT pins
Connections:
- net PA2 renamed PC13
Changed lines of the file:
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@@
     (effects (font (size 1.27 1.27)) (justify left))
   )
-  (hierarchical_label "PA2" (shape input) (at 86.995 99.06 90) (fields_autoplaced)
+  (hierarchical_label "PC13" (shape input) (at 86.995 99.06 90) (fields_autoplaced)
     (effects (font (size 1.27 1.27)) (justify left))
   )

Commit message: added Tianda's suggestions
Connections:
- net PC13 renamed PA2
Changed lines of the file:
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@@
     (effects (font (size 1.27 1.27)) (justify left))
   )
-  (hierarchical_label "PC13" (shape input) (at 86.995 99.06 90) (fields_autoplaced)
+  (hierarchical_label "PA2" (shape input) (at 86.995 99.06 90) (fields_autoplaced)
     (effects (font (size 1.27 1.27)) (justify left))
   )
