File: Leds.kicad_sch (KiCad schematic)
At the start: 8 parts

Commit message: FUCK capacitors
Parts:
- D12: value LED -> LED3; P/N APTD2012LCGCK -> APTD2012LVBC/D
- D13: value LED -> LED2; P/N APTD2012LCGCK -> APTD2012LVBC/D
- D14: value LED -> LED1; P/N APTD2012LCGCK -> APTD2012LVBC/D
- D4: P/N APTD2012LCGCK -> APTD2012LVBC/D
Changed lines of the file:
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@@
 			)
 		)
-		(property "Datasheet" "~"
+		(property "Datasheet" "https://www.kingbrightusa.com/images/catalog/SPEC/APTD2012LVBC-D.pdf"
 			(at 72.39 45.72 0)
 			(effects
@@
 			)
 		)
-		(property "P/N" "APTD2012LCGCK"
+		(property "P/N" "APTD2012LVBC/D"
 			(at 72.39 45.72 90)
 			(effects
@@
 		)
 		(property "Mouser Part Number" "604-APTD2012LCGCK"
+			(at 72.39 45.72 0)
+			(effects
+				(font
+					(size 1.27 1.27)
+				)
+				(hide yes)
+			)
+		)
+		(property "Sim.Pins" "1=K 2=A"
 			(at 72.39 45.72 0)
 			(effects
@@
 	)
 	(symbol
+		(lib_name "LED_2")
 		(lib_id "Device:LED")
 		(at 38.1 45.72 90)
@@
 		(fields_autoplaced yes)
 		(property "Reference" "D13"
-			(at 41.91 46.6725 90)
+			(at 41.91 46.0374 90)
 			(effects
 				(font
@@
 			)
 		)
-		(property "Value" "LED"
-			(at 41.91 49.2125 90)
+		(property "Value" "LED2"
+			(at 41.91 48.5774 90)
 			(effects
 				(font
@@
 			)
 		)
-		(property "Datasheet" "~"
+		(property "Datasheet" "https://www.kingbrightusa.com/images/catalog/SPEC/APTD2012LVBC-D.pdf"
 			(at 38.1 45.72 0)
 			(effects
@@
 			)
 		)
-		(property "P/N" "APTD2012LCGCK"
+		(property "P/N" "APTD2012LVBC/D"
+			(at 38.1 45.72 0)
+			(effects
+				(font
+					(size 1.27 1.27)
+				)
+				(hide yes)
+			)
+		)
+		(property "Sim.Pins" "1=K 2=A"
 			(at 38.1 45.72 0)
 			(effects
@@
 	)
 	(symbol
+		(lib_name "LED_3")
 		(lib_id "Device:LED")
 		(at 50.8 45.72 90)
@@
 		(fields_autoplaced yes)
 		(property "Reference" "D14"
-			(at 54.61 46.6725 90)
+			(at 54.61 46.0374 90)
 			(effects
 				(font
@@
 			)
 		)
-		(property "Value" "LED"
-			(at 54.61 49.2125 90)
+		(property "Value" "LED1"
+			(at 54.61 48.5774 90)
 			(effects
 				(font
@@
 			)
 		)
-		(property "Datasheet" "~"
+		(property "Datasheet" "https://www.kingbrightusa.com/images/catalog/SPEC/APTD2012LVBC-D.pdf"
 			(at 50.8 45.72 0)
 			(effects
@@
 			)
 		)
-		(property "P/N" "APTD2012LCGCK"
+		(property "P/N" "APTD2012LVBC/D"
+			(at 50.8 45.72 0)
+			(effects
+				(font
+					(size 1.27 1.27)
+				)
+				(hide yes)
+			)
+		)
+		(property "Sim.Pins" "1=K 2=A"
 			(at 50.8 45.72 0)
 			(effects
@@
 	)
 	(symbol
+		(lib_name "LED_1")
 		(lib_id "Device:LED")
 		(at 25.4 45.72 90)
@@
 		(fields_autoplaced yes)
 		(property "Reference" "D12"
-			(at 29.21 46.6725 90)
+			(at 29.21 46.0374 90)
 			(effects
 				(font
@@
 			)
 		)
-		(property "Value" "LED"
-			(at 29.21 49.2125 90)
+		(property "Value" "LED3"
+			(at 29.21 48.5774 90)
 			(effects
 				(font
@@
 			)
 		)
-		(property "Datasheet" "~"
+		(property "Datasheet" "https://www.kingbrightusa.com/images/catalog/SPEC/APTD2012LVBC-D.pdf"
 			(at 25.4 45.72 0)
 			(effects
@@
 			)
 		)
-		(property "P/N" "APTD2012LCGCK"
+		(property "P/N" "APTD2012LVBC/D"
 			(at 25.4 45.72 0)
 			(effects
+				(font
+					(size 1.27 1.27)
+				)
+				(hide yes)
+			)
+		)
+		(property "Sim.Pins" "1=K 2=A"
+			(at 25.4 45.72 0)
+			(effects

Commit message: all parts selected
Parts:
- R11, R17, R18, R6: P/N (none) -> CRCW0603120RFKEC
Changed lines of the file:
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@@
 			)
 		)
-		(property "P/N" ""
+		(property "P/N" "CRCW0603120RFKEC "
 			(at 50.8 36.83 0)
 			(effects
@@
 			)
 		)
-		(property "P/N" ""
+		(property "P/N" "CRCW0603120RFKEC "
 			(at 38.1 36.83 0)
 			(effects
@@
 			)
 		)
-		(property "P/N" ""
+		(property "P/N" "CRCW0603120RFKEC "
 			(at 25.4 36.83 0)
 			(effects
@@
 			)
 		)
-		(property "P/N" ""
+		(property "P/N" "CRCW0603120RFKEC "
 			(at 72.39 36.83 0)
 			(effects

Commit message: add some footprints
Parts:
- R11, R17, R18, R6: footprint (none) -> Resistor_SMD:R_0603_1608Metric_Pad0.98x0.95mm_HandSolder
Changed lines of the file:
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@@
 			)
 		)
-		(property "Footprint" ""
+		(property "Footprint" "Resistor_SMD:R_0603_1608Metric_Pad0.98x0.95mm_HandSolder"
 			(at 49.022 36.83 90)
 			(effects
@@
 			)
 		)
-		(property "Footprint" ""
+		(property "Footprint" "Resistor_SMD:R_0603_1608Metric_Pad0.98x0.95mm_HandSolder"
 			(at 36.322 36.83 90)
 			(effects
@@
 			)
 		)
-		(property "Footprint" ""
+		(property "Footprint" "Resistor_SMD:R_0603_1608Metric_Pad0.98x0.95mm_HandSolder"
 			(at 23.622 36.83 90)
 			(effects
@@
 			)
 		)
-		(property "Footprint" ""
+		(property "Footprint" "Resistor_SMD:R_0603_1608Metric_Pad0.98x0.95mm_HandSolder"
 			(at 70.612 36.83 90)
 			(effects

Commit message: all footprints assigned
Parts:
- D12, D13, D14, D4: footprint (none) -> LED_SMD:LED_0805_2012Metric_Pad1.15x1.40mm_HandSolder
Changed lines of the file:
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@@
 			)
 		)
-		(property "Footprint" ""
+		(property "Footprint" "LED_SMD:LED_0805_2012Metric_Pad1.15x1.40mm_HandSolder"
 			(at 72.39 45.72 0)
 			(effects
@@
 			)
 		)
-		(property "Footprint" ""
+		(property "Footprint" "LED_SMD:LED_0805_2012Metric_Pad1.15x1.40mm_HandSolder"
 			(at 38.1 45.72 0)
 			(effects
@@
 			)
 		)
-		(property "Footprint" ""
+		(property "Footprint" "LED_SMD:LED_0805_2012Metric_Pad1.15x1.40mm_HandSolder"
 			(at 50.8 45.72 0)
 			(effects
@@
 			)
 		)
-		(property "Footprint" ""
+		(property "Footprint" "LED_SMD:LED_0805_2012Metric_Pad1.15x1.40mm_HandSolder"
 			(at 25.4 45.72 0)
 			(effects

Commit message: address some stuff
Parts:
- D12, D13, D14, D4: Mouser Part Number 604-APTD2012LCGCK -> (none)
- R11, R17, R18, R6: Mouser Part Number Inventory -> (none)
Changed lines of the file:
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@@
-			)
-		)
-		(property "Mouser Part Number" "604-APTD2012LCGCK"
-			(at 72.39 45.72 0)
-			(effects
-				(font
-					(size 1.27 1.27)
-				)
-				(hide yes)
 			)
 		)
@@
 			)
 		)
-		(property "Mouser Part Number" "Inventory"
-			(at 50.8 36.83 0)
-			(effects
-				(font
-					(size 1.27 1.27)
-				)
-				(hide yes)
-			)
-		)
 		(property "P/N" "CRCW0603120RFKEC "
 			(at 50.8 36.83 0)
@@
 			)
 		)
-		(property "Mouser Part Number" "Inventory"
-			(at 38.1 36.83 0)
-			(effects
-				(font
-					(size 1.27 1.27)
-				)
-				(hide yes)
-			)
-		)
 		(property "P/N" "CRCW0603120RFKEC "
 			(at 38.1 36.83 0)
@@
 			)
 		)
-		(property "Mouser Part Number" "Inventory"
-			(at 25.4 36.83 0)
-			(effects
-				(font
-					(size 1.27 1.27)
-				)
-				(hide yes)
-			)
-		)
 		(property "P/N" "CRCW0603120RFKEC "
 			(at 25.4 36.83 0)
@@
 			)
 		)
-		(property "Mouser Part Number" "Inventory"
-			(at 72.39 36.83 0)
-			(effects
-				(font
-					(size 1.27 1.27)
-				)
-				(hide yes)
-			)
-		)
 		(property "P/N" "CRCW0603120RFKEC "
 			(at 72.39 36.83 0)
@@
 			)
 		)
-		(property "Mouser Part Number" "604-APTD2012LCGCK"
-			(at 38.1 45.72 0)
-			(effects
-				(font
-					(size 1.27 1.27)
-				)
-				(hide yes)
-			)
-		)
 		(property "P/N" "APTD2012LVBC/D"
 			(at 38.1 45.72 0)
@@
 			)
 		)
-		(property "Mouser Part Number" "604-APTD2012LCGCK"
-			(at 50.8 45.72 0)
-			(effects
-				(font
-					(size 1.27 1.27)
-				)
-				(hide yes)
-			)
-		)
 		(property "P/N" "APTD2012LVBC/D"
 			(at 50.8 45.72 0)
@@
 			(at 25.4 45.72 0)
 			(effects
-				(font
-					(size 1.27 1.27)
-				)
-				(hide yes)
-			)
-		)
-		(property "Mouser Part Number" "604-APTD2012LCGCK"
-			(at 25.4 45.72 0)
-			(effects

Commit message: WTF IS A SILKSCREEN OVERLAPPP
Parts:
- D12: value LED3 -> LED2
- D13: value LED2 -> LED1
- D14: value LED1 -> LED0
Changed lines of the file:
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@@
 			)
 		)
-		(property "Value" "LED2"
+		(property "Value" "LED1"
 			(at 41.91 48.5774 90)
 			(effects
@@
 			)
 		)
-		(property "Value" "LED1"
+		(property "Value" "LED0"
 			(at 54.61 48.5774 90)
 			(effects
@@
 			)
 		)
-		(property "Value" "LED3"
+		(property "Value" "LED2"
 			(at 29.21 48.5774 90)
 			(effects

Commit message: reroute uart, change leds to 0603
Parts:
- D12, D13, D14, D4: footprint LED_SMD:LED_0805_2012Metric_Pad1.15x1.40mm_HandSolder -> LED_SMD:LED_0603_1608Metric_Pad1.05x0.95mm_HandSolder
Changed lines of the file:
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@@
 			)
 		)
-		(property "Footprint" "LED_SMD:LED_0805_2012Metric_Pad1.15x1.40mm_HandSolder"
+		(property "Footprint" "LED_SMD:LED_0603_1608Metric_Pad1.05x0.95mm_HandSolder"
 			(at 72.39 45.72 0)
 			(effects
@@
 			)
 		)
-		(property "Footprint" "LED_SMD:LED_0805_2012Metric_Pad1.15x1.40mm_HandSolder"
+		(property "Footprint" "LED_SMD:LED_0603_1608Metric_Pad1.05x0.95mm_HandSolder"
 			(at 38.1 45.72 0)
 			(effects
@@
 			)
 		)
-		(property "Footprint" "LED_SMD:LED_0805_2012Metric_Pad1.15x1.40mm_HandSolder"
+		(property "Footprint" "LED_SMD:LED_0603_1608Metric_Pad1.05x0.95mm_HandSolder"
 			(at 50.8 45.72 0)
 			(effects
@@
 			)
 		)
-		(property "Footprint" "LED_SMD:LED_0805_2012Metric_Pad1.15x1.40mm_HandSolder"
+		(property "Footprint" "LED_SMD:LED_0603_1608Metric_Pad1.05x0.95mm_HandSolder"
 			(at 25.4 45.72 0)
 			(effects

Commit message: LED lcsc p/n
Parts:
- D12, D13, D14, D4: P/N APTD2012LVBC/D -> XL-1608UBC-06A
Changed lines of the file:
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@@
 			)
 		)
-		(property "P/N" "APTD2012LVBC/D"
+		(property "P/N" "XL-1608UBC-06A"
 			(at 72.39 45.72 90)
 			(effects
@@
 			)
 		)
-		(property "P/N" "APTD2012LVBC/D"
+		(property "P/N" "XL-1608UBC-06A"
 			(at 38.1 45.72 0)
 			(effects
@@
 			)
 		)
-		(property "P/N" "APTD2012LVBC/D"
+		(property "P/N" "XL-1608UBC-06A"
 			(at 50.8 45.72 0)
 			(effects
@@
 			)
 		)
-		(property "P/N" "APTD2012LVBC/D"
+		(property "P/N" "XL-1608UBC-06A"
 			(at 25.4 45.72 0)
 			(effects
