File: BPS-PeripheralSOM.kicad_pcb (KiCad board)
At the start: 2 copper layers, 83 parts, among them J1 SWD, J2 Can_In, J3 USB_B_Micro, J5 Conn_02x10_Counter_Clockwise, J6 CAN_OUT, Q1 Q_PMOS_GSD, SW1 Reset, SW3 SW_Push, U1 STM32L431CBTx, U2 ADM3055E, U3 CDSOT23-T24CAN, U4 CP2102N-A01-GQFN24, U5 NCP1117-3.3_SOT223, U6 RI3-1205S, Y1 8M

Commit message: ready for PCB layout
Parts:
- added SW4: SW_SPDT, UTSVT_Mechanical:CJS-1200B_NDC, F.Cu at (76.9, 102.5)
- J5: footprint UTSVT_Connectors:2039550203 -> UTSVT_Connectors:Molex_52465-2070
- R12: value 1.5k -> 1k
- moved C23 85.1 mm to (74.4, 107.3)
- moved C24 85.1 mm to (74.4, 110.3)
- moved C1 80.4 mm to (110.0, 43.4)
- moved C2 80.4 mm to (110.0, 46.4)
- moved C3 80.4 mm to (110.0, 49.4)
- moved C4 80.4 mm to (110.0, 52.4)
- moved C5 80.4 mm to (110.0, 55.4)
- moved C6 80.4 mm to (110.0, 58.4)
- moved C7 80.4 mm to (110.0, 61.5)
- moved C8 80.4 mm to (110.0, 64.5)
- moved J6 80.4 mm to (117.3, 45.5)
- moved L1 80.4 mm to (126.9, 60.6)
- moved L2 80.4 mm to (126.9, 63.4)
- moved R1 80.4 mm to (131.8, 50.6)
- moved R11 80.4 mm to (131.8, 53.6)
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
Commit message: Started layout
Parts:
- moved C14 118.4 mm to (217.0, 53.0), turned to -90 degrees
- moved C17 118.0 mm to (221.1, 53.0), turned to -90 degrees
- moved C15 114.2 mm to (213.0, 53.0), turned to -90 degrees
- moved C13 110.3 mm to (204.8, 53.0), turned to -90 degrees
- moved C16 110.1 mm to (209.0, 53.0), turned to -90 degrees
- moved D3 109.5 mm to (210.3, 31.9), turned to 180 degrees
- moved R7 105.0 mm to (223.0, 38.3)
- moved TP3 105.0 mm to (204.0, 23.1)
- moved TP4 105.0 mm to (204.0, 28.2)
- moved U6 105.0 mm to (212.8, 27.6)
- moved J2 103.4 mm to (162.3, 20.8)
- moved D8 95.2 mm to (208.8, 36.2), turned to -90 degrees
- moved U1 94.0 mm to (193.9, 77.9)
- moved C20 71.3 mm to (174.2, 26.7), turned to 180 degrees
- moved FB1 59.0 mm to (161.9, 25.7), turned to 90 degrees
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
Commit message: Seperated components in layout
Parts:
- moved J3 120.3 mm to (213.7, 86.4)
- moved C10 120.3 mm to (217.2, 95.1)
- moved C9 120.3 mm to (217.2, 92.0)
- moved D1 120.3 mm to (206.5, 94.5)
- moved U4 120.3 mm to (211.9, 93.7)
- moved R3 120.3 mm to (206.5, 84.9)
- moved R4 120.3 mm to (206.5, 87.8)
- moved R5 120.3 mm to (206.5, 90.8)
- moved C23 112.3 mm to (185.7, 122.4)
- moved C24 112.3 mm to (185.7, 125.4)
- moved D10 112.3 mm to (181.3, 116.6)
- moved D11 112.3 mm to (181.3, 119.6)
- moved D6 112.3 mm to (181.3, 107.5)
- moved D7 112.3 mm to (181.3, 110.5)
- moved D9 112.3 mm to (181.3, 113.5)
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
Commit message: USB routing
Parts:
- moved J5 151.4 mm to (231.6, 77.4), turned to 90 degrees
- moved J1 128.9 mm to (204.9, 68.5)
- moved J3 20.9 mm to (232.4, 95.6), turned to -90 degrees
- moved R5 18.5 mm to (223.9, 97.2)
- moved R3 15.5 mm to (216.2, 97.0), turned to -90 degrees
- moved D1 12.8 mm to (219.1, 97.0), turned to 180 degrees
- moved R4 11.8 mm to (213.9, 97.0), turned to -90 degrees
- moved C10 9.48 mm to (208.3, 91.9), turned to 180 degrees
- moved C9 7.52 mm to (210.5, 95.5), turned to 180 degrees
- moved U4 2.38 mm to (213.1, 91.6)

Commit message: STM32 peripheral routing + LED routing
Parts:
- R10, R9: moved to B.Cu
- moved CR1 136.9 mm to (202.8, 79.5)
- moved CR2 123.8 mm to (189.2, 92.0)
- moved Y1 111.4 mm to (177.7, 73.4), turned to 90 degrees
- moved R9 104.1 mm to (196.2, 79.3), turned to -90 degrees
- moved R10 101.0 mm to (193.2, 79.3), turned to -90 degrees
- moved R20 99.0 mm to (191.1, 86.3), turned to -90 degrees
- moved R15 96.0 mm to (188.0, 86.7), turned to -90 degrees
- moved C21 75.6 mm to (173.2, 75.4), turned to 180 degrees
- moved R2 75.2 mm to (167.2, 72.8)
- moved R8 75.2 mm to (167.2, 75.7)
- moved C22 73.0 mm to (173.1, 71.3), turned to 180 degrees
- moved LOGO2 61.0 mm to (33.7, 45.2)
- moved C24 58.0 mm to (185.6, 67.4), turned to 180 degrees
- moved SW4 56.2 mm to (178.9, 61.7), turned to 90 degrees
- moved R16 53.6 mm to (195.7, 66.1), turned to 90 degrees
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
Commit message: Started power routing (going to sleep :sob: )
Parts:
- moved U6 48.6 mm to (162.3, 23.2)
- moved C20 44.1 mm to (211.1, 47.1)
- moved FB1 44.1 mm to (198.8, 46.1)
- moved J2 44.1 mm to (199.2, 41.2)
- moved Q1 44.1 mm to (203.0, 47.6)
- moved U5 44.1 mm to (202.2, 55.0)
- moved C13 37.7 mm to (242.3, 48.9)
- moved C14 37.7 mm to (254.5, 48.9)
- moved C15 37.7 mm to (250.5, 48.9)
- moved C16 37.7 mm to (246.5, 48.8)
- moved C17 37.7 mm to (258.6, 48.9)
- moved C18 31.5 mm to (195.7, 57.5), turned to 180 degrees
- moved C19 28.6 mm to (195.7, 55.0), turned to 180 degrees
- moved TP6 22.4 mm to (194.8, 51.1)
- moved TP3 0.70 mm to (202.0, 22.0)
Changed lines of the file:
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@@
   )
   (footprint "Capacitor_SMD:C_0805_2012Metric" (layer "F.Cu")
-    (at 217.02 53.05 -90)
+    (at 254.52 48.9 -90)
     (descr "Capacitor SMD 0805 (2012 Metric), square (rectangular) end terminal, IPC_7351 nominal, (Body size source: IPC-SM-782 page 76, https://www.pcb-3d.com/wordpress/wp-content/uploads/ipc-sm-782a_amendment_1_and_2.pdf, https://docs.google.com/spreadsheets/d/1BsfQQcO9C6DZCsRaXUlFlo91Tg2WpOkGARC1WS5S8t0/edit?usp=sharing), generated with kicad-footprint-generator")
     (tags "capacitor")
@@
   )
   (footprint "Capacitor_SMD:C_0805_2012Metric" (layer "F.Cu")
-    (at 170.48 38.63)
+    (at 195.71 57.45 180)
     (descr "Capacitor SMD 0805 (2012 Metric), square (rectangular) end terminal, IPC_7351 nominal, (Body size source: IPC-SM-782 page 76, https://www.pcb-3d.com/wordpress/wp-content/uploads/ipc-sm-782a_amendment_1_and_2.pdf, https://docs.google.com/spreadsheets/d/1BsfQQcO9C6DZCsRaXUlFlo91Tg2WpOkGARC1WS5S8t0/edit?usp=sharing), generated with kicad-footprint-generator")
     (tags "capacitor")
@@
     (property "ki_keywords" "cap capacitor")
     (attr smd)
-    (fp_text reference "C18" (at 0 -1.68) (layer "F.SilkS")
+    (fp_text reference "C18" (at 3.22 0.06) (layer "F.SilkS")
         (effects (font (size 1 1) (thickness 0.15)))
     )
@@
     (fp_line (start 1 0.625) (end -1 0.625)
       (stroke (width 0.1) (type solid)) (layer "F.Fab"))
-    (pad "1" smd roundrect (at -0.95 0) (size 1 1.45) (layers "F.Cu" "F.Paste" "F.Mask") (roundrect_rratio 0.25)
+    (pad "1" smd roundrect (at -0.95 0 180) (size 1 1.45) (layers "F.Cu" "F.Paste" "F.Mask") (roundrect_rratio 0.25)
       (net 1 "+5V") (pintype "passive"))
-    (pad "2" smd roundrect (at 0.95 0) (size 1 1.45) (layers "F.Cu" "F.Paste" "F.Mask") (roundrect_rratio 0.25)
+    (pad "2" smd roundrect (at 0.95 0 180) (size 1 1.45) (layers "F.Cu" "F.Paste" "F.Mask") (roundrect_rratio 0.25)
       (net 2 "GND") (pintype "passive"))
     (model "${KICAD6_3DMODEL_DIR}/Capacitor_SMD.3dshapes/C_0805_2012Metric.wrl"
@@
   )
   (footprint "Package_TO_SOT_SMD:SOT-223-3_TabPin2" (layer "F.Cu")
-    (at 163.33 34.18)
+    (at 202.24 55.02)
     (descr "module CMS SOT223 4 pins")
     (tags "CMS SOT")
@@
   )
   (footprint "Inductor_SMD:L_0805_2012Metric" (layer "F.Cu")
-    (at 159.87 25.28 90)
+    (at 198.78 46.12 90)
     (descr "Inductor SMD 0805 (2012 Metric), square (rectangular) end terminal, IPC_7351 nominal, (Body size source: IPC-SM-782 page 80, https://www.pcb-3d.com/wordpress/wp-content/uploads/ipc-sm-782a_amendment_1_and_2.pdf), generated with kicad-footprint-generator")
     (tags "inductor")
@@
   )
   (footprint "Package_TO_SOT_SMD:SuperSOT-3" (layer "F.Cu")
-    (at 164.06 26.76)
+    (at 202.97 47.6)
     (descr "3-pin SuperSOT package https://www.fairchildsemi.com/package-drawings/MA/MA03B.pdf")
     (tags "SuperSOT-3 SSOT-3")
@@
   )
   (footprint "UTSVT_Passive:C_2220_5750Metric" (layer "F.Cu")
-    (at 172.19 26.3 180)
+    (at 211.1 47.14 180)
     (descr "Capacitor SMD 2220In_5750Metrix")
     (tags "Capacitor, 5750")
@@
   )
   (footprint "TestPoint:TestPoint_Keystone_5005-5009_Compact" (layer "F.Cu")
-    (at 201.92 22.73)
+    (at 201.98 22.03)
     (descr "Keystone Miniature THM Test Point 5005-5009, http://www.keyelco.com/product-pdf.cfm?p=1314")
     (tags "Through Hole Mount Test Points")
@@
   )
   (footprint "UTSVT_Connectors:Molex_MicroFit3.0_1x4xP3.00mm_PolarizingPeg_Vertical" (layer "F.Cu")
-    (at 160.29 20.37)
+    (at 199.2 41.21)
     (property "Sheetfile" "BPS-PeripheralSOM.kicad_sch")
     (property "Sheetname" "")
@@
   )
   (footprint "UTSVT_ICs:RI3_DC_Converter" (layer "F.Cu")
-    (at 210.77 27.24)
+    (at 162.31 23.24)
     (property "Sheetfile" "PowerDist.kicad_sch")
     (property "Sheetname" "PowerDist")
@@
   )
   (footprint "Capacitor_SMD:C_0805_2012Metric" (layer "F.Cu")
-    (at 209.04 52.99 -90)
+    (at 246.54 48.84 -90)
     (descr "Capacitor SMD 0805 (2012 Metric), square (rectangular) end terminal, IPC_7351 nominal, (Body size source: IPC-SM-782 page 76, https://www.pcb-3d.com/wordpress/wp-content/uploads/ipc-sm-782a_amendment_1_and_2.pdf, https://docs.google.com/spreadsheets/d/1BsfQQcO9C6DZCsRaXUlFlo91Tg2WpOkGARC1WS5S8t0/edit?usp=sharing), generated with kicad-footprint-generator")
     (tags "capacitor")
@@
   )
   (footprint "TestPoint:TestPoint_Keystone_5005-5009_Compact" (layer "F.Cu")
-    (at 185.79 30.63)
+    (at 194.8 51.14)
     (descr "Keystone Miniature THM Test Point 5005-5009, http://www.keyelco.com/product-pdf.cfm?p=1314")
     (tags "Through Hole Mount Test Points")
@@
   )
   (footprint "Capacitor_SMD:C_0805_2012Metric" (layer "F.Cu")
-    (at 170.48 41.64)
+    (at 195.73 55.03 180)
     (descr "Capacitor SMD 0805 (2012 Metric), square (rectangular) end terminal, IPC_7351 nominal, (Body size source: IPC-SM-782 page 76, https://www.pcb-3d.com/wordpress/wp-content/uploads/ipc-sm-782a_amendment_1_and_2.pdf, https://docs.google.com/spreadsheets/d/1BsfQQcO9C6DZCsRaXUlFlo91Tg2WpOkGARC1WS5S8t0/edit?usp=sharing), generated with kicad-footprint-generator")
     (tags "capacitor")
@@
     (property "ki_keywords" "cap capacitor")
     (attr smd)
-    (fp_text reference "C19" (at 0 -1.68) (layer "F.SilkS")
+    (fp_text reference "C19" (at 3.2 0.01) (layer "F.SilkS")
         (effects (font (size 1 1) (thickness 0.15)))
     )
@@
     (fp_line (start 1 0.625) (end -1 0.625)
       (stroke (width 0.1) (type solid)) (layer "F.Fab"))
-    (pad "1" smd roundrect (at -0.95 0) (size 1 1.45) (layers "F.Cu" "F.Paste" "F.Mask") (roundrect_rratio 0.25)
+    (pad "1" smd roundrect (at -0.95 0 180) (size 1 1.45) (layers "F.Cu" "F.Paste" "F.Mask") (roundrect_rratio 0.25)
       (net 3 "+3.3V") (pintype "passive"))
-    (pad "2" smd roundrect (at 0.95 0) (size 1 1.45) (layers "F.Cu" "F.Paste" "F.Mask") (roundrect_rratio 0.25)
+    (pad "2" smd roundrect (at 0.95 0 180) (size 1 1.45) (layers "F.Cu" "F.Paste" "F.Mask") (roundrect_rratio 0.25)
       (net 2 "GND") (pintype "passive"))
     (model "${KICAD6_3DMODEL_DIR}/Capacitor_SMD.3dshapes/C_0805_2012Metric.wrl"
@@
   )
   (footprint "Capacitor_SMD:C_0805_2012Metric" (layer "F.Cu")
-    (at 204.79 53.02 -90)
+    (at 242.29 48.87 -90)
     (descr "Capacitor SMD 0805 (2012 Metric), square (rectangular) end terminal, IPC_7351 nominal, (Body size source: IPC-SM-782 page 76, https://www.pcb-3d.com/wordpress/wp-content/uploads/ipc-sm-782a_amendment_1_and_2.pdf, https://docs.google.com/spreadsheets/d/1BsfQQcO9C6DZCsRaXUlFlo91Tg2WpOkGARC1WS5S8t0/edit?usp=sharing), generated with kicad-footprint-generator")
     (tags "capacitor")
@@
   )
   (footprint "Capacitor_SMD:C_0805_2012Metric" (layer "F.Cu")
-    (at 212.98 53.05 -90)
+    (at 250.48 48.9 -90)
     (descr "Capacitor SMD 0805 (2012 Metric), square (rectangular) end terminal, IPC_7351 nominal, (Body size source: IPC-SM-782 page 76, https://www.pcb-3d.com/wordpress/wp-content/uploads/ipc-sm-782a_amendment_1_and_2.pdf, https://docs.google.com/spreadsheets/d/1BsfQQcO9C6DZCsRaXUlFlo91Tg2WpOkGARC1WS5S8t0/edit?usp=sharing), generated with kicad-footprint-generator")
     (tags "capacitor")
@@
   )
   (footprint "Capacitor_SMD:C_0805_2012Metric" (layer "F.Cu")
-    (at 221.06 53.02 -90)
+    (at 258.56 48.87 -90)
     (descr "Capacitor SMD 0805 (2012 Metric), square (rectangular) end terminal, IPC_7351 nominal, (Body size source: IPC-SM-782 page 76, https://www.pcb-3d.com/wordpress/wp-content/uploads/ipc-sm-782a_amendment_1_and_2.pdf, https://docs.google.com/spreadsheets/d/1BsfQQcO9C6DZCsRaXUlFlo91Tg2WpOkGARC1WS5S8t0/edit?usp=sharing), generated with kicad-footprint-generator")
     (tags "capacitor")

Commit message: cleaned up layout now that i have sleep
Parts:
- J5: moved to B.Cu
- R10, R9: moved to F.Cu
- moved C11 88.9 mm to (176.0, 79.0), turned to 180 degrees
- moved R12 57.6 mm to (199.1, 60.7), turned to -90 degrees
- moved D10 57.1 mm to (196.1, 61.5)
- moved C20 26.8 mm to (234.3, 33.6)
- moved D3 26.8 mm to (231.4, 18.0)
- moved J2 26.8 mm to (222.4, 27.7)
- moved R7 26.8 mm to (244.1, 24.3)
- moved TP4 26.8 mm to (225.1, 14.3)
- moved D8 26.8 mm to (230.0, 22.3)
- moved FB1 26.8 mm to (222.0, 32.6)
- moved Q1 26.8 mm to (226.2, 34.1)
- moved TP6 26.8 mm to (218.0, 37.6)
- moved C12 22.4 mm to (114.6, 36.3)
- moved R9 10.9 mm to (204.2, 86.6), turned to 90 degrees
- moved R10 10.8 mm to (201.2, 86.5), turned to 90 degrees
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
Commit message: power layout + started can + cleaned up a little bit
Parts:
- moved J6 79.7 mm to (194.0, 47.7)
- moved U6 61.4 mm to (207.8, 64.5), turned to 180 degrees
- moved U2 57.4 mm to (168.5, 60.6)
- moved TP2 56.1 mm to (182.9, 47.8)
- moved TP1 54.3 mm to (178.3, 47.8)
- moved U3 53.4 mm to (179.6, 60.9)
- moved R7 49.4 mm to (209.8, 59.8), turned to -90 degrees
- moved D3 46.5 mm to (217.2, 62.2)
- moved TP6 45.7 mm to (173.5, 47.8)
- moved D8 41.0 mm to (213.6, 59.9), turned to 90 degrees
- moved TP3 40.6 mm to (233.4, 47.8)
- moved TP4 33.7 mm to (228.9, 47.8)
- moved R8 33.7 mm to (200.9, 75.2), turned to 180 degrees
- moved R2 32.0 mm to (199.3, 72.1), turned to 180 degrees
- moved C20 27.5 mm to (220.1, 57.1), turned to 0 degrees
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