File: BPS-PeripheralSOM.kicad_pcb (KiCad board)
At the start: 2 copper layers, 40 x 50 mm, 84 parts, among them J1 SWD, J2 CAN_In, J3 USB_B_Micro, J5 CAN_Out, J6 Conn_02x10_Counter_Clockwise, Q1 Q_PMOS_GSD, SW1 Reset, SW3 SW_Push, SW4 SW_SPDT, U1 STM32L431CBTx, U2 RI3-0505S, U3 LD1117-3.3_SOT223, U4 CP2102N-A01-GQFN24, U7 ADM3055E, U8 CDSOT23-T24CAN, Y1 8M

Commit message: Prelim layout v2 final draft (ahhhhhhhhh), also connected GPIO to STDBY and SILENT pins
Parts:
- removed C23, C24: 10nF, Capacitor_SMD:C_0805_2012Metric
- removed D11: Heartbeat, LED_SMD:LED_0805_2012Metric
- removed D6, D7, D9: LED, LED_SMD:LED_0805_2012Metric
- removed R13, R6: 220, Resistor_SMD:R_0805_2012Metric
- removed R16, R17, R18, R19: 1k, Resistor_SMD:R_0805_2012Metric
- removed SW3: SW_Push, Button_Switch_SMD:SW_SPST_B3SL-1002P
- removed SW4: SW_SPDT, UTSVT_Mechanical:CJS-1200B_NDC
- added C4: 10nF, Capacitor_SMD:C_0805_2012Metric, B.Cu at (138.0, 74.0)
- added C5: 10nF, Capacitor_SMD:C_0805_2012Metric, B.Cu at (127.6, 76.7)
- added D12: LED, LED_SMD:LED_0805_2012Metric, F.Cu at (113.0, 63.3)
- added D13: LED, LED_SMD:LED_0805_2012Metric, F.Cu at (113.0, 60.6)
- added D14: LED, LED_SMD:LED_0805_2012Metric, F.Cu at (113.0, 57.9)
- added D4: Heartbeat, LED_SMD:LED_0805_2012Metric, F.Cu at (113.0, 55.2)
- added R11: 1k, Resistor_SMD:R_0805_2012Metric, B.Cu at (114.7, 55.2)
- added R12: 220, Resistor_SMD:R_0805_2012Metric, B.Cu at (135.0, 74.0)
- added R22: 220, Resistor_SMD:R_0805_2012Metric, B.Cu at (122.6, 76.7)
- added R23: 1k, Resistor_SMD:R_0805_2012Metric, B.Cu at (114.7, 63.3)
- added R24: 1k, Resistor_SMD:R_0805_2012Metric, B.Cu at (114.6, 60.6)
- added R25: 1k, Resistor_SMD:R_0805_2012Metric, B.Cu at (114.7, 57.9)
- added SW2: SW_SPDT, UTSVT_Mechanical:CJS-1200B_NDC, F.Cu at (136.2, 74.1)
- added SW5: SW_Push, Button_Switch_SMD:SW_SPST_B3SL-1002P, F.Cu at (125.0, 78.0)
- C10, C14, C16, C17, C9, CR1, D1, R1, R15, R20, R3, R4, R5, U4: moved to B.Cu
- moved D2 114.1 mm to (113.0, 66.1)
- moved R1 112.0 mm to (115.0, 66.0)
- moved C10 100.7 mm to (124.0, 61.0), turned to -90 degrees
- moved C9 95.8 mm to (134.0, 48.0), turned to -90 degrees
- moved D1 90.4 mm to (131.0, 48.0), turned to 180 degrees
- moved R5 88.3 mm to (129.0, 52.0), turned to 180 degrees
- moved R21 83.1 mm to (119.0, 53.0), turned to 180 degrees
- moved R4 83.0 mm to (133.0, 53.0)
- moved R3 82.5 mm to (133.0, 51.0)
- moved C14 62.8 mm to (118.0, 65.0), turned to -90 degrees
- moved C17 62.4 mm to (118.0, 55.0), turned to 90 degrees
- moved R20 60.8 mm to (128.3, 60.7), turned to -90 degrees
- moved R15 58.5 mm to (130.3, 60.7), turned to -90 degrees
- moved C16 54.9 mm to (126.0, 55.0), turned to 90 degrees
- moved C13 53.7 mm to (128.0, 65.0), turned to 180 degrees
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Connections:
- U1 pad 11: unconnected-(U1-PA1-Pad11) -> /PA1
- U1 pad 18: /PB0 -> unconnected-(U1-PB0-Pad18)
- U1 pad 19: /PB1 -> unconnected-(U1-PB1-Pad19)
- U1 pad 2: unconnected-(U1-PC13-Pad2) -> /PC13
- U1 pad 20: /PB2 -> unconnected-(U1-PB2-Pad20)
- U1 pad 32: unconnected-(U1-PA11-Pad32) -> /SILENT
- U1 pad 33: unconnected-(U1-PA12-Pad33) -> /STDBY
- U1 pad 38: unconnected-(U1-PA15-Pad38) -> /PA15
- U7 pad 6: unconnected-(U7-SILENT-Pad6) -> /SILENT
- U7 pad 8: unconnected-(U7-STDBY-Pad8) -> /STDBY
Routing:
- net /SWCLK: track 0.00 -> 0.86 mm

Commit message: alligned components
Parts:
- C13: moved to B.Cu
- moved C14 11.1 mm to (129.0, 66.0), turned to 0 degrees
- moved TP6 3.07 mm to (137.0, 44.0)
- moved D3 3.00 mm to (114.0, 82.0), turned to 180 degrees
- moved R5 2.00 mm to (129.0, 54.0)
- moved C11 1.96 mm to (115.0, 69.0), turned to 180 degrees
- moved C13 1.41 mm to (129.0, 64.0), turned to 0 degrees
- moved Q1 1.41 mm to (112.0, 85.0)
- moved C5 1.30 mm to (127.6, 78.0)
- moved R22 1.30 mm to (122.6, 78.0)
- moved C15 1.13 mm to (132.0, 78.5)
- moved C12 1.06 mm to (138.0, 78.5)
- moved C10 1.00 mm to (124.0, 60.0)
- moved FB1 1.00 mm to (135.0, 83.0)
- moved FB4 1.00 mm to (138.0, 83.0)
- moved J1 1.00 mm to (137.0, 48.9)
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
Commit message: redo layout again >>:(
Parts:
- C2, C3, CR1: moved to F.Cu
- R21, U3: moved to B.Cu
- moved C11 20.5 mm to (129.0, 83.9), turned to -90 degrees
- moved J1 20.1 mm to (117.5, 53.5), turned to 90 degrees
- moved SW1 18.3 mm to (127.0, 84.9), turned to -90 degrees
- moved C2 17.5 mm to (112.0, 77.5)
- moved U3 16.6 mm to (112.5, 80.0)
- moved C3 15.4 mm to (112.0, 79.5)
- moved C16 13.5 mm to (117.5, 65.5), turned to -90 degrees
- moved C10 12.2 mm to (133.9, 53.0)
- moved CR1 11.8 mm to (130.6, 62.0), turned to 180 degrees
- moved R5 9.14 mm to (138.1, 53.0), turned to -90 degrees
- moved C14 9.11 mm to (128.0, 57.0), turned to 90 degrees
- moved L4 8.51 mm to (106.5, 44.4), turned to 90 degrees
- moved R22 8.04 mm to (128.0, 72.0), turned to 0 degrees
- moved C17 7.83 mm to (120.4, 62.5), turned to 180 degrees
- moved D3 7.52 mm to (106.5, 82.5), turned to 90 degrees
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Connections:
- J1 pad 1: +3V3 -> +3.3V
- U1 pad 24: +3V3 -> +3.3V
- U1 pad 36: +3V3 -> +3.3V
- U1 pad 48: +3V3 -> +3.3V
Routing:
- net /SWCLK: track 0.86 -> 0.00 mm
Other:
- board text added: "Grid size is .5mm"
- board text removed: "Grid size is 1.000m"

Commit message: aligned components
Parts:
- removed J6: Conn_02x10_Counter_Clockwise, UTSVT_Connectors:Molex_52465-2070
- added J4: Conn_02x10_Odd_Even, UTSVT_Connectors:Molex_52465-2070, B.Cu at (136.5, 62.0)
- moved C4 21.1 mm to (117.0, 72.5), turned to -90 degrees
- moved R12 20.6 mm to (114.5, 72.5)
- moved SW2 20.6 mm to (113.5, 71.5)
- moved C1 15.2 mm to (127.0, 86.5)
- moved FB1 14.3 mm to (126.5, 71.5)
- moved FB4 14.3 mm to (129.5, 71.5)
- moved C11 10.2 mm to (121.0, 77.5)
- moved C5 9.07 mm to (137.0, 77.5), turned to 90 degrees
- moved SW5 8.63 mm to (134.5, 78.5), turned to 180 degrees
- moved SW1 7.27 mm to (123.5, 78.5), turned to 0 degrees
- moved C12 6.97 mm to (138.0, 71.5)
- moved C15 6.97 mm to (132.0, 71.5)
- moved C7 6.97 mm to (135.0, 71.5)
- moved R22 6.76 mm to (132.0, 77.4), turned to 90 degrees
- moved JP1 1.46 mm to (122.5, 49.5)
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
Commit message: moved bypass caps and cleaned annotations
Parts:
- moved LOGO2 64.7 mm to (157.0, 65.0)
- moved C1 10.4 mm to (120.4, 78.5)
- moved C11 9.60 mm to (127.0, 85.0)
- moved SW1 9.60 mm to (129.5, 86.0)
- moved C17 6.67 mm to (117.5, 56.5)
- moved C3 0.50 mm to (112.0, 80.0)
- moved U4 0.23 mm to (129.8, 52.4)
- moved C10 0.07 mm to (134.0, 53.0)
- moved L4 0.06 mm to (106.5, 44.5)
- turned C4 to 90 degrees
Changed lines of the file:
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@@
   )
   (footprint "Connector_PinHeader_2.54mm:PinHeader_1x04_P2.54mm_Vertical" (layer "F.Cu")
-    (at 117.46 53.5 90)
+    (at 117.5 53.5 90)
     (descr "Through hole straight pin header, 1x04, 2.54mm pitch, single row")
     (tags "Through hole pin header THT 1x04 2.54mm single row")
@@
   )
   (footprint "Button_Switch_SMD:SW_SPST_B3SL-1002P" (layer "F.Cu")
-    (at 123.5 78.5)
+    (at 129.5 86)
     (descr "Middle Stroke Tactile Switch, B3SL")
     (tags "Middle Stroke Tactile Switch")
@@
   )
   (footprint "Capacitor_SMD:C_0805_2012Metric" (layer "F.Cu")
-    (at 112 79.5)
+    (at 112.05 80)
     (descr "Capacitor SMD 0805 (2012 Metric), square (rectangular) end terminal, IPC_7351 nominal, (Body size source: IPC-SM-782 page 76, https://www.pcb-3d.com/wordpress/wp-content/uploads/ipc-sm-782a_amendment_1_and_2.pdf, https://docs.google.com/spreadsheets/d/1BsfQQcO9C6DZCsRaXUlFlo91Tg2WpOkGARC1WS5S8t0/edit?usp=sharing), generated with kicad-footprint-generator")
     (tags "capacitor")
@@
   )
   (footprint "UTSVT_Passive:C_2220_5750Metric" (layer "F.Cu")
-    (at 127 86.5)
+    (at 120.3758 78.5)
     (descr "Capacitor SMD 2220In_5750Metrix")
     (tags "Capacitor, 5750")
@@
   )
   (footprint "Capacitor_SMD:C_0805_2012Metric" (layer "B.Cu")
-    (at 120.4125 62.5 180)
+    (at 117.5 56.5 180)
     (descr "Capacitor SMD 0805 (2012 Metric), square (rectangular) end terminal, IPC_7351 nominal, (Body size source: IPC-SM-782 page 76, https://www.pcb-3d.com/wordpress/wp-content/uploads/ipc-sm-782a_amendment_1_and_2.pdf, https://docs.google.com/spreadsheets/d/1BsfQQcO9C6DZCsRaXUlFlo91Tg2WpOkGARC1WS5S8t0/edit?usp=sharing), generated with kicad-footprint-generator")
     (tags "capacitor")
@@
   )
   (footprint "Capacitor_SMD:C_0805_2012Metric" (layer "B.Cu")
-    (at 121 77.55 -90)
+    (at 127 85.05 -90)
     (descr "Capacitor SMD 0805 (2012 Metric), square (rectangular) end terminal, IPC_7351 nominal, (Body size source: IPC-SM-782 page 76, https://www.pcb-3d.com/wordpress/wp-content/uploads/ipc-sm-782a_amendment_1_and_2.pdf, https://docs.google.com/spreadsheets/d/1BsfQQcO9C6DZCsRaXUlFlo91Tg2WpOkGARC1WS5S8t0/edit?usp=sharing), generated with kicad-footprint-generator")
     (tags "capacitor")
@@
   )
   (footprint "UTSVT_Special:UTSVT_Logo_Symbol" (layer "B.Cu")
-    (at 158.369 129.667 180)
+    (at 157 65 180)
     (property "Sheetfile" "BPS-PeripheralSOM.kicad_sch")
     (property "Sheetname" "")
@@
   )
   (footprint "Capacitor_SMD:C_0805_2012Metric" (layer "B.Cu")
-    (at 133.95 52.95 -90)
+    (at 134 53 -90)
     (descr "Capacitor SMD 0805 (2012 Metric), square (rectangular) end terminal, IPC_7351 nominal, (Body size source: IPC-SM-782 page 76, https://www.pcb-3d.com/wordpress/wp-content/uploads/ipc-sm-782a_amendment_1_and_2.pdf, https://docs.google.com/spreadsheets/d/1BsfQQcO9C6DZCsRaXUlFlo91Tg2WpOkGARC1WS5S8t0/edit?usp=sharing), generated with kicad-footprint-generator")
     (tags "capacitor")
@@
   )
   (footprint "Capacitor_SMD:C_0805_2012Metric" (layer "B.Cu")
-    (at 108.5 44.55 -90)
+    (at 108.5 44.5 -90)
     (descr "Capacitor SMD 0805 (2012 Metric), square (rectangular) end terminal, IPC_7351 nominal, (Body size source: IPC-SM-782 page 76, https://www.pcb-3d.com/wordpress/wp-content/uploads/ipc-sm-782a_amendment_1_and_2.pdf, https://docs.google.com/spreadsheets/d/1BsfQQcO9C6DZCsRaXUlFlo91Tg2WpOkGARC1WS5S8t0/edit?usp=sharing), generated with kicad-footprint-generator")
     (tags "capacitor")
@@
   )
   (footprint "Capacitor_SMD:C_0805_2012Metric" (layer "B.Cu")
-    (at 117 72.5 -90)
+    (at 117 72.5 90)
     (descr "Capacitor SMD 0805 (2012 Metric), square (rectangular) end terminal, IPC_7351 nominal, (Body size source: IPC-SM-782 page 76, https://www.pcb-3d.com/wordpress/wp-content/uploads/ipc-sm-782a_amendment_1_and_2.pdf, https://docs.google.com/spreadsheets/d/1BsfQQcO9C6DZCsRaXUlFlo91Tg2WpOkGARC1WS5S8t0/edit?usp=sharing), generated with kicad-footprint-generator")
     (tags "capacitor")
@@
     (fp_line (start 1 0.625) (end 1 -0.625)
       (stroke (width 0.1) (type solid)) (layer "B.Fab"))
-    (pad "1" smd roundrect (at -0.95 0 270) (size 1 1.45) (layers "B.Cu" "B.Paste" "B.Mask") (roundrect_rratio 0.25)
+    (pad "1" smd roundrect (at -0.95 0 90) (size 1 1.45) (layers "B.Cu" "B.Paste" "B.Mask") (roundrect_rratio 0.25)
       (net 79 "/PC13") (pintype "passive"))
-    (pad "2" smd roundrect (at 0.95 0 270) (size 1 1.45) (layers "B.Cu" "B.Paste" "B.Mask") (roundrect_rratio 0.25)
+    (pad "2" smd roundrect (at 0.95 0 90) (size 1 1.45) (layers "B.Cu" "B.Paste" "B.Mask") (roundrect_rratio 0.25)
       (net 20 "Net-(SW2-B)") (pintype "passive"))
     (model "${KICAD6_3DMODEL_DIR}/Capacitor_SMD.3dshapes/C_0805_2012Metric.wrl"
@@
   )
   (footprint "Capacitor_SMD:C_0805_2012Metric" (layer "B.Cu")
-    (at 110.5 44.55 -90)
+    (at 110.5 44.5 -90)
     (descr "Capacitor SMD 0805 (2012 Metric), square (rectangular) end terminal, IPC_7351 nominal, (Body size source: IPC-SM-782 page 76, https://www.pcb-3d.com/wordpress/wp-content/uploads/ipc-sm-782a_amendment_1_and_2.pdf, https://docs.google.com/spreadsheets/d/1BsfQQcO9C6DZCsRaXUlFlo91Tg2WpOkGARC1WS5S8t0/edit?usp=sharing), generated with kicad-footprint-generator")
     (tags "capacitor")
@@
   )
   (footprint "Package_DFN_QFN:QFN-24-1EP_4x4mm_P0.5mm_EP2.6x2.6mm" (layer "B.Cu")
-    (at 129.8875 52.25 -90)
+    (at 129.75 52.4375 -90)
     (descr "QFN, 24 Pin (http://ww1.microchip.com/downloads/en/PackagingSpec/00000049BQ.pdf#page=278), generated with kicad-footprint-generator ipc_noLead_generator.py")
     (tags "QFN NoLead")
@@
   )
   (footprint "Inductor_SMD:L_0805_2012Metric" (layer "B.Cu")
-    (at 106.5 44.4375 90)
+    (at 106.5 44.5 90)
     (descr "Inductor SMD 0805 (2012 Metric), square (rectangular) end terminal, IPC_7351 nominal, (Body size source: IPC-SM-782 page 80, https://www.pcb-3d.com/wordpress/wp-content/uploads/ipc-sm-782a_amendment_1_and_2.pdf), generated with kicad-footprint-generator")
     (tags "inductor")
@@
   )
   (footprint "Capacitor_SMD:C_0805_2012Metric" (layer "B.Cu")
-    (at 112.54 44.55 -90)
+    (at 112.54 44.5 -90)
     (descr "Capacitor SMD 0805 (2012 Metric), square (rectangular) end terminal, IPC_7351 nominal, (Body size source: IPC-SM-782 page 76, https://www.pcb-3d.com/wordpress/wp-content/uploads/ipc-sm-782a_amendment_1_and_2.pdf, https://docs.google.com/spreadsheets/d/1BsfQQcO9C6DZCsRaXUlFlo91Tg2WpOkGARC1WS5S8t0/edit?usp=sharing), generated with kicad-footprint-generator")
     (tags "capacitor")
@@
   )
   (footprint "Capacitor_SMD:C_0805_2012Metric" (layer "B.Cu")
-    (at 114.54 44.55 -90)
+    (at 114.54 44.5 -90)
     (descr "Capacitor SMD 0805 (2012 Metric), square (rectangular) end terminal, IPC_7351 nominal, (Body size source: IPC-SM-782 page 76, https://www.pcb-3d.com/wordpress/wp-content/uploads/ipc-sm-782a_amendment_1_and_2.pdf, https://docs.google.com/spreadsheets/d/1BsfQQcO9C6DZCsRaXUlFlo91Tg2WpOkGARC1WS5S8t0/edit?usp=sharing), generated with kicad-footprint-generator")
     (tags "capacitor")

Commit message: aligned components to .5 mm
Parts:
- moved C1 11.1 mm to (128.5, 86.0), turned to 180 degrees
- moved C11 10.6 mm to (119.5, 77.5)
- moved SW1 10.6 mm to (122.0, 78.5)
- moved J2 1.00 mm to (106.0, 56.0)
- moved J5 0.94 mm to (106.0, 70.0)
- moved U4 0.26 mm to (130.0, 52.5)
- moved D1 0.25 mm to (130.0, 48.0)
- moved CR2 0.16 mm to (131.0, 66.0)
- moved CR1 0.15 mm to (131.0, 62.0)
- moved R10 0.09 mm to (130.0, 60.5)
- moved R15 0.09 mm to (130.0, 64.0)
- moved R20 0.09 mm to (128.0, 64.0)
- moved R9 0.09 mm to (128.0, 60.5)
- moved R3 0.05 mm to (134.0, 49.0)
- moved R4 0.05 mm to (136.0, 49.0)
Changed lines of the file:
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@@
   )
   (footprint "Button_Switch_SMD:SW_SPST_B3SL-1002P" (layer "F.Cu")
-    (at 129.5 86)
+    (at 122 78.5)
     (descr "Middle Stroke Tactile Switch, B3SL")
     (tags "Middle Stroke Tactile Switch")
@@
   )
   (footprint "Connector_Molex:Molex_Micro-Fit_3.0_43045-0612_2x03_P3.00mm_Vertical" placed (layer "F.Cu")
-    (at 107 56 -90)
+    (at 106 56 -90)
     (descr "Molex Micro-Fit 3.0 Connector System, 43045-0612 (compatible alternatives: 43045-0613, 43045-0624), 3 Pins per row (http://www.molex.com/pdm_docs/sd/430450212_sd.pdf), generated with kicad-footprint-generator")
     (tags "connector Molex Micro-Fit_3.0 side entry")
@@
   )
   (footprint "Connector_USB:USB_Micro-B_Molex-105017-0001" (layer "F.Cu")
-    (at 131 43.5375 180)
+    (at 131 43.5 180)
     (descr "http://www.molex.com/pdm_docs/sd/1050170001_sd.pdf")
     (tags "Micro-USB SMD Typ-B")
@@
   )
   (footprint "UTSVT_Passive:C_2220_5750Metric" (layer "F.Cu")
-    (at 120.3758 78.5)
+    (at 128.5 86 180)
     (descr "Capacitor SMD 2220In_5750Metrix")
     (tags "Capacitor, 5750")
@@
     (fp_circle (center -2.9972 0) (end -2.921 0)
       (stroke (width 0.1524) (type solid)) (fill none) (layer "F.Fab"))
-    (pad "1" smd rect (at -3.1242 0) (size 0.5588 5.4102) (layers "F.Cu" "F.Paste" "F.Mask")
+    (pad "1" smd rect (at -3.1242 0 180) (size 0.5588 5.4102) (layers "F.Cu" "F.Paste" "F.Mask")
       (net 91 "Net-(D8-K)") (pintype "passive"))
-    (pad "2" smd rect (at 3.1242 0) (size 0.5588 5.4102) (layers "F.Cu" "F.Paste" "F.Mask")
+    (pad "2" smd rect (at 3.1242 0 180) (size 0.5588 5.4102) (layers "F.Cu" "F.Paste" "F.Mask")
       (net 5 "GNDPWR") (pintype "passive"))
   )
@@
   )
   (footprint "UTSVT_ICs:SOT26_DIO" (layer "F.Cu")
-    (at 130.85255 66.049999)
+    (at 131 66)
     (tags "D5V0P4UR6SO-7 ")
     (property "Sheetfile" "BPS-PeripheralSOM.kicad_sch")
@@
   )
   (footprint "Connector_Molex:Molex_Micro-Fit_3.0_43045-0612_2x03_P3.00mm_Vertical" (layer "F.Cu")
-    (at 106.94 70 -90)
+    (at 106 70 -90)
     (descr "Molex Micro-Fit 3.0 Connector System, 43045-0612 (compatible alternatives: 43045-0613, 43045-0624), 3 Pins per row (http://www.molex.com/pdm_docs/sd/430450212_sd.pdf), generated with kicad-footprint-generator")
     (tags "connector Molex Micro-Fit_3.0 side entry")
@@
   )
   (footprint "UTSVT_ICs:SOT26_DIO" (layer "F.Cu")
-    (at 130.85255 62.049999)
+    (at 131 62.049999)
     (tags "D5V0P4UR6SO-7 ")
     (property "Sheetfile" "BPS-PeripheralSOM.kicad_sch")
@@
   )
   (footprint "Capacitor_SMD:C_0805_2012Metric" (layer "B.Cu")
-    (at 127 85.05 -90)
+    (at 119.5 77.55 -90)
     (descr "Capacitor SMD 0805 (2012 Metric), square (rectangular) end terminal, IPC_7351 nominal, (Body size source: IPC-SM-782 page 76, https://www.pcb-3d.com/wordpress/wp-content/uploads/ipc-sm-782a_amendment_1_and_2.pdf, https://docs.google.com/spreadsheets/d/1BsfQQcO9C6DZCsRaXUlFlo91Tg2WpOkGARC1WS5S8t0/edit?usp=sharing), generated with kicad-footprint-generator")
     (tags "capacitor")
@@
   )
   (footprint "Resistor_SMD:R_0805_2012Metric" (layer "B.Cu")
-    (at 130 60.4125 -90)
+    (at 130 60.5 -90)
     (descr "Resistor SMD 0805 (2012 Metric), square (rectangular) end terminal, IPC_7351 nominal, (Body size source: IPC-SM-782 page 72, https://www.pcb-3d.com/wordpress/wp-content/uploads/ipc-sm-782a_amendment_1_and_2.pdf), generated with kicad-footprint-generator")
     (tags "resistor")
@@
   )
   (footprint "Package_TO_SOT_SMD:SOT-143" (layer "B.Cu")
-    (at 130.25 48 -90)
+    (at 130 48 -90)
     (descr "SOT-143 https://www.nxp.com/docs/en/package-information/SOT143B.pdf")
     (tags "SOT-143")
@@
   )
   (footprint "Resistor_SMD:R_0805_2012Metric" (layer "B.Cu")
-    (at 135.95 49 90)
+    (at 136 49 90)
     (descr "Resistor SMD 0805 (2012 Metric), square (rectangular) end terminal, IPC_7351 nominal, (Body size source: IPC-SM-782 page 72, https://www.pcb-3d.com/wordpress/wp-content/uploads/ipc-sm-782a_amendment_1_and_2.pdf), generated with kicad-footprint-generator")
     (tags "resistor")
@@
   )
   (footprint "Package_DFN_QFN:QFN-24-1EP_4x4mm_P0.5mm_EP2.6x2.6mm" (layer "B.Cu")
-    (at 129.75 52.4375 -90)
+    (at 130 52.5 -90)
     (descr "QFN, 24 Pin (http://ww1.microchip.com/downloads/en/PackagingSpec/00000049BQ.pdf#page=278), generated with kicad-footprint-generator ipc_noLead_generator.py")
     (tags "QFN NoLead")
@@
   )
   (footprint "Resistor_SMD:R_0805_2012Metric" (layer "B.Cu")
-    (at 128 63.9125 -90)
+    (at 128 64 -90)
     (descr "Resistor SMD 0805 (2012 Metric), square (rectangular) end terminal, IPC_7351 nominal, (Body size source: IPC-SM-782 page 72, https://www.pcb-3d.com/wordpress/wp-content/uploads/ipc-sm-782a_amendment_1_and_2.pdf), generated with kicad-footprint-generator")
     (tags "resistor")
@@
   )
   (footprint "Resistor_SMD:R_0805_2012Metric" (layer "B.Cu")
-    (at 128 60.4125 -90)
+    (at 128 60.5 -90)
     (descr "Resistor SMD 0805 (2012 Metric), square (rectangular) end terminal, IPC_7351 nominal, (Body size source: IPC-SM-782 page 72, https://www.pcb-3d.com/wordpress/wp-content/uploads/ipc-sm-782a_amendment_1_and_2.pdf), generated with kicad-footprint-generator")
     (tags "resistor")
@@
   )
   (footprint "Resistor_SMD:R_0805_2012Metric" (layer "B.Cu")
-    (at 133.95 49 90)
+    (at 134 49 90)
     (descr "Resistor SMD 0805 (2012 Metric), square (rectangular) end terminal, IPC_7351 nominal, (Body size source: IPC-SM-782 page 72, https://www.pcb-3d.com/wordpress/wp-content/uploads/ipc-sm-782a_amendment_1_and_2.pdf), generated with kicad-footprint-generator")
     (tags "resistor")
@@
   )
   (footprint "Resistor_SMD:R_0805_2012Metric" (layer "B.Cu")
-    (at 130 63.9125 -90)
+    (at 130 64 -90)
     (descr "Resistor SMD 0805 (2012 Metric), square (rectangular) end terminal, IPC_7351 nominal, (Body size source: IPC-SM-782 page 72, https://www.pcb-3d.com/wordpress/wp-content/uploads/ipc-sm-782a_amendment_1_and_2.pdf), generated with kicad-footprint-generator")
     (tags "resistor")
