File: BPS-PeripheralSOM.kicad_pcb (KiCad board)
At the start: 2 copper layers, 40 x 50 mm, 84 parts, among them J1 SWD, J2 CAN_In, J3 USB_B_Micro, J4 Conn_02x10_Odd_Even, J5 CAN_Out, Q1 Q_PMOS_GSD, SW1 Reset, SW2 SW_SPDT, SW5 SW_Push, U1 STM32L431CBTx, U2 RI3-0505S, U3 LD1117-3.3_SOT223, U4 CP2102N-A01-GQFN24, U7 ADM3055E, U8 CDSOT23-T24CAN, Y1 8M

Commit message: re-oriented i2c pullups to be closer to pins
Parts:
- moved C21 0.71 mm to (118.5, 72.5)
- moved C22 0.71 mm to (122.5, 72.5)
- moved Y1 0.16 mm to (120.5, 68.5)
- turned R10 to 90 degrees
- turned R9 to 90 degrees
Changed lines of the file:
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@@
   )
   (footprint "Capacitor_SMD:C_0805_2012Metric" (layer "F.Cu")
-    (at 122 72 -90)
+    (at 122.5 72.5 -90)
     (descr "Capacitor SMD 0805 (2012 Metric), square (rectangular) end terminal, IPC_7351 nominal, (Body size source: IPC-SM-782 page 76, https://www.pcb-3d.com/wordpress/wp-content/uploads/ipc-sm-782a_amendment_1_and_2.pdf, https://docs.google.com/spreadsheets/d/1BsfQQcO9C6DZCsRaXUlFlo91Tg2WpOkGARC1WS5S8t0/edit?usp=sharing), generated with kicad-footprint-generator")
     (tags "capacitor")
@@
   )
   (footprint "Crystal:Crystal_SMD_TXC_7A-2Pin_5x3.2mm" (layer "F.Cu")
-    (at 120.35 68.45)
+    (at 120.5 68.5)
     (descr "SMD Crystal TXC 7A http://txccrystal.com/images/pdf/7a.pdf")
     (tags "SMD SMT crystal")
@@
   )
   (footprint "Capacitor_SMD:C_0805_2012Metric" (layer "F.Cu")
-    (at 119 72 -90)
+    (at 118.5 72.5 -90)
     (descr "Capacitor SMD 0805 (2012 Metric), square (rectangular) end terminal, IPC_7351 nominal, (Body size source: IPC-SM-782 page 76, https://www.pcb-3d.com/wordpress/wp-content/uploads/ipc-sm-782a_amendment_1_and_2.pdf, https://docs.google.com/spreadsheets/d/1BsfQQcO9C6DZCsRaXUlFlo91Tg2WpOkGARC1WS5S8t0/edit?usp=sharing), generated with kicad-footprint-generator")
     (tags "capacitor")
@@
   )
   (footprint "Resistor_SMD:R_0805_2012Metric" (layer "B.Cu")
-    (at 130 60.5 -90)
+    (at 130 60.5 90)
     (descr "Resistor SMD 0805 (2012 Metric), square (rectangular) end terminal, IPC_7351 nominal, (Body size source: IPC-SM-782 page 72, https://www.pcb-3d.com/wordpress/wp-content/uploads/ipc-sm-782a_amendment_1_and_2.pdf), generated with kicad-footprint-generator")
     (tags "resistor")
@@
     (property "ki_keywords" "R res resistor")
     (attr smd)
-    (fp_text reference "R10" (at 0 1.65 -270) (layer "B.SilkS")
+    (fp_text reference "R10" (at 0 1.65 90) (layer "B.SilkS")
         (effects (font (size 1 1) (thickness 0.15)) (justify mirror))
     )
-    (fp_text value "10K" (at 0 -1.65 -270) (layer "B.Fab")
+    (fp_text value "10K" (at 0 -1.65 90) (layer "B.Fab")
         (effects (font (size 1 1) (thickness 0.15)) (justify mirror))
     )
-    (fp_text user "${REFERENCE}" (at 0 0 -270) (layer "B.Fab")
+    (fp_text user "${REFERENCE}" (at 0 0 90) (layer "B.Fab")
         (effects (font (size 0.5 0.5) (thickness 0.08)) (justify mirror))
     )
@@
     (fp_line (start 1 0.625) (end 1 -0.625)
       (stroke (width 0.1) (type solid)) (layer "B.Fab"))
-    (pad "1" smd roundrect (at -0.9125 0 270) (size 1.025 1.4) (layers "B.Cu" "B.Paste" "B.Mask") (roundrect_rratio 0.243902)
+    (pad "1" smd roundrect (at -0.9125 0 90) (size 1.025 1.4) (layers "B.Cu" "B.Paste" "B.Mask") (roundrect_rratio 0.243902)
       (net 3 "+3.3V") (pintype "passive"))
-    (pad "2" smd roundrect (at 0.9125 0 270) (size 1.025 1.4) (layers "B.Cu" "B.Paste" "B.Mask") (roundrect_rratio 0.243902)
+    (pad "2" smd roundrect (at 0.9125 0 90) (size 1.025 1.4) (layers "B.Cu" "B.Paste" "B.Mask") (roundrect_rratio 0.243902)
       (net 29 "/I2C2_SCL") (pintype "passive"))
     (model "${KICAD6_3DMODEL_DIR}/Resistor_SMD.3dshapes/R_0805_2012Metric.wrl"
@@
   )
   (footprint "Resistor_SMD:R_0805_2012Metric" (layer "B.Cu")
-    (at 128 60.5 -90)
+    (at 128 60.5 90)
     (descr "Resistor SMD 0805 (2012 Metric), square (rectangular) end terminal, IPC_7351 nominal, (Body size source: IPC-SM-782 page 72, https://www.pcb-3d.com/wordpress/wp-content/uploads/ipc-sm-782a_amendment_1_and_2.pdf), generated with kicad-footprint-generator")
     (tags "resistor")
@@
     (property "ki_keywords" "R res resistor")
     (attr smd)
-    (fp_text reference "R9" (at 0 1.65 -270) (layer "B.SilkS")
+    (fp_text reference "R9" (at 0 1.65 90) (layer "B.SilkS")
         (effects (font (size 1 1) (thickness 0.15)) (justify mirror))
     )
-    (fp_text value "10K" (at 0 -1.65 -270) (layer "B.Fab")
+    (fp_text value "10K" (at 0 -1.65 90) (layer "B.Fab")
         (effects (font (size 1 1) (thickness 0.15)) (justify mirror))
     )
-    (fp_text user "${REFERENCE}" (at 0 0 -270) (layer "B.Fab")
+    (fp_text user "${REFERENCE}" (at 0 0 90) (layer "B.Fab")
         (effects (font (size 0.5 0.5) (thickness 0.08)) (justify mirror))
     )
@@
     (fp_line (start 1 0.625) (end 1 -0.625)
       (stroke (width 0.1) (type solid)) (layer "B.Fab"))
-    (pad "1" smd roundrect (at -0.9125 0 270) (size 1.025 1.4) (layers "B.Cu" "B.Paste" "B.Mask") (roundrect_rratio 0.243902)
+    (pad "1" smd roundrect (at -0.9125 0 90) (size 1.025 1.4) (layers "B.Cu" "B.Paste" "B.Mask") (roundrect_rratio 0.243902)
       (net 3 "+3.3V") (pintype "passive"))
-    (pad "2" smd roundrect (at 0.9125 0 270) (size 1.025 1.4) (layers "B.Cu" "B.Paste" "B.Mask") (roundrect_rratio 0.243902)
+    (pad "2" smd roundrect (at 0.9125 0 90) (size 1.025 1.4) (layers "B.Cu" "B.Paste" "B.Mask") (roundrect_rratio 0.243902)
       (net 28 "/I2C2_SDA") (pintype "passive"))
     (model "${KICAD6_3DMODEL_DIR}/Resistor_SMD.3dshapes/R_0805_2012Metric.wrl"

Commit message: added Tianda's suggestions
Parts:
- moved TP6 52.0 mm to (102.5, 82.0)
- moved TP4 34.6 mm to (137.5, 84.5)
- moved J1 20.3 mm to (137.5, 50.2), turned to 0 degrees
- moved C4 20.0 mm to (137.0, 72.5)
- moved SW2 18.5 mm to (132.0, 71.5)
- moved R12 18.0 mm to (132.5, 72.5)
- moved C12 10.5 mm to (127.5, 72.5)
- moved C7 10.5 mm to (124.5, 72.5)
- moved C9 10.0 mm to (126.0, 53.0), turned to 180 degrees
- moved C10 8.33 mm to (126.0, 50.5), turned to 180 degrees
- moved R5 6.05 mm to (137.0, 47.0), turned to 180 degrees
- moved R3 5.93 mm to (136.0, 43.4)
- moved R4 5.93 mm to (138.0, 43.4)
- moved FB4 5.59 mm to (124.5, 69.0), turned to -90 degrees
- moved C15 5.17 mm to (127.5, 69.0), turned to 90 degrees
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Connections:
- C4 pad 1: /PC13 -> /PA2
- R12 pad 1: /PC13 -> /PA2
- U1 pad 12: unconnected-(U1-PA2-Pad12) -> /PA2
