File: BPS-PeripheralSOM.kicad_pcb (KiCad board)
At the start: 4 copper layers, 40 x 50 mm, 81 parts, among them J1 SWD, J2 CAN_In, J3 USB_B_Micro, J5 CAN_Out, J6 SOMConnector, Q1 Q_PMOS_GSD, SW1 Reset, SW2 SW_SPDT, SW5 SW_Push, U1 STM32L431CBTx, U2 RI3-0505S, U3 LD1117-3.3_SOT223, U4 CP2102N-A01-GQFN24, U7 ADM3055E, U8 CDSOT23-T24CAN, Y1 8M

Commit message: Cleaned up silkscreen more and made GND planes more whole
Parts:
- added IC1: TPS1120DR, UTSVT_ICs:SOIC127P600X175-8N, F.Cu at (136.1, 55.7)
Routing:
- net GNDPWR: track 4.24 -> 32.3 mm
- net GND: track 78.6 -> 84.1 mm, vias 24 -> 25
- net +5V: track 45.7 -> 47.2 mm, vias 2 -> 3
- net /5V_Ext: track 0.00 -> 1.44 mm
- net /I2C1_SCL: track 26.2 -> 25.1 mm
- net +3.3V: track 36.2 -> 37.2 mm
- net GND1: track 50.1 -> 51.0 mm
Other:
- board text added: "5V In"
- board text added: "C+"
- board text added: "C-"
- board text added: "GND PWR"
- board text added: "RST"
- board text added: "hello, kindly bridge this jumper if you'd like me to be the end"
- board text removed: "5v_In"
- board text removed: "GNDPWR"
- board text removed: "Jump if Terminating End"
- board text removed: "Reset"

Commit message: added more things to BOM and cleaned up silkscreen
Parts:
- moved SW2 1.17 mm to (134.5, 72.0), turned to 0 degrees
Connections:
- IC1 pad 1: unconnected-(IC1-1SOURCE-Pad1) -> Net-(IC1-1SOURCE)
- IC1 pad 2: unconnected-(IC1-1GATE-Pad2) -> /PA8
- IC1 pad 3: unconnected-(IC1-2SOURCE-Pad3) -> Net-(IC1-2SOURCE)
- IC1 pad 4: unconnected-(IC1-2GATE-Pad4) -> /PA8
- IC1 pad 5: unconnected-(IC1-2DRAIN_1-Pad5) -> GND
- IC1 pad 6: unconnected-(IC1-2DRAIN_2-Pad6) -> GND
- IC1 pad 7: unconnected-(IC1-1DRAIN_1-Pad7) -> GND
- IC1 pad 8: unconnected-(IC1-1DRAIN_2-Pad8) -> GND
- U1 pad 29: unconnected-(U1-PA8-Pad29) -> /PA8
Routing:
- net /PA2: track 15.4 -> 12.7 mm
- net GNDA: track 32.5 -> 35.2 mm
Other:
- board text added: "Champers and Lakshay Were here"
- board text added: "PeripheralSOM Fall 2023"

Commit message: Added more symbols for BOM and started sw pull downs
Parts:
- removed R10, R9: 10K, Resistor_SMD:R_0805_2012Metric
- added G***: LOGO, UTSVT_Special:vsus, B.Cu at (120.7, 71.1)
- added R12: 10K, Resistor_SMD:R_0805_2012Metric, B.Cu at (133.3, 55.9)
- added R13: 10K, Resistor_SMD:R_0805_2012Metric, B.Cu at (137.2, 55.9)
- moved C9 0.11 mm to (135.9, 50.5)
Connections:
- IC1 pad 5: GND -> /I2C2_SDA
- IC1 pad 6: GND -> /I2C2_SDA
- IC1 pad 7: GND -> /I2C2_SCL
- IC1 pad 8: GND -> /I2C2_SCL
Routing:
- net /PA8: track 0.00 -> 18.5 mm, vias 0 -> 2
- net /I2C2_SCL: track 17.3 -> 30.8 mm, vias 3 -> 4
- net +3.3V: track 37.2 -> 49.7 mm
- net /I2C2_SDA: track 16.2 -> 28.2 mm, vias 3 -> 4
- net Net-(IC1-2SOURCE): track 0.00 -> 3.10 mm, vias 0 -> 1
- net Net-(IC1-1SOURCE): track 0.00 -> 2.57 mm, vias 0 -> 1
- net /5V_Ext: track 1.44 -> 0.00 mm
- net GND: track 84.4 -> 83.4 mm, vias 25 -> 26

Commit message: added sw pull downs
Parts:
- added R9: 10k, Resistor_SMD:R_0805_2012Metric, B.Cu at (129.5, 56.0)
Connections:
- IC1 pad 1: Net-(IC1-1SOURCE) -> +3.3V
- IC1 pad 3: Net-(IC1-2SOURCE) -> +3.3V
- R12 pad 1: +3.3V -> +3V3
- R12 pad 2: Net-(IC1-1SOURCE) -> /I2C2_SCL
- R13 pad 1: +3.3V -> +3V3
- R13 pad 2: Net-(IC1-2SOURCE) -> /I2C2_SDA
Routing:
- net +3.3V: track 49.7 -> 42.6 mm, vias 15 -> 18
- net +3V3: track 0.00 -> 4.66 mm
- net Net-(IC1-2SOURCE): track 3.10 -> 0.00 mm, vias 1 -> 0
- net Net-(IC1-1SOURCE): track 2.57 -> 0.00 mm, vias 1 -> 0
- net /PowerDist/5V_Ferrite: track 6.16 -> 3.66 mm, vias 4 -> 3
- net (no net): track 1.54 -> 0.00 mm, vias 1 -> 0
- net /I2C2_SDA: track 28.2 -> 29.6 mm, vias 4 -> 3
- net /PA8: track 18.5 -> 19.8 mm, vias 2 -> 3
- net /I2C2_SCL: track 30.8 -> 31.5 mm, vias 4 -> 3

Commit message: fixed repeated items in BOMs and made molex connectors not backwards
Parts:
- U4: value CP2102N-A01-GQFN24 -> CP2102N-A02-GQFN24
- moved J2 6.71 mm to (103.0, 62.0), turned to 90 degrees
- moved J5 6.71 mm to (103.0, 76.0), turned to 90 degrees
Connections:
- J2 pad 1: /5V_Ext -> GNDPWR
- J2 pad 2: /CAN_H -> /CAN_L
- J2 pad 3: /V_CAN_IN -> GND1
- J2 pad 4: GND1 -> /V_CAN_IN
- J2 pad 5: /CAN_L -> /CAN_H
- J2 pad 6: GNDPWR -> /5V_Ext
- J5 pad 1: /5V_Ext -> GNDPWR
- J5 pad 2: /CAN_H -> /CAN_L
- J5 pad 3: /V_CAN_IN -> GND1
- J5 pad 4: GND1 -> /V_CAN_IN
- J5 pad 5: /CAN_L -> /CAN_H
- J5 pad 6: GNDPWR -> /5V_Ext
Routing:
- net +5V: track 46.9 -> 47.6 mm

Commit message: made 5V fill more whole, deleted not needed vias, made the vias bigger for bigger traces, changed 5V ferrite fill
Routing:
- net +5V: track 47.6 -> 31.2 mm
- net +3.3V: track 42.6 -> 52.6 mm, vias 18 -> 17
- net /PowerDist/5V_Ferrite: track 3.66 -> 0.05 mm
- net VDDA: track 34.3 -> 32.5 mm, vias 3 -> 2
- net GND: track 83.4 -> 85.1 mm, vias 26 -> 18
- net GNDA: track 35.2 -> 33.7 mm
Other:
- board text added: "3.3V"
- board text added: "SWCLK"
- board text added: "SWDIO"

Commit message: Made big planes have 2 layers
Routing:
- net VDDA: track 32.5 -> 31.2 mm
- net /V_CAN_IN: track 43.7 -> 44.3 mm
Changed lines of the file:
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@@
   (segment (start 117.5875 57.9125) (end 117.5875 57.3) (width 0.25) (layer "F.Cu") (net 24))
   (via (at 117.5875 57.3) (size 0.5) (drill 0.3) (layers "F.Cu" "B.Cu") (net 24))
-  (segment (start 120.19 54.65) (end 118.35 54.65) (width 0.5) (layer "In2.Cu") (net 24))
-  (segment (start 118.35 54.65) (end 117.5 55.5) (width 0.5) (layer "In2.Cu") (net 24))
-  (segment (start 117.5 55.5) (end 117.5 57.2125) (width 0.5) (layer "In2.Cu") (net 24))
-  (segment (start 117.5 57.2125) (end 117.5875 57.3) (width 0.5) (layer "In2.Cu") (net 24))
+  (segment (start 118.4 54.65) (end 117.5875 55.4625) (width 0.5) (layer "In2.Cu") (net 24))
+  (segment (start 120.19 54.65) (end 118.4 54.65) (width 0.5) (layer "In2.Cu") (net 24))
   (segment (start 121.49 53.35) (end 120.19 54.65) (width 0.5) (layer "In2.Cu") (net 24))
+  (segment (start 117.5875 55.4625) (end 117.5875 57.3) (width 0.5) (layer "In2.Cu") (net 24))
   (segment (start 120 57.7) (end 120 56.5) (width 0.25) (layer "F.Cu") (net 25))
   (via (at 120 57.7) (size 0.5) (drill 0.3) (layers "F.Cu" "B.Cu") (net 25))
@@
   (segment (start 126.3375 70.0625) (end 127.2755 71.0005) (width 0.25) (layer "In1.Cu") (net 62))
   (segment (start 139.0045 69.7205) (end 139.0045 64.6045) (width 0.25) (layer "In1.Cu") (net 62))
-  (segment (start 126.3375 70.0625) (end 126.5 70.225) (width 1.5) (layer "B.Cu") (net 62))
-  (segment (start 126.45 71.5) (end 126.5 71.55) (width 1.5) (layer "B.Cu") (net 62))
-  (segment (start 124.5 71.5) (end 126.45 71.5) (width 1.5) (layer "B.Cu") (net 62))
-  (segment (start 124.5 70.0625) (end 124.5 71.5) (width 1.5) (layer "B.Cu") (net 62))
-  (segment (start 126.5 70.225) (end 126.5 71.55) (width 1.5) (layer "B.Cu") (net 62))
-  (segment (start 126.3375 70.0625) (end 124.5 70.0625) (width 1.5) (layer "B.Cu") (net 62))
+  (segment (start 124.5 71.6) (end 124.5 70.0625) (width 0.25) (layer "B.Cu") (net 62))
+  (segment (start 124.5 70.0625) (end 126.3375 70.0625) (width 0.25) (layer "B.Cu") (net 62))
+  (segment (start 124.55 71.55) (end 124.5 71.6) (width 0.25) (layer "B.Cu") (net 62))
+  (segment (start 126.5 71.55) (end 124.55 71.55) (width 0.25) (layer "B.Cu") (net 62))
+  (segment (start 126.3375 70.0625) (end 126.5 69.9) (width 0.25) (layer "B.Cu") (net 62))
   (via (at 104.5 84.0625) (size 0.5) (drill 0.3) (layers "F.Cu" "B.Cu") (net 63))
   (via (at 106.5 82) (size 0.5) (drill 0.3) (layers "F.Cu" "B.Cu") (net 63))
@@
   (segment (start 106 62) (end 108.5 59.5) (width 0.5) (layer "In1.Cu") (net 64))
   (segment (start 108.5 46.875) (end 107.2 45.575) (width 0.5) (layer "In1.Cu") (net 64))
+  (segment (start 106 76) (end 107.819 74.181) (width 0.25) (layer "B.Cu") (net 64))
   (segment (start 108.315 42.6775) (end 109.2 43.5625) (width 1) (layer "B.Cu") (net 64))
-  (segment (start 104.925 63.075) (end 106 62) (width 0.25) (layer "B.Cu") (net 64))
+  (segment (start 107.819 63.819) (end 106 62) (width 0.25) (layer "B.Cu") (net 64))
   (segment (start 113.2 43.5625) (end 109.2 43.5625) (width 1) (layer "B.Cu") (net 64))
-  (segment (start 106 76) (end 104.925 74.925) (width 0.25) (layer "B.Cu") (net 64))
   (segment (start 108.315 41.5625) (end 108.315 42.6775) (width 1) (layer "B.Cu") (net 64))
-  (segment (start 104.925 74.925) (end 104.925 63.075) (width 0.25) (layer "B.Cu") (net 64))
+  (segment (start 107.819 74.181) (end 107.819 63.819) (width 0.25) (layer "B.Cu") (net 64))
   (segment (start 115.86967 44.568997) (end 104.168997 44.568997) (width 0.25) (layer "B.Cu") (net 65))
   (segment (start 118.96 47.659327) (end 115.86967 44.568997) (width 0.25) (layer "B.Cu") (net 65))
@@
   (segment (start 138.0725 55.88) (end 138 55.8075) (width 0.25) (layer "B.Cu") (net 92))
   (segment (start 138 55.8075) (end 138 53) (width 0.25) (layer "B.Cu") (net 92))
-  (zone (net 3) (net_name "+3.3V") (layer "F.Cu") (hatch edge 0.5)
+  (zone (net 3) (net_name "+3.3V") (layers "F.Cu" "In2.Cu") (hatch edge 0.5)
     (priority 2)
     (connect_pads (clearance 0.5))
@@
         (xy 140 90)
         (xy 100 90)
-      )
-    )
-  )
-  (zone (net 2) (net_name "GND") (layer "In1.Cu") (hatch edge 0.5)
-    (connect_pads (clearance 0.5))
-    (min_thickness 0.25) (filled_areas_thickness no)
-    (fill yes (thermal_gap 0.5) (thermal_bridge_width 0.5))
-    (polygon
-      (pts
-        (xy 140 90)
-        (xy 100 90)
-        (xy 100 40)
-        (xy 140 40)
       )
     )
@@
     )
   )
-  (zone (net 3) (net_name "+3.3V") (layer "In2.Cu") (hatch edge 0.5)
+  (zone (net 2) (net_name "GND") (layers "In1.Cu" "B.Cu") (hatch edge 0.5)
     (connect_pads (clearance 0.5))
     (min_thickness 0.25) (filled_areas_thickness no)
@@
     )
   )
-  (zone (net 2) (net_name "GND") (layer "B.Cu") (hatch edge 0.5)
-    (priority 1)
-    (connect_pads (clearance 0.5))
-    (min_thickness 0.25) (filled_areas_thickness no)
-    (fill yes (thermal_gap 0.5) (thermal_bridge_width 0.5))
-    (polygon
-      (pts
-        (xy 100 40)
-        (xy 140 40)
-        (xy 140 90)
-        (xy 100 90)
-      )
-    )
-  )
   (zone (net 5) (net_name "GNDPWR") (layer "B.Cu") (hatch edge 0.5)
     (priority 4)
@@
         (xy 112.5 89.5)
         (xy 104.4 89.55)
-        (xy 100.95 89.5)
-        (xy 100.8 78.45)
-        (xy 100.8 78.3)
-        (xy 100.5 60)
-      )
-    )
+        (xy 99.95 89.3)
+        (xy 99.8 78.25)
+        (xy 99.8 77.9)
+        (xy 99.75 59.85)
+      )
+    )

Commit message: i2c pullup & some fill/zone fixes
Parts:
- added R10: 10K, Resistor_SMD:R_0805_2012Metric, B.Cu at (135.0, 55.0)
- R12: value 10K -> 1k
- R9: value 10k -> 100k
- moved R9 1.80 mm to (131.0, 55.0), turned to 90 degrees
- moved R12 0.95 mm to (133.0, 55.0), turned to -90 degrees
- moved R13 0.89 mm to (137.0, 55.0), turned to 90 degrees
Connections:
- IC1 pad 2: /PA8 -> Net-(IC1-1GATE)
- IC1 pad 4: /PA8 -> Net-(IC1-1GATE)
- IC1 pad 5: /I2C2_SDA -> Net-(IC1-2DRAIN_1)
- IC1 pad 6: /I2C2_SDA -> Net-(IC1-2DRAIN_1)
- IC1 pad 7: /I2C2_SCL -> Net-(IC1-1DRAIN_1)
- IC1 pad 8: /I2C2_SCL -> Net-(IC1-1DRAIN_1)
- R12 pad 1: +3V3 -> /PA8
- R12 pad 2: /I2C2_SCL -> Net-(IC1-1GATE)
- R13 pad 1: +3V3 -> /I2C2_SDA
- R13 pad 2: /I2C2_SDA -> Net-(IC1-2DRAIN_1)
Routing:
- net +3.3V: track 52.6 -> 35.6 mm, vias 17 -> 16
- net GND: track 85.1 -> 73.0 mm
- net Net-(IC1-1GATE): track 0.00 -> 7.28 mm, vias 0 -> 1
- net /I2C2_SCL: track 31.5 -> 24.3 mm, vias 3 -> 2
- net /I2C2_SDA: track 29.6 -> 22.8 mm, vias 3 -> 2
- net /PA8: track 19.6 -> 13.0 mm, vias 3 -> 1
- net +3V3: track 4.66 -> 0.00 mm
- net Net-(IC1-1DRAIN_1): track 0.00 -> 2.56 mm, vias 0 -> 2
- net Net-(IC1-2DRAIN_1): track 0.00 -> 2.48 mm, vias 0 -> 1
- added copper zone on B.Cu, net +3.3V
