File: CAN.kicad_sch (KiCad schematic)
At the start: 15 parts, among them U17 ADM3055E, U18 CDSOT23-T24CAN

Commit message: v1.2 initial changes
Parts:
- removed C33, C38: 10uF, Capacitor_SMD:C_0805_2012Metric, symbol Device:C_Small
- removed C34: 100nF, Capacitor_SMD:C_0805_2012Metric, symbol Device:C_Small
- removed C36: 0.01uF, Capacitor_SMD:C_0805_2012Metric, symbol Device:C_Small
- removed C37: 0.22uF, Capacitor_SMD:C_0805_2012Metric, symbol Device:C_Small
- removed C40: 10nF, Capacitor_SMD:C_0805_2012Metric, symbol Device:C_Small
- removed JP2: Termination Resistors, Connector_PinHeader_2.54mm:PinHeader_1x02_P2.54mm_Vertical, symbol Device:Jumper_NC_Small
- removed L7, L8: 2kH, Inductor_SMD:L_0805_2012Metric, symbol Device:Ferrite_Bead_Small
- removed R34: 0, Resistor_SMD:R_0805_2012Metric, symbol Device:R
- removed U17: ADM3055E, UTSVT_ICs:SOIC-20W_7.5x15.4mm_Pitch1.27mm, symbol Dashboard-rescue:ADM3055E-utsvt-chips
- removed U18: CDSOT23-T24CAN, Package_TO_SOT_SMD:SOT-23W, symbol Dashboard-rescue:CDSOT23-T24CAN-utsvt-chips
- added JP2: Termination Resistors, Connector_PinHeader_2.54mm:PinHeader_1x02_P2.54mm_Vertical, symbol Jumper:Jumper_2_Open
- added U2: ISO1044BD, Package_SO:SSOP-8_3.9x5.05mm_P1.27mm, symbol utsvt-chips:ISO1044BD
- added U5: CDSOT23-T24CAN, Package_TO_SOT_SMD:SOT-23W, symbol utsvt-chips:CDSOT23-T24CAN
Connections:
- net +3.3V: now also U2.1 (VCC1)
- net CAN_HIGH: now also U2.6 (CANH), U5.1 (CAN_H)
- net CAN_LOW: now also JP2.1 (A), U2.5 (CANL), U5.2 (CAN_L)
- net CAN_RX: now also U2.3 (RXD)
- net CAN_TX: now also U2.2 (TXD)
- net GND: now also U2.4 (GND1)
- net GND1: now also U2.7 (GND2), U5.3 (GND)
- net TERM_H: now also JP2.2 (B)
- net V_CAN_IN: now also U2.8 (VCC2)
- no-connect marks 2 -> 0
Other:
- note removed: "Must be close to V_ISO_In"
- note removed: "Must be close to V_ISO_Out"
