File: CAN.kicad_sch (KiCad schematic)
At the start: 0 parts

Commit message: lower OVP
Parts:
- added U4: TCAN337, UTSVT_ICs:TCAN337DCNR, symbol utsvt_ics:TCAN337
Other:
- note removed: "add TCAN337 from other branch (check against ds)"
- title: (none) -> CAN
Changed lines of the file:
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@@
 	(generator "eeschema")
 	(generator_version "9.0")
-	(paper "A4")
-	(text "add TCAN337 from other branch (check against ds)"
+	(paper "A5")
+	(title_block
+		(title "CAN")
+	)
+	(symbol
+		(lib_id "utsvt_ics:TCAN337")
+		(at 66.04 55.88 0)
+		(unit 1)
 		(exclude_from_sim no)
-		(at 155.956 101.6 0)
-		(effects
-			(font
-				(size 1.27 1.27)
-				(color 255 0 0 1)
+		(in_bom yes)
+		(on_board yes)
+		(dnp no)
+		(fields_autoplaced yes)
+		(property "Reference" "U4"
+			(at 68.1833 43.18 0)
+			(effects
+				(font
+					(size 1.27 1.27)
+				)
+				(justify left)
 			)
 		)
+		(property "Value" "TCAN337"
+			(at 68.1833 45.72 0)
+			(effects
+				(font
+					(size 1.27 1.27)
+				)
+				(justify left)
+			)
+		)
+		(property "Footprint" "UTSVT_ICs:TCAN337DCNR"
+			(at 66.04 68.58 0)
+			(effects
+				(font
+					(size 1.27 1.27)
+					(italic yes)
+				)
+				(hide yes)
+			)
+		)
+		(property "Datasheet" "http://www.ti.com/lit/ds/symlink/tcan337.pdf"
+			(at 66.04 55.88 0)
+			(effects
+				(font
+					(size 1.27 1.27)
+				)
+				(hide yes)
+			)
+		)
+		(property "Description" "High-Speed CAN Transceiver, 1Mbps, 3.3V supply, silent mode, fault output, SOT-23-8/SOIC-8"
+			(at 66.04 55.88 0)
+			(effects
+				(font
+					(size 1.27 1.27)
+				)
+				(hide yes)
+			)
+		)
+		(property "P/N" "TCAN337DCNR"
+			(at 66.04 55.88 0)
+			(effects
+				(font
+					(size 1.27 1.27)
+				)
+				(hide yes)
+			)
+		)
+		(pin "8"
+		)
+		(pin "3"
+		)
+		(pin "1"
+		)
+		(pin "4"
+		)
+		(pin "5"
+		)
+		(pin "2"
+		)
+		(pin "6"
+		)
+		(pin "7"
+		)
+		(instances
+			(project ""
+				(path "/d5ebd247-5a7c-47c2-8aee-beabaef72d6d/1d0c269d-60cf-499b-bfd2-5087981d6678"
+					(reference "U4")
+					(unit 1)
+				)
+			)
+		)

Commit message: add CAN
Parts:
- added C19: 1uF, symbol Device:C
- added C24: 0.1uF, symbol Device:C
- added D3: FAULT, symbol Device:LED
- added JP1: CAN TERM, symbol Jumper:Jumper_2_Open
- added R4: 10k, symbol Device:R
- added R5: 2.1k, symbol Device:R
- added R7: 120, symbol Device:R
- added U5: CDSOT23-T24CAN, UTSVT_ICs:CDSOT23-T24CAN, symbol utsvt_ics:CDSOT23-T24CAN
Connections:
- net CAN_TX: now reaches U4.1 (TXD)
- net GND: now reaches U4.2 (GND)
- net GND: now also C19.2, C24.2, D3.1 (K), U5.3 (GND)
- net +3.3V: now reaches U4.3 (VCC)
- net +3.3V: now also C19.1, C24.1, R4.1
- net CAN_RX: now reaches U4.4 (RXD)
- net FAULT: now reaches U4.5 (FAULT)
- net FAULT: now also R4.2, R5.1
- net CAN_L: now reaches U4.6 (CANL)
- net CAN_L: now also R7.2, U5.2 (CAN_L)
- net CAN_H: now reaches U4.7 (CANH)
- net CAN_H: now also JP1.1 (A), U5.1 (CAN_H)
- new net: JP1.2 (B), R7.1
- new net: D3.2 (A), R5.2
- no-connect marks 0 -> 1
Other:
- note added: "CAN Bus Protection"
- note added: "CAN Bus Termination"
- note added: "CAN Transceiver"
- moved on the sheet: U4

Commit message: finish mcu breakouts
Connections:
- net CAN_RX renamed CAN1_RX
- net CAN_TX renamed CAN1_TX
Other:
- moved on the sheet: C19, C24, D3, R5, U4

Commit message: twinkle
Parts:
- R5: value 2.1k -> 120
Changed lines of the file:
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@@
 			)
 		)
-		(property "Value" "2.1k"
+		(property "Value" "120"
 			(at 114.3 40.6399 0)
 			(effects

Commit message: FUCK capacitors
Parts:
- C19: P/N (none) -> MLASU168SB5105KTNA01
- C24: P/N (none) -> MLASH168SB7104KTNA01
- D3: P/N (none) -> APTD2012LSURCK
Changed lines of the file:
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@@
+			)
+		)
+		(property "P/N" "MLASH168SB7104KTNA01"
+			(at 35.56 39.37 0)
+			(effects
+				(font
+					(size 1.27 1.27)
+				)
+				(hide yes)
 			)
 		)
@@
 			)
 		)
+		(property "P/N" "MLASU168SB5105KTNA01"
+			(at 24.13 39.37 0)
+			(effects
+				(font
+					(size 1.27 1.27)
+				)
+				(hide yes)
+			)
+		)
 		(pin "2"
 		)
@@
 			)
 		)
-		(property "Datasheet" "~"
+		(property "Datasheet" "https://www.kingbrightusa.com/images/catalog/spec/aptd2012lsurck.pdf"
 			(at 111.76 49.53 0)
 			(effects
@@
 			(effects
 				(font
+					(size 1.27 1.27)
+				)
+				(hide yes)
+			)
+		)
+		(property "P/N" "APTD2012LSURCK"
+			(at 111.76 49.53 90)
+			(effects
+				(font

Commit message: all parts selected
Parts:
- JP1: P/N (none) -> QPC02SXGN-RC
- R4: P/N (none) -> CRCW060310K0FKEI
- R5, R7: P/N (none) -> CRCW0603120RFKEC
Changed lines of the file:
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@@
+			)
+		)
+		(property "P/N" "CRCW0603120RFKEC "
+			(at 157.48 64.77 90)
+			(effects
+				(font
+					(size 1.27 1.27)
+				)
+				(hide yes)
 			)
 		)
@@
 			)
 		)
+		(property "P/N" "CRCW060310K0FKEI "
+			(at 49.53 39.37 0)
+			(effects
+				(font
+					(size 1.27 1.27)
+				)
+				(hide yes)
+			)
+		)
 		(pin "2"
 		)
@@
 			)
 		)
+		(property "P/N" "CRCW0603120RFKEC "
+			(at 111.76 39.37 0)
+			(effects
+				(font
+					(size 1.27 1.27)
+				)
+				(hide yes)
+			)
+		)
 		(pin "2"
 		)
@@
 			(at 144.78 64.77 0)
 			(effects
+				(font
+					(size 1.27 1.27)
+				)
+				(hide yes)
+			)
+		)
+		(property "P/N" "QPC02SXGN-RC "
+			(at 144.78 64.77 0)
+			(effects

Commit message: add some footprints
Parts:
- JP1: footprint (none) -> Connector_PinHeader_2.54mm:PinHeader_1x02_P2.54mm_Vertical
- R4, R5, R7: footprint (none) -> Resistor_SMD:R_0603_1608Metric_Pad0.98x0.95mm_HandSolder
Changed lines of the file:
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@@
 			)
 		)
-		(property "Footprint" ""
+		(property "Footprint" "Resistor_SMD:R_0603_1608Metric_Pad0.98x0.95mm_HandSolder"
 			(at 157.48 66.548 90)
 			(effects
@@
 			)
 		)
-		(property "Footprint" ""
+		(property "Footprint" "Resistor_SMD:R_0603_1608Metric_Pad0.98x0.95mm_HandSolder"
 			(at 47.752 39.37 90)
 			(effects
@@
 			)
 		)
-		(property "Footprint" ""
+		(property "Footprint" "Resistor_SMD:R_0603_1608Metric_Pad0.98x0.95mm_HandSolder"
 			(at 109.982 39.37 90)
 			(effects
@@
 			)
 		)
-		(property "Footprint" ""
+		(property "Footprint" "Connector_PinHeader_2.54mm:PinHeader_1x02_P2.54mm_Vertical"
 			(at 144.78 64.77 0)
 			(effects
