File: CAN.kicad_sch (KiCad schematic)
At the start: 9 parts, among them U4 TCAN337, U5 CDSOT23-T24CAN

Commit message: all footprints assigned
Parts:
- C19, C24: footprint (none) -> Capacitor_SMD:C_0603_1608Metric_Pad1.08x0.95mm_HandSolder
- D3: footprint (none) -> LED_SMD:LED_0805_2012Metric_Pad1.15x1.40mm_HandSolder
Changed lines of the file:
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@@
 			)
 		)
-		(property "Footprint" ""
+		(property "Footprint" "Capacitor_SMD:C_0603_1608Metric_Pad1.08x0.95mm_HandSolder"
 			(at 36.5252 43.18 0)
 			(effects
@@
 			)
 		)
-		(property "Footprint" ""
+		(property "Footprint" "Capacitor_SMD:C_0603_1608Metric_Pad1.08x0.95mm_HandSolder"
 			(at 25.0952 43.18 0)
 			(effects
@@
 			)
 		)
-		(property "Footprint" ""
+		(property "Footprint" "LED_SMD:LED_0805_2012Metric_Pad1.15x1.40mm_HandSolder"
 			(at 111.76 49.53 0)
 			(effects

Commit message: CAN layout
Parts:
- JP1: value CAN TERM -> TRM
Changed lines of the file:
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@@
 			)
 		)
-		(property "Value" "CAN TERM"
+		(property "Value" "TRM"
 			(at 144.78 60.96 0)
 			(effects

Commit message: erm hii
Connections:
- net CAN_H: now also R7.1; no longer JP1.1 (A)
- net CAN_L: now also JP1.2 (B); no longer R7.2
- new net: JP1.1 (A), R7.2
Other:
- moved on the sheet: JP1, R7
Changed lines of the file:
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@@
 	(wire
 		(pts
-			(xy 149.86 64.77) (xy 153.67 64.77)
+			(xy 147.32 64.77) (xy 151.13 64.77)
 		)
 		(stroke
@@
 	(symbol
 		(lib_id "Device:R")
-		(at 157.48 64.77 90)
+		(at 143.51 64.77 90)
 		(unit 1)
 		(exclude_from_sim no)
@@
 		(fields_autoplaced yes)
 		(property "Reference" "R7"
-			(at 157.48 58.42 90)
+			(at 143.51 58.42 90)
 			(effects
 				(font
@@
 		)
 		(property "Value" "120"
-			(at 157.48 60.96 90)
+			(at 143.51 60.96 90)
 			(effects
 				(font
@@
 		)
 		(property "Footprint" "Resistor_SMD:R_0603_1608Metric_Pad0.98x0.95mm_HandSolder"
-			(at 157.48 66.548 90)
+			(at 143.51 66.548 90)
 			(effects
 				(font
@@
 		)
 		(property "Datasheet" "~"
-			(at 157.48 64.77 0)
+			(at 143.51 64.77 0)
 			(effects
 				(font
@@
 		)
 		(property "Description" "Resistor"
-			(at 157.48 64.77 0)
+			(at 143.51 64.77 0)
 			(effects
 				(font
@@
 		)
 		(property "P/N" "CRCW0603120RFKEC "
-			(at 157.48 64.77 90)
+			(at 143.51 64.77 90)
 			(effects
 				(font
@@
 	(symbol
 		(lib_id "Jumper:Jumper_2_Open")
-		(at 144.78 64.77 0)
+		(at 156.21 64.77 0)
 		(unit 1)
 		(exclude_from_sim no)
@@
 		(fields_autoplaced yes)
 		(property "Reference" "JP1"
-			(at 144.78 58.42 0)
+			(at 156.21 58.42 0)
 			(effects
 				(font
@@
 		)
 		(property "Value" "TRM"
-			(at 144.78 60.96 0)
+			(at 156.21 60.96 0)
 			(effects
 				(font
@@
 		)
 		(property "Footprint" "Connector_PinHeader_2.54mm:PinHeader_1x02_P2.54mm_Vertical"
-			(at 144.78 64.77 0)
+			(at 156.21 64.77 0)
 			(effects
 				(font
@@
 		)
 		(property "Datasheet" "~"
-			(at 144.78 64.77 0)
+			(at 156.21 64.77 0)
 			(effects
 				(font
@@
 		)
 		(property "Description" "Jumper, 2-pole, open"
-			(at 144.78 64.77 0)
+			(at 156.21 64.77 0)
 			(effects
 				(font
@@
 		)
 		(property "P/N" "QPC02SXGN-RC "
-			(at 144.78 64.77 0)
-			(effects
-				(font
+			(at 156.21 64.77 0)
+			(effects
+				(font

Commit message: add some lcsc parts
Parts:
- D3: value FAULT -> FLT
Changed lines of the file:
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@@
 			)
 		)
-		(property "Value" "FAULT"
+		(property "Value" "FLT"
 			(at 115.57 52.3874 90)
 			(effects

Commit message: type shi
Parts:
- D3: value FLT -> CFLT
Changed lines of the file:
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@@
 			)
 		)
-		(property "Value" "FLT"
+		(property "Value" "CFLT"
 			(at 115.57 52.3874 90)
 			(effects

Commit message: reroute uart, change leds to 0603
Parts:
- D3: footprint LED_SMD:LED_0805_2012Metric_Pad1.15x1.40mm_HandSolder -> LED_SMD:LED_0603_1608Metric_Pad1.05x0.95mm_HandSolder
Changed lines of the file:
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@@
 			)
 		)
-		(property "Footprint" "LED_SMD:LED_0805_2012Metric_Pad1.15x1.40mm_HandSolder"
+		(property "Footprint" "LED_SMD:LED_0603_1608Metric_Pad1.05x0.95mm_HandSolder"
 			(at 111.76 49.53 0)
 			(effects

Commit message: skill issue
Parts:
- D3: P/N APTD2012LSURCK -> NCD0603R1
Changed lines of the file:
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@@
 			)
 		)
-		(property "Datasheet" "https://www.kingbrightusa.com/images/catalog/spec/aptd2012lsurck.pdf"
+		(property "Datasheet" "https://www.lcsc.com/datasheet/C84263.pdf"
 			(at 111.76 49.53 0)
 			(effects
@@
 			)
 		)
-		(property "P/N" "APTD2012LSURCK"
+		(property "P/N" "NCD0603R1"
 			(at 111.76 49.53 90)
 			(effects
