File: PowerDist.kicad_sch (KiCad schematic)
At the start: 18 parts, among them P2 1769405141, Q1 PBSS4330X,135, Q1 Q_PMOS_GSD, U6 LP5912-3.3DRV

Commit message: neato
Parts:
- removed FB1: 5VFB, Inductor_SMD:L_0805_2012Metric, symbol Device:FerriteBead_Small
- C5, C6: value 10uF -> 1uF; Mouser Part Number 581-0805YC106KAT2A -> Inventory; P/N 0805YC106KAT2A -> Inventory
- R5: value 1k -> 2.2k; Mouser Part Number 71-CRCW0805-21.5K-E3 -> Inventory; P/N CRCW080521K5FKEA -> Inventory
- TP1, TP2, TP3, TP4: footprint TestPoint:TestPoint_Pad_1.5x1.5mm -> Connector_PinHeader_2.54mm:PinHeader_1x01_P2.54mm_Vertical
- U6: footprint Package_SON:WSON-6-1EP_2x2mm_P0.65mm_EP1x1.6mm_ThermalVias -> Package_SON:WSON-6-1EP_2x2mm_P0.65mm_EP1x1.6mm
Connections:
- net 5V_Ferrite is gone; now on net 5V_Ext: D6.2 (A2), Q1.3 (D)
Changed lines of the file:
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@@
-    (stroke (width 0) (type default))
-  )
-  (wire (pts (xy 76.2 83.82) (xy 80.01 83.82))
     (stroke (width 0) (type default))
   )
@@
     (stroke (width 0) (type default))
   )
-  (wire (pts (xy 60.325 83.82) (xy 71.12 83.82))
+  (wire (pts (xy 60.325 83.82) (xy 80.01 83.82))
     (stroke (width 0) (type default))
   )
@@
       (effects (font (size 1.27 1.27)) (justify left))
     )
-    (property "Footprint" "TestPoint:TestPoint_Pad_1.5x1.5mm" (at 174.625 70.485 0)
+    (property "Footprint" "Connector_PinHeader_2.54mm:PinHeader_1x01_P2.54mm_Vertical" (at 174.625 70.485 0)
       (effects (font (size 1.27 1.27)) hide)
     )
@@
       (effects (font (size 1.27 1.27)) (justify left))
     )
-    (property "Value" "10uF" (at 275.336 88.773 0)
+    (property "Value" "1uF" (at 275.336 88.773 0)
       (effects (font (size 1.27 1.27)) (justify left))
     )
@@
       (effects (font (size 1.27 1.27)) hide)
     )
-    (property "Datasheet" "https://www.mouser.com/datasheet/2/40/AVX_X7RDielectric_777024-1853642.pdf" (at 272.415 87.63 0)
-      (effects (font (size 1.27 1.27)) hide)
-    )
-    (property "P/N" "0805YC106KAT2A" (at 272.415 87.63 0)
-      (effects (font (size 1.27 1.27)) hide)
-    )
-    (property "Mouser Part Number" "581-0805YC106KAT2A" (at 272.415 87.63 0)
+    (property "Datasheet" "" (at 272.415 87.63 0)
+      (effects (font (size 1.27 1.27)) hide)
+    )
+    (property "P/N" "Inventory" (at 272.415 87.63 0)
+      (effects (font (size 1.27 1.27)) hide)
+    )
+    (property "Mouser Part Number" "Inventory" (at 272.415 87.63 0)
       (effects (font (size 1.27 1.27)) hide)
     )
@@
     )
   )
-  (symbol (lib_id "Device:FerriteBead_Small") (at 73.66 83.82 270) (unit 1)
-    (in_bom yes) (on_board yes) (dnp no)
-    (property "Reference" "FB1" (at 73.025 89.535 90)
-      (effects (font (size 1.27 1.27)))
-    )
-    (property "Value" "5VFB" (at 73.025 86.995 90)
-      (effects (font (size 1.27 1.27)))
-    )
-    (property "Footprint" "Inductor_SMD:L_0805_2012Metric" (at 73.66 82.042 90)
-      (effects (font (size 1.27 1.27)) hide)
-    )
-    (property "Datasheet" "https://www.mouser.com/datasheet/2/87/eaton_mfbw1v2012_high_impedance_multilayer_ferrite-1916871.pdf" (at 73.66 83.82 0)
-      (effects (font (size 1.27 1.27)) hide)
-    )
-    (property "P/N" "MFBW1V2012-121-R" (at 73.66 83.82 90)
-      (effects (font (size 1.27 1.27)) hide)
-    )
-    (property "Mouser Part Number" "704-MFBW1V2012-121-R" (at 73.66 83.82 0)
-      (effects (font (size 1.27 1.27)) hide)
-    )
-    (pin "1")
-    (pin "2")
-    (instances
-      (project "Controls-LightingPCB"
-        (path "/229b82f0-5048-47d6-8bc8-0bcee42eb4bc"
-          (reference "FB1") (unit 1)
-        )
-      )
-      (project "BPS-PeripheralSOM"
-        (path "/d5ebd247-5a7c-47c2-8aee-beabaef72d6d"
-          (reference "FB2") (unit 1)
-        )
-        (path "/d5ebd247-5a7c-47c2-8aee-beabaef72d6d/60a4ab70-544e-48ed-aa76-f39bfcac39df"
-          (reference "FB2") (unit 1)
-        )
-      )
-    )
-  )
   (symbol (lib_id "Transistor_BJT:2N2219") (at 216.535 82.55 90) (unit 1)
     (in_bom yes) (on_board yes) (dnp no) (fields_autoplaced)
@@
       (effects (font (size 1.27 1.27)))
     )
-    (property "Footprint" "Package_SON:WSON-6-1EP_2x2mm_P0.65mm_EP1x1.6mm_ThermalVias" (at 252.095 73.66 0)
+    (property "Footprint" "Package_SON:WSON-6-1EP_2x2mm_P0.65mm_EP1x1.6mm" (at 252.095 73.66 0)
       (effects (font (size 1.27 1.27)) hide)
     )
@@
       (effects (font (size 1.27 1.27)) (justify right))
     )
-    (property "Footprint" "TestPoint:TestPoint_Pad_1.5x1.5mm" (at 172.72 120.015 0)
+    (property "Footprint" "Connector_PinHeader_2.54mm:PinHeader_1x01_P2.54mm_Vertical" (at 172.72 120.015 0)
       (effects (font (size 1.27 1.27)) hide)
     )
@@
       (effects (font (size 1.27 1.27)) (justify left))
     )
-    (property "Value" "10uF" (at 230.886 86.233 0)
+    (property "Value" "1uF" (at 230.886 86.233 0)
       (effects (font (size 1.27 1.27)) (justify left))
     )
@@
       (effects (font (size 1.27 1.27)) hide)
     )
-    (property "Datasheet" "https://www.mouser.com/datasheet/2/40/AVX_X7RDielectric_777024-1853642.pdf" (at 227.965 85.09 0)
-      (effects (font (size 1.27 1.27)) hide)
-    )
-    (property "P/N" "0805YC106KAT2A" (at 227.965 85.09 0)
-      (effects (font (size 1.27 1.27)) hide)
-    )
-    (property "Mouser Part Number" "581-0805YC106KAT2A" (at 227.965 85.09 0)
+    (property "Datasheet" "" (at 227.965 85.09 0)
+      (effects (font (size 1.27 1.27)) hide)
+    )
+    (property "P/N" "Inventory" (at 227.965 85.09 0)
+      (effects (font (size 1.27 1.27)) hide)
+    )
+    (property "Mouser Part Number" "Inventory" (at 227.965 85.09 0)
       (effects (font (size 1.27 1.27)) hide)
     )
@@
       (effects (font (size 1.27 1.27)) (justify left))
     )
-    (property "Value" "1k" (at 37.338 138.938 0)
+    (property "Value" "2.2k" (at 37.338 138.938 0)
       (effects (font (size 1.27 1.27)) (justify left))
     )
@@
       (effects (font (size 1.27 1.27)) hide)
     )
-    (property "Datasheet" "https://www.mouser.com/ProductDetail/Vishay-Dale/CRCW080521K5FKEA?qs=qpzLseAzoKqvp1KNYFXGvQ%3D%3D" (at 35.56 137.795 0)
-      (effects (font (size 1.27 1.27)) hide)
-    )
-    (property "P/N" "CRCW080521K5FKEA" (at 35.56 137.795 0)
-      (effects (font (size 1.27 1.27)) hide)
-    )
-    (property "Mouser Part Number" "71-CRCW0805-21.5K-E3" (at 35.56 137.795 0)
+    (property "Datasheet" "~" (at 35.56 137.795 0)
+      (effects (font (size 1.27 1.27)) hide)
+    )
+    (property "P/N" "Inventory" (at 35.56 137.795 0)
+      (effects (font (size 1.27 1.27)) hide)
+    )
+    (property "Mouser Part Number" "Inventory" (at 35.56 137.795 0)
       (effects (font (size 1.27 1.27)) hide)
     )
@@
       (effects (font (size 1.27 1.27)) (justify right))
     )
-    (property "Footprint" "TestPoint:TestPoint_Pad_1.5x1.5mm" (at 108.585 103.505 0)
+    (property "Footprint" "Connector_PinHeader_2.54mm:PinHeader_1x01_P2.54mm_Vertical" (at 108.585 103.505 0)
       (effects (font (size 1.27 1.27)) hide)
     )
@@
       (effects (font (size 1.27 1.27)) (justify left))
     )
-    (property "Footprint" "TestPoint:TestPoint_Pad_1.5x1.5mm" (at 112.395 81.28 0)
-      (effects (font (size 1.27 1.27)) hide)
-    )
+    (property "Footprint" "Connector_PinHeader_2.54mm:PinHeader_1x01_P2.54mm_Vertical" (at 112.395 81.28 0)
+      (effects (font (size 1.27 1.27)) hide)
+    )

Commit message: routed
Parts:
- Q1: symbol Transistor_BJT:2N2219 -> Transistor_BJT:2SC1815
- TP1: value +5V_TP -> +5V_ISO_TP
- TP3: value +5V_TP -> +3V3_TP
Connections:
- net +3.3V: now also TP3.1
- net +5V: now also Q1.2 (C); no longer Q1.3 (C), TP3.1
- net +5V_ISO: now reaches C21.1, P2.2 (+VIN), Q1.2 (S), TP1.1
- net at C4.1, R3.2: now also Q1.3 (B); no longer Q1.2 (B)
Changed lines of the file:
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@@
   (junction (at 170.18 117.475) (diameter 0) (color 0 0 0 0)
   )
-  (junction (at 165.1 71.755) (diameter 0) (color 0 0 0 0)
-  )
   (junction (at 107.315 83.82) (diameter 0) (color 0 0 0 0)
   )
   (junction (at 80.01 102.235) (diameter 0) (color 0 0 0 0)
+  )
+  (junction (at 264.16 80.01) (diameter 0) (color 0 0 0 0)
   )
   (junction (at 247.015 92.71) (diameter 0) (color 0 0 0 0)
@@
     (stroke (width 0) (type default))
   )
+  (wire (pts (xy 264.16 80.01) (xy 272.415 80.01))
+    (stroke (width 0) (type default))
+  )
   (wire (pts (xy 158.75 117.475) (xy 170.18 117.475))
     (stroke (width 0) (type default))
@@
     (stroke (width 0) (type default))
   )
-  (wire (pts (xy 262.255 80.01) (xy 272.415 80.01))
+  (wire (pts (xy 262.255 80.01) (xy 264.16 80.01))
     (stroke (width 0) (type default))
   )
@@
     (stroke (width 0) (type default))
   )
-  (wire (pts (xy 169.545 70.485) (xy 169.545 71.755))
-    (stroke (width 0) (type default))
-  )
   (wire (pts (xy 35.56 131.445) (xy 35.56 133.985))
     (stroke (width 0) (type default))
@@
   )
   (wire (pts (xy 35.56 142.875) (xy 35.56 141.605))
-    (stroke (width 0) (type default))
-  )
-  (wire (pts (xy 165.1 71.755) (xy 169.545 71.755))
     (stroke (width 0) (type default))
   )
@@
     (effects (font (size 1.27 1.27)) (justify left bottom))
   )
+  (global_label "+5V_ISO" (shape output) (at 107.315 83.82 0) (fields_autoplaced)
+    (effects (font (size 1.27 1.27)) (justify left))
+    (property "Intersheetrefs" "${INTERSHEET_REFS}" (at 118.2037 83.82 0)
+      (effects (font (size 1.27 1.27)) (justify left) hide)
+    )
+  )
   (hierarchical_label "5V_Ext" (shape input) (at 55.245 83.82 180) (fields_autoplaced)
     (effects (font (size 1.27 1.27)) (justify right))
@@
     )
   )
-  (symbol (lib_id "Connector:TestPoint") (at 169.545 70.485 0) (unit 1)
-    (in_bom yes) (on_board yes) (dnp no)
-    (property "Reference" "TP3" (at 171.0182 67.437 0)
-      (effects (font (size 1.27 1.27)) (justify left))
-    )
-    (property "Value" "+5V_TP" (at 171.0182 69.7484 0)
-      (effects (font (size 1.27 1.27)) (justify left))
-    )
-    (property "Footprint" "Connector_PinHeader_2.54mm:PinHeader_1x01_P2.54mm_Vertical" (at 174.625 70.485 0)
-      (effects (font (size 1.27 1.27)) hide)
-    )
-    (property "Datasheet" "https://www.mouser.com/datasheet/2/215/5005_5009-741322.pdf" (at 174.625 70.485 0)
-      (effects (font (size 1.27 1.27)) hide)
-    )
-    (property "P/N" "5005" (at 169.545 70.485 0)
-      (effects (font (size 1.27 1.27)) hide)
-    )
-    (property "Mouser Part Number" "534-5005" (at 169.545 70.485 0)
-      (effects (font (size 1.27 1.27)) hide)
-    )
-    (pin "1")
-    (instances
-      (project "Telemetry-Primary"
-        (path "/7f2a449b-14af-42b3-8d38-5f0f8a5ee7ce/00000000-0000-0000-0000-00005f6cdfd6"
-          (reference "TP3") (unit 1)
-        )
-      )
-      (project "BPS-PeripheralSOM"
-        (path "/d5ebd247-5a7c-47c2-8aee-beabaef72d6d/60a4ab70-544e-48ed-aa76-f39bfcac39df"
-          (reference "TP5") (unit 1)
-        )
-      )
-    )
-  )
   (symbol (lib_id "Device:C") (at 272.415 87.63 0) (unit 1)
     (in_bom yes) (on_board yes) (dnp no)
@@
     )
   )
-  (symbol (lib_id "Transistor_BJT:2N2219") (at 216.535 82.55 90) (unit 1)
+  (symbol (lib_id "Transistor_BJT:2SC1815") (at 216.535 82.55 90) (unit 1)
     (in_bom yes) (on_board yes) (dnp no) (fields_autoplaced)
     (property "Reference" "Q1" (at 216.535 74.93 90)
@@
         (path "/d5ebd247-5a7c-47c2-8aee-beabaef72d6d/60a4ab70-544e-48ed-aa76-f39bfcac39df"
           (reference "Q2") (unit 1)
+        )
+      )
+    )
+  )
+  (symbol (lib_id "Connector:TestPoint") (at 264.16 80.01 0) (unit 1)
+    (in_bom yes) (on_board yes) (dnp no)
+    (property "Reference" "TP3" (at 265.6332 76.962 0)
+      (effects (font (size 1.27 1.27)) (justify left))
+    )
+    (property "Value" "+3V3_TP" (at 265.6332 79.2734 0)
+      (effects (font (size 1.27 1.27)) (justify left))
+    )
+    (property "Footprint" "Connector_PinHeader_2.54mm:PinHeader_1x01_P2.54mm_Vertical" (at 269.24 80.01 0)
+      (effects (font (size 1.27 1.27)) hide)
+    )
+    (property "Datasheet" "https://www.mouser.com/datasheet/2/215/5005_5009-741322.pdf" (at 269.24 80.01 0)
+      (effects (font (size 1.27 1.27)) hide)
+    )
+    (property "P/N" "5005" (at 264.16 80.01 0)
+      (effects (font (size 1.27 1.27)) hide)
+    )
+    (property "Mouser Part Number" "534-5005" (at 264.16 80.01 0)
+      (effects (font (size 1.27 1.27)) hide)
+    )
+    (pin "1")
+    (instances
+      (project "Telemetry-Primary"
+        (path "/7f2a449b-14af-42b3-8d38-5f0f8a5ee7ce/00000000-0000-0000-0000-00005f6cdfd6"
+          (reference "TP3") (unit 1)
+        )
+      )
+      (project "BPS-PeripheralSOM"
+        (path "/d5ebd247-5a7c-47c2-8aee-beabaef72d6d/60a4ab70-544e-48ed-aa76-f39bfcac39df"
+          (reference "TP1") (unit 1)
         )
       )
@@
       (effects (font (size 1.27 1.27)) (justify left))
     )
-    (property "Value" "+5V_TP" (at 108.585 80.645 0)
-      (effects (font (size 1.27 1.27)) (justify left))
-    )
+    (property "Value" "+5V_ISO_TP" (at 108.585 80.645 0)
+      (effects (font (size 1.27 1.27)) (justify left))
+    )
