File: PowerDist.kicad_sch (KiCad schematic)
At the start: 22 parts, among them U3 TPS562231DRLR, U4 CME0303S3C

Commit message: idk anymore man
Parts:
- removed L2: 10uH, Inductor_SMD:L_0805_2012Metric_Pad1.15x1.40mm_HandSolder, symbol Device:L
- removed U4: CME0303S3C, UTSVT_Power:CME0303S3C, symbol utsvt-power-regulators:CME0303S3C
Connections:
- net +12V: now also C24.1, C9.1
- net 3V3_Bus: no longer C24.1, C9.1
- net fault renamed Fault
Other:
- sheet PowerProtection ports: added 3V3_Bus; removed 3.3V_Uniso
Changed lines of the file:
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@@
 	)
 	(junction
-		(at 200.66 128.27)
-		(diameter 0)
-		(color 0 0 0 0)
-	)
-	(junction
 		(at 38.1 116.84)
 		(diameter 0)
@@
 	(wire
 		(pts
-			(xy 190.5 128.27) (xy 200.66 128.27)
-		)
-		(stroke
-			(width 0)
-			(type default)
-		)
-	)
-	(wire
-		(pts
 			(xy 52.07 116.84) (xy 52.07 119.38)
 		)
@@
 	(wire
 		(pts
-			(xy 132.08 120.65) (xy 134.62 120.65)
+			(xy 208.28 118.11) (xy 208.28 120.65)
 		)
 		(stroke
@@
 	(wire
 		(pts
-			(xy 208.28 118.11) (xy 208.28 120.65)
+			(xy 41.91 71.12) (xy 59.69 71.12)
 		)
 		(stroke
@@
 	(wire
 		(pts
-			(xy 41.91 71.12) (xy 59.69 71.12)
+			(xy 38.1 114.3) (xy 38.1 116.84)
 		)
 		(stroke
@@
 	(wire
 		(pts
-			(xy 38.1 114.3) (xy 38.1 116.84)
+			(xy 251.46 109.22) (xy 250.19 109.22)
 		)
 		(stroke
@@
 	(wire
 		(pts
-			(xy 251.46 109.22) (xy 250.19 109.22)
+			(xy 200.66 120.65) (xy 208.28 120.65)
 		)
 		(stroke
@@
 	(wire
 		(pts
-			(xy 200.66 120.65) (xy 208.28 120.65)
+			(xy 39.37 64.77) (xy 59.69 64.77)
 		)
 		(stroke
@@
 	(wire
 		(pts
-			(xy 39.37 64.77) (xy 59.69 64.77)
+			(xy 190.5 63.5) (xy 190.5 62.23)
 		)
 		(stroke
@@
 	(wire
 		(pts
-			(xy 190.5 63.5) (xy 190.5 62.23)
+			(xy 127 120.65) (xy 134.62 120.65)
+		)
+		(stroke
+			(width 0)
+			(type default)
+		)
+	)
+	(wire
+		(pts
+			(xy 127 118.11) (xy 127 120.65)
 		)
 		(stroke
@@
 	(text "Isolation"
 		(exclude_from_sim no)
-		(at 170.434 113.284 0)
+		(at 170.18 107.95 0)
 		(effects
 			(font
@@
 	(text "3.3V -> 3.3V (Isolated)"
 		(exclude_from_sim no)
-		(at 136.906 105.664 0)
+		(at 134.112 105.918 0)
 		(effects
 			(font
@@
 		)
 	)
-	(label "fault"
+	(label "Fault"
 		(at 245.11 139.7 0)
 		(fields_autoplaced yes)
@@
 		)
 	)
-	(label "fault"
+	(label "Fault"
 		(at 41.91 76.2 180)
 		(fields_autoplaced yes)
@@
 		)
 	)
-	(hierarchical_label "3V3_Uniso"
+	(hierarchical_label "3V3_Bus"
 		(shape output)
 		(at 41.91 71.12 180)
@@
 	(hierarchical_label "3V3_Bus"
 		(shape output)
-		(at 132.08 120.65 180)
-		(fields_autoplaced yes)
-		(effects
-			(font
-				(size 1.27 1.27)
-			)
-			(justify right)
-		)
-	)
-	(hierarchical_label "3V3_Bus"
-		(shape output)
 		(at 207.01 59.69 0)
 		(fields_autoplaced yes)
@@
 	)
 	(symbol
+		(lib_id "power:+12V")
+		(at 127 118.11 0)
+		(unit 1)
+		(exclude_from_sim no)
+		(in_bom yes)
+		(on_board yes)
+		(dnp no)
+		(fields_autoplaced yes)
+		(property "Reference" "#PWR065"
+			(at 127 121.92 0)
+			(effects
+				(font
+					(size 1.27 1.27)
+				)
+				(hide yes)
+			)
+		)
+		(property "Value" "+12V"
+			(at 127 113.03 0)
+			(effects
+				(font
+					(size 1.27 1.27)
+				)
+			)
+		)
+		(property "Footprint" ""
+			(at 127 118.11 0)
+			(effects
+				(font
+					(size 1.27 1.27)
+				)
+				(hide yes)
+			)
+		)
+		(property "Datasheet" ""
+			(at 127 118.11 0)
+			(effects
+				(font
+					(size 1.27 1.27)
+				)
+				(hide yes)
+			)
+		)
+		(property "Description" "Power symbol creates a global label with name \"+12V\""
+			(at 127 118.11 0)
+			(effects
+				(font
+					(size 1.27 1.27)
+				)
+				(hide yes)
+			)
+		)
+		(pin "1"
+		)
+		(instances
+			(project "BPS-PeripheralSOM"
+				(path "/d5ebd247-5a7c-47c2-8aee-beabaef72d6d/60a4ab70-544e-48ed-aa76-f39bfcac39df"
+					(reference "#PWR065")
+					(unit 1)
+				)
+			)
+		)
+	)
+	(symbol
 		(lib_id "power:GNDPWR")
 		(at 97.79 138.43 0)
@@
 	)
 	(symbol
-		(lib_id "Device:L")
-		(at 194.31 120.65 90)
-		(unit 1)
-		(exclude_from_sim no)
-		(in_bom yes)
-		(on_board yes)
-		(dnp no)
-		(fields_autoplaced yes)
-		(property "Reference" "L2"
-			(at 194.31 115.57 90)
-			(effects
-				(font
-					(size 1.27 1.27)
-				)
-			)
-		)
-		(property "Value" "10uH"
-			(at 194.31 118.11 90)
-			(effects
-				(font
-					(size 1.27 1.27)
-				)
-			)
-		)
-		(property "Footprint" "Inductor_SMD:L_0805_2012Metric_Pad1.15x1.40mm_HandSolder"
-			(at 194.31 120.65 0)
-			(effects
-				(font
-					(size 1.27 1.27)
-				)
-				(hide yes)
-			)
-		)
-		(property "Datasheet" "~"
-			(at 194.31 120.65 0)
-			(effects
-				(font
-					(size 1.27 1.27)
-				)
-				(hide yes)
-			)
-		)
-		(property "Description" "Inductor"
-			(at 194.31 120.65 0)
-			(effects
-				(font
-					(size 1.27 1.27)
-				)
-				(hide yes)
-			)
-		)
-		(property "P/N" "MLZ2012N100LT000 "
-			(at 194.31 120.65 90)
-			(effects
-				(font
-					(size 1.27 1.27)
-				)
-				(hide yes)
-			)
-		)
-		(pin "1"
-		)
-		(pin "2"
-		)
-		(instances
-			(project "BPS-PeripheralSOM"
-				(path "/d5ebd247-5a7c-47c2-8aee-beabaef72d6d/60a4ab70-544e-48ed-aa76-f39bfcac39df"
-					(reference "L2")
-					(unit 1)
-				)
-			)
-		)
-	)
-	(symbol
 		(lib_id "Connector:TestPoint")
 		(at 186.69 71.12 90)
@@
 		)
 	)
-	(symbol
-		(lib_id "utsvt-power-regulators:CME0303S3C")
-		(at 170.18 116.84 0)
-		(unit 1)
-		(exclude_from_sim no)
-		(in_bom yes)
-		(on_board yes)
-		(dnp no)
-		(property "Reference" "U4"
-			(at 170.18 108.712 0)
-			(effects
-				(font
-					(size 1.27 1.27)
-				)
-			)
-		)
-		(property "Value" "CME0303S3C"
-			(at 170.18 111.252 0)
-			(effects
-				(font
-					(size 1.27 1.27)
-				)
-			)
-		)
-		(property "Footprint" "UTSVT_Power:CME0303S3C"
-			(at 170.18 116.84 0)
-			(effects
-				(font
-					(size 1.27 1.27)
-				)
-				(hide yes)
-			)
-		)
-		(property "Datasheet" "https://www.murata.com/products/productdata/8807029342238/kdc-cme.pdf"
-			(at 170.18 116.84 0)
-			(effects
-				(font
-					(size 1.27 1.27)
-				)
-				(hide yes)
-			)
-		)
-		(property "Description" ""
-			(at 170.18 116.84 0)
-			(effects
-				(font
-					(size 1.27 1.27)
-				)
-				(hide yes)
-			)
-		)
-		(property "PN" "CME0303S3C"
-			(at 170.18 115.57 0)
-			(effects
-				(font
-					(size 1.27 1.27)
-				)
-				(hide yes)
-			)
-		)
-		(property "P/N" "CME0303S3C"
-			(at 170.18 116.84 0)
-			(effects
-				(font
-					(size 1.27 1.27)
-				)
-				(hide yes)
-			)
-		)
-		(pin "2"
-		)
-		(pin "4"
-		)
-		(pin "3"
-		)
-		(pin "1"
-		)
-		(instances
-			(project "BPS-PeripheralSOM"
-				(path "/d5ebd247-5a7c-47c2-8aee-beabaef72d6d/60a4ab70-544e-48ed-aa76-f39bfcac39df"
-					(reference "U4")
-					(unit 1)
-				)
-			)
-		)
-	)
 	(sheet
 		(at 59.69 60.452)
@@
 			)
 		)
-		(pin "3.3V_Uniso" output
+		(pin "3V3_Bus" output
 			(at 59.69 71.12 180)
 			(effects

Commit message: hi ishannnnnn
Parts:
- added U4: RO-123.3S, UTSVT_ICs:RI3_DC_Converter, symbol utsvt-power-regulators:RO-123.3S_HP
Connections:
- net +12V: now also U4.2 (+Vin)
- net +3.3V: now also U4.4 (+Vout)
- net GND: now also U4.3 (-Vout)
- net GNDPWR: now also U4.1 (-Vin)
Other:
- note added: "12V -> 3.3V (Isolated)"
- note added: "Max draw: 303 mA"
- note removed: "3.3V -> 3.3V (Isolated)"
- note removed: "Max draw: 227 mA"
- moved on the sheet: C8
Changed lines of the file:
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@@
 	)
 	(junction
+		(at 200.66 121.92)
+		(diameter 0)
+		(color 0 0 0 0)
+	)
+	(junction
+		(at 200.66 129.54)
+		(diameter 0)
+		(color 0 0 0 0)
+	)
+	(junction
 		(at 38.1 116.84)
 		(diameter 0)
@@
 	)
 	(junction
-		(at 200.66 120.65)
-		(diameter 0)
-		(color 0 0 0 0)
-	)
-	(junction
 		(at 48.26 124.46)
 		(diameter 0)
@@
 	(wire
 		(pts
-			(xy 92.71 129.54) (xy 97.79 129.54)
+			(xy 149.86 128.27) (xy 149.86 127)
 		)
 		(stroke
@@
 	(wire
 		(pts
-			(xy 200.66 128.27) (xy 200.66 129.54)
+			(xy 92.71 129.54) (xy 97.79 129.54)
 		)
 		(stroke
@@
 	(wire
 		(pts
+			(xy 149.86 121.92) (xy 149.86 120.65)
+		)
+		(stroke
+			(width 0)
+			(type default)
+		)
+	)
+	(wire
+		(pts
 			(xy 97.79 114.3) (xy 97.79 119.38)
 		)
@@
 	(wire
 		(pts
+			(xy 195.58 129.54) (xy 200.66 129.54)
+		)
+		(stroke
+			(width 0)
+			(type default)
+		)
+	)
+	(wire
+		(pts
 			(xy 190.5 71.12) (xy 186.69 71.12)
 		)
@@
 	(wire
 		(pts
+			(xy 181.61 127) (xy 195.58 127)
+		)
+		(stroke
+			(width 0)
+			(type default)
+		)
+	)
+	(wire
+		(pts
 			(xy 97.79 129.54) (xy 97.79 128.27)
 		)
@@
 	(wire
 		(pts
-			(xy 208.28 118.11) (xy 208.28 120.65)
+			(xy 208.28 118.11) (xy 208.28 121.92)
 		)
 		(stroke
@@
 	(wire
 		(pts
+			(xy 181.61 121.92) (xy 200.66 121.92)
+		)
+		(stroke
+			(width 0)
+			(type default)
+		)
+	)
+	(wire
+		(pts
 			(xy 38.1 114.3) (xy 38.1 116.84)
 		)
@@
 	(wire
 		(pts
-			(xy 200.66 120.65) (xy 208.28 120.65)
+			(xy 200.66 121.92) (xy 208.28 121.92)
 		)
 		(stroke
@@
 	(wire
 		(pts
+			(xy 158.75 121.92) (xy 149.86 121.92)
+		)
+		(stroke
+			(width 0)
+			(type default)
+		)
+	)
+	(wire
+		(pts
 			(xy 190.5 63.5) (xy 190.5 62.23)
 		)
@@
 	(wire
 		(pts
-			(xy 60.96 135.89) (xy 57.15 135.89)
+			(xy 149.86 127) (xy 158.75 127)
 		)
 		(stroke
@@
 	(wire
 		(pts
-			(xy 198.12 120.65) (xy 200.66 120.65)
+			(xy 60.96 135.89) (xy 57.15 135.89)
 		)
 		(stroke
@@
 	(wire
 		(pts
+			(xy 200.66 132.08) (xy 200.66 129.54)
+		)
+		(stroke
+			(width 0)
+			(type default)
+		)
+	)
+	(wire
+		(pts
 			(xy 134.62 120.65) (xy 146.05 120.65)
 		)
@@
 	(wire
 		(pts
+			(xy 195.58 127) (xy 195.58 129.54)
+		)
+		(stroke
+			(width 0)
+			(type default)
+		)
+	)
+	(wire
+		(pts
 			(xy 250.19 109.22) (xy 250.19 118.11)
 		)
@@
 		)
 	)
-	(text "3.3V -> 3.3V (Isolated)"
+	(text "12V -> 3.3V (Isolated)"
 		(exclude_from_sim no)
-		(at 134.112 105.918 0)
+		(at 133.604 105.918 0)
 		(effects
 			(font
@@
 		)
 	)
-	(text "Max draw: 227 mA"
+	(text "Max draw: 303 mA"
 		(exclude_from_sim no)
 		(at 131.064 153.416 0)
@@
 	(symbol
 		(lib_id "Device:C")
-		(at 200.66 124.46 0)
+		(at 200.66 125.73 0)
 		(unit 1)
 		(exclude_from_sim no)
@@
 		(fields_autoplaced yes)
 		(property "Reference" "C8"
-			(at 204.47 123.825 0)
+			(at 204.47 125.095 0)
 			(effects
 				(font
@@
 		)
 		(property "Value" "4.7uF"
-			(at 204.47 126.365 0)
+			(at 204.47 127.635 0)
 			(effects
 				(font
@@
 		)
 		(property "Footprint" "Capacitor_SMD:C_0805_2012Metric"
-			(at 201.6252 128.27 0)
+			(at 201.6252 129.54 0)
 			(effects
 				(font
@@
 		)
 		(property "Datasheet" "~"
-			(at 200.66 124.46 0)
+			(at 200.66 125.73 0)
 			(effects
 				(font
@@
 		)
 		(property "Description" "Unpolarized capacitor"
-			(at 200.66 124.46 0)
+			(at 200.66 125.73 0)
 			(effects
 				(font
@@
 		)
 		(property "Mouser Part Number" "81-GRM219R6YA475KA3D"
-			(at 200.66 124.46 0)
+			(at 200.66 125.73 0)
 			(effects
 				(font
@@
 		)
 		(property "P/N" "GRM219R6YA475KA73D"
-			(at 200.66 124.46 0)
+			(at 200.66 125.73 0)
 			(effects
 				(font
@@
 	(symbol
 		(lib_id "power:GND")
-		(at 200.66 129.54 0)
+		(at 200.66 132.08 0)
 		(unit 1)
 		(exclude_from_sim no)
@@
 		(fields_autoplaced yes)
 		(property "Reference" "#PWR06"
-			(at 200.66 135.89 0)
+			(at 200.66 138.43 0)
 			(effects
 				(font
@@
 		)
 		(property "Value" "GND"
-			(at 200.66 134.62 0)
+			(at 200.66 137.16 0)
 			(effects
 				(font
@@
 		)
 		(property "Footprint" ""
-			(at 200.66 129.54 0)
+			(at 200.66 132.08 0)
 			(effects
 				(font
@@
 		)
 		(property "Datasheet" ""
-			(at 200.66 129.54 0)
+			(at 200.66 132.08 0)
 			(effects
 				(font
@@
 		)
 		(property "Description" "Power symbol creates a global label with name \"GND\" , ground"
-			(at 200.66 129.54 0)
+			(at 200.66 132.08 0)
 			(effects
 				(font
@@
 					(unit 1)
 				)
+			)
+		)
+	)
+	(symbol
+		(lib_id "utsvt-power-regulators:RO-123.3S_HP")
+		(at 170.18 124.46 0)
+		(unit 1)
+		(exclude_from_sim no)
+		(in_bom yes)
+		(on_board yes)
+		(dnp no)
+		(property "Reference" "U4"
+			(at 169.926 110.236 0)
+			(effects
+				(font
+					(size 1.27 1.27)
+				)
+			)
+		)
+		(property "Value" "RO-123.3S"
+			(at 169.926 112.776 0)
+			(effects
+				(font
+					(size 1.27 1.27)
+				)
+			)
+		)
+		(property "Footprint" "UTSVT_ICs:RI3_DC_Converter"
+			(at 170.18 132.08 0)
+			(effects
+				(font
+					(size 1.27 1.27)
+				)
+				(hide yes)
+			)
+		)
+		(property "Datasheet" "https://www.mouser.com/datasheet/2/468/RO-1711124.pdf"
+			(at 170.18 132.08 0)
+			(effects
+				(font
+					(size 1.27 1.27)
+				)
+				(hide yes)
+			)
+		)
+		(property "Description" "Isolated DC/DC Converters 1W DC/DC 2kV UNREG 12Vin 3.3Vout"
+			(at 170.18 124.46 0)
+			(effects
+				(font
+					(size 1.27 1.27)
+				)
+				(hide yes)
+			)
+		)
+		(pin "1"
+		)
+		(pin "3"
+		)
+		(pin "4"
+		)
+		(pin "2"
+		)
+		(instances
+			(project "BPS-PeripheralSOM"
+				(path "/d5ebd247-5a7c-47c2-8aee-beabaef72d6d/60a4ab70-544e-48ed-aa76-f39bfcac39df"
+					(reference "U4")
+					(unit 1)
+				)
