File: PowerDist.kicad_sch (KiCad schematic)
At the start: 36 parts, among them U2 TPS5405DR, U3 LT1963AEST-3.3#TRPBF, U6 TPS2115ADRBR

Commit message: add some footprints
Parts:
- R25, R26, R28, R3, R8, R9: footprint (none) -> Resistor_SMD:R_0603_1608Metric_Pad0.98x0.95mm_HandSolder
Changed lines of the file:
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@@
 			)
 		)
-		(property "Footprint" ""
+		(property "Footprint" "Resistor_SMD:R_0603_1608Metric_Pad0.98x0.95mm_HandSolder"
 			(at 220.472 116.84 90)
 			(effects
@@
 			)
 		)
-		(property "Footprint" ""
+		(property "Footprint" "Resistor_SMD:R_0603_1608Metric_Pad0.98x0.95mm_HandSolder"
 			(at 71.882 132.08 90)
 			(effects
@@
 			)
 		)
-		(property "Footprint" ""
+		(property "Footprint" "Resistor_SMD:R_0603_1608Metric_Pad0.98x0.95mm_HandSolder"
 			(at 177.292 36.83 90)
 			(effects
@@
 			)
 		)
-		(property "Footprint" ""
+		(property "Footprint" "Resistor_SMD:R_0603_1608Metric_Pad0.98x0.95mm_HandSolder"
 			(at 266.7 98.552 90)
 			(effects
@@
 			)
 		)
-		(property "Footprint" ""
+		(property "Footprint" "Resistor_SMD:R_0603_1608Metric_Pad0.98x0.95mm_HandSolder"
 			(at 156.972 36.83 90)
 			(effects
@@
 			)
 		)
-		(property "Footprint" ""
+		(property "Footprint" "Resistor_SMD:R_0603_1608Metric_Pad0.98x0.95mm_HandSolder"
 			(at 167.132 36.83 90)
 			(effects

Commit message: all footprints assigned
Parts:
- C10, C18, C3, C34, C35, C8, C9: footprint (none) -> Capacitor_SMD:C_0805_2012Metric_Pad1.18x1.45mm_HandSolder
- C26, C27, C28, C4, C5, C6: footprint (none) -> Capacitor_SMD:C_0603_1608Metric_Pad1.08x0.95mm_HandSolder
- D1: footprint (none) -> Diode_SMD:D_SOD-123F
- D7, D8, D9: footprint (none) -> LED_SMD:LED_0805_2012Metric_Pad1.15x1.40mm_HandSolder
- L1: footprint (none) -> Inductor_SMD:L_Coilcraft_MSS1246-XXX
Changed lines of the file:
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@@
 			)
 		)
-		(property "Footprint" ""
+		(property "Footprint" "Capacitor_SMD:C_0603_1608Metric_Pad1.08x0.95mm_HandSolder"
 			(at 65.7352 119.38 0)
 			(effects
@@
 			)
 		)
-		(property "Footprint" ""
+		(property "Footprint" "Capacitor_SMD:C_0805_2012Metric_Pad1.18x1.45mm_HandSolder"
 			(at 238.4552 45.72 0)
 			(effects
@@
 			)
 		)
-		(property "Footprint" ""
+		(property "Footprint" "Capacitor_SMD:C_0805_2012Metric_Pad1.18x1.45mm_HandSolder"
 			(at 53.0352 109.22 0)
 			(effects
@@
 			)
 		)
-		(property "Footprint" ""
+		(property "Footprint" "Capacitor_SMD:C_0603_1608Metric_Pad1.08x0.95mm_HandSolder"
 			(at 131.7752 109.22 0)
 			(effects
@@
 			)
 		)
-		(property "Footprint" ""
+		(property "Footprint" "LED_SMD:LED_0805_2012Metric_Pad1.15x1.40mm_HandSolder"
 			(at 158.75 46.99 0)
 			(effects
@@
 			)
 		)
-		(property "Footprint" ""
+		(property "Footprint" "Capacitor_SMD:C_0805_2012Metric_Pad1.18x1.45mm_HandSolder"
 			(at 197.8152 45.72 0)
 			(effects
@@
 			)
 		)
-		(property "Footprint" ""
+		(property "Footprint" "Capacitor_SMD:C_0603_1608Metric_Pad1.08x0.95mm_HandSolder"
 			(at 204.1652 111.76 0)
 			(effects
@@
 			)
 		)
-		(property "Footprint" ""
+		(property "Footprint" "Capacitor_SMD:C_0603_1608Metric_Pad1.08x0.95mm_HandSolder"
 			(at 192.7352 111.76 0)
 			(effects
@@
 			)
 		)
-		(property "Footprint" ""
+		(property "Footprint" "Inductor_SMD:L_Coilcraft_MSS1246-XXX"
 			(at 142.24 110.49 0)
 			(effects
@@
 			)
 		)
-		(property "Footprint" ""
+		(property "Footprint" "Capacitor_SMD:C_0603_1608Metric_Pad1.08x0.95mm_HandSolder"
 			(at 74.6252 125.73 0)
 			(effects
@@
 			)
 		)
-		(property "Footprint" ""
+		(property "Footprint" "LED_SMD:LED_0805_2012Metric_Pad1.15x1.40mm_HandSolder"
 			(at 179.07 46.99 0)
 			(effects
@@
 			)
 		)
-		(property "Footprint" ""
+		(property "Footprint" "LED_SMD:LED_0805_2012Metric_Pad1.15x1.40mm_HandSolder"
 			(at 168.91 46.99 0)
 			(effects
@@
 			)
 		)
-		(property "Footprint" ""
+		(property "Footprint" "Capacitor_SMD:C_0805_2012Metric_Pad1.18x1.45mm_HandSolder"
 			(at 149.5552 120.65 0)
 			(effects
@@
 			)
 		)
-		(property "Footprint" ""
+		(property "Footprint" "Capacitor_SMD:C_0805_2012Metric_Pad1.18x1.45mm_HandSolder"
 			(at 172.4152 120.65 0)
 			(effects
@@
 			)
 		)
-		(property "Footprint" ""
+		(property "Footprint" "Capacitor_SMD:C_0805_2012Metric_Pad1.18x1.45mm_HandSolder"
 			(at 160.9852 120.65 0)
 			(effects
@@
 			)
 		)
-		(property "Footprint" ""
+		(property "Footprint" "Diode_SMD:D_SOD-123F"
 			(at 130.81 114.3 0)
 			(effects
@@
 			)
 		)
-		(property "Footprint" ""
+		(property "Footprint" "Capacitor_SMD:C_0805_2012Metric_Pad1.18x1.45mm_HandSolder"
 			(at 63.1952 109.22 0)
 			(effects
@@
 			)
 		)
-		(property "Footprint" ""
+		(property "Footprint" "Capacitor_SMD:C_0603_1608Metric_Pad1.08x0.95mm_HandSolder"
 			(at 274.0152 111.76 0)
 			(effects

Commit message: more layout
Parts:
- R2: footprint (none) -> Resistor_SMD:R_0603_1608Metric_Pad0.98x0.95mm_HandSolder
- U6: footprint TPS2115ADRBR:SON65P300X300X100-9N -> Package_SON:VSON-8-1EP_3x3mm_P0.65mm_EP1.65x2.4mm
Connections:
- net ILIM: now reaches R8.1, U6.4 (ILIM)
- net STAT: now reaches R9.2, U6.1 (STAT)
Other:
- moved on the sheet: C26, R8, R9
Changed lines of the file:
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@@
 	)
 	(junction
-		(at 273.05 95.25)
-		(diameter 0)
-		(color 0 0 0 0)
-	)
-	(junction
 		(at 160.02 110.49)
 		(diameter 0)
@@
 	)
 	(junction
-		(at 273.05 100.33)
-		(diameter 0)
-		(color 0 0 0 0)
-	)
-	(junction
-		(at 219.71 121.92)
+		(at 218.44 121.92)
 		(diameter 0)
 		(color 0 0 0 0)
@@
 	)
 	(junction
+		(at 274.32 95.25)
+		(diameter 0)
+		(color 0 0 0 0)
+	)
+	(junction
 		(at 217.17 48.26)
 		(diameter 0)
@@
 	)
 	(junction
+		(at 274.32 100.33)
+		(diameter 0)
+		(color 0 0 0 0)
+	)
+	(junction
 		(at 148.59 123.19)
 		(diameter 0)
@@
 	(wire
 		(pts
-			(xy 224.79 110.49) (xy 222.25 110.49)
+			(xy 220.98 110.49) (xy 224.79 110.49)
 		)
 		(stroke
@@
 	(wire
 		(pts
-			(xy 273.05 115.57) (xy 265.43 115.57)
+			(xy 274.32 115.57) (xy 265.43 115.57)
 		)
 		(stroke
@@
 	(wire
 		(pts
-			(xy 273.05 100.33) (xy 273.05 95.25)
+			(xy 274.32 100.33) (xy 274.32 95.25)
 		)
 		(stroke
@@
 	(wire
 		(pts
-			(xy 273.05 111.76) (xy 273.05 115.57)
+			(xy 274.32 111.76) (xy 274.32 115.57)
 		)
 		(stroke
@@
 	(wire
 		(pts
-			(xy 222.25 120.65) (xy 222.25 121.92)
+			(xy 220.98 120.65) (xy 220.98 121.92)
 		)
 		(stroke
@@
 	(wire
 		(pts
-			(xy 273.05 100.33) (xy 273.05 104.14)
+			(xy 274.32 100.33) (xy 274.32 104.14)
 		)
 		(stroke
@@
 	(wire
 		(pts
-			(xy 219.71 121.92) (xy 219.71 123.19)
+			(xy 218.44 121.92) (xy 218.44 123.19)
 		)
 		(stroke
@@
 	(wire
 		(pts
-			(xy 260.35 100.33) (xy 262.89 100.33)
+			(xy 260.35 100.33) (xy 265.43 100.33)
 		)
 		(stroke
@@
 	(wire
 		(pts
-			(xy 222.25 121.92) (xy 219.71 121.92)
+			(xy 220.98 121.92) (xy 218.44 121.92)
 		)
 		(stroke
@@
 	(wire
 		(pts
-			(xy 270.51 100.33) (xy 273.05 100.33)
+			(xy 273.05 100.33) (xy 274.32 100.33)
 		)
 		(stroke
@@
 	(wire
 		(pts
-			(xy 224.79 105.41) (xy 219.71 105.41)
+			(xy 218.44 105.41) (xy 224.79 105.41)
 		)
 		(stroke
@@
 	(wire
 		(pts
-			(xy 222.25 110.49) (xy 222.25 113.03)
+			(xy 220.98 110.49) (xy 220.98 113.03)
 		)
 		(stroke
@@
 	(wire
 		(pts
-			(xy 260.35 95.25) (xy 273.05 95.25)
+			(xy 260.35 95.25) (xy 274.32 95.25)
 		)
 		(stroke
@@
 	(wire
 		(pts
-			(xy 273.05 92.71) (xy 273.05 95.25)
+			(xy 274.32 92.71) (xy 274.32 95.25)
 		)
 		(stroke
@@
 	(wire
 		(pts
-			(xy 219.71 105.41) (xy 219.71 121.92)
+			(xy 218.44 105.41) (xy 218.44 121.92)
 		)
 		(stroke
@@
 		)
 	)
+	(label "ILIM"
+		(at 220.98 110.49 0)
+		(effects
+			(font
+				(size 1.27 1.27)
+			)
+			(justify left bottom)
+		)
+	)
+	(label "STAT"
+		(at 260.35 100.33 0)
+		(effects
+			(font
+				(size 1.27 1.27)
+			)
+			(justify left bottom)
+		)
+	)
 	(hierarchical_label "IMON_OUT"
 		(shape output)
@@
 	(symbol
 		(lib_id "Device:R")
-		(at 222.25 116.84 0)
+		(at 220.98 116.84 0)
 		(unit 1)
 		(exclude_from_sim no)
@@
 		(fields_autoplaced yes)
 		(property "Reference" "R8"
-			(at 224.79 115.5699 0)
+			(at 223.52 115.5699 0)
 			(effects
 				(font
@@
 		)
 		(property "Value" "332"
-			(at 224.79 118.1099 0)
+			(at 223.52 118.1099 0)
 			(effects
 				(font
@@
 		)
 		(property "Footprint" "Resistor_SMD:R_0603_1608Metric_Pad0.98x0.95mm_HandSolder"
-			(at 220.472 116.84 90)
+			(at 219.202 116.84 90)
 			(effects
 				(font
@@
 		)
 		(property "Datasheet" "~"
-			(at 222.25 116.84 0)
+			(at 220.98 116.84 0)
 			(effects
 				(font
@@
 		)
 		(property "Description" "Resistor"
-			(at 222.25 116.84 0)
+			(at 220.98 116.84 0)
 			(effects
 				(font
@@
 		)
 		(property "P/N" "CRCW0603332RFKEAHP "
-			(at 222.25 116.84 0)
+			(at 220.98 116.84 0)
 			(effects
 				(font
@@
 	(symbol
 		(lib_id "Device:R")
-		(at 266.7 100.33 270)
+		(at 269.24 100.33 270)
 		(unit 1)
 		(exclude_from_sim no)
@@
 		(dnp no)
 		(property "Reference" "R9"
-			(at 266.7 103.124 90)
+			(at 269.24 103.124 90)
 			(effects
 				(font
@@
 		)
 		(property "Value" "10k"
-			(at 266.7 105.664 90)
+			(at 269.24 105.664 90)
 			(effects
 				(font
@@
 		)
 		(property "Footprint" "Resistor_SMD:R_0603_1608Metric_Pad0.98x0.95mm_HandSolder"
-			(at 266.7 98.552 90)
+			(at 269.24 98.552 90)
 			(effects
 				(font
@@
 		)
 		(property "Datasheet" "~"
-			(at 266.7 100.33 0)
+			(at 269.24 100.33 0)
 			(effects
 				(font
@@
 		)
 		(property "Description" "Resistor"
-			(at 266.7 100.33 0)
+			(at 269.24 100.33 0)
 			(effects
 				(font
@@
 		)
 		(property "P/N" "CRCW060310K0FKEI "
-			(at 266.7 100.33 90)
+			(at 269.24 100.33 90)
 			(effects
 				(font
@@
 	(symbol
 		(lib_id "power:PWR_FLAG")
-		(at 273.05 95.25 270)
+		(at 274.32 95.25 270)
 		(unit 1)
 		(exclude_from_sim no)
@@
 		(dnp no)
 		(property "Reference" "#FLG05"
-			(at 274.955 95.25 0)
+			(at 276.225 95.25 0)
 			(effects
 				(font
@@
 		)
 		(property "Value" "PWR_FLAG"
-			(at 276.225 95.25 0)
+			(at 277.495 95.25 0)
 			(effects
 				(font
@@
 		)
 		(property "Footprint" ""
-			(at 273.05 95.25 0)
+			(at 274.32 95.25 0)
 			(effects
 				(font
@@
 		)
 		(property "Datasheet" "~"
-			(at 273.05 95.25 0)
+			(at 274.32 95.25 0)
 			(effects
 				(font
@@
 		)
 		(property "Description" "Special symbol for telling ERC where power comes from"
-			(at 273.05 95.25 0)
+			(at 274.32 95.25 0)
 			(effects
 				(font
@@
 	(symbol
 		(lib_id "power:+24V")
-		(at 273.05 92.71 0)
+		(at 274.32 92.71 0)
 		(unit 1)
 		(exclude_from_sim no)
@@
 		(dnp no)
 		(property "Reference" "#PWR043"
-			(at 273.05 96.52 0)
+			(at 274.32 96.52 0)
 			(effects
 				(font
@@
 		)
 		(property "Value" "+5V"
-			(at 272.796 88.9 0)
+			(at 274.066 88.9 0)
 			(effects
 				(font
@@
 		)
 		(property "Footprint" ""
-			(at 273.05 92.71 0)
+			(at 274.32 92.71 0)
 			(effects
 				(font
@@
 		)
 		(property "Datasheet" ""
-			(at 273.05 92.71 0)
+			(at 274.32 92.71 0)
 			(effects
 				(font
@@
 		)
 		(property "Description" "Power symbol creates a global label with name \"+24V\""
-			(at 273.05 92.71 0)
+			(at 274.32 92.71 0)
 			(effects
 				(font
@@
 	(symbol
 		(lib_id "power:GND")
-		(at 219.71 123.19 0)
+		(at 218.44 123.19 0)
 		(unit 1)
 		(exclude_from_sim no)
@@
 		(fields_autoplaced yes)
 		(property "Reference" "#PWR044"
-			(at 219.71 129.54 0)
+			(at 218.44 129.54 0)
 			(effects
 				(font
@@
 		)
 		(property "Value" "GND"
-			(at 219.71 128.27 0)
+			(at 218.44 128.27 0)
 			(effects
 				(font
@@
 		)
 		(property "Footprint" ""
-			(at 219.71 123.19 0)
+			(at 218.44 123.19 0)
 			(effects
 				(font
@@
 		)
 		(property "Datasheet" ""
-			(at 219.71 123.19 0)
+			(at 218.44 123.19 0)
 			(effects
 				(font
@@
 		)
 		(property "Description" "Power symbol creates a global label with name \"GND\" , ground"
-			(at 219.71 123.19 0)
+			(at 218.44 123.19 0)
 			(effects
 				(font
@@
 			)
 		)
-		(property "Footprint" "TPS2115ADRBR:SON65P300X300X100-9N"
+		(property "Footprint" "Package_SON:VSON-8-1EP_3x3mm_P0.65mm_EP1.65x2.4mm"
 			(at 242.57 105.41 0)
 			(effects
@@
 		(exclude_from_sim no)
 		(in_bom no)
-		(on_board no)
+		(on_board yes)
 		(dnp yes)
 		(property "Reference" "R2"
@@
 			)
 		)
-		(property "Footprint" ""
+		(property "Footprint" "Resistor_SMD:R_0603_1608Metric_Pad0.98x0.95mm_HandSolder"
 			(at 87.122 137.16 90)
 			(effects
@@
 	(symbol
 		(lib_id "Device:C")
-		(at 273.05 107.95 0)
+		(at 274.32 107.95 0)
 		(unit 1)
 		(exclude_from_sim no)
@@
 		(dnp no)
 		(property "Reference" "C26"
-			(at 276.0472 106.7816 0)
+			(at 277.3172 106.7816 0)
 			(effects
 				(font
@@
 		)
 		(property "Value" "1uF"
-			(at 276.0472 109.093 0)
+			(at 277.3172 109.093 0)
 			(effects
 				(font
@@
 		)
 		(property "Footprint" "Capacitor_SMD:C_0603_1608Metric_Pad1.08x0.95mm_HandSolder"
-			(at 274.0152 111.76 0)
+			(at 275.2852 111.76 0)
 			(effects
 				(font
@@
 		)
 		(property "Datasheet" "~"
-			(at 273.05 107.95 0)
+			(at 274.32 107.95 0)
 			(effects
 				(font
@@
 		)
 		(property "Description" "Unpolarized capacitor"
-			(at 273.05 107.95 0)
+			(at 274.32 107.95 0)
 			(effects
 				(font
@@
 		)
 		(property "P/N" "MLASU168SB5105KTNA01"
-			(at 273.05 107.95 0)
+			(at 274.32 107.95 0)
 			(effects
 				(font
@@
 		)
 		(property "Mouser Part Number" "581-22201C106KAT2A"
-			(at 273.05 107.95 0)
+			(at 274.32 107.95 0)
 			(effects
 				(font

Commit message: address some stuff
Parts:
- removed TP5: 5V, TestPoint:TestPoint_Pad_1.0x1.0mm, symbol Connector:TestPoint
- added D11: BUCK, LED_SMD:LED_0805_2012Metric_Pad1.15x1.40mm_HandSolder, symbol Device:LED
- added R32: 768, Resistor_SMD:R_0603_1608Metric_Pad0.98x0.95mm_HandSolder, symbol Device:R
- C10, C18, C26, C27, C28, C3, C34, C35, C4, C5, C6, C8: Mouser Part Number 581-22201C106KAT2A -> (none)
- C9: value 10uF -> 1uF; footprint Capacitor_SMD:C_0805_2012Metric_Pad1.18x1.45mm_HandSolder -> Capacitor_SMD:C_0603_1608Metric_Pad1.08x0.95mm_HandSolder; Mouser Part Number 581-22201C106KAT2A -> (none); P/N GRM21BR61H106KE43K -> MLASU168SB5105KTNA01
- D1: P/N MBR230S1F-7 -> SS24FL
- D9: value PG -> FLT
- R2, R25, R26, R28, R3: Mouser Part Number 71-CRCW0805100KFKEAC -> (none)
- U6: Availability In Stock -> (none); MF Texas Instruments -> (none); MP TPS2115ADRBR -> (none); Price None -> (none)
Connections:
- net 24V is gone; now on net +24V: TP2.1
- net 24V_EXT is gone; now on net +24V_EXT: TP1.1
- net 3.3V is gone; now on net +3.3V: TP6.1
- net 5V_BUCK is gone; now on net +5V_BUCK: TP3.1
- net 5V_VBUS is gone; now on net +5V_VBUS: TP4.1
- net +24V: now also R28.1
- net +5V: now also R32.1
- net FAULT: now also D9.1 (K); no longer R28.1
- net GND: no longer D9.1 (K)
- net STAT: now also D11.1 (K)
- new net: D11.2 (A), R32.2
Other:
- moved on the sheet: C10, C18, U3

Commit message: erm hii
Parts:
- TP3: value 5V_BUCK -> 5V_BK
Changed lines of the file:
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@@
 			)
 		)
-		(property "Value" "5V_BUCK"
+		(property "Value" "5V_BK"
 			(at 124.46 52.8319 0)
 			(effects

Commit message: add some lcsc parts
Parts:
- D9: P/N APTD2012LVBC/D -> APTD2012LSURCK
Changed lines of the file:
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@@
 			)
 		)
-		(property "P/N" "APTD2012LVBC/D"
+		(property "P/N" "APTD2012LSURCK"
 			(at 179.07 46.99 90)
 			(effects

Commit message: type shi
Parts:
- D9: value FLT -> PFLT
Changed lines of the file:
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@@
 			)
 		)
-		(property "Value" "FLT"
+		(property "Value" "PFLT"
 			(at 182.88 49.8474 90)
 			(effects

Commit message: boo lakshay
Parts:
- TP2: value 24V_PROT -> 24V
Changed lines of the file:
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@@
 			)
 		)
-		(property "Value" "24V_PROT"
+		(property "Value" "24V"
 			(at 110.49 52.8319 0)
 			(effects
