File: USB.kicad_sch (KiCad schematic)
At the start: 8 parts, among them J23 USB_B_Micro, U19 CP2102N-A02-GQFN24

Commit message: v1.2 initial changes
Parts:
- removed D15: SP0503BAHT, Package_TO_SOT_SMD:SOT-143, symbol Dash2-rescue:SP0503BAHT-Power_Protection
- removed J23: USB_B_Micro, Connector_USB:USB_Micro-B_Molex-105017-0001, symbol Dashboard-rescue:USB_B_Micro-Connector
- removed U19: CP2102N-A02-GQFN24, Package_DFN_QFN:QFN-24-1EP_4x4mm_P0.5mm_EP2.6x2.6mm, symbol Interface_USB:CP2102N-A01-GQFN24
- added D1: SP0503BAHT, Package_TO_SOT_SMD:SOT-143, symbol Power_Protection:SP0503BAHT
- added J3: USB_B_Micro, Connector_USB:USB_Micro-B_Molex-105017-0001, symbol Connector:USB_B_Micro
- added U4: CP2102N-Axx-xQFN24, Package_DFN_QFN:QFN-24-1EP_4x4mm_P0.5mm_EP2.6x2.6mm, symbol Interface_USB:CP2102N-Axx-xQFN24
Connections:
- net +3.3V: now also U4.5 (VIO), U4.6 (VDD), U4.7 (VREGIN)
- net GND: now also D1.1 (A), J3.5 (GND), J3.6 (Shield), U4.2 (GND), U4.25 (GND)
- net UART_RX: now also U4.20 (RXD)
- net UART_TX: now also U4.21 (TXD)
- net at R36.1, R37.1: now also U4.8 (VBUS)
- net at R36.2: now also D1.2 (K), J3.1 (VBUS)
- net at R38.2: now also U4.9 (~{RST})
- new net: D1.3 (K), J3.2 (D-), U4.3 (D+)
- new net: D1.4 (K), J3.3 (D+), U4.4 (D-)
Other:
- moved on the sheet: C41, C42, R36, R37, R38

Commit message: Fix broken USB (ノಠ益ಠ)ノ彡┻━┻
Connections:
- net at D1.3 (K), J3.2 (D-): now also U4.4 (D-); no longer U4.3 (D+)
- net at D1.4 (K), J3.3 (D+): now also U4.3 (D+); no longer U4.4 (D-)
Changed lines of the file:
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@@
 (kicad_sch (version 20230121) (generator eeschema)
   (paper "A4")
+  (junction (at 93.98 97.79) (diameter 0) (color 0 0 0 0)
+  )
   (junction (at 135.255 62.865) (diameter 0) (color 0 0 0 0)
   )
@@
   )
   (junction (at 130.81 77.47) (diameter 0) (color 0 0 0 0)
-  )
-  (junction (at 93.98 100.33) (diameter 0) (color 0 0 0 0)
   )
   (junction (at 128.27 77.47) (diameter 0) (color 0 0 0 0)
@@
   (junction (at 69.85 111.76) (diameter 0) (color 0 0 0 0)
   )
+  (junction (at 96.52 100.33) (diameter 0) (color 0 0 0 0)
+  )
   (junction (at 128.27 62.865) (diameter 0) (color 0 0 0 0)
   )
@@
   )
   (junction (at 147.955 73.025) (diameter 0) (color 0 0 0 0)
-  )
-  (junction (at 96.52 97.79) (diameter 0) (color 0 0 0 0)
   )
   (no_connect (at 143.51 95.25))
@@
     (stroke (width 0) (type default))
   )
-  (wire (pts (xy 77.47 102.87) (xy 82.55 102.87))
+  (wire (pts (xy 93.98 97.79) (xy 82.55 97.79))
     (stroke (width 0) (type default))
   )
-  (wire (pts (xy 96.52 97.79) (xy 118.11 97.79))
+  (wire (pts (xy 77.47 102.87) (xy 82.55 102.87))
     (stroke (width 0) (type default))
   )
@@
     (stroke (width 0) (type default))
   )
-  (wire (pts (xy 80.01 100.33) (xy 77.47 100.33))
+  (wire (pts (xy 77.47 100.33) (xy 96.52 100.33))
     (stroke (width 0) (type default))
   )
   (wire (pts (xy 118.11 71.12) (xy 128.27 71.12))
+    (stroke (width 0) (type default))
+  )
+  (wire (pts (xy 93.98 97.79) (xy 93.98 107.95))
     (stroke (width 0) (type default))
   )
@@
     (stroke (width 0) (type default))
   )
-  (wire (pts (xy 93.98 107.95) (xy 93.98 100.33))
-    (stroke (width 0) (type default))
-  )
   (wire (pts (xy 91.44 107.95) (xy 91.44 95.25))
     (stroke (width 0) (type default))
@@
     (stroke (width 0) (type default))
   )
-  (wire (pts (xy 82.55 100.33) (xy 93.98 100.33))
-    (stroke (width 0) (type default))
-  )
   (wire (pts (xy 69.85 111.76) (xy 69.85 113.03))
     (stroke (width 0) (type default))
   )
-  (wire (pts (xy 82.55 102.87) (xy 82.55 100.33))
+  (wire (pts (xy 82.55 97.79) (xy 82.55 102.87))
     (stroke (width 0) (type default))
   )
   (wire (pts (xy 128.27 77.47) (xy 130.81 77.47))
-    (stroke (width 0) (type default))
-  )
-  (wire (pts (xy 80.01 97.79) (xy 80.01 100.33))
     (stroke (width 0) (type default))
   )
@@
     (stroke (width 0) (type default))
   )
-  (wire (pts (xy 93.98 100.33) (xy 118.11 100.33))
+  (wire (pts (xy 96.52 100.33) (xy 118.11 100.33))
     (stroke (width 0) (type default))
   )
@@
     (stroke (width 0) (type default))
   )
-  (wire (pts (xy 80.01 97.79) (xy 96.52 97.79))
+  (wire (pts (xy 118.11 97.79) (xy 93.98 97.79))
     (stroke (width 0) (type default))
   )
@@
     (stroke (width 0) (type default))
   )
-  (wire (pts (xy 96.52 107.95) (xy 96.52 97.79))
-    (stroke (width 0) (type default))
-  )
   (wire (pts (xy 69.85 111.76) (xy 69.85 110.49))
     (stroke (width 0) (type default))
   )
+  (wire (pts (xy 96.52 100.33) (xy 96.52 107.95))
+    (stroke (width 0) (type default))
+  )

Commit message: Added BOM + Mouser + Docs (#7)
* Updated Readme

* fixed schematic name

* Fixed connector numbers and pinouts on readme

* Added part numbers and BOM

* Added mouser cart

* Fixed Readme spacing

* forgot to add step file :cry:

* whoops, forgot to push :/
Parts:
- D1: value SP0503BAHT -> SP0503BAHTG; Mouser Part Number (none) -> 576-SP0503BAHTG; P/N (none) -> SP0503BAHTG
- J3: Mouser Part Number (none) -> 538-105017-0001; P/N (none) -> 105017-0001
- U4: Mouser Part Number (none) -> 634-CP2102NA02QFN24R; P/N (none) -> CP2102N-A02-GQFN24R
Changed lines of the file:
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@@
+      (effects (font (size 1.27 1.27)) hide)
+    )
+    (property "Mouser Part Number" "634-CP2102NA02QFN24R" (at 130.81 105.41 0)
+      (effects (font (size 1.27 1.27)) hide)
+    )
+    (property "P/N" "CP2102N-A02-GQFN24R" (at 130.81 105.41 0)
       (effects (font (size 1.27 1.27)) hide)
     )
@@
       (effects (font (size 1.27 1.27)) (justify left))
     )
-    (property "Value" "SP0503BAHT" (at 100.33 114.3 0)
+    (property "Value" "SP0503BAHTG" (at 100.33 114.3 0)
       (effects (font (size 1.27 1.27)) (justify left))
     )
@@
     )
     (property "Datasheet" "http://www.littelfuse.com/~/media/files/littelfuse/technical%20resources/documents/data%20sheets/sp05xxba.pdf" (at 97.155 109.855 0)
+      (effects (font (size 1.27 1.27)) hide)
+    )
+    (property "Mouser Part Number" "576-SP0503BAHTG" (at 93.98 113.03 0)
+      (effects (font (size 1.27 1.27)) hide)
+    )
+    (property "P/N" "SP0503BAHTG" (at 93.98 113.03 0)
       (effects (font (size 1.27 1.27)) hide)
     )
@@
       (effects (font (size 1.27 1.27)) hide)
     )
+    (property "Mouser Part Number" "538-105017-0001" (at 69.85 100.33 0)
+      (effects (font (size 1.27 1.27)) hide)
+    )
+    (property "P/N" "105017-0001" (at 69.85 100.33 0)
+      (effects (font (size 1.27 1.27)) hide)
+    )

Commit message: started v2 changes
Parts:
- removed C41: 4.7uF, Capacitor_SMD:C_0805_2012Metric, symbol Device:C
- removed C42: 100nF, Capacitor_SMD:C_0805_2012Metric, symbol Device:C
- removed R36: 22.1k, Resistor_SMD:R_0805_2012Metric, symbol Device:R
- removed R37: 47.5k, Resistor_SMD:R_0805_2012Metric, symbol Device:R
- removed R38: 1k, Resistor_SMD:R_0805_2012Metric, symbol Device:R
- added C8: 4.7uF, Capacitor_SMD:C_0805_2012Metric, symbol Device:C
- added C9: 100nF, Capacitor_SMD:C_0805_2012Metric, symbol Device:C
- added R3: 22.1k, Resistor_SMD:R_0805_2012Metric, symbol Device:R
- added R4: 47.5k, Resistor_SMD:R_0805_2012Metric, symbol Device:R
- added R5: 1k, Resistor_SMD:R_0805_2012Metric, symbol Device:R
- added U6: FT230XS-R, Package_SO:SSOP-16_3.9x4.9mm_P0.635mm, symbol utsvt-chips:FT230XS-R
Connections:
- net +3.3V: now also C8.1, C9.1, R5.1, U6.12 (VCC), U6.3 (VCCIO)
- net GND: now also C8.2, C9.2, R4.2, U6.13 (AGND), U6.5 (GND); no longer D1.1 (A)
- net at U4.8 (VBUS): now also R3.1, R4.1
- net at U4.9 (~{RST}): now also R5.2
- net at J3.1 (VBUS): no longer D1.2 (K)
- new net: J3.2 (D-), U6.8 (USBDP)
- new net: J3.3 (D+), U6.9 (USBDM)
- now unconnected: D1.3 (K), D1.4 (K), U4.3 (D+), U4.4 (D-)
Other:
- moved on the sheet: J3

Commit message: wahoooooo
Parts:
- removed C8: 4.7uF, Capacitor_SMD:C_0805_2012Metric, symbol Device:C
- removed C9: 100nF, Capacitor_SMD:C_0805_2012Metric, symbol Device:C
- removed D1: SP0503BAHTG, Package_TO_SOT_SMD:SOT-143, symbol Power_Protection:SP0503BAHT
- removed R3: 22.1k, Resistor_SMD:R_0805_2012Metric, symbol Device:R
- removed R4: 47.5k, Resistor_SMD:R_0805_2012Metric, symbol Device:R
- removed R5: 1k, Resistor_SMD:R_0805_2012Metric, symbol Device:R
- removed U4: CP2102N-Axx-xQFN24, Package_DFN_QFN:QFN-24-1EP_4x4mm_P0.5mm_EP2.6x2.6mm, symbol Interface_USB:CP2102N-Axx-xQFN24
- added C1, C10, C18, C19: 100nF, Capacitor_SMD:C_0805_2012Metric, symbol Device:C
- added C28, C29: 47pF, Capacitor_SMD:C_0805_2012Metric, symbol Device:C
- added R1, R25, R26, R7: 27, symbol Device:R
Connections:
- net +3.3V: now also U6.10 (3V3OUT), U6.11 (RESET), C1.1, C10.1, C18.1, C19.1, R26.1
- net GND: now also C1.2, C10.2, C18.2, C19.2, C28.2, C29.2, R25.2
- net UART_RX: now also U6.4 (RXD)
- net UART_TX: now also U6.1 (TXD)
- net at U6.16 (CBUS3): now also R25.1, R26.2
- net at U6.8 (USBDP): now also R7.1; no longer J3.2 (D-)
- net at U6.9 (USBDM): now also R1.1; no longer J3.3 (D+)
- net vbus: now reaches J3.1 (VBUS)
- new net D+: C28.1, J3.3 (D+), R7.2
- new net D-: C29.1, J3.2 (D-), R1.2
- no-connect marks 13 -> 6
Other:
- note added: "Used for sensing presence of USB cable"
- note removed: "The microcontroller should have Rx connected to UART_TX and Tx connected to UART_RX"
- moved on the sheet: J3

Commit message: fixed symbols
Parts:
- U6: P/N (none) -> FT230XS-R
Changed lines of the file:
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@@
+			)
+		)
+		(property "P/N" "FT230XS-R"
+			(at 135.89 87.63 0)
+			(effects
+				(font
+					(size 1.27 1.27)
+				)
+				(hide yes)
 			)
 		)

Commit message: updated footprints and added caps
Parts:
- R1, R7: footprint (none) -> Resistor_SMD:R_0805_2012Metric
- R25: value 27 -> 10k; footprint (none) -> Resistor_SMD:R_0805_2012Metric
- R26: value 27 -> 4.7k; footprint (none) -> Resistor_SMD:R_0805_2012Metric
Changed lines of the file:
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@@
 			)
 		)
-		(property "Footprint" ""
+		(property "Footprint" "Resistor_SMD:R_0805_2012Metric"
 			(at 104.14 99.822 90)
 			(effects
@@
 			)
 		)
-		(property "Value" "27"
+		(property "Value" "4.7k"
 			(at 166.37 111.7599 0)
 			(effects
@@
 			)
 		)
-		(property "Footprint" ""
+		(property "Footprint" "Resistor_SMD:R_0805_2012Metric"
 			(at 162.052 110.49 90)
 			(effects
@@
 			)
 		)
-		(property "Footprint" ""
+		(property "Footprint" "Resistor_SMD:R_0805_2012Metric"
 			(at 113.03 97.282 90)
 			(effects
@@
 			)
 		)
-		(property "Value" "27"
+		(property "Value" "10k"
 			(at 166.37 121.9199 0)
 			(effects
@@
 			)
 		)
-		(property "Footprint" ""
+		(property "Footprint" "Resistor_SMD:R_0805_2012Metric"
 			(at 162.052 120.65 90)
 			(effects
