File: USB.kicad_sch (KiCad schematic)
At the start: 12 parts, among them J3 USB_B_Micro, U6 FT230XS-R

Commit message: pp
Connections:
- net +3.3V: no longer R26.1
- net vbus: now also R26.1
Other:
- moved on the sheet: R7
Changed lines of the file:
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@@
 	(wire
 		(pts
-			(xy 100.33 101.6) (xy 96.52 101.6)
+			(xy 102.87 101.6) (xy 96.52 101.6)
 		)
 		(stroke
@@
 	(wire
 		(pts
+			(xy 163.83 105.41) (xy 166.37 105.41)
+		)
+		(stroke
+			(width 0)
+			(type default)
+		)
+	)
+	(wire
+		(pts
 			(xy 67.31 133.35) (xy 55.88 133.35)
 		)
@@
 	(wire
 		(pts
-			(xy 107.95 101.6) (xy 119.38 101.6)
+			(xy 110.49 101.6) (xy 119.38 101.6)
 		)
 		(stroke
@@
 	(text "Used for sensing \npresence of USB cable"
 		(exclude_from_sim no)
-		(at 180.086 114.808 0)
+		(at 180.34 114.3 0)
 		(effects
 			(font
@@
 	(label "D+"
 		(at 68.58 102.87 0)
+		(fields_autoplaced yes)
+		(effects
+			(font
+				(size 1.27 1.27)
+			)
+			(justify left bottom)
+		)
+	)
+	(label "vbus"
+		(at 166.37 105.41 0)
 		(fields_autoplaced yes)
 		(effects
@@
 	(symbol
 		(lib_id "Device:R")
-		(at 104.14 101.6 270)
+		(at 106.68 101.6 270)
 		(unit 1)
 		(exclude_from_sim no)
@@
 		(fields_autoplaced yes)
 		(property "Reference" "R7"
-			(at 104.14 95.25 90)
+			(at 106.68 95.25 90)
 			(effects
 				(font
@@
 		)
 		(property "Value" "27"
-			(at 104.14 97.79 90)
+			(at 106.68 97.79 90)
 			(effects
 				(font
@@
 		)
 		(property "Footprint" "Resistor_SMD:R_0805_2012Metric"
-			(at 104.14 99.822 90)
+			(at 106.68 99.822 90)
 			(effects
 				(font
@@
 		)
 		(property "Datasheet" "~"
-			(at 104.14 101.6 0)
+			(at 106.68 101.6 0)
 			(effects
 				(font
@@
 		)
 		(property "Description" "Resistor"
-			(at 104.14 101.6 0)
+			(at 106.68 101.6 0)
 			(effects
 				(font
@@
 					(unit 1)
 				)
-			)
-		)
-	)
-	(symbol
-		(lib_id "power:+3.3V")
-		(at 163.83 105.41 0)
-		(unit 1)
-		(exclude_from_sim no)
-		(in_bom yes)
-		(on_board yes)
-		(dnp no)
-		(fields_autoplaced yes)
-		(property "Reference" "#PWR032"
-			(at 163.83 109.22 0)
-			(effects
-				(font
-					(size 1.27 1.27)
-				)
-				(hide yes)
-			)
-		)
-		(property "Value" "+3.3V"
-			(at 163.83 100.33 0)
-			(effects
-				(font
-					(size 1.27 1.27)
-				)
-			)
-		)
-		(property "Footprint" ""
-			(at 163.83 105.41 0)
-			(effects
-				(font
-					(size 1.27 1.27)
-				)
-				(hide yes)
-			)
-		)
-		(property "Datasheet" ""
-			(at 163.83 105.41 0)
-			(effects
-				(font
-					(size 1.27 1.27)
-				)
-				(hide yes)
-			)
-		)
-		(property "Description" "Power symbol creates a global label with name \"+3.3V\""
-			(at 163.83 105.41 0)
-			(effects
-				(font
-					(size 1.27 1.27)
-				)
-				(hide yes)
-			)
-		)
-		(pin "1"
-		)
-		(instances
-			(project "BPS-PeripheralSOM"
-				(path "/d5ebd247-5a7c-47c2-8aee-beabaef72d6d/94125b35-79a1-41d0-8b6c-f77e699b83b8"
-					(reference "#PWR032")
-					(unit 1)
-				)

Commit message: DRC go brrr (need to change text thickness)
Connections:
- net UART_RX renamed CHIP_RX
- net UART_TX renamed CHIP_TX
Changed lines of the file:
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@@
 		)
 	)
-	(hierarchical_label "UART_TX"
+	(hierarchical_label "CHIP_TX"
 		(shape output)
 		(at 154.94 91.44 0)
@@
 		)
 	)
-	(hierarchical_label "UART_RX"
+	(hierarchical_label "CHIP_RX"
 		(shape input)
 		(at 154.94 93.98 0)

Commit message: BOOM
Parts:
- C28, C29: P/N (none) -> 0805N470G160CT
- R1, R7: P/N (none) -> CR0805-FX-27R0ELF
- R25: P/N (none) -> RT0603FRE0710KL
- R26: P/N (none) -> CRCW08054K70FKEAC
Changed lines of the file:
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@@
+			)
+		)
+		(property "P/N" "CR0805-FX-27R0ELF"
+			(at 106.68 101.6 0)
+			(effects
+				(font
+					(size 1.27 1.27)
+				)
+				(hide yes)
 			)
 		)
@@
 			)
 		)
+		(property "P/N" "0805N470G160CT"
+			(at 86.36 105.41 0)
+			(effects
+				(font
+					(size 1.27 1.27)
+				)
+				(hide yes)
+			)
+		)
 		(pin "1"
 		)
@@
 			)
 		)
+		(property "P/N" "CRCW08054K70FKEAC"
+			(at 163.83 110.49 0)
+			(effects
+				(font
+					(size 1.27 1.27)
+				)
+				(hide yes)
+			)
+		)
 		(pin "1"
 		)
@@
 			)
 		)
+		(property "P/N" "CR0805-FX-27R0ELF"
+			(at 113.03 99.06 0)
+			(effects
+				(font
+					(size 1.27 1.27)
+				)
+				(hide yes)
+			)
+		)
 		(pin "1"
 		)
@@
 			)
 		)
+		(property "P/N" "0805N470G160CT"
+			(at 96.52 105.41 0)
+			(effects
+				(font
+					(size 1.27 1.27)
+				)
+				(hide yes)
+			)
+		)
 		(pin "1"
 		)
@@
 			(at 163.83 120.65 0)
 			(effects
+				(font
+					(size 1.27 1.27)
+				)
+				(hide yes)
+			)
+		)
+		(property "P/N" "RT0603FRE0710KL "
+			(at 163.83 120.65 0)
+			(effects

Commit message: V2.1 (#17)
* womp womp

* woop woop

* can+power layout

* and so it begins...

* wahoo?

* routing done mayhaps

* fixed LED traces

* switched green and yellow traces

* better LED ordering + silkscreen stuff

* less via in pad

* addressed prat

* womp womp

* it's gerbing time

* i'm so dumb

* new dc-dc

* change max draw on iso dc-dc

* gerbers

* update ibom

* bom
Parts:
- added J5: Conn_01x02_Pin, Connector_PinHeader_2.54mm:PinHeader_1x02_P2.54mm_Vertical, symbol Connector:Conn_01x02_Pin
Connections:
- net CHIP_RX: now also J5.1 (Pin_1)
- net CHIP_TX: now also J5.2 (Pin_2)
Changed lines of the file:
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@@
+	(wire
+		(pts
+			(xy 180.34 83.185) (xy 180.34 87.63)
+		)
+		(stroke
+			(width 0)
+			(type default)
+		)
+	)
 	(wire
 		(pts
@@
 	(wire
 		(pts
+			(xy 177.8 83.185) (xy 177.8 87.63)
+		)
+		(stroke
+			(width 0)
+			(type default)
+		)
+	)
+	(wire
+		(pts
 			(xy 55.88 132.08) (xy 55.88 133.35)
 		)
@@
 	(wire
 		(pts
-			(xy 66.04 97.79) (xy 69.85 97.79)
+			(xy 66.04 97.79) (xy 71.755 97.79)
 		)
 		(stroke
@@
 		)
 	)
-	(label "vbus"
-		(at 69.85 97.79 0)
+	(label "D+"
+		(at 68.58 102.87 0)
 		(fields_autoplaced yes)
 		(effects
@@
 		)
 	)
-	(label "D+"
-		(at 68.58 102.87 0)
+	(label "vbus"
+		(at 166.37 105.41 0)
 		(fields_autoplaced yes)
 		(effects
@@
 	)
 	(label "vbus"
-		(at 166.37 105.41 0)
+		(at 71.755 97.79 0)
 		(fields_autoplaced yes)
 		(effects
@@
 	(hierarchical_label "CHIP_RX"
 		(shape input)
-		(at 154.94 93.98 0)
+		(at 180.34 87.63 270)
 		(fields_autoplaced yes)
 		(effects
@@
 				(size 1.27 1.27)
 			)
+			(justify right)
+		)
+	)
+	(hierarchical_label "CHIP_RX"
+		(shape input)
+		(at 154.94 93.98 0)
+		(fields_autoplaced yes)
+		(effects
+			(font
+				(size 1.27 1.27)
+			)
 			(justify left)
+		)
+	)
+	(hierarchical_label "CHIP_TX"
+		(shape output)
+		(at 177.8 87.63 270)
+		(fields_autoplaced yes)
+		(effects
+			(font
+				(size 1.27 1.27)
+			)
+			(justify right)
 		)
 	)
@@
 					(unit 1)
 				)
+			)
+		)
+	)
+	(symbol
+		(lib_id "Connector:Conn_01x02_Pin")
+		(at 180.34 78.105 270)
+		(unit 1)
+		(exclude_from_sim no)
+		(in_bom yes)
+		(on_board yes)
+		(dnp no)
+		(fields_autoplaced yes)
+		(property "Reference" "J5"
+			(at 181.61 77.4699 90)
+			(effects
+				(font
+					(size 1.27 1.27)
+				)
+				(justify left)
+			)
+		)
+		(property "Value" "Conn_01x02_Pin"
+			(at 181.61 80.0099 90)
+			(effects
+				(font
+					(size 1.27 1.27)
+				)
+				(justify left)
+			)
+		)
+		(property "Footprint" "Connector_PinHeader_2.54mm:PinHeader_1x02_P2.54mm_Vertical"
+			(at 180.34 78.105 0)
+			(effects
+				(font
+					(size 1.27 1.27)
+				)
+				(hide yes)
+			)
+		)
+		(property "Datasheet" "~"
+			(at 180.34 78.105 0)
+			(effects
+				(font
+					(size 1.27 1.27)
+				)
+				(hide yes)
+			)
+		)
+		(property "Description" "Generic connector, single row, 01x02, script generated"
+			(at 180.34 78.105 0)
+			(effects
+				(font
+					(size 1.27 1.27)
+				)
+				(hide yes)
+			)
+		)
+		(pin "2"
+		)
+		(pin "1"
+		)
+		(instances
+			(project "BPS-PeripheralSOM"
+				(path "/d5ebd247-5a7c-47c2-8aee-beabaef72d6d/94125b35-79a1-41d0-8b6c-f77e699b83b8"
+					(reference "J5")
+					(unit 1)
+				)

Commit message: skibbidi
Parts:
- removed J3: USB_B_Micro, Connector_USB:USB_Micro-B_Molex-105017-0001, symbol Connector:USB_B_Micro
- added D10: D_Schottky, Diode_SMD:D_SOD-323_HandSoldering, symbol Device:D_Schottky
- added D7: SP0503BAHT, Package_TO_SOT_SMD:SOT-143, symbol utsvt-chips:SP0503BAHT-Power_Protection
- added J6: UJ31-CH-G2-SMT-TR, UTSVT_Connectors:CUI_UJ31-CH-G2-SMT-TR, symbol UJ31-CH-G2-SMT-TR:UJ31-CH-G2-SMT-TR
- added R22, R30: 5.1k, Resistor_SMD:R_0805_2012Metric, symbol Device:R
Connections:
- net D+: now also D7.2 (K), J6.A6 (DP1)
- net D-: now also D7.3 (K), J6.A7 (DN1)
- net GND: now also D7.1 (A), J6.A1 (GND), J6.A12 (GND__1), J6.B1 (GND__2), J6.B12 (GND__3), J6.SH1 (SHIELD), J6.SH2 (SHIELD__1), J6.SH4 (SHIELD__3), R22.1, R30.1
- net vbus renamed VBUS
- net VBUS: now also D10.1 (K), D7.4 (K)
- new net: J6.A5 (CC1), R22.2
- new net: D10.2 (A), J6.A4 (VBUS)
- new net: J6.A9 (VBUS__1), J6.B4 (VBUS__2), J6.B9 (VBUS__3)
- new net: J6.B5 (CC2), R30.2
- no-connect marks 6 -> 17
Other:
- note added: "vbus should be ~5V"
- moved on the sheet: C1, C10, C18, C19, C28, C29, J5, R1, R25, R26, R7, U6

Commit message: poop and farts
Connections:
- net GND: now also J6.SH3 (SHIELD__2)
- net CC1: now reaches J6.A5 (CC1), R22.2
- net CC2: now reaches J6.B5 (CC2), R30.2
Changed lines of the file:
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@@
+	)
+	(junction
+		(at 59.055 156.845)
+		(diameter 0)
+		(color 0 0 0 0)
 	)
 	(junction
@@
 	(wire
 		(pts
+			(xy 57.15 156.845) (xy 59.055 156.845)
+		)
+		(stroke
+			(width 0)
+			(type default)
+		)
+	)
+	(wire
+		(pts
 			(xy 156.21 116.84) (xy 158.75 116.84)
 		)
@@
 	(wire
 		(pts
+			(xy 59.055 156.845) (xy 59.055 154.305)
+		)
+		(stroke
+			(width 0)
+			(type default)
+		)
+	)
+	(wire
+		(pts
 			(xy 139.7 95.25) (xy 142.24 95.25)
 		)
@@
 	(wire
 		(pts
-			(xy 59.055 159.385) (xy 59.055 154.305)
+			(xy 59.055 159.385) (xy 59.055 156.845)
 		)
 		(stroke
@@
 		(effects
 			(font
+				(size 1.27 1.27)
+			)
+			(justify left bottom)
+		)
+	)
+	(label "CC2"
+		(at 60.96 131.445 0)
+		(effects
+			(font
+				(size 1.27 1.27)
+			)
+			(justify left bottom)
+		)
+	)
+	(label "CC1"
+		(at 59.69 113.665 0)
+		(effects
+			(font
