File: USB.kicad_sch (KiCad schematic)
At the start: 15 parts, among them J2 USB4215-03-A, U8 CP2102N-A02-GQFN24

Commit message: finish mcu breakouts
Connections:
- net UART_RX renamed USART1_TX
- net UART_TX renamed USART1_RX
Other:
- moved on the sheet: R21, R22, R24, U8

Commit message: FUCK capacitors
Parts:
- C29: P/N (none) -> GRM21BR61H106KE43K
- C30, C32: P/N (none) -> 08055D475KAT4A
- C31, C33: P/N (none) -> MLASH168SB7104KTNA01
Changed lines of the file:
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@@
+			)
+		)
+		(property "P/N" "08055D475KAT4A"
+			(at 100.33 39.37 0)
+			(effects
+				(font
+					(size 1.27 1.27)
+				)
+				(hide yes)
 			)
 		)
@@
 			)
 		)
+		(property "P/N" "MLASH168SB7104KTNA01"
+			(at 113.03 66.04 0)
+			(effects
+				(font
+					(size 1.27 1.27)
+				)
+				(hide yes)
+			)
+		)
 		(pin "1"
 		)
@@
 			)
 		)
+		(property "P/N" "08055D475KAT4A"
+			(at 100.33 66.04 0)
+			(effects
+				(font
+					(size 1.27 1.27)
+				)
+				(hide yes)
+			)
+		)
 		(pin "1"
 		)
@@
 			)
 		)
+		(property "P/N" "MLASH168SB7104KTNA01"
+			(at 113.03 39.37 0)
+			(effects
+				(font
+					(size 1.27 1.27)
+				)
+				(hide yes)
+			)
+		)
 		(pin "1"
 		)
@@
 			(at 80.01 34.29 0)
 			(effects
+				(font
+					(size 1.27 1.27)
+				)
+				(hide yes)
+			)
+		)
+		(property "P/N" "GRM21BR61H106KE43K"
+			(at 80.01 34.29 0)
+			(effects

Commit message: all parts selected
Parts:
- R10: P/N (none) -> CRCW06030000Z0EI
- R14, R16: P/N (none) -> CRCW06035K10FKEC
- R21: P/N (none) -> CRCW06031K00FKEI
- R22: P/N (none) -> CRCW060322K1FKEBC
- R24: P/N (none) -> CRCW060347K5FKEAHP
Changed lines of the file:
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@@
+			)
+		)
+		(property "P/N" "CRCW06030000Z0EI "
+			(at 33.02 72.39 0)
+			(effects
+				(font
+					(size 1.27 1.27)
+				)
+				(hide yes)
 			)
 		)
@@
 		)
 		(property "Description" "Resistor"
+			(at 134.62 59.69 0)
+			(effects
+				(font
+					(size 1.27 1.27)
+				)
+				(hide yes)
+			)
+		)
+		(property "P/N" "CRCW060347K5FKEAHP "
 			(at 134.62 59.69 0)
 			(effects
@@
 			)
 		)
+		(property "P/N" "CRCW06035K10FKEC "
+			(at 31.75 106.68 0)
+			(effects
+				(font
+					(size 1.27 1.27)
+				)
+				(hide yes)
+			)
+		)
 		(pin "1"
 		)
@@
 		(property "Description" "Resistor"
 			(at 128.27 49.53 0)
+			(effects
+				(font
+					(size 1.27 1.27)
+				)
+				(hide yes)
+			)
+		)
+		(property "P/N" "CRCW060322K1FKEBC "
+			(at 128.27 49.53 90)
 			(effects
 				(font
@@
 			)
 		)
+		(property "P/N" "CRCW06031K00FKEI "
+			(at 138.43 30.48 0)
+			(effects
+				(font
+					(size 1.27 1.27)
+				)
+				(hide yes)
+			)
+		)
 		(pin "1"
 		)
@@
 			(at 21.59 106.68 0)
 			(effects
+				(font
+					(size 1.27 1.27)
+				)
+				(hide yes)
+			)
+		)
+		(property "P/N" "CRCW06035K10FKEC "
+			(at 21.59 106.68 0)
+			(effects

Commit message: add some footprints
Parts:
- R10, R14, R16, R21, R22, R24: footprint (none) -> Resistor_SMD:R_0603_1608Metric_Pad0.98x0.95mm_HandSolder
Changed lines of the file:
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@@
 			)
 		)
-		(property "Footprint" ""
+		(property "Footprint" "Resistor_SMD:R_0603_1608Metric_Pad0.98x0.95mm_HandSolder"
 			(at 31.242 72.39 90)
 			(effects
@@
 			)
 		)
-		(property "Footprint" ""
+		(property "Footprint" "Resistor_SMD:R_0603_1608Metric_Pad0.98x0.95mm_HandSolder"
 			(at 132.842 59.69 90)
 			(effects
@@
 			)
 		)
-		(property "Footprint" ""
+		(property "Footprint" "Resistor_SMD:R_0603_1608Metric_Pad0.98x0.95mm_HandSolder"
 			(at 29.972 106.68 90)
 			(effects
@@
 			)
 		)
-		(property "Footprint" ""
+		(property "Footprint" "Resistor_SMD:R_0603_1608Metric_Pad0.98x0.95mm_HandSolder"
 			(at 128.27 51.308 90)
 			(effects
@@
 			)
 		)
-		(property "Footprint" ""
+		(property "Footprint" "Resistor_SMD:R_0603_1608Metric_Pad0.98x0.95mm_HandSolder"
 			(at 136.652 30.48 90)
 			(effects
@@
 			)
 		)
-		(property "Footprint" ""
+		(property "Footprint" "Resistor_SMD:R_0603_1608Metric_Pad0.98x0.95mm_HandSolder"
 			(at 19.812 106.68 90)
 			(effects

Commit message: more stuff
Parts:
- J2: footprint (none) -> USB4215-03-A:GCT_USB4215-03-A_REVA
Changed lines of the file:
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@@
 			)
 		)
-		(property "Footprint" ""
+		(property "Footprint" "USB4215-03-A:GCT_USB4215-03-A_REVA"
 			(at 44.45 43.18 0)
 			(effects

Commit message: all footprints assigned
Parts:
- C29, C30, C32: footprint (none) -> Capacitor_SMD:C_0805_2012Metric_Pad1.18x1.45mm_HandSolder
- C31, C33: footprint (none) -> Capacitor_SMD:C_0603_1608Metric_Pad1.08x0.95mm_HandSolder
- D5: footprint (none) -> Diode_SMD:D_SOD-123
Changed lines of the file:
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@@
 			)
 		)
-		(property "Footprint" ""
+		(property "Footprint" "Diode_SMD:D_SOD-123"
 			(at 69.85 27.94 0)
 			(effects
@@
 			)
 		)
-		(property "Footprint" ""
+		(property "Footprint" "Capacitor_SMD:C_0805_2012Metric_Pad1.18x1.45mm_HandSolder"
 			(at 101.2952 43.18 0)
 			(effects
@@
 			)
 		)
-		(property "Footprint" ""
+		(property "Footprint" "Capacitor_SMD:C_0603_1608Metric_Pad1.08x0.95mm_HandSolder"
 			(at 113.9952 69.85 0)
 			(effects
@@
 			)
 		)
-		(property "Footprint" ""
+		(property "Footprint" "Capacitor_SMD:C_0805_2012Metric_Pad1.18x1.45mm_HandSolder"
 			(at 101.2952 69.85 0)
 			(effects
@@
 			)
 		)
-		(property "Footprint" ""
+		(property "Footprint" "Capacitor_SMD:C_0603_1608Metric_Pad1.08x0.95mm_HandSolder"
 			(at 113.9952 43.18 0)
 			(effects
@@
 			)
 		)
-		(property "Footprint" ""
+		(property "Footprint" "Capacitor_SMD:C_0805_2012Metric_Pad1.18x1.45mm_HandSolder"
 			(at 80.9752 38.1 0)
 			(effects

Commit message: CAN layout
Parts:
- J2: footprint USB4215-03-A:GCT_USB4215-03-A_REVA -> Connector_USB:USB_C_Receptacle_GCT_USB4105-xx-A_16P_TopMnt_Horizontal
Connections:
- net D+: now also D6.3 (K); no longer D6.2 (K)
- net D-: now also D6.2 (K); no longer D6.3 (K)
- net SH: now reaches J2.S1 (SHIELD), R10.1
- net VBUS: now reaches R22.2, R24.1, U8.8 (VBUS)
- net RST: now reaches R21.2, U8.9 (~{RST})
Other:
- moved on the sheet: R21
Changed lines of the file:
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@@
 	(text "Voltage divider\nper datasheet\npg. 9"
 		(exclude_from_sim no)
-		(at 135.636 45.466 0)
+		(at 135.636 42.926 0)
 		(effects
 			(font
@@
 	(wire
 		(pts
-			(xy 138.43 25.4) (xy 151.13 25.4)
+			(xy 137.16 25.4) (xy 151.13 25.4)
 		)
 		(stroke
@@
 	(wire
 		(pts
-			(xy 138.43 26.67) (xy 138.43 25.4)
-		)
-		(stroke
-			(width 0)
-			(type default)
-		)
-	)
-	(wire
-		(pts
-			(xy 138.43 36.83) (xy 140.97 36.83)
+			(xy 137.16 26.67) (xy 137.16 25.4)
+		)
+		(stroke
+			(width 0)
+			(type default)
+		)
+	)
+	(wire
+		(pts
+			(xy 137.16 36.83) (xy 140.97 36.83)
 		)
 		(stroke
@@
 	(wire
 		(pts
-			(xy 138.43 34.29) (xy 138.43 36.83)
+			(xy 137.16 34.29) (xy 137.16 36.83)
 		)
 		(stroke
@@
 		)
 	)
+	(label "VBUS"
+		(at 135.89 49.53 0)
+		(effects
+			(font
+				(size 1.27 1.27)
+			)
+			(justify left bottom)
+		)
+	)
 	(label "USART1_TX"
 		(at 177.8 39.37 180)
@@
 		)
 	)
-	(label "D-"
+	(label "D+"
 		(at 50.8 97.79 270)
 		(effects
@@
 			)
 			(justify right bottom)
+		)
+	)
+	(label "D-"
+		(at 48.26 97.79 270)
+		(effects
+			(font
+				(size 1.27 1.27)
+			)
+			(justify right bottom)
+		)
+	)
+	(label "SH"
+		(at 33.02 68.58 90)
+		(effects
+			(font
+				(size 1.27 1.27)
+			)
+			(justify left bottom)
 		)
 	)
@@
 		)
 	)
-	(label "CC1"
-		(at 64.77 33.02 180)
+	(label "RST"
+		(at 137.16 36.83 0)
 		(effects
 			(font
 				(size 1.27 1.27)
 			)
-			(justify right bottom)
-		)
-	)
-	(label "D+"
-		(at 48.26 97.79 270)
+			(justify left bottom)
+		)
+	)
+	(label "CC1"
+		(at 64.77 33.02 180)
 		(effects
 			(font
@@
 			)
 		)
-		(property "Footprint" "USB4215-03-A:GCT_USB4215-03-A_REVA"
+		(property "Footprint" "Connector_USB:USB_C_Receptacle_GCT_USB4105-xx-A_16P_TopMnt_Horizontal"
 			(at 44.45 43.18 0)
 			(effects
@@
 	(symbol
 		(lib_id "Device:R")
-		(at 138.43 30.48 0)
+		(at 137.16 30.48 0)
 		(unit 1)
 		(exclude_from_sim no)
@@
 		(fields_autoplaced yes)
 		(property "Reference" "R21"
-			(at 140.97 29.2099 0)
+			(at 139.7 29.2099 0)
 			(effects
 				(font
@@
 		)
 		(property "Value" "1k"
-			(at 140.97 31.7499 0)
+			(at 139.7 31.7499 0)
 			(effects
 				(font
@@
 		)
 		(property "Footprint" "Resistor_SMD:R_0603_1608Metric_Pad0.98x0.95mm_HandSolder"
-			(at 136.652 30.48 90)
+			(at 135.382 30.48 90)
 			(effects
 				(font
@@
 		)
 		(property "Datasheet" "~"
-			(at 138.43 30.48 0)
+			(at 137.16 30.48 0)
 			(effects
 				(font
@@
 		)
 		(property "Description" "Resistor"
-			(at 138.43 30.48 0)
+			(at 137.16 30.48 0)
 			(effects
 				(font
@@
 		)
 		(property "P/N" "CRCW06031K00FKEI "
-			(at 138.43 30.48 0)
-			(effects
-				(font
+			(at 137.16 30.48 0)
+			(effects
+				(font

Commit message: address some stuff
Parts:
- removed R10: 0, Resistor_SMD:R_0603_1608Metric_Pad0.98x0.95mm_HandSolder, symbol Device:R
- D6: Mouser Part Number 576-SP0503BAHTG -> (none)
Connections:
- net SH is gone; now on net GND: J2.S1 (SHIELD)
Other:
- note removed: "0 ohm cause ground loops can be fucky"
Changed lines of the file:
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@@
-		)
-	)
-	(text "0 ohm cause ground\nloops can be fucky"
-		(exclude_from_sim no)
-		(at 28.702 80.772 0)
-		(effects
-			(font
-				(size 1.27 1.27)
-			)
 		)
 	)
@@
 	(wire
 		(pts
-			(xy 33.02 76.2) (xy 33.02 77.47)
+			(xy 33.02 66.04) (xy 33.02 77.47)
 		)
 		(stroke
@@
 		(pts
 			(xy 100.33 43.18) (xy 100.33 44.45)
-		)
-		(stroke
-			(width 0)
-			(type default)
-		)
-	)
-	(wire
-		(pts
-			(xy 33.02 66.04) (xy 33.02 68.58)
 		)
 		(stroke
@@
 			)
 			(justify right bottom)
-		)
-	)
-	(label "SH"
-		(at 33.02 68.58 90)
-		(effects
-			(font
-				(size 1.27 1.27)
-			)
-			(justify left bottom)
 		)
 	)
@@
 			)
 		)
-		(property "Mouser Part Number" "576-SP0503BAHTG "
-			(at 50.8 107.95 0)
-			(effects
-				(font
-					(size 1.27 1.27)
-				)
-				(hide yes)
-			)
-		)
 		(property "P/N" "SP0503BAHTG"
 			(at 50.8 107.95 0)
@@
 					(unit 1)
 				)
-			)
-		)
-	)
-	(symbol
-		(lib_id "Device:R")
-		(at 33.02 72.39 0)
-		(unit 1)
-		(exclude_from_sim no)
-		(in_bom yes)
-		(on_board yes)
-		(dnp no)
-		(fields_autoplaced yes)
-		(property "Reference" "R10"
-			(at 35.56 71.1199 0)
-			(effects
-				(font
-					(size 1.27 1.27)
-				)
-				(justify left)
-			)
-		)
-		(property "Value" "0"
-			(at 35.56 73.6599 0)
-			(effects
-				(font
-					(size 1.27 1.27)
-				)
-				(justify left)
-			)
-		)
-		(property "Footprint" "Resistor_SMD:R_0603_1608Metric_Pad0.98x0.95mm_HandSolder"
-			(at 31.242 72.39 90)
-			(effects
-				(font
-					(size 1.27 1.27)
-				)
-				(hide yes)
-			)
-		)
-		(property "Datasheet" "~"
-			(at 33.02 72.39 0)
-			(effects
-				(font
-					(size 1.27 1.27)
-				)
-				(hide yes)
-			)
-		)
-		(property "Description" "Resistor"
-			(at 33.02 72.39 0)
-			(effects
-				(font
-					(size 1.27 1.27)
-				)
-				(hide yes)
-			)
-		)
-		(property "P/N" "CRCW06030000Z0EI "
-			(at 33.02 72.39 0)
-			(effects
-				(font
-					(size 1.27 1.27)
-				)
-				(hide yes)
-			)
-		)
-		(pin "1"
-		)
-		(pin "2"
-		)
-		(instances
-			(project ""
-				(path "/d5ebd247-5a7c-47c2-8aee-beabaef72d6d/94125b35-79a1-41d0-8b6c-f77e699b83b8"
-					(reference "R10")
-					(unit 1)
-				)
