File: PowerProtection.kicad_sch (KiCad schematic)
At the start: 11 parts, among them U7 LM76202QPWPRQ1

Commit message: idk anymore man
Connections:
- net 3.3V_Uniso renamed 3V3_Bus
Changed lines of the file:
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@@
 		)
 	)
-	(hierarchical_label "3.3V_Uniso"
+	(hierarchical_label "3V3_Bus"
 		(shape output)
 		(at 116.84 85.09 0)

Commit message: lakshay learns algebra + BOM
Parts:
- R22: value 10K -> 1k
- R4: value 100k -> 10k
- R5: value 3k -> 200
Changed lines of the file:
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@@
 		(fields_autoplaced yes)
 		(property "Reference" "R22"
-			(at 109.22 108.585 0)
-			(effects
-				(font
-					(size 1.27 1.27)
-				)
-				(justify left)
-			)
-		)
-		(property "Value" "10K"
-			(at 109.22 111.125 0)
+			(at 109.22 107.9499 0)
+			(effects
+				(font
+					(size 1.27 1.27)
+				)
+				(justify left)
+			)
+		)
+		(property "Value" "1k"
+			(at 109.22 110.4899 0)
 			(effects
 				(font
@@
 		)
 		(property "P/N" "CRCW080510K0FKEAC"
+			(at 106.68 109.22 0)
+			(effects
+				(font
+					(size 1.27 1.27)
+				)
+				(hide yes)
+			)
+		)
+		(property "PN" ""
+			(at 106.68 109.22 0)
+			(effects
+				(font
+					(size 1.27 1.27)
+				)
+				(hide yes)
+			)
+		)
+		(property "p/n" ""
 			(at 106.68 109.22 0)
 			(effects
@@
 			)
 		)
-		(property "Value" "100k"
+		(property "Value" "10k"
 			(at 108.458 90.043 0)
 			(effects
@@
 		)
 		(property "P/N" "CRCW0805100KFKEAC"
+			(at 106.68 88.9 0)
+			(effects
+				(font
+					(size 1.27 1.27)
+				)
+				(hide yes)
+			)
+		)
+		(property "PN" ""
+			(at 106.68 88.9 0)
+			(effects
+				(font
+					(size 1.27 1.27)
+				)
+				(hide yes)
+			)
+		)
+		(property "p/n" ""
 			(at 106.68 88.9 0)
 			(effects
@@
 			)
 		)
+		(property "PN" ""
+			(at 179.07 97.79 0)
+			(effects
+				(font
+					(size 1.27 1.27)
+				)
+				(hide yes)
+			)
+		)
+		(property "p/n" ""
+			(at 179.07 97.79 0)
+			(effects
+				(font
+					(size 1.27 1.27)
+				)
+				(hide yes)
+			)
+		)
 		(pin "1"
 		)
@@
 		)
 		(property "P/N" ""
+			(at 87.63 87.63 0)
+			(effects
+				(font
+					(size 1.27 1.27)
+				)
+				(hide yes)
+			)
+		)
+		(property "PN" ""
+			(at 87.63 87.63 0)
+			(effects
+				(font
+					(size 1.27 1.27)
+				)
+				(hide yes)
+			)
+		)
+		(property "p/n" ""
 			(at 87.63 87.63 0)
 			(effects
@@
 			)
 		)
-		(property "Value" "3k"
+		(property "Value" "200"
 			(at 109.22 100.3299 0)
 			(effects
@@
 		)
 		(property "Description" "Resistor"
+			(at 106.68 99.06 0)
+			(effects
+				(font
+					(size 1.27 1.27)
+				)
+				(hide yes)
+			)
+		)
+		(property "P/N" ""
+			(at 106.68 99.06 0)
+			(effects
+				(font
+					(size 1.27 1.27)
+				)
+				(hide yes)
+			)
+		)
+		(property "PN" ""
+			(at 106.68 99.06 0)
+			(effects
+				(font
+					(size 1.27 1.27)
+				)
+				(hide yes)
+			)
+		)
+		(property "p/n" ""
 			(at 106.68 99.06 0)
 			(effects
@@
 			)
 		)
+		(property "PN" ""
+			(at 175.26 85.09 0)
+			(effects
+				(font
+					(size 1.27 1.27)
+				)
+				(hide yes)
+			)
+		)
+		(property "p/n" ""
+			(at 175.26 85.09 0)
+			(effects
+				(font
+					(size 1.27 1.27)
+				)
+				(hide yes)
+			)
+		)
 		(pin "1"
 		)
@@
 		)
 		(property "P/N" "CRCW0805100KFKEAC"
+			(at 162.56 85.09 0)
+			(effects
+				(font
+					(size 1.27 1.27)
+				)
+				(hide yes)
+			)
+		)
+		(property "PN" ""
+			(at 162.56 85.09 0)
+			(effects
+				(font
+					(size 1.27 1.27)
+				)
+				(hide yes)
+			)
+		)
+		(property "p/n" ""
 			(at 162.56 85.09 0)
 			(effects
@@
 			)
 		)
+		(property "PN" ""
+			(at 115.57 95.25 0)
+			(effects
+				(font
+					(size 1.27 1.27)
+				)
+				(hide yes)
+			)
+		)
+		(property "p/n" ""
+			(at 115.57 95.25 0)
+			(effects
+				(font
+					(size 1.27 1.27)
+				)
+				(hide yes)
+			)
+		)
 		(pin "1"
 		)
@@
 			)
 		)
+		(property "PN" ""
+			(at 167.64 100.33 0)
+			(effects
+				(font
+					(size 1.27 1.27)
+				)
+				(hide yes)
+			)
+		)
+		(property "p/n" ""
+			(at 167.64 100.33 0)
+			(effects
+				(font
+					(size 1.27 1.27)
+				)
+				(hide yes)
+			)
+		)
 		(pin "1"
 		)
@@
 			)
 		)
+		(property "PN" ""
+			(at 100.33 87.63 0)
+			(effects
+				(font
+					(size 1.27 1.27)
+				)
+				(hide yes)
+			)
+		)
+		(property "p/n" ""
+			(at 100.33 87.63 0)
+			(effects
+				(font
+					(size 1.27 1.27)
+				)
+				(hide yes)
+			)
+		)
 		(pin "1"
 		)
@@
 			(at 143.51 78.74 0)
 			(effects
+				(font
+					(size 1.27 1.27)
+				)
+				(hide yes)
+			)
+		)
+		(property "PN" ""
+			(at 143.51 78.74 0)
+			(effects
+				(font
+					(size 1.27 1.27)
+				)
+				(hide yes)
+			)
+		)
+		(property "p/n" ""
+			(at 143.51 78.74 0)
+			(effects

Commit message: BOOM
Parts:
- C20, C23: value 47uF -> 10uF; Mouser Part Number (none) -> 581-22201C106KAT2A; P/N (none) -> TMK212BBJ106MGHT
- R22: P/N CRCW080510K0FKEAC -> CRCW08051K00FKEAC
- R5: P/N (none) -> CR0805-JW-201ELF

Commit message: V2.1 (#17)
* womp womp

* woop woop

* can+power layout

* and so it begins...

* wahoo?

* routing done mayhaps

* fixed LED traces

* switched green and yellow traces

* better LED ordering + silkscreen stuff

* less via in pad

* addressed prat

* womp womp

* it's gerbing time

* i'm so dumb

* new dc-dc

* change max draw on iso dc-dc

* gerbers

* update ibom

* bom
Parts:
- removed R22: 1k, Resistor_SMD:R_0805_2012Metric, symbol Device:R
- removed R4: 10k, Resistor_SMD:R_0805_2012Metric, symbol Device:R
- removed R5: 200, Resistor_SMD:R_0805_2012Metric, symbol Device:R
- added R12: 10k, Resistor_SMD:R_0805_2012Metric, symbol Device:R
- added R13: 200, Resistor_SMD:R_0805_2012Metric, symbol Device:R
- added R15: 1k, Resistor_SMD:R_0805_2012Metric, symbol Device:R
- added R20: 402k, Resistor_SMD:R_0805_2012Metric, symbol Device:R
- R24: value 100k -> 10k; Mouser Part Number 71-CRCW0805100KFKEAC -> (none); P/N CRCW0805100KFKEAC -> CRCW080510K0FKEAC
Connections:
- net 12V_Ext: now also R12.1
- net OVP: now also R13.2, R15.1
- net RTN: now also R15.2, R20.2; no longer U7.6 (MODE)
- net UVLO: now also R12.2, R13.1
- new net MODE: R20.1, U7.6 (MODE)
Other:
- note added: "Set to circuit breaker Auto-retry"

Commit message: purge shit
Parts:
- C20, C23, C25: footprint Capacitor_SMD:C_0805_2012Metric -> (none)
- D2: footprint Diode_SMD:D_SOD-323 -> (none)
- R12, R13, R15, R20, R23, R24, R27: footprint Resistor_SMD:R_0805_2012Metric -> (none)
- U7: footprint UTSVT_ICs:SOP65P640X120-17N -> (none)
Changed lines of the file:
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@@
 			)
 		)
-		(property "Footprint" "Capacitor_SMD:C_0805_2012Metric"
+		(property "Footprint" ""
 			(at 180.0352 101.6 0)
 			(effects
@@
 			)
 		)
-		(property "Footprint" "Capacitor_SMD:C_0805_2012Metric"
+		(property "Footprint" ""
 			(at 86.0552 91.44 0)
 			(effects
@@
 			)
 		)
-		(property "Footprint" "Resistor_SMD:R_0805_2012Metric"
+		(property "Footprint" ""
 			(at 160.782 85.09 90)
 			(effects
@@
 			)
 		)
-		(property "Footprint" "Resistor_SMD:R_0805_2012Metric"
+		(property "Footprint" ""
 			(at 44.577 114.935 90)
 			(effects
@@
 			)
 		)
-		(property "Footprint" "Resistor_SMD:R_0805_2012Metric"
+		(property "Footprint" ""
 			(at 41.402 163.83 90)
 			(effects
@@
 			)
 		)
-		(property "Footprint" "Capacitor_SMD:C_0805_2012Metric"
+		(property "Footprint" ""
 			(at 178.7652 88.9 0)
 			(effects
@@
 			)
 		)
-		(property "Footprint" "Resistor_SMD:R_0805_2012Metric"
+		(property "Footprint" ""
 			(at 113.792 95.25 90)
 			(effects
@@
 			)
 		)
-		(property "Footprint" "Resistor_SMD:R_0805_2012Metric"
+		(property "Footprint" ""
 			(at 165.862 100.33 90)
 			(effects
@@
 			)
 		)
-		(property "Footprint" "Diode_SMD:D_SOD-323"
+		(property "Footprint" ""
 			(at 105.41 87.63 0)
 			(effects
@@
 			)
 		)
-		(property "Footprint" "UTSVT_ICs:SOP65P640X120-17N"
+		(property "Footprint" ""
 			(at 143.51 78.74 0)
 			(effects
@@
 			)
 		)
-		(property "Footprint" "Resistor_SMD:R_0805_2012Metric"
+		(property "Footprint" ""
 			(at 41.402 153.67 90)
 			(effects
@@
 			)
 		)
-		(property "Footprint" "Resistor_SMD:R_0805_2012Metric"
+		(property "Footprint" ""
 			(at 41.402 143.51 90)
 			(effects

Commit message: initial PP changes
Parts:
- C20, C23: P/N TMK212BBJ106MGHT -> (none)
- C25: P/N C0805C104M5RACTU -> (none)
- D2: value SD12_SOD323 -> TVS; Mouser Part Number 771-PESD15VL1BA-T/R -> (none); Mouser Price/Stock https://www.mouser.com/ProductDetail/Nexperia/PESD15VL1BA11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 -> (none); P/N PESD15VL1BA,115 -> SD24C-01FTG
- R12: P/N CRCW0805100KFKEAC -> (none)
- R13: P/N CR0805-JW-201ELF -> (none)
- R15: P/N CRCW08051K00FKEAC -> (none)
- R20: P/N RC0805FR-07402KL -> (none)
- R23, R24, R27: P/N CRCW080510K0FKEAC -> (none)
Connections:
- net +12V renamed +24V
- net 12V_Ext renamed 24V_Ext
- net GNDPWR renamed GND
Other:
- note added: "TODO: change ILIM to 1.5A Current lim(A) = 12/Rilim(k) 1.2A = 12/10k ohms"
- note added: "add more decoupling caps both sides"
- note added: "check val"
- note added: "fix vals"
- note added: "sufficient current limit?"
- note added: "want PTC as well?"
- note added: "why pu to 3v3?"
- note removed: "Current lim(A) = 12/Rilim(k) 1.2A = 12/10k ohms"
- moved on the sheet: C20, C23, C25, D2, R12, R13, R15, R20, R23, R24, R27, U7
