File: PowerProtection.kicad_sch (KiCad schematic)
At the start: 12 parts, among them U7 LM76202QPWPRQ1

Commit message: completed PP
Parts:
- removed R24: 10k, symbol Device:R
- added C1, C2: 1uF, symbol Device:C
- added R1: 10k, symbol Device:R
- R12: value 10k -> 45.3k
- R13: value 200 -> 590
- R15: value 1k -> 2k
- U7: footprint (none) -> UTSVT_Power:LM76202QPWPRQ1; symbol utsvt-chips:LM76202QPWPRQ1 -> utsvt_power:LM76202QPWPRQ1; Height (none) -> 1.2; Manufacturer_Name (none) -> Texas Instruments; Mouser Part Number (none) -> 595-LM76202QPWPRQ1
Connections:
- net +24V: now also C2.1, R1.1
- net 24V_Ext: now also C1.1
- net Fault: now also R1.2
- net GND: now also C1.2, C2.2
- net SHDN: now reaches R23.2, U7.7 (~{SHDN})
- net ILIM: now reaches R27.1, U7.11 (ILIM)
Other:
- note added: "20.88 ms ramp time"
- note added: "Functional Mode Selection"
- note added: "ILim(A) = 12/R(k) 1.2A = 12/10kΩ"
- note added: "Overcurrent Protection"
- note added: "Pullups"
- note added: "Set to circuit breaker (latchoff) Use 0 ohm resistor for auto-retry (540ms)"
- note added: "Under/Overvoltage Protection"
- note removed: "Set to circuit breaker Auto-retry"
- note removed: "TODO: change ILIM to 1.5A Current lim(A) = 12/Rilim(k) 1.2A = 12/10k ohms"
- note removed: "UVLO rising voltage: 1.1V OVLO divider voltage: 1.19V"
- note removed: "add more decoupling caps both sides"
- note removed: "check val"
- note removed: "fix vals"
- note removed: "sufficient current limit?"
- note removed: "want PTC as well?"
- note removed: "why pu to 3v3?"
- title: (none) -> Power Protection
- moved on the sheet: C20, C23, C25, D2, R12, R13, R15, R20, R23, R27, U7

Commit message: kinda add buck
Connections:
- net 3V3_Bus renamed +3.3V
Other:
- note added: "SHDN has weak internal pullup - pulled up to MCU voltage after initial power on"
- moved on the sheet: R1, R23
Changed lines of the file:
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@@
 	)
 	(rectangle
-		(start 150.495 43.18)
-		(end 175.26 76.2)
+		(start 147.955 43.18)
+		(end 194.945 76.2)
 		(stroke
 			(width 0)
@@
 	(text "Pullups"
 		(exclude_from_sim no)
-		(at 151.638 46.228 0)
+		(at 149.098 46.228 0)
 		(effects
 			(font
@@
 		)
 	)
+	(text "SHDN has weak internal\npullup - pulled up to\nMCU voltage after initial\npower on"
+		(exclude_from_sim no)
+		(at 180.34 58.674 0)
+		(effects
+			(font
+				(size 1.27 1.27)
+			)
+		)
+	)
 	(junction
 		(at 45.72 31.75)
@@
 	(wire
 		(pts
-			(xy 165.1 97.79) (xy 165.1 93.98)
+			(xy 165.1 96.52) (xy 165.1 93.98)
 		)
 		(stroke
@@
 	(wire
 		(pts
-			(xy 154.94 72.39) (xy 154.94 68.58)
+			(xy 152.4 72.39) (xy 152.4 68.58)
 		)
 		(stroke
@@
 	(wire
 		(pts
-			(xy 172.72 72.39) (xy 166.37 72.39)
+			(xy 165.1 83.82) (xy 165.1 86.36)
+		)
+		(stroke
+			(width 0)
+			(type default)
+		)
+	)
+	(wire
+		(pts
+			(xy 170.18 72.39) (xy 163.83 72.39)
 		)
 		(stroke
@@
 	(wire
 		(pts
-			(xy 157.48 72.39) (xy 154.94 72.39)
+			(xy 154.94 72.39) (xy 152.4 72.39)
 		)
 		(stroke
@@
 	(wire
 		(pts
-			(xy 132.08 97.79) (xy 129.54 97.79)
+			(xy 135.89 97.79) (xy 129.54 97.79)
 		)
 		(stroke
@@
 	(wire
 		(pts
-			(xy 166.37 72.39) (xy 166.37 68.58)
+			(xy 163.83 72.39) (xy 163.83 68.58)
 		)
 		(stroke
@@
 	(wire
 		(pts
-			(xy 154.94 58.42) (xy 154.94 60.96)
+			(xy 152.4 58.42) (xy 152.4 60.96)
 		)
 		(stroke
@@
 	(wire
 		(pts
+			(xy 170.18 83.82) (xy 165.1 83.82)
+		)
+		(stroke
+			(width 0)
+			(type default)
+		)
+	)
+	(wire
+		(pts
 			(xy 21.59 106.68) (xy 21.59 107.95)
 		)
@@
 	(wire
 		(pts
-			(xy 166.37 58.42) (xy 166.37 60.96)
+			(xy 163.83 58.42) (xy 163.83 60.96)
 		)
 		(stroke
@@
 	(wire
 		(pts
-			(xy 21.59 107.95) (xy 30.48 107.95)
+			(xy 129.54 87.63) (xy 135.89 87.63)
 		)
 		(stroke
@@
 	(wire
 		(pts
-			(xy 111.76 41.91) (xy 102.87 41.91)
+			(xy 21.59 107.95) (xy 30.48 107.95)
 		)
 		(stroke
@@
 	(wire
 		(pts
-			(xy 165.1 81.28) (xy 165.1 86.36)
+			(xy 111.76 41.91) (xy 102.87 41.91)
 		)
 		(stroke
@@
 	(wire
 		(pts
-			(xy 170.18 97.79) (xy 165.1 97.79)
+			(xy 170.18 96.52) (xy 165.1 96.52)
 		)
 		(stroke
@@
 	(wire
 		(pts
+			(xy 129.54 87.63) (xy 129.54 88.9)
+		)
+		(stroke
+			(width 0)
+			(type default)
+		)
+	)
+	(wire
+		(pts
 			(xy 135.89 31.75) (xy 135.89 34.29)
 		)
@@
 	)
 	(label "RTN"
-		(at 132.08 97.79 0)
+		(at 135.89 97.79 180)
 		(effects
 			(font
 				(size 1.27 1.27)
 			)
-			(justify left bottom)
+			(justify right bottom)
 		)
 	)
 	(label "SHDN"
-		(at 172.72 72.39 180)
+		(at 170.18 72.39 180)
 		(effects
 			(font
@@
 	)
 	(label "RTN"
-		(at 170.18 97.79 180)
+		(at 170.18 96.52 180)
 		(effects
 			(font
@@
 	)
 	(label "ILIM"
-		(at 165.1 81.28 270)
+		(at 170.18 83.82 180)
 		(effects
 			(font
@@
 	)
 	(label "MODE"
-		(at 129.54 88.9 0)
+		(at 135.89 87.63 180)
 		(effects
 			(font
 				(size 1.27 1.27)
 			)
-			(justify left bottom)
+			(justify right bottom)
 		)
 	)
@@
 	)
 	(hierarchical_label "Fault"
-		(shape input)
-		(at 107.95 36.83 0)
-		(effects
-			(font
-				(size 1.27 1.27)
-			)
-			(justify left)
-		)
-	)
-	(hierarchical_label "3V3_Bus"
 		(shape output)
-		(at 166.37 58.42 90)
+		(at 107.95 36.83 0)
 		(effects
 			(font
@@
 	)
 	(hierarchical_label "Fault"
-		(shape input)
-		(at 157.48 72.39 0)
+		(shape output)
+		(at 154.94 72.39 0)
 		(effects
 			(font
@@
 	(symbol
 		(lib_id "power:+12V")
-		(at 154.94 58.42 0)
+		(at 152.4 58.42 0)
 		(unit 1)
 		(exclude_from_sim no)
@@
 		(fields_autoplaced yes)
 		(property "Reference" "#PWR04"
-			(at 154.94 62.23 0)
+			(at 152.4 62.23 0)
 			(effects
 				(font
@@
 		)
 		(property "Value" "+24V"
-			(at 154.94 53.34 0)
+			(at 152.4 53.34 0)
 			(effects
 				(font
@@
 		)
 		(property "Footprint" ""
-			(at 154.94 58.42 0)
+			(at 152.4 58.42 0)
 			(effects
 				(font
@@
 		)
 		(property "Datasheet" ""
-			(at 154.94 58.42 0)
+			(at 152.4 58.42 0)
 			(effects
 				(font
@@
 		)
 		(property "Description" "Power symbol creates a global label with name \"+12V\""
-			(at 154.94 58.42 0)
+			(at 152.4 58.42 0)
 			(effects
 				(font
@@
 	)
 	(symbol
+		(lib_id "power:+3.3V")
+		(at 163.83 58.42 0)
+		(unit 1)
+		(exclude_from_sim no)
+		(in_bom yes)
+		(on_board yes)
+		(dnp no)
+		(fields_autoplaced yes)
+		(property "Reference" "#PWR05"
+			(at 163.83 62.23 0)
+			(effects
+				(font
+					(size 1.27 1.27)
+				)
+				(hide yes)
+			)
+		)
+		(property "Value" "+3.3V"
+			(at 163.83 53.34 0)
+			(effects
+				(font
+					(size 1.27 1.27)
+				)
+			)
+		)
+		(property "Footprint" ""
+			(at 163.83 58.42 0)
+			(effects
+				(font
+					(size 1.27 1.27)
+				)
+				(hide yes)
+			)
+		)
+		(property "Datasheet" ""
+			(at 163.83 58.42 0)
+			(effects
+				(font
+					(size 1.27 1.27)
+				)
+				(hide yes)
+			)
+		)
+		(property "Description" "Power symbol creates a global label with name \"+3.3V\""
+			(at 163.83 58.42 0)
+			(effects
+				(font
+					(size 1.27 1.27)
+				)
+				(hide yes)
+			)
+		)
+		(pin "1"
+		)
+		(instances
+			(project "PeripheralSOM"
+				(path "/d5ebd247-5a7c-47c2-8aee-beabaef72d6d/60a4ab70-544e-48ed-aa76-f39bfcac39df/e2d9692e-b475-45c2-ba25-1b5b4c5e9a86"
+					(reference "#PWR05")
+					(unit 1)
+				)
+			)
+		)
+	)
+	(symbol
 		(lib_id "Device:R")
 		(at 129.54 92.71 0)
@@
 	(symbol
 		(lib_id "Device:R")
-		(at 154.94 64.77 0)
+		(at 152.4 64.77 0)
 		(unit 1)
 		(exclude_from_sim no)
@@
 		(dnp no)
 		(property "Reference" "R1"
-			(at 156.718 63.6016 0)
+			(at 154.178 63.6016 0)
 			(effects
 				(font
@@
 		)
 		(property "Value" "10k"
-			(at 156.718 65.913 0)
+			(at 154.178 65.913 0)
 			(effects
 				(font
@@
 		)
 		(property "Footprint" ""
-			(at 153.162 64.77 90)
+			(at 150.622 64.77 90)
 			(effects
 				(font
@@
 		)
 		(property "Datasheet" "~"
-			(at 154.94 64.77 0)
+			(at 152.4 64.77 0)
 			(effects
 				(font
@@
 		)
 		(property "Description" "Resistor"
-			(at 154.94 64.77 0)
+			(at 152.4 64.77 0)
 			(effects
 				(font
@@
 		)
 		(property "Mouser Part Number" ""
-			(at 154.94 64.77 0)
+			(at 152.4 64.77 0)
 			(effects
 				(font
@@
 		)
 		(property "P/N" ""
-			(at 154.94 64.77 0)
+			(at 152.4 64.77 0)
 			(effects
 				(font
@@
 		)
 		(property "PN" ""
-			(at 154.94 64.77 0)
+			(at 152.4 64.77 0)
 			(effects
 				(font
@@
 		)
 		(property "p/n" ""
-			(at 154.94 64.77 0)
+			(at 152.4 64.77 0)
 			(effects
 				(font
@@
 	(symbol
 		(lib_id "Device:R")
-		(at 166.37 64.77 0)
+		(at 163.83 64.77 0)
 		(unit 1)
 		(exclude_from_sim no)
@@
 		(fields_autoplaced yes)
 		(property "Reference" "R23"
-			(at 168.91 64.135 0)
+			(at 166.37 64.135 0)
 			(effects
 				(font
@@
 		)
 		(property "Value" "10K"
-			(at 168.91 66.675 0)
+			(at 166.37 66.675 0)
 			(effects
 				(font
@@
 		)
 		(property "Footprint" ""
-			(at 164.592 64.77 90)
+			(at 162.052 64.77 90)
 			(effects
 				(font
@@
 		)
 		(property "Datasheet" "~"
-			(at 166.37 64.77 0)
+			(at 163.83 64.77 0)
 			(effects
 				(font
@@
 		)
 		(property "Description" "Resistor"
-			(at 166.37 64.77 0)
+			(at 163.83 64.77 0)
 			(effects
 				(font
@@
 		)
 		(property "Mouser Part Number" "71-CRCW080510K0FKEAC"
-			(at 166.37 64.77 0)
+			(at 163.83 64.77 0)
 			(effects
 				(font
@@
 		)
 		(property "P/N" ""
-			(at 166.37 64.77 0)
+			(at 163.83 64.77 0)
 			(effects
 				(font
@@
 		)
 		(property "PN" ""
-			(at 166.37 64.77 0)
+			(at 163.83 64.77 0)
 			(effects
 				(font
@@
 		)
 		(property "p/n" ""
-			(at 166.37 64.77 0)
+			(at 163.83 64.77 0)
 			(effects
 				(font

Commit message: finish buck sch
Parts:
- U7: Height 1.2 -> (none)

Commit message: lower OVP
Parts:
- C1, C20: Mouser Part Number 581-22201C106KAT2A -> (none)
- R15: value 2k -> 2.1k
Other:
- note added: "OVP set to 27v for buck max voltage of 28v"

Commit message: FUCK capacitors
Parts:
- C1, C2: P/N (none) -> MLASU168SB5105KTNA01
- C20, C23: P/N (none) -> GRM21BR61H106KE43K
- C25: P/N (none) -> MLASH168SB7104KTNA01
Changed lines of the file:
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@@
 			)
 		)
-		(property "P/N" ""
+		(property "P/N" "MLASH168SB7104KTNA01"
 			(at 111.76 46.99 0)
 			(effects
@@
 			)
 		)
-		(property "P/N" ""
+		(property "P/N" "GRM21BR61H106KE43K"
 			(at 34.29 36.83 0)
 			(effects
@@
 			)
 		)
-		(property "P/N" ""
+		(property "P/N" "GRM21BR61H106KE43K"
 			(at 135.89 38.1 0)
 			(effects
@@
 			)
 		)
-		(property "P/N" ""
+		(property "P/N" "MLASU168SB5105KTNA01"
 			(at 125.73 38.1 0)
 			(effects
@@
 			)
 		)
-		(property "P/N" ""
+		(property "P/N" "MLASU168SB5105KTNA01"
 			(at 45.72 36.83 0)
 			(effects

Commit message: all parts selected
Parts:
- R1: P/N (none) -> CRCW060310K0FKEI
- R12: P/N (none) -> CRCW060345K3FKEAHP
- R13: P/N (none) -> CRCW0603590RFKEA
- R15: P/N (none) -> CRCW06032K10FKEA
- R20: P/N (none) -> CRCW0603402KFKEAC
- R23, R27: value 10K -> 10k; P/N (none) -> CRCW060310K0FKEI
Changed lines of the file:
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@@
 			)
 		)
-		(property "P/N" ""
+		(property "P/N" "CRCW0603402KFKEAC "
 			(at 129.54 92.71 0)
 			(effects
@@
 			)
 		)
-		(property "P/N" ""
+		(property "P/N" "CRCW06032K10FKEA "
 			(at 21.59 123.19 0)
 			(effects
@@
 			)
 		)
-		(property "P/N" ""
+		(property "P/N" "CRCW060310K0FKEI "
 			(at 152.4 64.77 0)
 			(effects
@@
 			)
 		)
-		(property "Value" "10K"
+		(property "Value" "10k"
 			(at 166.37 66.675 0)
 			(effects
@@
 			)
 		)
-		(property "P/N" ""
+		(property "P/N" "CRCW060310K0FKEI "
 			(at 163.83 64.77 0)
 			(effects
@@
 			)
 		)
-		(property "Value" "10K"
+		(property "Value" "10k"
 			(at 167.64 92.075 0)
 			(effects
@@
 			)
 		)
-		(property "P/N" ""
+		(property "P/N" "CRCW060310K0FKEI "
 			(at 165.1 90.17 0)
 			(effects
@@
 			)
 		)
-		(property "P/N" ""
+		(property "P/N" "CRCW0603590RFKEA"
 			(at 21.59 113.03 0)
 			(effects
@@
 			)
 		)
-		(property "P/N" ""
+		(property "P/N" "CRCW060345K3FKEAHP "
 			(at 21.59 102.87 0)
 			(effects

Commit message: add IMON, change conn pinout
Parts:
- added D10: TVS, symbol Device:D_Zener
- added R30: 24m, symbol Device:R
- added R31: 100k, symbol Device:R
Connections:
- net GND: now also D10.2 (A)
- net RTN: now also R30.2
- net IMON: now reaches U7.10 (IMON)
- net IMON: now also R30.1, R31.1
- new net IMON_OUT: D10.1 (K), R31.2
- no-connect marks 3 -> 2
Other:
- note added: "Current Monitoring"
- note added: "DNP until validated"
- note added: "Typical gain: 78.28 uA/A Vout @ 1.3A = 2.407v R(imon) = 23.7 mΩ"
- moved on the sheet: C1, C2, C20, C23, C25, D2, R1, R23, R27, U7

Commit message: add some footprints
Parts:
- R1, R12, R13, R15, R20, R23, R27, R30: footprint (none) -> Resistor_SMD:R_0603_1608Metric_Pad0.98x0.95mm_HandSolder
- R31: footprint (none) -> Resistor_SMD:R_0603_1608Metric_Pad0.98x0.95mm_HandSolder; P/N (none) -> CRCW0603100KFKEE
Changed lines of the file:
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@@
 			)
 		)
-		(property "Footprint" ""
+		(property "Footprint" "Resistor_SMD:R_0603_1608Metric_Pad0.98x0.95mm_HandSolder"
 			(at 153.67 32.258 90)
 			(effects
@@
 		(property "Description" "Resistor"
 			(at 153.67 30.48 0)
+			(effects
+				(font
+					(size 1.27 1.27)
+				)
+				(hide yes)
+			)
+		)
+		(property "P/N" "CRCW0603100KFKEE "
+			(at 153.67 30.48 90)
 			(effects
 				(font
@@
 			)
 		)
-		(property "Footprint" ""
+		(property "Footprint" "Resistor_SMD:R_0603_1608Metric_Pad0.98x0.95mm_HandSolder"
 			(at 127.762 92.71 90)
 			(effects
@@
 			)
 		)
-		(property "Footprint" ""
+		(property "Footprint" "Resistor_SMD:R_0603_1608Metric_Pad0.98x0.95mm_HandSolder"
 			(at 19.812 123.19 90)
 			(effects
@@
 			)
 		)
-		(property "Footprint" ""
+		(property "Footprint" "Resistor_SMD:R_0603_1608Metric_Pad0.98x0.95mm_HandSolder"
 			(at 144.272 88.9 90)
 			(effects
@@
 			)
 		)
-		(property "Footprint" ""
+		(property "Footprint" "Resistor_SMD:R_0603_1608Metric_Pad0.98x0.95mm_HandSolder"
 			(at 155.702 88.9 90)
 			(effects
@@
 			)
 		)
-		(property "Footprint" ""
+		(property "Footprint" "Resistor_SMD:R_0603_1608Metric_Pad0.98x0.95mm_HandSolder"
 			(at 35.052 68.58 90)
 			(effects
@@
 			)
 		)
-		(property "Footprint" ""
+		(property "Footprint" "Resistor_SMD:R_0603_1608Metric_Pad0.98x0.95mm_HandSolder"
 			(at 140.462 36.83 90)
 			(effects
@@
 			)
 		)
-		(property "Footprint" ""
+		(property "Footprint" "Resistor_SMD:R_0603_1608Metric_Pad0.98x0.95mm_HandSolder"
 			(at 19.812 113.03 90)
 			(effects
@@
 			)
 		)
-		(property "Footprint" ""
+		(property "Footprint" "Resistor_SMD:R_0603_1608Metric_Pad0.98x0.95mm_HandSolder"
 			(at 19.812 102.87 90)
 			(effects
