File: PowerProtection.kicad_sch (KiCad schematic)
At the start: 17 parts, among them U7 LM76202QPWPRQ1

Commit message: all footprints assigned
Parts:
- C1, C2, C25: footprint (none) -> Capacitor_SMD:C_0603_1608Metric_Pad1.08x0.95mm_HandSolder
- C20, C23: footprint (none) -> Capacitor_SMD:C_0805_2012Metric_Pad1.18x1.45mm_HandSolder
- D10: footprint (none) -> Diode_SMD:D_SOD-923
- D2: footprint (none) -> Diode_SMD:D_SOD-323_HandSoldering
Changed lines of the file:
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@@
 			)
 		)
-		(property "Footprint" ""
+		(property "Footprint" "Diode_SMD:D_SOD-923"
 			(at 158.75 36.83 0)
 			(effects
@@
 			)
 		)
-		(property "Datasheet" "~"
+		(property "Datasheet" "https://www.onsemi.com/pdf/datasheet/esd9101-d.pdf"
 			(at 158.75 36.83 0)
 			(effects
@@
 			)
 		)
-		(property "Footprint" ""
+		(property "Footprint" "Capacitor_SMD:C_0603_1608Metric_Pad1.08x0.95mm_HandSolder"
 			(at 107.6452 50.8 0)
 			(effects
@@
 			)
 		)
-		(property "Footprint" ""
+		(property "Footprint" "Capacitor_SMD:C_0805_2012Metric_Pad1.18x1.45mm_HandSolder"
 			(at 30.1752 40.64 0)
 			(effects
@@
 			)
 		)
-		(property "Footprint" ""
+		(property "Footprint" "Capacitor_SMD:C_0805_2012Metric_Pad1.18x1.45mm_HandSolder"
 			(at 131.7752 41.91 0)
 			(effects
@@
 			)
 		)
-		(property "Footprint" ""
+		(property "Footprint" "Capacitor_SMD:C_0603_1608Metric_Pad1.08x0.95mm_HandSolder"
 			(at 121.6152 41.91 0)
 			(effects
@@
 			)
 		)
-		(property "Footprint" ""
+		(property "Footprint" "Capacitor_SMD:C_0603_1608Metric_Pad1.08x0.95mm_HandSolder"
 			(at 41.6052 40.64 0)
 			(effects
@@
 			)
 		)
-		(property "Footprint" ""
+		(property "Footprint" "Diode_SMD:D_SOD-323_HandSoldering"
 			(at 57.15 36.83 0)
 			(effects

Commit message: address some stuff
Parts:
- C2, C23: Mouser Part Number 581-22201C106KAT2A -> (none)
- C25: Mouser Part Number 80-C0805C104M5R -> (none)
- D10: footprint Diode_SMD:D_SOD-923 -> Diode_SMD:D_SOD-123F; P/N ESD9101P2T5G -> SMF3.3
- R12: Mouser Part Number 71-CRCW0805100KFKEAC -> (none)
- R15, R23, R27: Mouser Part Number 71-CRCW080510K0FKEAC -> (none)
- U7: Manufacturer_Name Texas Instruments -> (none); Mouser Part Number 595-LM76202QPWPRQ1 -> (none)
Changed lines of the file:
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@@
 			)
 		)
-		(property "Footprint" "Diode_SMD:D_SOD-923"
+		(property "Footprint" "Diode_SMD:D_SOD-123F"
 			(at 158.75 36.83 0)
 			(effects
@@
 			)
 		)
-		(property "Datasheet" "https://www.onsemi.com/pdf/datasheet/esd9101-d.pdf"
+		(property "Datasheet" "https://www.littelfuse.com/assetdocs/tvs-diodes-smf3?assetguid=2e80cd26-b0c3-442f-9d77-27a283ccff4f"
 			(at 158.75 36.83 0)
 			(effects
@@
 			)
 		)
-		(property "P/N" "ESD9101P2T5G"
+		(property "P/N" "SMF3.3"
 			(at 158.75 36.83 90)
 			(effects
@@
 			)
 		)
-		(property "Mouser Part Number" "80-C0805C104M5R"
-			(at 106.68 46.99 0)
-			(effects
-				(font
-					(size 1.27 1.27)
-				)
-				(hide yes)
-			)
-		)
 		(property "P/N" "MLASH168SB7104KTNA01"
 			(at 106.68 46.99 0)
@@
 			)
 		)
-		(property "Mouser Part Number" ""
-			(at 29.21 36.83 0)
-			(effects
-				(font
-					(size 1.27 1.27)
-				)
-				(hide yes)
-			)
-		)
 		(pin "1"
 		)
@@
 			)
 		)
-		(property "Mouser Part Number" "71-CRCW080510K0FKEAC"
-			(at 21.59 123.19 0)
-			(effects
-				(font
-					(size 1.27 1.27)
-				)
-				(hide yes)
-			)
-		)
 		(property "P/N" "CRCW06032K10FKEA "
 			(at 21.59 123.19 0)
@@
 			)
 		)
-		(property "Mouser Part Number" "581-22201C106KAT2A"
-			(at 130.81 38.1 0)
-			(effects
-				(font
-					(size 1.27 1.27)
-				)
-				(hide yes)
-			)
-		)
 		(pin "1"
 		)
@@
 		)
 		(property "Description" "Resistor"
-			(at 146.05 88.9 0)
-			(effects
-				(font
-					(size 1.27 1.27)
-				)
-				(hide yes)
-			)
-		)
-		(property "Mouser Part Number" ""
 			(at 146.05 88.9 0)
 			(effects
@@
 			)
 		)
-		(property "Mouser Part Number" "71-CRCW080510K0FKEAC"
-			(at 157.48 88.9 0)
-			(effects
-				(font
-					(size 1.27 1.27)
-				)
-				(hide yes)
-			)
-		)
 		(property "P/N" "CRCW060310K0FKEI "
 			(at 157.48 88.9 0)
@@
 			)
 		)
-		(property "Mouser Part Number" "581-22201C106KAT2A"
-			(at 120.65 38.1 0)
-			(effects
-				(font
-					(size 1.27 1.27)
-				)
-				(hide yes)
-			)
-		)
 		(pin "1"
 		)
@@
 		)
 		(property "P/N" "MLASU168SB5105KTNA01"
-			(at 40.64 36.83 0)
-			(effects
-				(font
-					(size 1.27 1.27)
-				)
-				(hide yes)
-			)
-		)
-		(property "Mouser Part Number" ""
 			(at 40.64 36.83 0)
 			(effects
@@
 			)
 		)
-		(property "Mouser Part Number" "71-CRCW080510K0FKEAC"
-			(at 36.83 68.58 0)
-			(effects
-				(font
-					(size 1.27 1.27)
-				)
-				(hide yes)
-			)
-		)
 		(property "P/N" "CRCW060310K0FKEI "
 			(at 36.83 68.58 0)
@@
 		(property "P/N" "SD24C-01FTG"
 			(at 52.07 36.83 90)
-			(effects
-				(font
-					(size 1.27 1.27)
-				)
-				(hide yes)
-			)
-		)
-		(property "Mouser Part Number" ""
-			(at 52.07 36.83 0)
 			(effects
 				(font
@@
 			)
 		)
-		(property "Mouser Part Number" "595-LM76202QPWPRQ1"
-			(at 93.98 526.67 0)
-			(effects
-				(font
-					(size 1.27 1.27)
-				)
-				(justify left top)
-				(hide yes)
-			)
-		)
-		(property "Manufacturer_Name" "Texas Instruments"
-			(at 93.98 726.67 0)
-			(effects
-				(font
-					(size 1.27 1.27)
-				)
-				(justify left top)
-				(hide yes)
-			)
-		)
 		(pin "12"
 		)
@@
 			(at 21.59 102.87 0)
 			(effects
-				(font
-					(size 1.27 1.27)
-				)
-				(hide yes)
-			)
-		)
-		(property "Mouser Part Number" "71-CRCW0805100KFKEAC"
-			(at 21.59 102.87 0)
-			(effects

Commit message: Rev B Fixes + PCBA (#23)
* add or gate for boot

* 2 unrouted

* holy chopped 🥀

* bom changes

* add solder jumper for 3v3

* new prod files
Parts:
- R30: value 24m -> 19k; P/N WFCP0603R0240FE66 -> CRCW060320K0FKEA
Other:
- note added: "Typical gain: 78.28 uA/A Vout @ 1.5A = 2.231v R(imon) = 19 kΩ"
- note removed: "Typical gain: 78.28 uA/A Vout @ 1.3A = 2.407v R(imon) = 23.7 mΩ"
Changed lines of the file:
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@@
 		)
 	)
-	(text "Typical gain: 78.28 uA/A\nVout @ 1.3A = 2.407v\nR(imon) = 23.7 mΩ"
+	(text "Typical gain: 78.28 uA/A\nVout @ 1.5A = 2.231v\nR(imon) = 19 kΩ"
 		(exclude_from_sim no)
 		(at 179.324 35.814 0)
@@
 			)
 		)
-		(property "Value" "24m"
+		(property "Value" "19k"
 			(at 144.78 38.0999 0)
 			(effects
@@
 			)
 		)
-		(property "P/N" "WFCP0603R0240FE66"
+		(property "P/N" "CRCW060320K0FKEA"
 			(at 142.24 36.83 0)
 			(effects
