File: PeripheralSOM.kicad_sch (KiCad schematic)
At the start: 7 parts, among them J4 52465-2470

Commit message: initial PP changes
Parts:
- removed LOGO2: UTSVT Logo, symbol utsvt-misc:Logo_Placeholder
Connections:
- net GNDPWR is gone; now on net GND: J4.24
- net +3.3V: no longer J4.9
- net 12V_Ext renamed 24V_Ext
- net CAN_H: no longer names the net of J4.23
- net CAN_L: no longer names the net of J4.21
- net I2C1_SCL: no longer names the net of J4.14
- net I2C1_SDA: no longer names the net of J4.16
- net I2C2_SCL: no longer names the net of J4.8
- net I2C2_SDA: no longer names the net of J4.6
- net PA1: no longer names the net of J4.20
- net PA2: no longer names the net of J4.18
- net SPI1_MISO: no longer names the net of J4.15
- net SPI1_MOSI: no longer names the net of J4.17
- net SPI1_NSS: no longer names the net of J4.19
- net SPI1_SCK: no longer names the net of J4.13
- net SPI2_MISO: no longer names the net of J4.3
- net SPI2_MOSI: no longer names the net of J4.1
- net SPI2_NSS: no longer names the net of J4.7
- net SPI2_SCK: no longer names the net of J4.5
Other:
- sheet Switches and LEDs renamed LEDs
- sheet LEDs ports: added none; removed SW_PUSH
- note added: "DONT CHANGE PWR/GND recheck pinout with prev"

Commit message: completed PP
Parts:
- MH1, MH2, MH3, MH4: value M.3 -> M3
Changed lines of the file:
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@@
 			)
 		)
-		(property "Value" "M.3"
+		(property "Value" "M3"
 			(at 190.5 90.678 0)
 			(effects
@@
 			)
 		)
-		(property "Value" "M.3"
+		(property "Value" "M3"
 			(at 180.34 90.678 0)
 			(effects
@@
 			)
 		)
-		(property "Value" "M.3"
+		(property "Value" "M3"
 			(at 190.5 98.933 0)
 			(effects
@@
 			)
 		)
-		(property "Value" "M.3"
+		(property "Value" "M3"
 			(at 180.34 98.933 0)
 			(effects

Commit message: kinda add buck
Other:
- note added: "Todo: - Finish microcontroller breakouts - Double check pins for UART and CAN bootloader - Swap out buck converter for 25 - 5V converter - Spec LDO for a little bit higher currnet - Swap out Micro USB for USB-C - Swap out FTDI chip for Sci Labs chip - Get rid of push button - Change all testpoints to pad testpoints - Swap out 2 extra ADC pins for the better ones - Remove isolation - Swap out CAN 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"
- note removed: "Todo: - Finish microcontroller breakouts - Double check pins for UART and CAN bootloader - Need to change pp values to be 24V - Swap out buck converter for 25 - 5V converter - Spec LDO for a little bit higher currnet - Swap out Micro USB for USB-C - Swap out FTDI chip for Sci Labs chip - Get rid of push button - Change all testpoints to pad testpoints - Swap out 2 extra ADC pins for the better on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"
Changed lines of the file:
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@@
 		)
 	)
-	(text "Todo:\n- Finish microcontroller breakouts\n- Double check pins for UART and CAN bootloader\n- Need to change pp values to be 24V\n- Swap out buck converter for 25 - 5V converter\n- Spec LDO for a little bit higher currnet\n- Swap out Micro USB for USB-C\n- Swap out FTDI chip for Sci Labs chip\n- Get rid of push button\n- Change all testpoints to pad testpoints\n- Swap out 2 extra ADC pins for the better ones\n- Remove isolation\n- Swap out CAN chip for TCAN (noniso)\n- CubeMX to try and get the internal STM32 PGA (programmable gain amplifier)\n- Add new logo footprint\nDone:"
+	(text "Todo:\n- Finish microcontroller breakouts\n- Double check pins for UART and CAN bootloader\n- Swap out buck converter for 25 - 5V converter\n- Spec LDO for a little bit higher currnet\n- Swap out Micro USB for USB-C\n- Swap out FTDI chip for Sci Labs chip\n- Get rid of push button\n- Change all testpoints to pad testpoints\n- Swap out 2 extra ADC pins for the better ones\n- Remove isolation\n- Swap out CAN chip for TCAN (noniso)\n- CubeMX to try and get the internal STM32 PGA (programmable gain amplifier)\n- Add new logo footprint\nDone:\n- Need to change pp values to be 24V"
 		(exclude_from_sim no)
 		(at 69.088 79.248 0)

Commit message: finish buck sch
Parts:
- J4: Height 3.55 -> (none); Mouser Price/Stock https://www.mouser.co.uk/ProductDetail/Molex/52465-2470?qs=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 -> (none)
Changed lines of the file:
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@@
-			)
-		)
-		(property "PN" ""
-			(at 187.96 89.535 0)
-			(effects
-				(font
-					(size 1.27 1.27)
-				)
-				(hide yes)
-			)
-		)
-		(property "p/n" ""
-			(at 187.96 89.535 0)
-			(effects
-				(font
-					(size 1.27 1.27)
-				)
-				(hide yes)
 			)
 		)
@@
 			)
 		)
-		(property "Height" "3.55"
-			(at 168.91 435.56 0)
-			(effects
-				(font
-					(size 1.27 1.27)
-				)
-				(justify left top)
-				(hide yes)
-			)
-		)
 		(property "Mouser Part Number" "538-52465-2470"
 			(at 168.91 535.56 0)
@@
 			)
 		)
-		(property "Mouser Price/Stock" "https://www.mouser.co.uk/ProductDetail/Molex/52465-2470?qs=sEN%2FkO1EG6Yhu4DkZwbE7Q%3D%3D"
-			(at 168.91 635.56 0)
-			(effects
-				(font
-					(size 1.27 1.27)
-				)
-				(justify left top)
-				(hide yes)
-			)
-		)
 		(property "Manufacturer_Name" "Molex"
 			(at 168.91 735.56 0)
@@
 				)
 				(justify left top)
-				(hide yes)
-			)
-		)
-		(property "PN" ""
-			(at 149.86 40.64 0)
-			(effects
-				(font
-					(size 1.27 1.27)
-				)
-				(hide yes)
-			)
-		)
-		(property "p/n" ""
-			(at 149.86 40.64 0)
-			(effects
-				(font
-					(size 1.27 1.27)
-				)
 				(hide yes)
 			)
@@
 			)
 		)
-		(property "PN" ""
-			(at 157.48 89.535 0)
-			(effects
-				(font
-					(size 1.27 1.27)
-				)
-				(hide yes)
-			)
-		)
-		(property "p/n" ""
-			(at 157.48 89.535 0)
-			(effects
-				(font
-					(size 1.27 1.27)
-				)
-				(hide yes)
-			)
-		)
 		(instances
 			(project "BPS-Leader"
@@
 			)
 		)
-		(property "PN" ""
-			(at 177.8 89.535 0)
-			(effects
-				(font
-					(size 1.27 1.27)
-				)
-				(hide yes)
-			)
-		)
-		(property "p/n" ""
-			(at 177.8 89.535 0)
-			(effects
-				(font
-					(size 1.27 1.27)
-				)
-				(hide yes)
-			)
-		)
 		(instances
 			(project "BPS-Leader"
@@
 			)
 		)
-		(property "PN" ""
-			(at 187.96 97.79 0)
-			(effects
-				(font
-					(size 1.27 1.27)
-				)
-				(hide yes)
-			)
-		)
-		(property "p/n" ""
-			(at 187.96 97.79 0)
-			(effects
-				(font
-					(size 1.27 1.27)
-				)
-				(hide yes)
-			)
-		)
 		(instances
 			(project "BPS-PeripheralSOM"
@@
 			(at 177.8 97.79 0)
 			(effects
-				(font
-					(size 1.27 1.27)
-				)
-				(hide yes)
-			)
-		)
-		(property "PN" ""
-			(at 177.8 97.79 0)
-			(effects
-				(font
-					(size 1.27 1.27)
-				)
-				(hide yes)
-			)
-		)
-		(property "p/n" ""
-			(at 177.8 97.79 0)
-			(effects

Commit message: add LDO
Other:
- note added: "Todo: - Finish microcontroller breakouts - Double check pins for UART and CAN bootloader - Swap out Micro USB for USB-C - Swap out FTDI chip for Sci Labs chip - Get rid of push button - Change all testpoints to pad testpoints - Swap out 2 extra ADC pins for the better ones - Remove isolation - Swap out CAN chip for TCAN (noniso) - CubeMX to try and get the internal STM32 PGA (programmable gain am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"
- note removed: "Todo: - Finish microcontroller breakouts - Double check pins for UART and CAN bootloader - Swap out buck converter for 25 - 5V converter - Spec LDO for a little bit higher currnet - Swap out Micro USB for USB-C - Swap out FTDI chip for Sci Labs chip - Get rid of push button - Change all testpoints to pad testpoints - Swap out 2 extra ADC pins for the better ones - Remove isolation - Swap out CAN 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"
Changed lines of the file:
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@@
 		)
 	)
-	(text "Todo:\n- Finish microcontroller breakouts\n- Double check pins for UART and CAN bootloader\n- Swap out buck converter for 25 - 5V converter\n- Spec LDO for a little bit higher currnet\n- Swap out Micro USB for USB-C\n- Swap out FTDI chip for Sci Labs chip\n- Get rid of push button\n- Change all testpoints to pad testpoints\n- Swap out 2 extra ADC pins for the better ones\n- Remove isolation\n- Swap out CAN chip for TCAN (noniso)\n- CubeMX to try and get the internal STM32 PGA (programmable gain amplifier)\n- Add new logo footprint\nDone:\n- Need to change pp values to be 24V"
+	(text "Todo:\n- Finish microcontroller breakouts\n- Double check pins for UART and CAN bootloader\n- Swap out Micro USB for USB-C\n- Swap out FTDI chip for Sci Labs chip\n- Get rid of push button\n- Change all testpoints to pad testpoints\n- Swap out 2 extra ADC pins for the better ones\n- Remove isolation\n- Swap out CAN chip for TCAN (noniso)\n- CubeMX to try and get the internal STM32 PGA (programmable gain amplifier)\n- Add new logo footprint\nDone:\n- Need to change pp values to be 24V\n- Swap out buck converter for 25 - 5V converter\n- Spec LDO for a little bit higher current"
 		(exclude_from_sim no)
 		(at 69.088 79.248 0)

Commit message: lower OVP
Other:
- note added: "Todo: - Finish microcontroller breakouts - Double check pins for UART and CAN bootloader - Swap out Micro USB for USB-C - Swap out FTDI chip for Sci Labs chip - Change all testpoints to pad testpoints - Swap out 2 extra ADC pins for the better ones - Swap out CAN chip for TCAN (noniso) - CubeMX to try and get the internal STM32 PGA (programmable gain amplifier) - Add new logo footprint (KiCAD-Bil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"
- note removed: "Todo: - Finish microcontroller breakouts - Double check pins for UART and CAN bootloader - Swap out Micro USB for USB-C - Swap out FTDI chip for Sci Labs chip - Get rid of push button - Change all testpoints to pad testpoints - Swap out 2 extra ADC pins for the better ones - Remove isolation - Swap out CAN chip for TCAN (noniso) - CubeMX to try and get the internal STM32 PGA (programmable gain am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"
Changed lines of the file:
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@@
 		)
 	)
-	(text "Todo:\n- Finish microcontroller breakouts\n- Double check pins for UART and CAN bootloader\n- Swap out Micro USB for USB-C\n- Swap out FTDI chip for Sci Labs chip\n- Get rid of push button\n- Change all testpoints to pad testpoints\n- Swap out 2 extra ADC pins for the better ones\n- Remove isolation\n- Swap out CAN chip for TCAN (noniso)\n- CubeMX to try and get the internal STM32 PGA (programmable gain amplifier)\n- Add new logo footprint\nDone:\n- Need to change pp values to be 24V\n- Swap out buck converter for 25 - 5V converter\n- Spec LDO for a little bit higher current"
+	(text "Todo:\n- Finish microcontroller breakouts\n- Double check pins for UART and CAN bootloader\n- Swap out Micro USB for USB-C\n- Swap out FTDI chip for Sci Labs chip\n- Change all testpoints to pad testpoints\n- Swap out 2 extra ADC pins for the better ones\n- Swap out CAN chip for TCAN (noniso)\n- CubeMX to try and get the internal STM32 PGA (programmable gain amplifier)\n- Add new logo footprint (KiCAD-Bild)\nDone:\n- Need to change pp values to be 24V\n- Swap out buck converter for 25 - 5V converter\n- Spec LDO for a little bit higher current\n- Get rid of push button\n- Remove isolation\n"
 		(exclude_from_sim no)
 		(at 69.088 79.248 0)

Commit message: add CAN
Other:
- sheet CAN ports: added CAN_H, CAN_L, CAN_RX, CAN_TX; removed none
Changed lines of the file:
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@@
+			)
+		)
+		(pin "CAN_H" bidirectional
+			(at 53.34 41.91 0)
+			(effects
+				(font
+					(size 1.27 1.27)
+				)
+				(justify right)
+			)
+		)
+		(pin "CAN_L" bidirectional
+			(at 53.34 44.45 0)
+			(effects
+				(font
+					(size 1.27 1.27)
+				)
+				(justify right)
+			)
+		)
+		(pin "CAN_RX" output
+			(at 53.34 50.8 0)
+			(effects
+				(font
+					(size 1.27 1.27)
+				)
+				(justify right)
+			)
+		)
+		(pin "CAN_TX" input
+			(at 53.34 48.26 0)
+			(effects
+				(font
+					(size 1.27 1.27)
+				)
+				(justify right)
 			)
 		)

Commit message: add 5v power mux
Other:
- note added: "Todo: - Finish microcontroller breakouts - Double check pins for UART and CAN bootloader - Swap out Micro USB for USB-C - Swap out FTDI chip for Sci Labs chip - Change all testpoints to pad testpoints - Swap out 2 extra ADC pins for the better ones - CubeMX to try and get the internal STM32 PGA (programmable gain amplifier) - Add new logo footprint (KiCAD-Bild) Done: - Need to change pp values to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"
- note removed: "Todo: - Finish microcontroller breakouts - Double check pins for UART and CAN bootloader - Swap out Micro USB for USB-C - Swap out FTDI chip for Sci Labs chip - Change all testpoints to pad testpoints - Swap out 2 extra ADC pins for the better ones - Swap out CAN chip for TCAN (noniso) - CubeMX to try and get the internal STM32 PGA (programmable gain amplifier) - Add new logo footprint (KiCAD-Bil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"
Changed lines of the file:
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@@
 		)
 	)
-	(text "Todo:\n- Finish microcontroller breakouts\n- Double check pins for UART and CAN bootloader\n- Swap out Micro USB for USB-C\n- Swap out FTDI chip for Sci Labs chip\n- Change all testpoints to pad testpoints\n- Swap out 2 extra ADC pins for the better ones\n- Swap out CAN chip for TCAN (noniso)\n- CubeMX to try and get the internal STM32 PGA (programmable gain amplifier)\n- Add new logo footprint (KiCAD-Bild)\nDone:\n- Need to change pp values to be 24V\n- Swap out buck converter for 25 - 5V converter\n- Spec LDO for a little bit higher current\n- Get rid of push button\n- Remove isolation\n"
+	(text "Todo:\n- Finish microcontroller breakouts\n- Double check pins for UART and CAN bootloader\n- Swap out Micro USB for USB-C\n- Swap out FTDI chip for Sci Labs chip\n- Change all testpoints to pad testpoints\n- Swap out 2 extra ADC pins for the better ones\n- CubeMX to try and get the internal STM32 PGA (programmable gain amplifier)\n- Add new logo footprint (KiCAD-Bild)\nDone:\n- Need to change pp values to be 24V\n- Swap out buck converter for 25 - 5V converter\n- Spec LDO for a little bit higher current\n- Get rid of push button\n- Remove isolation\n- Swap out CAN chip for TCAN (noniso)\n- Add 5v power mux"
 		(exclude_from_sim no)
 		(at 69.088 79.248 0)
