File: PeripheralSOM.kicad_sch (KiCad schematic)
At the start: 6 parts, among them J4 52465-2470

Commit message: add USB
Connections:
- net 24V_Ext renamed +24V_EXT
Other:
- sheet USB ports: added UART_RX, UART_TX; removed none
- note added: "Todo: - Finish microcontroller breakouts - Double check pins for UART and CAN bootloader - Change all testpoints to pad testpoints - Swap out 2 extra ADC pins for the better ones - CubeMX to try and get the internal STM32 PGA (programmable gain amplifier) - Add new logo footprint (KiCAD-Bild) Done: - Need to change pp values to be 24V - Swap out buck converter for 25 - 5V converter - Spec LDO for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"
- note removed: "Todo: - Finish microcontroller breakouts - Double check pins for UART and CAN bootloader - Swap out Micro USB for USB-C - Swap out FTDI chip for Sci Labs chip - Change all testpoints to pad testpoints - Swap out 2 extra ADC pins for the better ones - CubeMX to try and get the internal STM32 PGA (programmable gain amplifier) - Add new logo footprint (KiCAD-Bild) Done: - Need to change pp values to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"
Changed lines of the file:
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@@
 		)
 	)
-	(text "Todo:\n- Finish microcontroller breakouts\n- Double check pins for UART and CAN bootloader\n- Swap out Micro USB for USB-C\n- Swap out FTDI chip for Sci Labs chip\n- Change all testpoints to pad testpoints\n- Swap out 2 extra ADC pins for the better ones\n- CubeMX to try and get the internal STM32 PGA (programmable gain amplifier)\n- Add new logo footprint (KiCAD-Bild)\nDone:\n- Need to change pp values to be 24V\n- Swap out buck converter for 25 - 5V converter\n- Spec LDO for a little bit higher current\n- Get rid of push button\n- Remove isolation\n- Swap out CAN chip for TCAN (noniso)\n- Add 5v power mux"
+	(text "Todo:\n- Finish microcontroller breakouts\n- Double check pins for UART and CAN bootloader\n- Change all testpoints to pad testpoints\n- Swap out 2 extra ADC pins for the better ones\n- CubeMX to try and get the internal STM32 PGA (programmable gain amplifier)\n- Add new logo footprint (KiCAD-Bild)\nDone:\n- Need to change pp values to be 24V\n- Swap out buck converter for 25 - 5V converter\n- Spec LDO for a little bit higher current\n- Get rid of push button\n- Remove isolation\n- Swap out CAN chip for TCAN (noniso)\n- Add 5v power mux\n- Swap out Micro USB for USB-C\n- Swap out FTDI chip for Sci Labs chip"
 		(exclude_from_sim no)
 		(at 69.088 79.248 0)
@@
 	(wire
 		(pts
-			(xy 172.72 43.18) (xy 181.61 43.18)
+			(xy 172.72 43.18) (xy 180.34 43.18)
 		)
 		(stroke
@@
 		)
 	)
-	(label "24V_Ext"
-		(at 181.61 43.18 180)
-		(effects
-			(font
-				(size 1.27 1.27)
-			)
-			(justify right bottom)
-		)
-	)
 	(label "PA0"
 		(at 59.69 80.01 0)
@@
 		)
 		(property "Value" "GND"
-			(at 189.8142 40.513 0)
+			(at 190.754 40.64 90)
 			(effects
 				(font
@@
 		)
 		(property "Value" "VDDA"
-			(at 191.77 58.42 0)
+			(at 193.548 58.42 90)
 			(effects
 				(font
@@
 		)
 		(property "Value" "GND"
-			(at 145.4658 56.007 0)
+			(at 144.526 55.88 90)
 			(effects
 				(font
@@
 		)
 		(property "Value" "GND"
-			(at 182.1942 65.913 0)
+			(at 183.134 66.04 90)
 			(effects
 				(font
@@
 				(path "/d5ebd247-5a7c-47c2-8aee-beabaef72d6d"
 					(reference "#PWR067")
+					(unit 1)
+				)
+			)
+		)
+	)
+	(symbol
+		(lib_id "power:+3.3V")
+		(at 180.34 43.18 270)
+		(unit 1)
+		(exclude_from_sim no)
+		(in_bom yes)
+		(on_board yes)
+		(dnp no)
+		(property "Reference" "#PWR052"
+			(at 176.53 43.18 0)
+			(effects
+				(font
+					(size 1.27 1.27)
+				)
+				(hide yes)
+			)
+		)
+		(property "Value" "+24V_EXT"
+			(at 183.388 43.18 90)
+			(effects
+				(font
+					(size 1.27 1.27)
+				)
+				(justify left)
+			)
+		)
+		(property "Footprint" ""
+			(at 180.34 43.18 0)
+			(effects
+				(font
+					(size 1.27 1.27)
+				)
+				(hide yes)
+			)
+		)
+		(property "Datasheet" ""
+			(at 180.34 43.18 0)
+			(effects
+				(font
+					(size 1.27 1.27)
+				)
+				(hide yes)
+			)
+		)
+		(property "Description" "Power symbol creates a global label with name \"+3.3V\""
+			(at 180.34 43.18 0)
+			(effects
+				(font
+					(size 1.27 1.27)
+				)
+				(hide yes)
+			)
+		)
+		(pin "1"
+		)
+		(instances
+			(project "PeripheralSOM"
+				(path "/d5ebd247-5a7c-47c2-8aee-beabaef72d6d"
+					(reference "#PWR052")
 					(unit 1)
 				)
@@
 		)
 		(property "Value" "GNDA"
-			(at 187.325 55.88 0)
+			(at 188.468 55.88 90)
 			(effects
 				(font
@@
 	(sheet
 		(at 13.97 60.325)
-		(size 39.37 6.985)
+		(size 39.37 8.255)
 		(exclude_from_sim no)
 		(in_bom yes)
@@
 		)
 		(property "Sheetfile" "USB.kicad_sch"
-			(at 13.97 67.8946 0)
+			(at 13.97 69.1646 0)
 			(effects
 				(font
@@
 			)
 		)
+		(pin "UART_RX" input
+			(at 53.34 63.5 0)
+			(effects
+				(font
+					(size 1.27 1.27)
+				)
+				(justify right)
+			)
+		)
+		(pin "UART_TX" output
+			(at 53.34 66.04 0)
+			(effects
+				(font
+					(size 1.27 1.27)
+				)
+				(justify right)
+			)
+		)

Commit message: stuf
Other:
- note added: "Todo: - Finish microcontroller breakouts - Check over and redo MCU pins - Double check pins for UART and CAN bootloader - Swap out 2 extra ADC pins for the better ones - CubeMX to try and get the internal STM32 PGA (programmable gain amplifier) - Add new logo footprint (KiCAD-Bild) - Part & Footprint selection Done: - Need to change pp values to be 24V - Swap out buck converter for 25 - 5V conver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"
- note removed: "Todo: - Finish microcontroller breakouts - Double check pins for UART and CAN bootloader - Change all testpoints to pad testpoints - Swap out 2 extra ADC pins for the better ones - CubeMX to try and get the internal STM32 PGA (programmable gain amplifier) - Add new logo footprint (KiCAD-Bild) Done: - Need to change pp values to be 24V - Swap out buck converter for 25 - 5V converter - Spec LDO for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"
Changed lines of the file:
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@@
 		)
 	)
-	(text "Todo:\n- Finish microcontroller breakouts\n- Double check pins for UART and CAN bootloader\n- Change all testpoints to pad testpoints\n- Swap out 2 extra ADC pins for the better ones\n- CubeMX to try and get the internal STM32 PGA (programmable gain amplifier)\n- Add new logo footprint (KiCAD-Bild)\nDone:\n- Need to change pp values to be 24V\n- Swap out buck converter for 25 - 5V converter\n- Spec LDO for a little bit higher current\n- Get rid of push button\n- Remove isolation\n- Swap out CAN chip for TCAN (noniso)\n- Add 5v power mux\n- Swap out Micro USB for USB-C\n- Swap out FTDI chip for Sci Labs chip"
+	(text "Todo:\n- Finish microcontroller breakouts\n- Check over and redo MCU pins\n- Double check pins for UART and CAN bootloader\n- Swap out 2 extra ADC pins for the better ones\n- CubeMX to try and get the internal STM32 PGA (programmable gain amplifier)\n- Add new logo footprint (KiCAD-Bild)\n- Part & Footprint selection\nDone:\n- Need to change pp values to be 24V\n- Swap out buck converter for 25 - 5V converter\n- Spec LDO for a little bit higher current\n- Get rid of push button\n- Remove isolation\n- Swap out CAN chip for TCAN (noniso)\n- Add 5v power mux\n- Swap out Micro USB for USB-C\n- Swap out FTDI chip for Sci Labs chip\n- Change all testpoints to pad testpoints\n"
 		(exclude_from_sim no)
 		(at 69.088 79.248 0)
@@
 			(font
 				(size 2.54 2.54)
-				(thickness 0.508)
-				(bold yes)
+				(thickness 0.3175)
 			)
 			(justify left bottom)

Commit message: control but micro
Other:
- sheet MCU ports: added USART1; removed SPI1, UART1
- note added: "Todo: - Check over and redo MCU pins - Add new logo footprint (KiCAD-Bild) - Part & Footprint selection Done: - Need to change pp values to be 24V - Swap out buck converter for 25 - 5V converter - Spec LDO for a little bit higher current - Get rid of push button - Remove isolation - Swap out CAN chip for TCAN (noniso) - Add 5v power mux - Swap out Micro USB for USB-C - Swap out FTDI chip for Sci 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"
- note removed: "Todo: - Finish microcontroller breakouts - Check over and redo MCU pins - Double check pins for UART and CAN bootloader - Swap out 2 extra ADC pins for the better ones - CubeMX to try and get the internal STM32 PGA (programmable gain amplifier) - Add new logo footprint (KiCAD-Bild) - Part & Footprint selection Done: - Need to change pp values to be 24V - Swap out buck converter for 25 - 5V conver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"
Changed lines of the file:
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@@
 		)
 	)
-	(text "Todo:\n- Finish microcontroller breakouts\n- Check over and redo MCU pins\n- Double check pins for UART and CAN bootloader\n- Swap out 2 extra ADC pins for the better ones\n- CubeMX to try and get the internal STM32 PGA (programmable gain amplifier)\n- Add new logo footprint (KiCAD-Bild)\n- Part & Footprint selection\nDone:\n- Need to change pp values to be 24V\n- Swap out buck converter for 25 - 5V converter\n- Spec LDO for a little bit higher current\n- Get rid of push button\n- Remove isolation\n- Swap out CAN chip for TCAN (noniso)\n- Add 5v power mux\n- Swap out Micro USB for USB-C\n- Swap out FTDI chip for Sci Labs chip\n- Change all testpoints to pad testpoints\n"
+	(text "Todo:\n- Check over and redo MCU pins\n- Add new logo footprint (KiCAD-Bild)\n- Part & Footprint selection\nDone:\n- Need to change pp values to be 24V\n- Swap out buck converter for 25 - 5V converter\n- Spec LDO for a little bit higher current\n- Get rid of push button\n- Remove isolation\n- Swap out CAN chip for TCAN (noniso)\n- Add 5v power mux\n- Swap out Micro USB for USB-C\n- Swap out FTDI chip for Sci Labs chip\n- Change all testpoints to pad testpoints\n- Double check pins for UART and CAN bootloader\n- Swap out 2 extra ADC pins for the better ones\n- CubeMX to try and get the internal STM32 PGA (programmable gain amplifier)"
 		(exclude_from_sim no)
 		(at 69.088 79.248 0)
@@
 		)
 	)
-	(bus
+	(wire
 		(pts
-			(xy 53.34 77.47) (xy 66.04 77.47)
+			(xy 172.72 55.88) (xy 182.88 55.88)
 		)
 		(stroke
@@
 		)
 	)
-	(wire
+	(bus
 		(pts
-			(xy 172.72 55.88) (xy 182.88 55.88)
+			(xy 118.11 25.4) (xy 128.27 25.4)
 		)
 		(stroke
@@
 	(wire
 		(pts
-			(xy 59.69 80.01) (xy 53.34 80.01)
+			(xy 172.72 58.42) (xy 187.96 58.42)
 		)
 		(stroke
@@
 	(wire
 		(pts
-			(xy 172.72 58.42) (xy 187.96 58.42)
+			(xy 172.72 68.58) (xy 179.07 68.58)
 		)
 		(stroke
@@
 	(wire
 		(pts
-			(xy 172.72 68.58) (xy 179.07 68.58)
+			(xy 172.72 66.04) (xy 177.8 66.04)
 		)
 		(stroke
@@
 		)
 	)
-	(wire
-		(pts
-			(xy 172.72 66.04) (xy 177.8 66.04)
-		)
-		(stroke
-			(width 0)
-			(type default)
-		)
-	)
-	(label "PB[3..5]"
-		(at 66.04 77.47 180)
+	(label "{USART1}"
+		(at 128.27 25.4 180)
 		(effects
 			(font
@@
 			)
 			(justify right bottom)
-		)
-	)
-	(label "PA0"
-		(at 59.69 80.01 0)
-		(effects
-			(font
-				(size 1.27 1.27)
-			)
-			(justify left bottom)
 		)
 	)
@@
 	(sheet
 		(at 13.97 39.37)
-		(size 39.37 13.97)
+		(size 21.59 13.97)
 		(exclude_from_sim no)
 		(in_bom yes)
@@
 		)
 		(property "Sheetfile" "CAN.kicad_sch"
-			(at 13.97 54.5596 0)
+			(at 13.97 53.9246 0)
 			(effects
 				(font
@@
 		)
 		(pin "CAN_H" bidirectional
-			(at 53.34 41.91 0)
+			(at 35.56 41.91 0)
 			(effects
 				(font
@@
 		)
 		(pin "CAN_L" bidirectional
-			(at 53.34 44.45 0)
+			(at 35.56 44.45 0)
 			(effects
 				(font
@@
 		)
 		(pin "CAN_RX" output
-			(at 53.34 50.8 0)
+			(at 35.56 50.8 0)
 			(effects
 				(font
@@
 		)
 		(pin "CAN_TX" input
-			(at 53.34 48.26 0)
+			(at 35.56 48.26 0)
 			(effects
 				(font
@@
 	)
 	(sheet
-		(at 75.184 21.59)
-		(size 44.45 22.606)
+		(at 74.295 21.59)
+		(size 44.45 22.86)
 		(exclude_from_sim no)
 		(in_bom yes)
@@
 		)
 		(property "Sheetname" "MCU"
-			(at 75.184 20.8784 0)
+			(at 74.295 20.8784 0)
 			(effects
 				(font
@@
 		)
 		(property "Sheetfile" "STM32L431CBT6.kicad_sch"
-			(at 75.184 44.7806 0)
+			(at 74.295 44.7806 0)
 			(effects
 				(font
@@
 			)
 		)
-		(pin "UART1" bidirectional
-			(at 119.634 40.64 0)
-			(effects
-				(font
-					(size 1.27 1.27)
-				)
-				(justify right)
-			)
-		)
-		(pin "SPI1" bidirectional
-			(at 119.634 24.13 0)
+		(pin "USART1" bidirectional
+			(at 118.745 25.4 0)
 			(effects
 				(font
@@
 	(sheet
 		(at 13.97 74.93)
-		(size 39.37 10.16)
+		(size 21.59 10.16)
 		(exclude_from_sim no)
 		(in_bom yes)
@@
 		)
 		(pin "LED[1..3]" input
-			(at 53.34 77.47 0)
+			(at 35.56 77.47 0)
 			(effects
 				(font
@@
 		)
 		(pin "LED_HB" input
-			(at 53.34 80.01 0)
+			(at 35.56 80.01 0)
 			(effects
 				(font
@@
 	(sheet
 		(at 13.97 22.098)
-		(size 39.37 9.652)
+		(size 24.765 9.652)
 		(exclude_from_sim no)
 		(in_bom yes)
@@
 	(sheet
 		(at 13.97 60.325)
-		(size 39.37 8.255)
+		(size 21.59 8.255)
 		(exclude_from_sim no)
 		(in_bom yes)
@@
 		)
 		(pin "UART_RX" input
-			(at 53.34 63.5 0)
+			(at 35.56 63.5 0)
 			(effects
 				(font
@@
 		)
 		(pin "UART_TX" output
-			(at 53.34 66.04 0)
-			(effects
-				(font
+			(at 35.56 66.04 0)
+			(effects
+				(font

Commit message: finish mcu breakouts
Other:
- sheet CAN ports: added {CAN1}; removed CAN_RX, CAN_TX
- sheet MCU ports: added OPAMP1_VINP, {ADC1}, {CAN1}, {I2C1}, {SPI1}, {SPI2}, {USART1}; removed USART1
- sheet USB ports: added {USART1}; removed UART_RX, UART_TX
- note added: "Todo: - Check over and redo MCU pins - Add new logo footprint (KiCAD-Bild) - Part & Footprint selection Done: - Need to change pp values to be 24V - Swap out buck converter for 25 - 5V converter - Spec LDO for a little bit higher current - Get rid of push button - Remove isolation - Swap out CAN chip for TCAN (noniso) - Add 5v power mux - Swap out Micro USB for USB-C - Swap out FTDI chip for SiLa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"
- note removed: "Todo: - Check over and redo MCU pins - Add new logo footprint (KiCAD-Bild) - Part & Footprint selection Done: - Need to change pp values to be 24V - Swap out buck converter for 25 - 5V converter - Spec LDO for a little bit higher current - Get rid of push button - Remove isolation - Swap out CAN chip for TCAN (noniso) - Add 5v power mux - Swap out Micro USB for USB-C - Swap out FTDI chip for Sci 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"

Commit message: populate conn
Parts:
- J4: footprint (none) -> UTSVT_Connectors:524652470; symbol utsvt-connectors:52465-2470 -> utsvt_connectors:52465-2470; Height (none) -> 3.55; Mouser Price/Stock (none) -> https://www.mouser.co.uk/ProductDetail/Molex/52465-2470?qs=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
Connections:
- net ADC1_IN10: now also J4.18
- net ADC1_IN11: now also J4.20
- net ADC1_IN7: now also J4.14
- net ADC1_IN9: now also J4.16
- net I2C1_SCL: now also J4.8
- net I2C1_SDA: now also J4.6
- net OPAMP1_VINP: now also J4.9
- net SPI1_MISO: now also J4.17
- net SPI1_MOSI: now also J4.19
- net SPI1_NSS: now also J4.23
- net SPI1_SCK: now also J4.21
- net SPI2_MISO: now also J4.7
- net SPI2_MOSI: now also J4.5
- net SPI2_NSS: now also J4.1
- net SPI2_SCK: now also J4.3
- net CAN_H: now reaches J4.13
- net CAN_L: now reaches J4.15
Other:
- note added: "Todo: - Add new logo footprint (KiCAD-Bild) - Part & Footprint selection Done: - Need to change pp values to be 24V - Swap out buck converter for 25 - 5V converter - Spec LDO for a little bit higher current - Get rid of push button - Remove isolation - Swap out CAN chip for TCAN (noniso) - Add 5v power mux - Swap out Micro USB for USB-C - Swap out FTDI chip for SiLabs chip - Change all testpoints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"
- note removed: "Peripherals"
- note removed: "Todo: - Check over and redo MCU pins - Add new logo footprint (KiCAD-Bild) - Part & Footprint selection Done: - Need to change pp values to be 24V - Swap out buck converter for 25 - 5V converter - Spec LDO for a little bit higher current - Get rid of push button - Remove isolation - Swap out CAN chip for TCAN (noniso) - Add 5v power mux - Swap out Micro USB for USB-C - Swap out FTDI chip for SiLa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"
- moved on the sheet: J4

Commit message: twinkle
Other:
- sheet MCU ports: added LED[1..3], LED_HB; removed none
- note added: "Board Notes"
- note added: "Connector mates with 53307-2471 Consult README for pin usage guide *Always verify pin functions with CubeMX*"
- note added: "Ext 24v -> Protected 24v -> 5v -> 3.3v"
- note added: "Graphics/Mounting"
- note added: "Todo: - Add new logo footprint (KiCAD-Bild) - Part & Footprint selection - Add datasheet links for all Done: - Need to change pp values to be 24V - Swap out buck converter for 25 - 5V converter - Spec LDO for a little bit higher current - Get rid of push button - Remove isolation - Swap out CAN chip for TCAN (noniso) - Add 5v power mux - Swap out Micro USB for USB-C - Swap out FTDI chip for SiLab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"
- note removed: "Connector mates with 53307-2471 Please consult README for pin usage guide ** Note that the pin naming scheme is not indicative of proper usage guidelines **"
- note removed: "DONT CHANGE PWR/GND recheck pinout with prev"
- note removed: "Graphics/Logos"
- note removed: "Todo: - Add new logo footprint (KiCAD-Bild) - Part & Footprint selection Done: - Need to change pp values to be 24V - Swap out buck converter for 25 - 5V converter - Spec LDO for a little bit higher current - Get rid of push button - Remove isolation - Swap out CAN chip for TCAN (noniso) - Add 5v power mux - Swap out Micro USB for USB-C - Swap out FTDI chip for SiLabs chip - Change all testpoints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"
- company: LHRs -> Longhorn Racing Solar
- moved on the sheet: J4, MH1, MH2, MH3, MH4

Commit message: FUCK capacitors
Parts:
- added LOGO2: LHRs, UTSVT_Logos:Hallock_Image_Small, symbol utsvt_misc:Logo_Placeholder
- LOGO1: footprint (none) -> UTSVT_Logos:Hallock_Image_Small; symbol utsvt-misc:Logo_Placeholder -> utsvt_misc:Logo_Placeholder; now left out of the parts list
- MH1, MH2, MH3, MH4: now left out of the parts list
Other:
- note added: "Todo: - Part & Footprint selection - Add datasheet links for all Done: - Need to change pp values to be 24V - Swap out buck converter for 25 - 5V converter - Spec LDO for a little bit higher current - Get rid of push button - Remove isolation - Swap out CAN chip for TCAN (noniso) - Add 5v power mux - Swap out Micro USB for USB-C - Swap out FTDI chip for SiLabs chip - Change all testpoints to pad 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"
- note added: "idk figure it out"
- note removed: "Todo: - Add new logo footprint (KiCAD-Bild) - Part & Footprint selection - Add datasheet links for all Done: - Need to change pp values to be 24V - Swap out buck converter for 25 - 5V converter - Spec LDO for a little bit higher current - Get rid of push button - Remove isolation - Swap out CAN chip for TCAN (noniso) - Add 5v power mux - Swap out Micro USB for USB-C - Swap out FTDI chip for SiLab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"
Changed lines of the file:
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@@
 		)
 	)
-	(text "Todo:\n- Add new logo footprint (KiCAD-Bild)\n- Part & Footprint selection\n- Add datasheet links for all\nDone:\n- Need to change pp values to be 24V\n- Swap out buck converter for 25 - 5V converter\n- Spec LDO for a little bit higher current\n- Get rid of push button\n- Remove isolation\n- Swap out CAN chip for TCAN (noniso)\n- Add 5v power mux\n- Swap out Micro USB for USB-C\n- Swap out FTDI chip for SiLabs chip\n- Change all testpoints to pad testpoints\n- Double check pins for UART and CAN bootloader\n- Swap out 2 extra ADC pins for the better ones\n- CubeMX to try and get the internal STM32 PGA (programmable gain amplifier)\n- Check over and redo MCU pins\n"
+	(text "Todo:\n- Part & Footprint selection\n- Add datasheet links for all\nDone:\n- Need to change pp values to be 24V\n- Swap out buck converter for 25 - 5V converter\n- Spec LDO for a little bit higher current\n- Get rid of push button\n- Remove isolation\n- Swap out CAN chip for TCAN (noniso)\n- Add 5v power mux\n- Swap out Micro USB for USB-C\n- Swap out FTDI chip for SiLabs chip\n- Change all testpoints to pad testpoints\n- Double check pins for UART and CAN bootloader\n- Swap out 2 extra ADC pins for the better ones\n- CubeMX to try and get the internal STM32 PGA\n- Check over and redo MCU pins\n"
 		(exclude_from_sim no)
-		(at 222.758 146.812 0)
+		(at 14.986 114.808 0)
 		(effects
 			(font
@@
 		)
 	)
-	(text "Connector mates with 53307-2471\nConsult README for pin usage guide\n*Always verify pin functions with CubeMX*"
+	(text "idk figure it out"
 		(exclude_from_sim no)
-		(at 152.4 82.804 0)
+		(at 152.654 78.74 0)
 		(effects
 			(font
@@
 		(unit 1)
 		(exclude_from_sim no)
-		(in_bom yes)
+		(in_bom no)
 		(on_board yes)
 		(dnp no)
@@
 				(path "/d5ebd247-5a7c-47c2-8aee-beabaef72d6d"
 					(reference "#PWR013")
+					(unit 1)
+				)
+			)
+		)
+	)
+	(symbol
+		(lib_id "utsvt_misc:Logo_Placeholder")
+		(at 109.22 91.44 0)
+		(unit 1)
+		(exclude_from_sim no)
+		(in_bom no)
+		(on_board yes)
+		(dnp no)
+		(property "Reference" "LOGO2"
+			(at 109.22 87.63 0)
+			(effects
+				(font
+					(size 1.27 1.27)
+				)
+				(hide yes)
+			)
+		)
+		(property "Value" "LHRs"
+			(at 112.776 91.44 0)
+			(effects
+				(font
+					(size 1.27 1.27)
+				)
+				(justify left)
+			)
+		)
+		(property "Footprint" "UTSVT_Logos:Hallock_Image_Small"
+			(at 109.22 89.535 0)
+			(effects
+				(font
+					(size 1.27 1.27)
+				)
+				(hide yes)
+			)
+		)
+		(property "Datasheet" ""
+			(at 109.22 89.535 0)
+			(effects
+				(font
+					(size 1.27 1.27)
+				)
+				(hide yes)
+			)
+		)
+		(property "Description" "Graph footprint placeholder"
+			(at 109.22 91.44 0)
+			(effects
+				(font
+					(size 1.27 1.27)
+				)
+				(hide yes)
+			)
+		)
+		(property "PN" ""
+			(at 109.22 91.44 0)
+			(effects
+				(font
+					(size 1.27 1.27)
+				)
+				(hide yes)
+			)
+		)
+		(property "p/n" ""
+			(at 109.22 91.44 0)
+			(effects
+				(font
+					(size 1.27 1.27)
+				)
+				(hide yes)
+			)
+		)
+		(instances
+			(project "PeripheralSOM"
+				(path "/d5ebd247-5a7c-47c2-8aee-beabaef72d6d"
+					(reference "LOGO2")
 					(unit 1)
 				)
@@
 	)
 	(symbol
-		(lib_id "utsvt-misc:Logo_Placeholder")
+		(lib_id "utsvt_misc:Logo_Placeholder")
 		(at 109.22 83.185 0)
 		(unit 1)
 		(exclude_from_sim no)
-		(in_bom yes)
+		(in_bom no)
 		(on_board yes)
 		(dnp no)
@@
 			)
 		)
-		(property "Footprint" ""
+		(property "Footprint" "UTSVT_Logos:Hallock_Image_Small"
 			(at 109.22 81.28 0)
 			(effects
@@
 		)
 		(property "Description" "Graph footprint placeholder"
+			(at 109.22 83.185 0)
+			(effects
+				(font
+					(size 1.27 1.27)
+				)
+				(hide yes)
+			)
+		)
+		(property "PN" ""
+			(at 109.22 83.185 0)
+			(effects
+				(font
+					(size 1.27 1.27)
+				)
+				(hide yes)
+			)
+		)
+		(property "p/n" ""
 			(at 109.22 83.185 0)
 			(effects
@@
 		(unit 1)
 		(exclude_from_sim no)
-		(in_bom yes)
+		(in_bom no)
 		(on_board yes)
 		(dnp no)
@@
 		(unit 1)
 		(exclude_from_sim no)
-		(in_bom yes)
+		(in_bom no)
 		(on_board yes)
 		(dnp no)
@@
 		(unit 1)
 		(exclude_from_sim no)
-		(in_bom yes)
+		(in_bom no)
 		(on_board yes)
 		(dnp no)
