File: PeripheralSOM.kicad_sch (KiCad schematic)
At the start: 7 parts, among them J4 52465-2470

Commit message: all parts selected
Other:
- note added: "Todo: - Move power/gnd to diff sides of conn - Connect IMON to MCU - Part & Footprint selection - Add datasheet links for all Done: - Need to change pp values to be 24V - Swap out buck converter for 25 - 5V converter - Spec LDO for a little bit higher current - Get rid of push button - Remove isolation - Swap out CAN chip for TCAN (noniso) - Add 5v power mux - Swap out Micro USB for USB-C - Swap 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"
- note removed: "Todo: - Part & Footprint selection - Add datasheet links for all Done: - Need to change pp values to be 24V - Swap out buck converter for 25 - 5V converter - Spec LDO for a little bit higher current - Get rid of push button - Remove isolation - Swap out CAN chip for TCAN (noniso) - Add 5v power mux - Swap out Micro USB for USB-C - Swap out FTDI chip for SiLabs chip - Change all testpoints to pad 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"
Changed lines of the file:
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@@
 		)
 	)
-	(text "Todo:\n- Part & Footprint selection\n- Add datasheet links for all\nDone:\n- Need to change pp values to be 24V\n- Swap out buck converter for 25 - 5V converter\n- Spec LDO for a little bit higher current\n- Get rid of push button\n- Remove isolation\n- Swap out CAN chip for TCAN (noniso)\n- Add 5v power mux\n- Swap out Micro USB for USB-C\n- Swap out FTDI chip for SiLabs chip\n- Change all testpoints to pad testpoints\n- Double check pins for UART and CAN bootloader\n- Swap out 2 extra ADC pins for the better ones\n- CubeMX to try and get the internal STM32 PGA\n- Check over and redo MCU pins\n"
+	(text "Todo:\n- Move power/gnd to diff sides of conn\n- Connect IMON to MCU\n- Part & Footprint selection\n- Add datasheet links for all\nDone:\n- Need to change pp values to be 24V\n- Swap out buck converter for 25 - 5V converter\n- Spec LDO for a little bit higher current\n- Get rid of push button\n- Remove isolation\n- Swap out CAN chip for TCAN (noniso)\n- Add 5v power mux\n- Swap out Micro USB for USB-C\n- Swap out FTDI chip for SiLabs chip\n- Change all testpoints to pad testpoints\n- Double check pins for UART and CAN bootloader\n- Swap out 2 extra ADC pins for the better ones\n- CubeMX to try and get the internal STM32 PGA\n- Check over and redo MCU pins\n"
 		(exclude_from_sim no)
-		(at 14.986 114.808 0)
+		(at 13.208 116.586 0)
 		(effects
 			(font
@@
 		)
 		(property "Description" "Graph footprint placeholder"
-			(at 109.22 91.44 0)
-			(effects
-				(font
-					(size 1.27 1.27)
-				)
-				(hide yes)
-			)
-		)
-		(property "PN" ""
-			(at 109.22 91.44 0)
-			(effects
-				(font
-					(size 1.27 1.27)
-				)
-				(hide yes)
-			)
-		)
-		(property "p/n" ""
 			(at 109.22 91.44 0)
 			(effects
@@
 			(at 109.22 83.185 0)
 			(effects
-				(font
-					(size 1.27 1.27)
-				)
-				(hide yes)
-			)
-		)
-		(property "PN" ""
-			(at 109.22 83.185 0)
-			(effects
-				(font
-					(size 1.27 1.27)
-				)
-				(hide yes)
-			)
-		)
-		(property "p/n" ""
-			(at 109.22 83.185 0)
-			(effects
