File: PeripheralSOM.kicad_sch (KiCad schematic)
At the start: 6 parts, among them J4 52465-2470

Commit message: more basic parts
Other:
- note added: "Changelog: - Change pp values to be 24V - Swap out buck converter for 24 - 5V converter - Spec LDO for a little bit higher current - Get rid of push button - Remove isolation - Swap out CAN chip for TCAN (noniso) - Add 5v power mux - Swap out Micro USB for USB-C - Swap out FTDI chip for SiLabs chip - Change all testpoints to pad testpoints - Double check pins for UART and CAN bootloader - Swap ou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"
- note removed: "Done: - Need to change pp values to be 24V - Swap out buck converter for 25 - 5V converter - Spec LDO for a little bit higher current - Get rid of push button - Remove isolation - Swap out CAN chip for TCAN (noniso) - Add 5v power mux - Swap out Micro USB for USB-C - Swap out FTDI chip for SiLabs chip - Change all testpoints to pad testpoints - Double check pins for UART and CAN bootloader - Swap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"
Changed lines of the file:
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@@
 		)
 	)
-	(text "Done:\n- Need to change pp values to be 24V\n- Swap out buck converter for 25 - 5V converter\n- Spec LDO for a little bit higher current\n- Get rid of push button\n- Remove isolation\n- Swap out CAN chip for TCAN (noniso)\n- Add 5v power mux\n- Swap out Micro USB for USB-C\n- Swap out FTDI chip for SiLabs chip\n- Change all testpoints to pad testpoints\n- Double check pins for UART and CAN bootloader\n- Swap out 2 extra ADC pins for the better ones\n- CubeMX to try and get the internal STM32 PGA\n- Check over and redo MCU pins\n- Connect IMON to MCU\n- Move power/gnd to diff sides of conn\n- Add datasheet links for all\n- Part selection\n- Footprint selection\n"
+	(text "Changelog:\n- Change pp values to be 24V\n- Swap out buck converter for 24 - 5V converter\n- Spec LDO for a little bit higher current\n- Get rid of push button\n- Remove isolation\n- Swap out CAN chip for TCAN (noniso)\n- Add 5v power mux\n- Swap out Micro USB for USB-C\n- Swap out FTDI chip for SiLabs chip\n- Change all testpoints to pad testpoints\n- Double check pins for UART and CAN bootloader\n- Swap out 2 extra ADC pins for the better ones\n- CubeMX to try and get the internal STM32 PGA\n- Check over and redo MCU pins\n- Connect IMON to MCU\n- Move power/gnd to diff sides of conn\n- Add datasheet links for all\n- Part selection\n- Footprint selection\n"
 		(exclude_from_sim no)
 		(at 22.098 107.442 0)
