File: STM32L431CBT6.kicad_sch (KiCad schematic)
At the start: 20 parts, among them J1 SWD, SW1 Reset, U1 STM32L431CBTx, Y1 8M

Commit message: purge shit
Parts:
- C11, C12, C13, C14, C15, C16, C17, C21, C22, C7: footprint Capacitor_SMD:C_0805_2012Metric -> (none)
- CR1, CR2: footprint UTSVT_ICs:SOT26_DIO -> (none)
- FB1, FB4: footprint Inductor_SMD:L_0805_2012Metric -> (none)
- J1: footprint Connector_PinHeader_2.54mm:PinHeader_1x04_P2.54mm_Vertical -> (none)
- R19, R29: footprint Resistor_SMD:R_0805_2012Metric -> (none)
- SW1: footprint Button_Switch_SMD:SW_SPST_B3SL-1002P -> (none)
- U1: footprint Package_QFP:LQFP-48_7x7mm_P0.5mm -> (none)
- Y1: footprint Crystal:Crystal_SMD_TXC_7A-2Pin_5x3.2mm -> (none)
Changed lines of the file:
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@@
 			)
 		)
-		(property "Footprint" "UTSVT_ICs:SOT26_DIO"
+		(property "Footprint" ""
 			(at 218.44 127 0)
 			(effects
@@
 			)
 		)
-		(property "Footprint" "Capacitor_SMD:C_0805_2012Metric"
+		(property "Footprint" ""
 			(at 100.0252 186.69 0)
 			(effects
@@
 			)
 		)
-		(property "Footprint" "Capacitor_SMD:C_0805_2012Metric"
+		(property "Footprint" ""
 			(at 115.2652 151.13 0)
 			(effects
@@
 			)
 		)
-		(property "Footprint" "Button_Switch_SMD:SW_SPST_B3SL-1002P"
+		(property "Footprint" ""
 			(at 115.57 182.88 0)
 			(effects
@@
 			)
 		)
-		(property "Footprint" "Capacitor_SMD:C_0805_2012Metric"
+		(property "Footprint" ""
 			(at 79.7052 151.13 0)
 			(effects
@@
 			)
 		)
-		(property "Footprint" "Inductor_SMD:L_0805_2012Metric"
+		(property "Footprint" ""
 			(at 55.88 182.118 90)
 			(effects
@@
 			)
 		)
-		(property "Footprint" "Capacitor_SMD:C_0805_2012Metric"
+		(property "Footprint" ""
 			(at 61.9252 187.96 0)
 			(effects
@@
 			)
 		)
-		(property "Footprint" "Capacitor_SMD:C_0805_2012Metric"
+		(property "Footprint" ""
 			(at 100.0252 151.13 0)
 			(effects
@@
 			)
 		)
-		(property "Footprint" "Resistor_SMD:R_0805_2012Metric"
+		(property "Footprint" ""
 			(at 110.998 50.8 90)
 			(effects
@@
 			)
 		)
-		(property "Footprint" "UTSVT_ICs:SOT26_DIO"
+		(property "Footprint" ""
 			(at 219.71 101.6 0)
 			(effects
@@
 			)
 		)
-		(property "Footprint" "Capacitor_SMD:C_0805_2012Metric"
+		(property "Footprint" ""
 			(at 67.0052 151.13 0)
 			(effects
@@
 			)
 		)
-		(property "Footprint" "Capacitor_SMD:C_0805_2012Metric"
+		(property "Footprint" ""
 			(at 88.9 39.0652 0)
 			(effects
@@
 			)
 		)
-		(property "Footprint" "Capacitor_SMD:C_0805_2012Metric"
+		(property "Footprint" ""
 			(at 55.5752 151.13 0)
 			(effects
@@
 			)
 		)
-		(property "Footprint" "Crystal:Crystal_SMD_TXC_7A-2Pin_5x3.2mm"
+		(property "Footprint" ""
 			(at 101.6 43.18 0)
 			(effects
@@
 			)
 		)
-		(property "Footprint" "Inductor_SMD:L_0805_2012Metric"
+		(property "Footprint" ""
 			(at 140.335 122.428 90)
 			(effects
@@
 			)
 		)
-		(property "Footprint" "Connector_PinHeader_2.54mm:PinHeader_1x04_P2.54mm_Vertical"
+		(property "Footprint" ""
 			(at 144.78 144.78 0)
 			(effects
@@
 			)
 		)
-		(property "Footprint" "Capacitor_SMD:C_0805_2012Metric"
+		(property "Footprint" ""
 			(at 88.9 49.2252 0)
 			(effects
@@
 			)
 		)
-		(property "Footprint" "Resistor_SMD:R_0805_2012Metric"
+		(property "Footprint" ""
 			(at 107.442 171.45 90)
 			(effects
@@
 			)
 		)
-		(property "Footprint" "Capacitor_SMD:C_0805_2012Metric"
+		(property "Footprint" ""
 			(at 44.1452 151.13 0)
 			(effects
@@
 			)
 		)
-		(property "Footprint" "Package_QFP:LQFP-48_7x7mm_P0.5mm"
+		(property "Footprint" ""
 			(at 128.27 105.41 0)
 			(effects

Commit message: initial PP changes
Parts:
- C11, C12, C14, C15, C16, C17, C7: P/N C0805C104M5RACTU -> (none)
- C13: P/N GRM219R6YA475KA73D -> (none)
- C21, C22: P/N C0805C120K5HACTU -> (none)
- CR1, CR2: P/N D5V0P4UR6SO-7 -> (none)
- R19: P/N CRCW08051K00FKEAC -> (none)
- R29: P/N CRCW080510K0FKEAC -> (none)
Changed lines of the file:
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@@
 			)
 		)
-		(property "P/N" "D5V0P4UR6SO-7"
+		(property "P/N" ""
 			(at 198.12 130.81 0)
 			(effects
@@
 			)
 		)
-		(property "P/N" "C0805C104M5RACTU"
+		(property "P/N" ""
 			(at 99.06 182.88 0)
 			(effects
@@
 			)
 		)
-		(property "P/N" "C0805C104M5RACTU"
+		(property "P/N" ""
 			(at 114.3 147.32 0)
 			(effects
@@
 			)
 		)
-		(property "P/N" "C0805C104M5RACTU"
+		(property "P/N" ""
 			(at 78.74 147.32 0)
 			(effects
@@
 			)
 		)
-		(property "P/N" "C0805C104M5RACTU"
+		(property "P/N" ""
 			(at 60.96 184.15 0)
 			(effects
@@
 			)
 		)
-		(property "P/N" "C0805C104M5RACTU"
+		(property "P/N" ""
 			(at 99.06 147.32 0)
 			(effects
@@
 			)
 		)
-		(property "P/N" "CRCW08051K00FKEAC"
+		(property "P/N" ""
 			(at 109.22 50.8 0)
 			(effects
@@
 			)
 		)
-		(property "P/N" "D5V0P4UR6SO-7"
+		(property "P/N" ""
 			(at 199.39 105.41 0)
 			(effects
@@
 			)
 		)
-		(property "P/N" "C0805C104M5RACTU"
+		(property "P/N" ""
 			(at 66.04 147.32 0)
 			(effects
@@
 			)
 		)
-		(property "P/N" "C0805C120K5HACTU"
+		(property "P/N" ""
 			(at 92.71 38.1 0)
 			(effects
@@
 			)
 		)
-		(property "P/N" "C0805C104M5RACTU"
+		(property "P/N" ""
 			(at 54.61 147.32 0)
 			(effects
@@
 			)
 		)
-		(property "P/N" "C0805C120K5HACTU"
+		(property "P/N" ""
 			(at 92.71 48.26 0)
 			(effects
@@
 			)
 		)
-		(property "P/N" "CRCW080510K0FKEAC"
+		(property "P/N" ""
 			(at 109.22 171.45 0)
 			(effects
@@
 			)
 		)
-		(property "P/N" "GRM219R6YA475KA73D"
+		(property "P/N" ""
 			(at 43.18 147.32 0)
 			(effects

Commit message: stuf
Parts:
- SW1: value Reset -> RST
- U1: footprint (none) -> Package_QFP:LQFP-48_7x7mm_P0.5mm
Other:
- note added: "Bypass/Separation"
- note added: "SPI Protection"
- note added: "confirm rst behavior"
- note added: "new part"
- note removed: "SPI TVS Diodes"
- title: (none) -> MCU
- moved on the sheet: C11, C12, C13, C14, C15, C16, C17, C21, C22, C7, CR1, CR2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

Commit message: control but micro
Parts:
- added SW2: BOOT, symbol Switch:SW_SPDT
- R19: value 1k -> 10k
Connections:
- net +3.3V: now also SW2.1 (A)
- net GND: now also SW2.3 (C); no longer R19.1
- net BOOT0: now reaches R19.2, U1.44 (PH3)
- new net: R19.1, SW2.2 (B)
Other:
- note added: "Boot Switch"
- note added: "Boot from..."
- note added: "CAN bootloader pins"
- note added: "Main flash (user code)"
- note added: "Pin Functions"
- note added: "System memory (bootloader)"
- note added: "UART bootloader pins"
- note added: "check where caps go (example)"
- note removed: "PH3 = boot"
- moved on the sheet: C21, C22, FB1, R19, U1, Y1

Commit message: control but micro
Connections:
- net I2C2_SCL is gone; now on net SPI2_SCK: U1.21 (PB10)
- net PB3 is gone; now on net SPI1_SCK: U1.39 (PB3)
- net SPI1_MISO: now also U1.32 (PA11); no longer U1.16 (PA6)
- net SPI1_MOSI: now also U1.33 (PA12); no longer U1.17 (PA7)
- net SPI1_NSS: now also U1.38 (PA15); no longer U1.14 (PA4)
- net SPI1_SCK: no longer U1.15 (PA5)
- net SPI2_SCK: no longer U1.26 (PB13)
- net OPAMP1_VOUT: now reaches U1.13 (PA3)
- net ADC1_IN15: now reaches U1.18 (PB0)
- net I2C2_SDA: no longer names the net of U1.22 (PB11)
- net PA0 renamed OPAMP1_VINP
- net PA1: no longer names the net of U1.11 (PA1)
- net PA2 renamed ADC1_IN7
- net PB1 renamed ADC1_IN16
- net PB4: no longer names the net of U1.40 (PB4)
- net PB5: no longer names the net of U1.41 (PB5)
- new net ADC1_IN10: U1.15 (PA5)
- new net ADC1_IN11: U1.16 (PA6)
- new net ADC1_IN12: U1.17 (PA7)
- new net ADC1_IN9: U1.14 (PA4)
Other:
- note added: "Internally connected to ADC1_IN8"
- note added: "NC OPAMP1_VINM (inverting input) -> using internal PGA"
- note added: "Primary Pin Functions"
- note added: "USART bootloader pins"
- note added: "add LEDs for unused pins"
- note added: "add list of alternate functions"
- note added: "new part + pinout?"
- note added: "shift pins for optimal routing"
- note removed: "Pin Functions"
- note removed: "UART bootloader pins"
- note removed: "new part"
- moved on the sheet: C21, CR1, CR2, R19, SW2

Commit message: prelim pin selection
Connections:
- net ADC1_IN15 is gone; now on net SPI1_NSS: U1.18 (PB0)
- net SPI1_NSS: no longer U1.38 (PA15)
- net ADC1_IN12: no longer names the net of U1.17 (PA7)
- net ADC1_IN16: no longer names the net of U1.19 (PB1)
- no-connect marks 11 -> 14

Commit message: bruh
Connections:
- net VDD is gone; now on net +3.3V: R29.1
- net +3.3V: now also U1.1 (VBAT)
- net CAN_RX renamed CAN1_RX
- net CAN_TX renamed CAN1_TX
- no-connect marks 14 -> 13
Changed lines of the file:
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@@
 	)
 	(junction
+		(at 137.16 26.67)
+		(diameter 0)
+		(color 0 0 0 0)
+	)
+	(junction
+		(at 138.43 26.67)
+		(diameter 0)
+		(color 0 0 0 0)
+	)
+	(junction
 		(at 21.59 63.5)
 		(diameter 0)
@@
 	)
 	(no_connect
-		(at 134.62 27.94)
-	)
-	(no_connect
 		(at 124.46 86.36)
 	)
@@
 	(wire
 		(pts
+			(xy 134.62 26.67) (xy 134.62 27.94)
+		)
+		(stroke
+			(width 0)
+			(type default)
+		)
+	)
+	(wire
+		(pts
 			(xy 139.7 26.67) (xy 139.7 27.94)
 		)
@@
 	(wire
 		(pts
+			(xy 134.62 26.67) (xy 137.16 26.67)
+		)
+		(stroke
+			(width 0)
+			(type default)
+		)
+	)
+	(wire
+		(pts
 			(xy 44.45 31.75) (xy 57.15 31.75)
 		)
@@
 	(wire
 		(pts
+			(xy 138.43 26.67) (xy 139.7 26.67)
+		)
+		(stroke
+			(width 0)
+			(type default)
+		)
+	)
+	(wire
+		(pts
 			(xy 113.03 76.2) (xy 124.46 76.2)
 		)
@@
 	(wire
 		(pts
-			(xy 137.16 26.67) (xy 139.7 26.67)
+			(xy 137.16 26.67) (xy 138.43 26.67)
 		)
 		(stroke
@@
 	(wire
 		(pts
-			(xy 139.7 24.13) (xy 139.7 26.67)
+			(xy 138.43 24.13) (xy 138.43 26.67)
 		)
 		(stroke
@@
 		)
 	)
-	(label "CAN_RX"
+	(label "CAN1_RX"
 		(at 113.03 78.74 0)
 		(effects
@@
 		)
 	)
-	(label "CAN_TX"
+	(label "CAN1_TX"
 		(at 113.03 81.28 0)
 		(effects
@@
 	)
 	(symbol
+		(lib_id "power:+3.3V")
+		(at 33.02 88.9 0)
+		(unit 1)
+		(exclude_from_sim no)
+		(in_bom yes)
+		(on_board yes)
+		(dnp no)
+		(property "Reference" "#PWR062"
+			(at 33.02 92.71 0)
+			(effects
+				(font
+					(size 1.27 1.27)
+				)
+				(hide yes)
+			)
+		)
+		(property "Value" "+3.3V"
+			(at 32.004 85.344 0)
+			(effects
+				(font
+					(size 1.27 1.27)
+				)
+			)
+		)
+		(property "Footprint" ""
+			(at 33.02 88.9 0)
+			(effects
+				(font
+					(size 1.27 1.27)
+				)
+				(hide yes)
+			)
+		)
+		(property "Datasheet" ""
+			(at 33.02 88.9 0)
+			(effects
+				(font
+					(size 1.27 1.27)
+				)
+				(hide yes)
+			)
+		)
+		(property "Description" "Power symbol creates a global label with name \"+3.3V\""
+			(at 33.02 88.9 0)
+			(effects
+				(font
+					(size 1.27 1.27)
+				)
+				(hide yes)
+			)
+		)
+		(pin "1"
+		)
+		(instances
+			(project "PeripheralSOM"
+				(path "/d5ebd247-5a7c-47c2-8aee-beabaef72d6d/1d53f8ef-8689-4a8b-8330-e806b7f39af5"
+					(reference "#PWR062")
+					(unit 1)
+				)
+			)
+		)
+	)
+	(symbol
 		(lib_id "utsvt-chips:D5V0P4UR6SO-7")
 		(at 33.02 167.64 0)
@@
 	(symbol
 		(lib_id "power:+3.3V")
-		(at 139.7 24.13 0)
+		(at 138.43 24.13 0)
 		(unit 1)
 		(exclude_from_sim no)
@@
 		(dnp no)
 		(property "Reference" "#PWR023"
-			(at 139.7 27.94 0)
+			(at 138.43 27.94 0)
 			(effects
 				(font
@@
 		)
 		(property "Value" "+3.3V"
-			(at 138.684 20.574 0)
+			(at 137.414 20.574 0)
 			(effects
 				(font
@@
 		)
 		(property "Footprint" ""
-			(at 139.7 24.13 0)
+			(at 138.43 24.13 0)
 			(effects
 				(font
@@
 		)
 		(property "Datasheet" ""
-			(at 139.7 24.13 0)
+			(at 138.43 24.13 0)
 			(effects
 				(font
@@
 		)
 		(property "Description" "Power symbol creates a global label with name \"+3.3V\""
-			(at 139.7 24.13 0)
+			(at 138.43 24.13 0)
 			(effects
 				(font
@@
 					(unit 1)
 				)
-			)
-		)
-	)
-	(symbol
-		(lib_id "power:VDD")
-		(at 33.02 88.9 0)
-		(unit 1)
-		(exclude_from_sim no)
-		(in_bom yes)
-		(on_board yes)
-		(dnp no)
-		(fields_autoplaced yes)
-		(property "Reference" "#PWR062"
-			(at 33.02 92.71 0)
-			(effects
-				(font
-					(size 1.27 1.27)
-				)
-				(hide yes)
-			)
-		)
-		(property "Value" "VDD"
-			(at 33.02 83.82 0)
-			(effects
-				(font
-					(size 1.27 1.27)
-				)
-			)
-		)
-		(property "Footprint" ""
-			(at 33.02 88.9 0)
-			(effects
-				(font
-					(size 1.27 1.27)
-				)
-				(hide yes)
-			)
-		)
-		(property "Datasheet" ""
-			(at 33.02 88.9 0)
-			(effects
-				(font
-					(size 1.27 1.27)
-				)
-				(hide yes)
-			)
-		)
-		(property "Description" "Power symbol creates a global label with name \"VDD\""
-			(at 33.02 88.9 0)
-			(effects
-				(font
-					(size 1.27 1.27)
-				)
-				(hide yes)
-			)
-		)
-		(pin "1"
-		)
-		(instances
-			(project "BPS-PeripheralSOM"
-				(path "/d5ebd247-5a7c-47c2-8aee-beabaef72d6d/1d53f8ef-8689-4a8b-8330-e806b7f39af5"
-					(reference "#PWR062")
-					(unit 1)
-				)
