File: STM32L431CBT6.kicad_sch (KiCad schematic)
At the start: 21 parts, among them J1 SWD, SW1 RST, SW2 BOOT, U1 STM32L431CBTx, Y1 8M

Commit message: finish mcu breakouts
Connections:
- net SPI2_MOSI: no longer CR1.4
- net SPI2_SCK: now also CR1.4
- net OPAMP1_VOUT: no longer names the net of U1.13 (PA3)
- no-connect marks 13 -> 14
Other:
- note added: "NC OPAMP1_VOUT -> internally connected to ADC1_IN8"
- note removed: "Internally connected to ADC1_IN8"

Commit message: twinkle
Connections:
- net LED1: now reaches U1.17 (PA7)
- net LED_HB: now reaches U1.22 (PB11)
- net LED2: now reaches U1.29 (PA8)
- net LED3: now reaches U1.38 (PA15)
- no-connect marks 14 -> 10
Other:
- note removed: "add LEDs for unused pins"
- note removed: "check where caps go (example)"
Changed lines of the file:
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@@
 	(text "The crystal and caps have to be as \nclose to the uC as possible and\nno traces should go underneath\nthese components or connections."
 		(exclude_from_sim no)
-		(at 83.312 28.194 0)
+		(at 80.518 31.496 0)
 		(effects
 			(font
@@
 		)
 	)
-	(text "check where caps go (example)"
-		(exclude_from_sim no)
-		(at 83.058 31.75 0)
-		(effects
-			(font
-				(size 1.27 1.27)
-				(color 255 0 0 1)
-			)
-			(justify left bottom)
-		)
-	)
 	(text "SPI Protection"
 		(exclude_from_sim no)
@@
 		)
 	)
-	(text "add LEDs for unused pins"
-		(exclude_from_sim no)
-		(at 154.94 76.708 0)
-		(effects
-			(font
-				(size 1.27 1.27)
-				(color 255 0 0 1)
-			)
-			(justify left bottom)
-		)
-	)
 	(text "VDDA Bypass Caps"
 		(exclude_from_sim no)
@@
 	)
 	(no_connect
-		(at 124.46 86.36)
-	)
-	(no_connect
 		(at 154.94 35.56)
 	)
 	(no_connect
-		(at 154.94 50.8)
-	)
-	(no_connect
-		(at 154.94 53.34)
-	)
-	(no_connect
 		(at 124.46 53.34)
 	)
@@
 		(at 124.46 91.44)
 	)
-	(no_connect
-		(at 154.94 71.12)
-	)
 	(bus_entry
 		(at 113.03 78.74)
@@
 	)
 	(bus_entry
+		(at 179.07 69.85)
+		(size 2.54 2.54)
+		(stroke
+			(width 0)
+			(type default)
+		)
+	)
+	(bus_entry
 		(at 88.9 99.06)
 		(size 2.54 -2.54)
@@
 	)
 	(bus_entry
+		(at 179.07 72.39)
+		(size 2.54 2.54)
+		(stroke
+			(width 0)
+			(type default)
+		)
+	)
+	(bus_entry
 		(at 168.91 55.88)
 		(size 2.54 2.54)
@@
 	)
 	(bus_entry
+		(at 179.07 74.93)
+		(size 2.54 2.54)
+		(stroke
+			(width 0)
+			(type default)
+		)
+	)
+	(bus_entry
 		(at 168.91 45.72)
 		(size 2.54 2.54)
@@
 	(wire
 		(pts
+			(xy 123.19 85.09) (xy 123.19 86.36)
+		)
+		(stroke
+			(width 0)
+			(type default)
+		)
+	)
+	(wire
+		(pts
+			(xy 173.99 72.39) (xy 179.07 72.39)
+		)
+		(stroke
+			(width 0)
+			(type default)
+		)
+	)
+	(wire
+		(pts
 			(xy 134.62 26.67) (xy 134.62 27.94)
 		)
@@
 	(wire
 		(pts
+			(xy 121.92 85.09) (xy 123.19 85.09)
+		)
+		(stroke
+			(width 0)
+			(type default)
+		)
+	)
+	(bus
+		(pts
+			(xy 181.61 72.39) (xy 181.61 74.93)
+		)
+		(stroke
+			(width 0)
+			(type default)
+		)
+	)
+	(wire
+		(pts
 			(xy 82.55 44.45) (xy 85.09 44.45)
 		)
@@
 	(wire
 		(pts
+			(xy 154.94 53.34) (xy 168.91 53.34)
+		)
+		(stroke
+			(width 0)
+			(type default)
+		)
+	)
+	(wire
+		(pts
 			(xy 54.61 97.79) (xy 54.61 93.98)
 		)
@@
 	(wire
 		(pts
+			(xy 173.99 69.85) (xy 179.07 69.85)
+		)
+		(stroke
+			(width 0)
+			(type default)
+		)
+	)
+	(wire
+		(pts
 			(xy 44.45 31.75) (xy 57.15 31.75)
 		)
@@
 	(wire
 		(pts
+			(xy 123.19 86.36) (xy 124.46 86.36)
+		)
+		(stroke
+			(width 0)
+			(type default)
+		)
+	)
+	(wire
+		(pts
+			(xy 173.99 74.93) (xy 179.07 74.93)
+		)
+		(stroke
+			(width 0)
+			(type default)
+		)
+	)
+	(wire
+		(pts
 			(xy 154.94 63.5) (xy 168.91 63.5)
 		)
@@
 		)
 	)
+	(bus
+		(pts
+			(xy 182.88 78.74) (xy 184.15 78.74)
+		)
+		(stroke
+			(width 0)
+			(type default)
+		)
+	)
 	(wire
 		(pts
@@
 		)
 	)
+	(bus
+		(pts
+			(xy 182.88 78.74) (xy 181.61 77.47)
+		)
+		(stroke
+			(width 0)
+			(type default)
+		)
+	)
 	(wire
 		(pts
@@
 	(wire
 		(pts
+			(xy 154.94 50.8) (xy 168.91 50.8)
+		)
+		(stroke
+			(width 0)
+			(type default)
+		)
+	)
+	(wire
+		(pts
 			(xy 33.02 88.9) (xy 33.02 90.17)
 		)
@@
 	(wire
 		(pts
+			(xy 154.94 71.12) (xy 168.91 71.12)
+		)
+		(stroke
+			(width 0)
+			(type default)
+		)
+	)
+	(wire
+		(pts
 			(xy 21.59 63.5) (xy 36.83 63.5)
 		)
@@
 		)
 	)
+	(bus
+		(pts
+			(xy 181.61 74.93) (xy 181.61 77.47)
+		)
+		(stroke
+			(width 0)
+			(type default)
+		)
+	)
 	(wire
 		(pts
@@
 		)
 	)
+	(label "LED3"
+		(at 173.99 74.93 0)
+		(effects
+			(font
+				(size 1.27 1.27)
+			)
+			(justify left bottom)
+		)
+	)
 	(label "ADC1_IN10"
 		(at 168.91 45.72 180)
@@
 		)
 	)
+	(label "LED1"
+		(at 168.91 50.8 180)
+		(effects
+			(font
+				(size 1.27 1.27)
+			)
+			(justify right bottom)
+		)
+	)
 	(label "SWCLK"
 		(at 55.88 91.44 0)
@@
 		)
 	)
+	(label "LED2"
+		(at 173.99 72.39 0)
+		(effects
+			(font
+				(size 1.27 1.27)
+			)
+			(justify left bottom)
+		)
+	)
 	(label "SPI2_MOSI"
 		(at 22.86 167.64 0)
@@
 		)
 	)
+	(label "LED1"
+		(at 173.99 69.85 0)
+		(effects
+			(font
+				(size 1.27 1.27)
+			)
+			(justify left bottom)
+		)
+	)
 	(label "SPI1_NSS"
 		(at 113.03 58.42 0)
@@
 		)
 	)
+	(label "LED2"
+		(at 168.91 53.34 180)
+		(effects
+			(font
+				(size 1.27 1.27)
+			)
+			(justify right bottom)
+		)
+	)
 	(label "OSC_IN"
 		(at 102.87 38.1 0)
@@
 		)
 	)
+	(label "LED3"
+		(at 168.91 71.12 180)
+		(effects
+			(font
+				(size 1.27 1.27)
+			)
+			(justify right bottom)
+		)
+	)
 	(hierarchical_label "{ADC1}"
 		(shape bidirectional)
@@
 		)
 	)
+	(hierarchical_label "LED[1..3]"
+		(shape output)
+		(at 184.15 78.74 0)
+		(effects
+			(font
+				(size 1.27 1.27)
+			)
+			(justify left)
+		)
+	)
 	(hierarchical_label "{SPI2}"
 		(shape bidirectional)
@@
 		)
 	)
+	(hierarchical_label "LED_HB"
+		(shape output)
+		(at 121.92 85.09 180)
+		(effects
+			(font
+				(size 1.27 1.27)
+			)
+			(justify right)
+		)
+	)
 	(hierarchical_label "{CAN1}"
 		(shape bidirectional)
@@
 		(dnp no)
 		(property "Reference" "C21"
-			(at 90.1954 37.338 0)
+			(at 86.868 38.0746 90)
 			(effects
 				(font
@@
 		)
 		(property "Value" "12p"
-			(at 87.884 37.338 0)
+			(at 86.868 40.386 90)
 			(effects
 				(font
@@
 		(dnp no)
 		(property "Reference" "C22"
-			(at 90.0684 47.371 0)
+			(at 87.0585 48.0441 90)
 			(effects
 				(font
@@
 		)
 		(property "Value" "12p"
-			(at 87.757 47.371 0)
+			(at 87.0585 50.3555 90)
 			(effects
 				(font

Commit message: FUCK capacitors
Parts:
- C11, C12, C14, C15, C16, C17, C7: P/N (none) -> MLASH168SB7104KTNA01
- C13: P/N (none) -> 08055D475KAT4A
- C21, C22: P/N (none) -> 06035U120FAT2A
- CR1, CR2: footprint (none) -> UTSVT_ICs:D5V0P4UR6SO-7; symbol utsvt-chips:D5V0P4UR6SO-7 -> utsvt_ics:D5V0P4UR6SO-7; P/N (none) -> D5V0P4UR6SO-7
Changed lines of the file:
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@@
 	)
 	(symbol
-		(lib_id "utsvt-chips:D5V0P4UR6SO-7")
+		(lib_id "utsvt_ics:D5V0P4UR6SO-7")
 		(at 33.02 167.64 0)
 		(unit 1)
@@
 			)
 		)
-		(property "Footprint" ""
+		(property "Footprint" "UTSVT_ICs:D5V0P4UR6SO-7"
 			(at 53.34 163.83 0)
 			(effects
@@
 			)
 		)
-		(property "P/N" ""
+		(property "P/N" "D5V0P4UR6SO-7"
+			(at 33.02 167.64 0)
+			(effects
+				(font
+					(size 1.27 1.27)
+				)
+				(hide yes)
+			)
+		)
+		(property "PN" ""
+			(at 33.02 167.64 0)
+			(effects
+				(font
+					(size 1.27 1.27)
+				)
+				(hide yes)
+			)
+		)
+		(property "p/n" ""
 			(at 33.02 167.64 0)
 			(effects
@@
 			)
 		)
-		(property "P/N" ""
+		(property "P/N" "MLASH168SB7104KTNA01"
 			(at 21.59 105.41 0)
 			(effects
@@
 			)
 		)
-		(property "P/N" ""
+		(property "P/N" "MLASH168SB7104KTNA01"
 			(at 36.83 59.69 0)
 			(effects
@@
 			)
 		)
-		(property "Datasheet" "~"
+		(property "Datasheet" "https://omronfs.omron.com/en_US/ecb/products/pdf/en-b3sl.pdf"
 			(at 38.1 105.41 0)
 			(effects
@@
 			)
 		)
-		(property "P/N" ""
+		(property "P/N" "MLASH168SB7104KTNA01"
 			(at 57.15 35.56 0)
 			(effects
@@
 			)
 		)
-		(property "Datasheet" "~"
+		(property "Datasheet" "https://www.eaton.com/content/dam/eaton/products/electronic-components/resources/data-sheet/eaton-mfbw1v2012-high-impedance-multilayer-ferrite-chip-bead-data-sheet.pdf"
 			(at 59.69 54.61 0)
 			(effects
@@
 			)
 		)
-		(property "P/N" ""
+		(property "P/N" "MLASH168SB7104KTNA01"
 			(at 64.77 58.42 0)
 			(effects
@@
 			)
 		)
-		(property "P/N" ""
+		(property "P/N" "MLASH168SB7104KTNA01"
 			(at 21.59 59.69 0)
 			(effects
@@
 	)
 	(symbol
-		(lib_id "utsvt-chips:D5V0P4UR6SO-7")
+		(lib_id "utsvt_ics:D5V0P4UR6SO-7")
 		(at 33.02 144.78 0)
 		(unit 1)
@@
 			)
 		)
-		(property "Footprint" ""
+		(property "Footprint" "UTSVT_ICs:D5V0P4UR6SO-7"
 			(at 53.34 140.97 0)
 			(effects
@@
 			)
 		)
-		(property "P/N" ""
+		(property "P/N" "D5V0P4UR6SO-7"
+			(at 33.02 144.78 0)
+			(effects
+				(font
+					(size 1.27 1.27)
+				)
+				(hide yes)
+			)
+		)
+		(property "PN" ""
+			(at 33.02 144.78 0)
+			(effects
+				(font
+					(size 1.27 1.27)
+				)
+				(hide yes)
+			)
+		)
+		(property "p/n" ""
 			(at 33.02 144.78 0)
 			(effects
@@
 			)
 		)
-		(property "P/N" ""
+		(property "P/N" "MLASH168SB7104KTNA01"
 			(at 44.45 35.56 0)
 			(effects
@@
 			)
 		)
-		(property "P/N" ""
+		(property "P/N" "06035U120FAT2A"
 			(at 88.9 34.29 0)
 			(effects
@@
 			)
 		)
-		(property "P/N" ""
+		(property "P/N" "MLASH168SB7104KTNA01"
 			(at 33.02 35.56 0)
 			(effects
@@
 			)
 		)
-		(property "Datasheet" "~"
+		(property "Datasheet" "https://abracon.com/Resonators/ABM3.pdf"
 			(at 96.52 39.37 0)
 			(effects
@@
 			)
 		)
-		(property "Datasheet" "~"
+		(property "Datasheet" "https://www.eaton.com/content/dam/eaton/products/electronic-components/resources/data-sheet/eaton-mfbw1v2012-high-impedance-multilayer-ferrite-chip-bead-data-sheet.pdf"
 			(at 139.065 113.03 0)
 			(effects
@@
 			)
 		)
-		(property "P/N" ""
+		(property "P/N" "06035U120FAT2A"
 			(at 88.9 44.45 0)
 			(effects
@@
 			)
 		)
-		(property "P/N" ""
+		(property "P/N" "08055D475KAT4A"
 			(at 21.59 35.56 0)
 			(effects

Commit message: all parts selected
Parts:
- J1: P/N (none) -> 0022232041
- R19: P/N (none) -> CRCW060310K0FKEI
- R29: value 10K -> 10k; P/N (none) -> CRCW060310K0FKEI
- SW2: P/N (none) -> CJS-1200TA
Changed lines of the file:
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@@
-			)
-		)
-		(property "PN" ""
-			(at 33.02 167.64 0)
-			(effects
-				(font
-					(size 1.27 1.27)
-				)
-				(hide yes)
-			)
-		)
-		(property "p/n" ""
-			(at 33.02 167.64 0)
-			(effects
-				(font
-					(size 1.27 1.27)
-				)
-				(hide yes)
 			)
 		)
@@
 			)
 		)
-		(property "Datasheet" "~"
+		(property "Datasheet" "https://www.mouser.com/datasheet/2/972/cjs-1827353.pdf"
 			(at 120.65 146.05 0)
 			(effects
@@
 			)
 		)
+		(property "P/N" "CJS-1200TA "
+			(at 120.65 138.43 0)
+			(effects
+				(font
+					(size 1.27 1.27)
+				)
+				(hide yes)
+			)
+		)
 		(pin "2"
 		)
@@
 			)
 		)
-		(property "P/N" ""
+		(property "P/N" "CRCW060310K0FKEI "
 			(at 110.49 138.43 0)
 			(effects
@@
 			)
 		)
-		(property "PN" ""
-			(at 33.02 144.78 0)
-			(effects
-				(font
-					(size 1.27 1.27)
-				)
-				(hide yes)
-			)
-		)
-		(property "p/n" ""
-			(at 33.02 144.78 0)
-			(effects
-				(font
-					(size 1.27 1.27)
-				)
-				(hide yes)
-			)
-		)
 		(pin "1"
 		)
@@
 			)
 		)
-		(property "Datasheet" "~"
+		(property "Datasheet" "https://www.molex.com/en-us/products/part-detail/22232041?display=pdf"
 			(at 68.58 91.44 0)
 			(effects
@@
 		)
 		(property "Description" "Generic connector, single row, 01x04, script generated (kicad-library-utils/schlib/autogen/connector/)"
+			(at 68.58 91.44 0)
+			(effects
+				(font
+					(size 1.27 1.27)
+				)
+				(hide yes)
+			)
+		)
+		(property "P/N" "0022232041"
 			(at 68.58 91.44 0)
 			(effects
@@
 			)
 		)
-		(property "Value" "10K"
+		(property "Value" "10k"
 			(at 35.56 95.885 0)
 			(effects
@@
 			)
 		)
-		(property "P/N" ""
+		(property "P/N" "CRCW060310K0FKEI "
 			(at 33.02 93.98 0)
 			(effects

Commit message: add IMON, change conn pinout
Connections:
- net ADC1_IN16: now reaches U1.19 (PB1)
- no-connect marks 10 -> 9

Commit message: add some footprints
Parts:
- R19, R29: footprint (none) -> Resistor_SMD:R_0603_1608Metric_Pad0.98x0.95mm_HandSolder
- SW1: footprint (none) -> Button_Switch_SMD:SW_SPST_B3SL-1002P
Changed lines of the file:
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@@
 			)
 		)
-		(property "Footprint" ""
+		(property "Footprint" "Button_Switch_SMD:SW_SPST_B3SL-1002P"
 			(at 38.1 105.41 0)
 			(effects
@@
 		(instances
 			(project ""
+				(path "/d5ebd247-5a7c-47c2-8aee-beabaef72d6d/1d0c269d-60cf-499b-bfd2-5087981d6678"
+					(reference "SW2")
+					(unit 1)
+				)
 				(path "/d5ebd247-5a7c-47c2-8aee-beabaef72d6d/1d53f8ef-8689-4a8b-8330-e806b7f39af5"
 					(reference "SW2")
@@
 			)
 		)
-		(property "Footprint" ""
+		(property "Footprint" "Resistor_SMD:R_0603_1608Metric_Pad0.98x0.95mm_HandSolder"
 			(at 110.49 136.652 90)
 			(effects
@@
 			)
 		)
-		(property "Footprint" ""
+		(property "Footprint" "Resistor_SMD:R_0603_1608Metric_Pad0.98x0.95mm_HandSolder"
 			(at 31.242 93.98 90)
 			(effects

Commit message: more stuff
Parts:
- J1: footprint (none) -> 0022232041:CONN_A-6373-04A_MOL
- SW2: footprint (none) -> CJS-1200TA:SW_CJS-1200TA
- Y1: footprint (none) -> Crystal:Crystal_SMD_Abracon_ABM3-2Pin_5.0x3.2mm
Changed lines of the file:
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@@
 			)
 		)
-		(property "Footprint" ""
+		(property "Footprint" "CJS-1200TA:SW_CJS-1200TA"
 			(at 120.65 138.43 0)
 			(effects
@@
 			)
 		)
-		(property "Footprint" ""
+		(property "Footprint" "Crystal:Crystal_SMD_Abracon_ABM3-2Pin_5.0x3.2mm"
 			(at 96.52 39.37 0)
 			(effects
@@
 			)
 		)
-		(property "Footprint" ""
+		(property "Footprint" "0022232041:CONN_A-6373-04A_MOL"
 			(at 68.58 91.44 0)
 			(effects

Commit message: all footprints assigned
Parts:
- C11, C12, C14, C15, C16, C17, C21, C22, C7: footprint (none) -> Capacitor_SMD:C_0603_1608Metric_Pad1.08x0.95mm_HandSolder
- C13: footprint (none) -> Capacitor_SMD:C_0805_2012Metric_Pad1.18x1.45mm_HandSolder
- FB1, FB4: footprint (none) -> Capacitor_SMD:C_0603_1608Metric_Pad1.08x0.95mm_HandSolder; P/N MFBW1V2012-121-R -> BLM18PG121SH1D
Changed lines of the file:
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@@
 			)
 		)
-		(property "Footprint" ""
+		(property "Footprint" "Capacitor_SMD:C_0603_1608Metric_Pad1.08x0.95mm_HandSolder"
 			(at 22.5552 109.22 0)
 			(effects
@@
 			)
 		)
-		(property "Footprint" ""
+		(property "Footprint" "Capacitor_SMD:C_0603_1608Metric_Pad1.08x0.95mm_HandSolder"
 			(at 37.7952 63.5 0)
 			(effects
@@
 			)
 		)
-		(property "Footprint" ""
+		(property "Footprint" "Capacitor_SMD:C_0603_1608Metric_Pad1.08x0.95mm_HandSolder"
 			(at 58.1152 39.37 0)
 			(effects
@@
 			)
 		)
-		(property "Footprint" ""
+		(property "Footprint" "Capacitor_SMD:C_0603_1608Metric_Pad1.08x0.95mm_HandSolder"
 			(at 59.69 56.388 90)
 			(effects
@@
 			)
 		)
-		(property "P/N" "MFBW1V2012-121-R"
+		(property "P/N" "BLM18PG121SH1D"
 			(at 59.69 54.61 0)
 			(effects
@@
 			)
 		)
-		(property "Footprint" ""
+		(property "Footprint" "Capacitor_SMD:C_0603_1608Metric_Pad1.08x0.95mm_HandSolder"
 			(at 65.7352 62.23 0)
 			(effects
@@
 			)
 		)
-		(property "Footprint" ""
+		(property "Footprint" "Capacitor_SMD:C_0603_1608Metric_Pad1.08x0.95mm_HandSolder"
 			(at 22.5552 63.5 0)
 			(effects
@@
 			)
 		)
-		(property "Footprint" ""
+		(property "Footprint" "Capacitor_SMD:C_0603_1608Metric_Pad1.08x0.95mm_HandSolder"
 			(at 45.4152 39.37 0)
 			(effects
@@
 			)
 		)
-		(property "Footprint" ""
+		(property "Footprint" "Capacitor_SMD:C_0603_1608Metric_Pad1.08x0.95mm_HandSolder"
 			(at 85.09 35.2552 0)
 			(effects
@@
 			)
 		)
-		(property "Footprint" ""
+		(property "Footprint" "Capacitor_SMD:C_0603_1608Metric_Pad1.08x0.95mm_HandSolder"
 			(at 33.9852 39.37 0)
 			(effects
@@
 			)
 		)
-		(property "Footprint" ""
+		(property "Footprint" "Capacitor_SMD:C_0603_1608Metric_Pad1.08x0.95mm_HandSolder"
 			(at 139.065 114.808 90)
 			(effects
@@
 			)
 		)
-		(property "P/N" "MFBW1V2012-121-R"
+		(property "P/N" "BLM18PG121SH1D"
 			(at 139.065 113.03 0)
 			(effects
@@
 			)
 		)
-		(property "Footprint" ""
+		(property "Footprint" "Capacitor_SMD:C_0603_1608Metric_Pad1.08x0.95mm_HandSolder"
 			(at 85.09 45.4152 0)
 			(effects
@@
 			)
 		)
-		(property "Footprint" ""
+		(property "Footprint" "Capacitor_SMD:C_0805_2012Metric_Pad1.18x1.45mm_HandSolder"
 			(at 22.5552 39.37 0)
 			(effects
