File: STM32L431CBT6.kicad_sch (KiCad schematic)
At the start: 21 parts, among them J1 SWD, SW1 RST, SW2 BOOT, U1 STM32L431CBTx, Y1 8M

Commit message: sch notes
Other:
- note removed: "confirm rst behavior"
- note removed: "new part + pinout?"
Changed lines of the file:
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@@
-		)
-	)
-	(text "confirm rst behavior"
-		(exclude_from_sim no)
-		(at 23.876 114.808 0)
-		(effects
-			(font
-				(size 1.27 1.27)
-				(color 255 0 0 1)
-			)
-			(justify left bottom)
 		)
 	)
@@
 		)
 	)
-	(text "new part + pinout?"
-		(exclude_from_sim no)
-		(at 56.642 86.614 0)
-		(effects
-			(font
-				(size 1.27 1.27)
-				(color 255 0 0 1)
-			)
-			(justify left bottom)
-		)
-	)

Commit message: start adding mcu
Connections:
- net SPI2_MISO: now also CR1.1; no longer CR1.6
- net SPI2_MOSI: now also CR1.6; no longer CR1.1
Other:
- note removed: "shift pins for optimal routing"
Changed lines of the file:
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@@
 		)
 	)
-	(text "shift pins for\noptimal routing"
-		(exclude_from_sim no)
-		(at 67.31 157.988 0)
-		(effects
-			(font
-				(size 1.27 1.27)
-				(color 255 0 0 1)
-			)
-			(justify left bottom)
-		)
-	)
 	(text "SWD Connector"
 		(exclude_from_sim no)
@@
 		)
 	)
-	(label "SPI2_MISO"
+	(label "SPI2_MOSI"
 		(at 83.82 167.64 180)
 		(effects
@@
 		)
 	)
-	(label "SPI2_MOSI"
+	(label "SPI2_MISO"
 		(at 22.86 167.64 0)
 		(effects

Commit message: address some stuff
Parts:
- C11, C12, C14, C15, C16, C17, C7: Mouser Part Number 80-C0805C104M5R -> (none)
- C13: Mouser Part Number 81-GRM219R6YA475KA3D -> (none)
- C21, C22: Mouser Part Number 80-C0805C120K5HACTU -> (none)
- CR1, CR2: Mouser Part Number 621-D5V0P4UR6SO-7 -> (none)
- FB1, FB4: Mouser Part Number 704-MFBW1V2012-121-R -> (none)
- R19, R29: Mouser Part Number 71-CRCW080510K0FKEAC -> (none)
- SW1: Mouser Part Number 653-B3SL-1002P -> (none)
- U1: Mouser Part Number 511-STM32L431CBT6 -> (none)
- Y1: Mouser Part Number 815-ABM3-8-D2Y-T -> (none)
Other:
- note added: "Mates with 0022013047"
Changed lines of the file:
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@@
 		)
 	)
+	(text "Mates with\n0022013047"
+		(exclude_from_sim no)
+		(at 58.928 103.632 0)
+		(effects
+			(font
+				(size 1.27 1.27)
+			)
+			(justify left bottom)
+		)
+	)
 	(text "Boot Switch"
 		(exclude_from_sim no)
@@
 			)
 		)
-		(property "Mouser Part Number" "621-D5V0P4UR6SO-7"
-			(at 33.02 167.64 0)
-			(effects
-				(font
-					(size 1.27 1.27)
-				)
-				(hide yes)
-			)
-		)
 		(property "P/N" "D5V0P4UR6SO-7"
 			(at 33.02 167.64 0)
@@
 			)
 		)
-		(property "Mouser Part Number" "80-C0805C104M5R"
-			(at 21.59 105.41 0)
-			(effects
-				(font
-					(size 1.27 1.27)
-				)
-				(hide yes)
-			)
-		)
 		(property "P/N" "MLASH168SB7104KTNA01"
 			(at 21.59 105.41 0)
@@
 			)
 		)
-		(property "Mouser Part Number" "80-C0805C104M5R"
-			(at 36.83 59.69 0)
-			(effects
-				(font
-					(size 1.27 1.27)
-				)
-				(hide yes)
-			)
-		)
 		(property "P/N" "MLASH168SB7104KTNA01"
 			(at 36.83 59.69 0)
@@
 			)
 		)
-		(property "Mouser Part Number" "653-B3SL-1002P"
-			(at 33.02 105.41 0)
-			(effects
-				(font
-					(size 1.27 1.27)
-				)
-				(hide yes)
-			)
-		)
 		(pin "1"
 		)
@@
 			)
 		)
-		(property "Mouser Part Number" "80-C0805C104M5R"
-			(at 57.15 35.56 0)
-			(effects
-				(font
-					(size 1.27 1.27)
-				)
-				(hide yes)
-			)
-		)
 		(property "P/N" "MLASH168SB7104KTNA01"
 			(at 57.15 35.56 0)
@@
 			)
 		)
-		(property "Mouser Part Number" "704-MFBW1V2012-121-R"
-			(at 59.69 54.61 0)
-			(effects
-				(font
-					(size 1.27 1.27)
-				)
-				(hide yes)
-			)
-		)
 		(property "P/N" "BLM18PG121SH1D"
 			(at 59.69 54.61 0)
@@
 			)
 		)
-		(property "Mouser Part Number" "80-C0805C104M5R"
-			(at 64.77 58.42 0)
-			(effects
-				(font
-					(size 1.27 1.27)
-				)
-				(hide yes)
-			)
-		)
 		(property "P/N" "MLASH168SB7104KTNA01"
 			(at 64.77 58.42 0)
@@
 			)
 		)
-		(property "Mouser Part Number" "80-C0805C104M5R"
-			(at 21.59 59.69 0)
-			(effects
-				(font
-					(size 1.27 1.27)
-				)
-				(hide yes)
-			)
-		)
 		(property "P/N" "MLASH168SB7104KTNA01"
 			(at 21.59 59.69 0)
@@
 			)
 		)
-		(property "Mouser Part Number" "71-CRCW080510K0FKEAC"
-			(at 110.49 138.43 0)
-			(effects
-				(font
-					(size 1.27 1.27)
-				)
-				(hide yes)
-			)
-		)
 		(property "P/N" "CRCW060310K0FKEI "
 			(at 110.49 138.43 0)
@@
 			)
 		)
-		(property "Mouser Part Number" "621-D5V0P4UR6SO-7"
-			(at 33.02 144.78 0)
-			(effects
-				(font
-					(size 1.27 1.27)
-				)
-				(hide yes)
-			)
-		)
 		(property "P/N" "D5V0P4UR6SO-7"
 			(at 33.02 144.78 0)
@@
 			)
 		)
-		(property "Mouser Part Number" "80-C0805C104M5R"
-			(at 44.45 35.56 0)
-			(effects
-				(font
-					(size 1.27 1.27)
-				)
-				(hide yes)
-			)
-		)
 		(property "P/N" "MLASH168SB7104KTNA01"
 			(at 44.45 35.56 0)
@@
 			)
 		)
-		(property "Mouser Part Number" "80-C0805C120K5HACTU"
-			(at 88.9 34.29 0)
-			(effects
-				(font
-					(size 1.27 1.27)
-				)
-				(hide yes)
-			)
-		)
 		(property "P/N" "06035U120FAT2A"
 			(at 88.9 34.29 0)
@@
 			)
 		)
-		(property "Mouser Part Number" "80-C0805C104M5R"
-			(at 33.02 35.56 0)
-			(effects
-				(font
-					(size 1.27 1.27)
-				)
-				(hide yes)
-			)
-		)
 		(property "P/N" "MLASH168SB7104KTNA01"
 			(at 33.02 35.56 0)
@@
 			)
 		)
-		(property "Mouser Part Number" "815-ABM3-8-D2Y-T"
-			(at 96.52 39.37 0)
-			(effects
-				(font
-					(size 1.27 1.27)
-				)
-				(hide yes)
-			)
-		)
 		(pin "1"
 		)
@@
 			)
 		)
-		(property "Mouser Part Number" "704-MFBW1V2012-121-R"
-			(at 139.065 113.03 0)
-			(effects
-				(font
-					(size 1.27 1.27)
-				)
-				(hide yes)
-			)
-		)
 		(property "P/N" "BLM18PG121SH1D"
 			(at 139.065 113.03 0)
@@
 			)
 		)
-		(property "Mouser Part Number" "80-C0805C120K5HACTU"
-			(at 88.9 44.45 0)
-			(effects
-				(font
-					(size 1.27 1.27)
-				)
-				(hide yes)
-			)
-		)
 		(property "P/N" "06035U120FAT2A"
 			(at 88.9 44.45 0)
@@
 			)
 		)
-		(property "Mouser Part Number" "71-CRCW080510K0FKEAC"
-			(at 33.02 93.98 0)
-			(effects
-				(font
-					(size 1.27 1.27)
-				)
-				(hide yes)
-			)
-		)
 		(property "P/N" "CRCW060310K0FKEI "
 			(at 33.02 93.98 0)
@@
 			)
 		)
-		(property "Mouser Part Number" "81-GRM219R6YA475KA3D"
-			(at 21.59 35.56 0)
-			(effects
-				(font
-					(size 1.27 1.27)
-				)
-				(hide yes)
-			)
-		)
 		(property "P/N" "08055D475KAT4A"
 			(at 21.59 35.56 0)
@@
 			(at 139.7 66.04 0)
 			(effects
-				(font
-					(size 1.27 1.27)
-				)
-				(hide yes)
-			)
-		)
-		(property "Mouser Part Number" "511-STM32L431CBT6"
-			(at 139.7 66.04 0)
-			(effects

Commit message: place mcu/usb-uart
Parts:
- J1: footprint 0022232041:CONN_A-6373-04A_MOL -> Connector_Molex:Molex_Nano-Fit_105309-xx04_1x04_P2.50mm_Vertical; P/N 0022232041 -> 1053091104
Changed lines of the file:
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@@
 			)
 		)
-		(property "Footprint" "0022232041:CONN_A-6373-04A_MOL"
+		(property "Footprint" "Connector_Molex:Molex_Nano-Fit_105309-xx04_1x04_P2.50mm_Vertical"
 			(at 68.58 91.44 0)
 			(effects
@@
 			)
 		)
-		(property "Datasheet" "https://www.molex.com/en-us/products/part-detail/22232041?display=pdf"
+		(property "Datasheet" "https://www.literature.molex.com/SQLImages/kelmscott/Molex/PDF_Images/987651-1223.PDF"
 			(at 68.58 91.44 0)
 			(effects
@@
 			)
 		)
-		(property "P/N" "0022232041"
+		(property "P/N" "1053091104"
 			(at 68.58 91.44 0)
 			(effects

Commit message: can't
Parts:
- SW1: footprint Button_Switch_SMD:SW_SPST_B3SL-1002P -> TL3365AF180QG:SW_TL3365AF180QG; P/N B3SL-1002P -> TL3365AF180QG
Changed lines of the file:
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@@
 			)
 		)
-		(property "Footprint" "Button_Switch_SMD:SW_SPST_B3SL-1002P"
+		(property "Footprint" "TL3365AF180QG:SW_TL3365AF180QG"
 			(at 38.1 105.41 0)
 			(effects
@@
 			)
 		)
-		(property "Datasheet" "https://omronfs.omron.com/en_US/ecb/products/pdf/en-b3sl.pdf"
+		(property "Datasheet" "https://configured-product-images.s3.amazonaws.com/Datasheets/TL3365.pdf"
 			(at 38.1 105.41 0)
 			(effects
@@
 			)
 		)
-		(property "P/N" "B3SL-1002P"
+		(property "P/N" "TL3365AF180QG"
 			(at 33.02 105.41 90)
 			(effects
