File: PeripheralSOM.kicad_pcb (KiCad board)
At the start: 4 copper layers, 0 parts

Commit message: add some footprints
Parts:
- added CR1: D5V0P4UR6SO-7, UTSVT_ICs:D5V0P4UR6SO-7, F.Cu at (173.8, 121.8)
- added CR2: D5V0P4UR6SO-7, UTSVT_ICs:D5V0P4UR6SO-7, F.Cu at (173.8, 126.6)
- added D6: SP0503BAHTG, Package_TO_SOT_SMD:SOT-143, F.Cu at (183.1, 92.1)
- added J4: 52465-2470, UTSVT_Connectors:524652470, F.Cu at (139.0, 112.5)
- added JP1: CAN TERM, Connector_PinHeader_2.54mm:PinHeader_1x02_P2.54mm_Vertical, F.Cu at (183.3, 102.8)
- added LOGO1: Dr. Hallock, UTSVT_Logos:Hallock_Image_Small, F.Cu at (141.6, 95.5)
- added LOGO2: LHRs, UTSVT_Logos:LHRs_LOGO, F.Cu at (163.1, 95.5)
- added MH1: M3, MountingHole:MountingHole_3.2mm_M3_Pad_TopBottom, F.Cu at (127.7, 87.4)
- added MH2: M3, MountingHole:MountingHole_3.2mm_M3_Pad_TopBottom, F.Cu at (127.7, 95.4)
- added MH3: M3, MountingHole:MountingHole_3.2mm_M3_Pad_TopBottom, F.Cu at (127.7, 103.3)
- added MH4: M3, MountingHole:MountingHole_3.2mm_M3_Pad_TopBottom, F.Cu at (127.7, 111.3)
- added R1: 10k, Resistor_SMD:R_0603_1608Metric_Pad0.98x0.95mm_HandSolder, F.Cu at (125.9, 120.7)
- added R10: 0, Resistor_SMD:R_0603_1608Metric_Pad0.98x0.95mm_HandSolder, F.Cu at (178.8, 84.7)
- added R11: 120, Resistor_SMD:R_0603_1608Metric_Pad0.98x0.95mm_HandSolder, F.Cu at (180.6, 123.2)
- added R12: 45.3k, Resistor_SMD:R_0603_1608Metric_Pad0.98x0.95mm_HandSolder, F.Cu at (125.9, 123.2)
- added R13: 590, Resistor_SMD:R_0603_1608Metric_Pad0.98x0.95mm_HandSolder, F.Cu at (125.9, 125.7)
- added R14: 5.1k, Resistor_SMD:R_0603_1608Metric_Pad0.98x0.95mm_HandSolder, F.Cu at (178.8, 87.2)
- added R15: 2.1k, Resistor_SMD:R_0603_1608Metric_Pad0.98x0.95mm_HandSolder, F.Cu at (125.9, 128.2)
- added R16: 5.1k, Resistor_SMD:R_0603_1608Metric_Pad0.98x0.95mm_HandSolder, F.Cu at (178.8, 89.7)
- added R17: 120, Resistor_SMD:R_0603_1608Metric_Pad0.98x0.95mm_HandSolder, F.Cu at (180.6, 125.7)
- added R18: 120, Resistor_SMD:R_0603_1608Metric_Pad0.98x0.95mm_HandSolder, F.Cu at (180.6, 128.2)
- added R19: 10k, Resistor_SMD:R_0603_1608Metric_Pad0.98x0.95mm_HandSolder, F.Cu at (171.9, 132.1)
- added R20: 402k, Resistor_SMD:R_0603_1608Metric_Pad0.98x0.95mm_HandSolder, F.Cu at (125.9, 130.8)
- added R21: 1k, Resistor_SMD:R_0603_1608Metric_Pad0.98x0.95mm_HandSolder, F.Cu at (178.8, 92.2)
- added R22: 22.1k, Resistor_SMD:R_0603_1608Metric_Pad0.98x0.95mm_HandSolder, F.Cu at (178.8, 94.7)
- added R23: 10k, Resistor_SMD:R_0603_1608Metric_Pad0.98x0.95mm_HandSolder, F.Cu at (125.9, 133.3)
- added R24: 47.5k, Resistor_SMD:R_0603_1608Metric_Pad0.98x0.95mm_HandSolder, F.Cu at (178.8, 97.2)
- added R25: 4.3k, Resistor_SMD:R_0603_1608Metric_Pad0.98x0.95mm_HandSolder, F.Cu at (141.2, 128.2)
- added R26: 120, Resistor_SMD:R_0603_1608Metric_Pad0.98x0.95mm_HandSolder, F.Cu at (141.2, 130.8)
- added R27: 10k, Resistor_SMD:R_0603_1608Metric_Pad0.98x0.95mm_HandSolder, F.Cu at (125.9, 135.8)
- added R28: 4.3k, Resistor_SMD:R_0603_1608Metric_Pad0.98x0.95mm_HandSolder, F.Cu at (141.2, 133.3)
- added R29: 10k, Resistor_SMD:R_0603_1608Metric_Pad0.98x0.95mm_HandSolder, F.Cu at (171.9, 134.6)
- added R3: 16k, Resistor_SMD:R_0603_1608Metric_Pad0.98x0.95mm_HandSolder, F.Cu at (141.2, 120.7)
- added R30: 24m, Resistor_SMD:R_0603_1608Metric_Pad0.98x0.95mm_HandSolder, F.Cu at (125.9, 138.3)
- added R31: 100k, Resistor_SMD:R_0603_1608Metric_Pad0.98x0.95mm_HandSolder, F.Cu at (125.9, 140.8)
- added R4: 10k, Resistor_SMD:R_0603_1608Metric_Pad0.98x0.95mm_HandSolder, F.Cu at (178.8, 101.8)
- added R5: 120, Resistor_SMD:R_0603_1608Metric_Pad0.98x0.95mm_HandSolder, F.Cu at (178.8, 104.3)
- added R6: 120, Resistor_SMD:R_0603_1608Metric_Pad0.98x0.95mm_HandSolder, F.Cu at (180.6, 120.7)
- added R7: 120, Resistor_SMD:R_0603_1608Metric_Pad0.98x0.95mm_HandSolder, F.Cu at (178.8, 106.8)
- added R8: 332, Resistor_SMD:R_0603_1608Metric_Pad0.98x0.95mm_HandSolder, F.Cu at (141.2, 123.2)
- added R9: 10k, Resistor_SMD:R_0603_1608Metric_Pad0.98x0.95mm_HandSolder, F.Cu at (141.2, 125.7)
- added SW1: RST, Button_Switch_SMD:SW_SPST_B3SL-1002P, F.Cu at (164.7, 135.0)
- added TP1: 24V_EXT, TestPoint:TestPoint_Pad_1.0x1.0mm, F.Cu at (144.9, 121.0)
- added TP2: 24V_PROT, TestPoint:TestPoint_Pad_1.0x1.0mm, F.Cu at (144.9, 124.0)
- added TP3: 5V_BUCK, TestPoint:TestPoint_Pad_1.0x1.0mm, F.Cu at (147.9, 121.0)
- added TP4: 5V_USB, TestPoint:TestPoint_Pad_1.0x1.0mm, F.Cu at (147.9, 124.0)
- added TP5: 5V, TestPoint:TestPoint_Pad_1.0x1.0mm, F.Cu at (151.0, 121.0)
- added TP6: 3V3, TestPoint:TestPoint_Pad_1.0x1.0mm, F.Cu at (151.0, 124.0)
- added TP7: GND, TestPoint:TestPoint_Pad_1.0x1.0mm, F.Cu at (154.0, 121.0)
- added TP8: GND, TestPoint:TestPoint_Pad_1.0x1.0mm, F.Cu at (154.0, 124.0)
- added U1: STM32L431CBTx, Package_QFP:LQFP-48_7x7mm_P0.5mm, F.Cu at (165.4, 125.1)
- added U2: TPS5405DR, UTSVT_Power:TPS5405DR, F.Cu at (147.6, 137.2)
- added U3: LT1963AEST-3.3#TRPBF, Package_TO_SOT_SMD:SOT-223-3_TabPin2, F.Cu at (148.3, 129.8)
- added U4: TCAN337, UTSVT_ICs:TCAN337DCNR, F.Cu at (179.2, 110.3)
- added U5: CDSOT23-T24CAN, UTSVT_ICs:CDSOT23-T24CAN, F.Cu at (184.3, 110.5)
- added U6: TPS2115ADRBR, TPS2115ADRBR:SON65P300X300X100-9N, F.Cu at (155.1, 136.2)
- added U7: LM76202QPWPRQ1, UTSVT_Power:LM76202QPWPRQ1, F.Cu at (132.6, 122.9)
- added U8: CP2102N-A02-GQFN24, UTSVT_ICs:CP2102N-A02-GQFN24, F.Cu at (184.1, 86.6)

Commit message: more stuff
Parts:
- added SW2: BOOT, CJS-1200TA:SW_CJS-1200TA, F.Cu at (165.0, 114.1)

Commit message: sch notes
Parts:
- added C1: 1uF, Capacitor_SMD:C_0603_1608Metric_Pad1.08x0.95mm_HandSolder, F.Cu at (236.0, 110.3)
- added C10: 10uF, Capacitor_SMD:C_0805_2012Metric_Pad1.18x1.45mm_HandSolder, F.Cu at (204.2, 103.2)
- added C11: 100nF, Capacitor_SMD:C_0603_1608Metric_Pad1.08x0.95mm_HandSolder, F.Cu at (204.0, 121.4)
- added C12: 100nF, Capacitor_SMD:C_0603_1608Metric_Pad1.08x0.95mm_HandSolder, F.Cu at (204.0, 123.9)
- added C13: 4.7uF, Capacitor_SMD:C_0805_2012Metric_Pad1.18x1.45mm_HandSolder, F.Cu at (220.5, 126.9)
- added C14: 100nF, Capacitor_SMD:C_0603_1608Metric_Pad1.08x0.95mm_HandSolder, F.Cu at (204.0, 126.4)
- added C15: 100nF, Capacitor_SMD:C_0603_1608Metric_Pad1.08x0.95mm_HandSolder, F.Cu at (204.0, 128.9)
- added C16: 100nF, Capacitor_SMD:C_0603_1608Metric_Pad1.08x0.95mm_HandSolder, F.Cu at (204.0, 131.4)
- added C17: 100nF, Capacitor_SMD:C_0603_1608Metric_Pad1.08x0.95mm_HandSolder, F.Cu at (208.4, 118.9)
- added C18: 10uF, Capacitor_SMD:C_0805_2012Metric_Pad1.18x1.45mm_HandSolder, F.Cu at (204.2, 106.3)
- added C19: 1uF, Capacitor_SMD:C_0603_1608Metric_Pad1.08x0.95mm_HandSolder, F.Cu at (229.2, 127.5)
- added C2: 1uF, Capacitor_SMD:C_0603_1608Metric_Pad1.08x0.95mm_HandSolder, F.Cu at (236.0, 112.8)
- added C20: 10uF, Capacitor_SMD:C_0805_2012Metric_Pad1.18x1.45mm_HandSolder, F.Cu at (240.6, 110.5)
- added C21: 12p, Capacitor_SMD:C_0603_1608Metric_Pad1.08x0.95mm_HandSolder, F.Cu at (208.4, 121.4)
- added C22: 12p, Capacitor_SMD:C_0603_1608Metric_Pad1.08x0.95mm_HandSolder, F.Cu at (208.4, 123.9)
- added C23: 10uF, Capacitor_SMD:C_0805_2012Metric_Pad1.18x1.45mm_HandSolder, F.Cu at (240.6, 113.5)
- added C24: 0.1uF, Capacitor_SMD:C_0603_1608Metric_Pad1.08x0.95mm_HandSolder, F.Cu at (229.2, 130.0)
- added C25: 100nF, Capacitor_SMD:C_0603_1608Metric_Pad1.08x0.95mm_HandSolder, F.Cu at (236.0, 115.3)
- added C26: 1uF, Capacitor_SMD:C_0603_1608Metric_Pad1.08x0.95mm_HandSolder, F.Cu at (208.8, 101.5)
- added C27: 0.1uF, Capacitor_SMD:C_0603_1608Metric_Pad1.08x0.95mm_HandSolder, F.Cu at (208.8, 104.0)
- added C28: 0.1uF, Capacitor_SMD:C_0603_1608Metric_Pad1.08x0.95mm_HandSolder, F.Cu at (208.8, 106.5)
- added C29: 10uF, Capacitor_SMD:C_0805_2012Metric_Pad1.18x1.45mm_HandSolder, F.Cu at (240.8, 94.2)
- added C3: 10uF, Capacitor_SMD:C_0805_2012Metric_Pad1.18x1.45mm_HandSolder, F.Cu at (204.2, 94.2)
- added C30: 4.7uF, Capacitor_SMD:C_0805_2012Metric_Pad1.18x1.45mm_HandSolder, F.Cu at (240.8, 97.2)
- added C31: 0.1uF, Capacitor_SMD:C_0603_1608Metric_Pad1.08x0.95mm_HandSolder, F.Cu at (235.0, 103.2)
- added C32: 4.7uF, Capacitor_SMD:C_0805_2012Metric_Pad1.18x1.45mm_HandSolder, F.Cu at (240.8, 100.2)
- added C33: 0.1uF, Capacitor_SMD:C_0603_1608Metric_Pad1.08x0.95mm_HandSolder, F.Cu at (235.0, 105.8)
- added C34: 10uF, Capacitor_SMD:C_0805_2012Metric_Pad1.18x1.45mm_HandSolder, F.Cu at (204.2, 109.3)
- added C35: 10uF, Capacitor_SMD:C_0805_2012Metric_Pad1.18x1.45mm_HandSolder, F.Cu at (204.2, 112.3)
- added C4: 0.1uF, Capacitor_SMD:C_0603_1608Metric_Pad1.08x0.95mm_HandSolder, F.Cu at (208.8, 94.0)
- added C5: 10nF, Capacitor_SMD:C_0603_1608Metric_Pad1.08x0.95mm_HandSolder, F.Cu at (208.8, 96.5)
- added C6: 3.3nF, Capacitor_SMD:C_0603_1608Metric_Pad1.08x0.95mm_HandSolder, F.Cu at (208.8, 99.0)
- added C7: 100nF, Capacitor_SMD:C_0603_1608Metric_Pad1.08x0.95mm_HandSolder, F.Cu at (204.0, 118.9)
- added C8: 10uF, Capacitor_SMD:C_0805_2012Metric_Pad1.18x1.45mm_HandSolder, F.Cu at (204.2, 97.2)
- added C9: 10uF, Capacitor_SMD:C_0805_2012Metric_Pad1.18x1.45mm_HandSolder, F.Cu at (204.2, 100.2)
- added D1: MBR230S1F, Diode_SMD:D_SOD-123F, F.Cu at (218.6, 108.2)
- added D10: TVS, Diode_SMD:D_SOD-923, F.Cu at (235.2, 117.5)
- added D12: LED3, LED_SMD:LED_0805_2012Metric_Pad1.15x1.40mm_HandSolder, F.Cu at (229.5, 113.6)
- added D13: LED2, LED_SMD:LED_0805_2012Metric_Pad1.15x1.40mm_HandSolder, F.Cu at (229.5, 116.6)
- added D14: LED1, LED_SMD:LED_0805_2012Metric_Pad1.15x1.40mm_HandSolder, F.Cu at (229.5, 119.6)
- added D2: TVS, Diode_SMD:D_SOD-323_HandSoldering, F.Cu at (240.8, 116.5)
- added D3: FAULT, LED_SMD:LED_0805_2012Metric_Pad1.15x1.40mm_HandSolder, F.Cu at (229.5, 124.7)
- added D4: Heartbeat, LED_SMD:LED_0805_2012Metric_Pad1.15x1.40mm_HandSolder, F.Cu at (229.5, 110.5)
- added D5: 1N5819HW, Diode_SMD:D_SOD-123, F.Cu at (230.0, 103.7)
- added D7: 24V, LED_SMD:LED_0805_2012Metric_Pad1.15x1.40mm_HandSolder, F.Cu at (213.4, 108.0)
- added D8: 3V3, LED_SMD:LED_0805_2012Metric_Pad1.15x1.40mm_HandSolder, F.Cu at (213.4, 111.0)
- added D9: PG, LED_SMD:LED_0805_2012Metric_Pad1.15x1.40mm_HandSolder, F.Cu at (213.4, 114.1)
- added FB1: FerriteBead, Capacitor_SMD:C_0603_1608Metric_Pad1.08x0.95mm_HandSolder, F.Cu at (208.4, 126.4)
- added FB4: FerriteBead, Capacitor_SMD:C_0603_1608Metric_Pad1.08x0.95mm_HandSolder, F.Cu at (208.4, 128.9)
- added J1: SWD, 0022232041:CONN_A-6373-04A_MOL, F.Cu at (214.8, 121.4)
- added J2: USB4215-03-A, USB4215-03-A:GCT_USB4215-03-A_REVA, F.Cu at (232.7, 99.1)
- added L1: 100uH, Inductor_SMD:L_Coilcraft_MSS1246-XXX, F.Cu at (218.0, 99.7)
- added Y1: 8M, Crystal:Crystal_SMD_Abracon_ABM3-2Pin_5.0x3.2mm, F.Cu at (214.3, 128.0)

Commit message: update usb footprint
Parts:
- J2: footprint USB4215-03-A:GCT_USB4215-03-A_REVA -> Connector_USB:USB_C_Receptacle_GCT_USB4105-xx-A_16P_TopMnt_Horizontal
- moved J2 208.4 mm to (30.2, 50.2)
- moved C29 205.0 mm to (49.7, 20.0)
- moved C30 205.0 mm to (49.7, 23.0)
- moved C31 205.0 mm to (43.9, 29.0)
- moved C32 205.0 mm to (49.7, 26.0)
- moved C33 205.0 mm to (43.9, 31.5)
- moved D5 205.0 mm to (38.8, 29.4)
- moved D3 196.6 mm to (34.1, 102.7)
- moved C19 196.6 mm to (33.9, 105.5)
- moved C24 196.6 mm to (33.9, 108.0)
- moved R10 168.3 mm to (23.4, 20.1)
- moved R14 168.3 mm to (23.4, 22.6)
- moved R16 168.3 mm to (23.4, 25.1)
- moved R21 168.3 mm to (23.4, 27.6)
- moved R22 168.3 mm to (23.4, 30.1)
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
Commit message: CAN layout
Parts:
- JP1: value CAN TERM -> TRM
- R10, R14, R16: moved to B.Cu
- moved R5 33.0 mm to (50.1, 118.0), turned to 180 degrees
- moved R4 32.9 mm to (47.0, 120.2), turned to 180 degrees
- moved R10 30.3 mm to (28.8, 49.9), turned to -90 degrees
- moved R14 30.1 mm to (31.8, 51.5)
- moved U5 28.8 mm to (54.6, 105.4)
- moved C29 27.6 mm to (30.5, 39.8), turned to 180 degrees
- moved R7 27.3 mm to (47.8, 106.4), turned to 180 degrees
- moved C30 26.7 mm to (23.0, 24.2), turned to -90 degrees
- moved R16 25.3 mm to (31.8, 49.0)
- moved JP1 23.0 mm to (47.9, 103.6), turned to 90 degrees
- moved U4 22.9 mm to (43.5, 105.5)
- moved C32 21.0 mm to (28.8, 26.8), turned to -90 degrees
- moved C31 19.5 mm to (25.0, 24.2), turned to -90 degrees
- moved D3 19.4 mm to (46.1, 118.0)
- moved C33 17.8 mm to (26.8, 26.8), turned to -90 degrees
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Connections:
- net Net-(J2-SHIELD) renamed /USB/SH
- net Net-(U8-VBUS) renamed /USB/VBUS
- net Net-(U8-~{RST}) renamed /USB/RST
- D6 pad 2: /USB/D+ -> /USB/D-
- D6 pad 3: /USB/D- -> /USB/D+
Routing:
- net /CAN_H: track 0.00 -> 10.6 mm
- net /CAN_L: track 0.00 -> 9.58 mm
- net /USB/D+: track 0.00 -> 5.65 mm
- net /USB/D-: track 0.00 -> 4.92 mm
- net +3.3V: track 0.00 -> 3.98 mm
- net GND: track 0.00 -> 3.96 mm
- net Net-(JP1-B): track 0.00 -> 3.50 mm

Commit message: more layout
Parts:
- added G***: LOGO, LOGO, F.Cu at (223.5, 104.5)
- added R2: ROSC, Resistor_SMD:R_0603_1608Metric_Pad0.98x0.95mm_HandSolder, F.Cu at (212.2, 117.2)
- C4, D1: moved to B.Cu
- LOGO1: footprint UTSVT_Logos:Hallock_Image_Small -> UTSVT_Logos:Hallock_Image_Tiny
- U6: footprint TPS2115ADRBR:SON65P300X300X100-9N -> Package_SON:VSON-8-1EP_3x3mm_P0.65mm_EP1.65x2.4mm
- moved R3 201.0 mm to (224.5, 113.2), turned to 180 degrees
- moved U2 194.8 mm to (218.8, 114.2)
- moved C35 183.1 mm to (220.3, 94.2), turned to 180 degrees
- moved C8 180.6 mm to (226.8, 96.5)
- moved C34 180.4 mm to (220.3, 96.5), turned to 180 degrees
- moved C6 167.7 mm to (224.5, 115.0)
- moved C9 163.5 mm to (213.8, 112.2), turned to 90 degrees
- moved L1 162.9 mm to (223.5, 104.5), turned to 90 degrees
- moved C4 162.2 mm to (218.8, 110.5)
- moved D1 159.7 mm to (218.0, 108.2), turned to 180 degrees
- moved C3 159.1 mm to (211.5, 112.2), turned to 90 degrees
- moved C5 156.2 mm to (214.0, 117.2), turned to -90 degrees
- moved Y1 129.8 mm to (126.0, 101.8), turned to -90 degrees
- moved R25 127.0 mm to (159.4, 183.9)
- moved R26 127.0 mm to (159.4, 186.4)
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Connections:
- net Net-(U6-ILIM) renamed /PowerDist/ILIM
- net Net-(U6-STAT) renamed /PowerDist/STAT
Routing:
- net +3.3V: track 3.98 -> 12.1 mm
- net /USB/SH: vias 0 -> 1
- added copper zone on F.Cu, net +3.3V
- added copper zone on F.Cu, net +5V
- added copper zone on F.Cu, net +5V_BUCK
- added copper zone on F.Cu, net +5V_VBUS
- added copper zone on F.Cu, net /USB/SH
- added copper zone on F.Cu, net /USB/VBUS_IN

Commit message: buck + mux + ldo
Parts:
- moved C18 183.2 mm to (256.5, 88.0), turned to 90 degrees
- moved U3 176.5 mm to (251.4, 88.0), turned to 90 degrees
- moved C10 170.0 mm to (246.5, 88.0), turned to 90 degrees
- moved R9 114.4 mm to (252.0, 104.2)
- moved R8 110.8 mm to (247.8, 102.8)
- moved C26 105.7 mm to (245.9, 91.0)
- moved C27 105.7 mm to (243.1, 88.2)
- moved C28 105.7 mm to (245.9, 92.8)
- moved U6 105.7 mm to (241.8, 91.9)
- moved LOGO1 95.2 mm to (234.3, 172.8)
- moved LOGO2 95.2 mm to (255.7, 172.8)
- moved R2 38.2 mm to (217.4, 79.4), turned to 180 degrees
- moved C5 36.3 mm to (217.4, 81.2), turned to 180 degrees
- moved C3 35.3 mm to (222.4, 78.7), turned to 0 degrees
- moved C9 32.5 mm to (222.4, 80.9), turned to 0 degrees
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Routing:
- net /PowerDist/ROSC: track 0.00 -> 4.39 mm
- net GND: track 3.96 -> 6.70 mm
- net Net-(U2-BOOT): track 0.00 -> 2.34 mm, vias 0 -> 1
- net Net-(U2-COMP): track 0.00 -> 2.22 mm
- net Net-(U2-SS): track 0.00 -> 2.14 mm
- net Net-(C6-Pad2): track 0.00 -> 1.77 mm
- net Net-(D1-K): vias 0 -> 2
- added copper zone on F.Cu, net +24V
- added copper zone on F.Cu, net GND
- added copper zone on B.Cu, net Net-(D1-K)
- added copper zone on F.Cu, net Net-(D1-K)

Commit message: start adding mcu
Parts:
- C12, C15, FB1, FB4, R8, R9: moved to B.Cu
- moved C29 216.4 mm to (244.0, 95.0)
- moved D5 216.4 mm to (247.8, 97.7)
- moved D6 216.4 mm to (244.2, 98.2)
- moved J2 216.4 mm to (243.7, 105.4)
- moved R10 216.4 mm to (240.3, 104.4)
- moved R14 216.4 mm to (243.3, 105.3)
- moved R16 216.4 mm to (245.5, 105.3)
- moved C22 52.1 mm to (126.9, 146.5), turned to 180 degrees
- moved C21 50.9 mm to (126.9, 142.5), turned to 180 degrees
- moved CR1 49.1 mm to (146.6, 147.6)
- moved C13 48.4 mm to (132.8, 139.0), turned to 135 degrees
- moved C12 44.7 mm to (138.2, 146.2), turned to 90 degrees
- moved U1 43.2 mm to (138.6, 145.0)
- moved Y1 43.0 mm to (130.9, 144.5)
- moved C17 42.7 mm to (144.0, 139.5), turned to 45 degrees
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Connections:
- CR1 pad 1: /MCU/SPI2_MOSI -> /MCU/SPI2_MISO
- CR1 pad 6: /MCU/SPI2_MISO -> /MCU/SPI2_MOSI
Routing:
- net +3.3V: track 12.1 -> 22.6 mm
- net /MCU/OSC_OUT: track 0.00 -> 7.77 mm
- net /MCU/OSC_IN: track 0.00 -> 7.47 mm
- net VDDA: track 0.00 -> 5.93 mm, vias 0 -> 1
- net GNDA: track 0.00 -> 5.75 mm, vias 0 -> 1
- net /MCU/SPI2_MOSI: track 0.00 -> 5.39 mm
- net /PowerDist/STAT: track 0.00 -> 3.57 mm, vias 0 -> 1
- net /MCU/SPI1_MOSI: track 0.00 -> 3.00 mm
- net /MCU/SPI2_NSS: track 0.00 -> 2.81 mm
- net /MCU/SPI1_MISO: track 0.00 -> 2.58 mm
- net /MCU/SPI2_MISO: track 0.00 -> 2.56 mm
- net /PowerDist/ILIM: track 0.00 -> 1.78 mm, vias 0 -> 1
- net +5V: vias 0 -> 1
Other:
- board text added: "24V->5V"
- board text added: "5V->3V3"
- board text added: "USB"
- board text added: "you've voided your warranty"
