File: PeripheralSOM.kicad_pcb (KiCad board)
At the start: 4 copper layers, 114 parts, among them J1 SWD, J2 USB4215-03-A, J4 52465-2470, SW1 RST, SW2 BOOT, U1 STM32L431CBTx, U2 TPS5405DR, U3 LT1963AEST-3.3#TRPBF, U4 TCAN337, U5 CDSOT23-T24CAN, U6 TPS2115ADRBR, U7 LM76202QPWPRQ1, U8 CP2102N-A02-GQFN24, Y1 8M

Commit message: almost all subsheets routed
Parts:
- C11, R19, R29: moved to B.Cu
- moved D12 175.3 mm to (132.2, 182.2)
- moved D13 175.3 mm to (132.2, 185.2)
- moved D14 175.3 mm to (132.2, 188.2)
- moved D4 175.3 mm to (132.2, 179.1)
- moved R11 175.3 mm to (124.5, 183.0)
- moved R17 175.3 mm to (124.5, 185.5)
- moved R18 175.3 mm to (124.5, 188.0)
- moved R6 175.3 mm to (124.5, 180.5)
- moved C30 174.3 mm to (194.7, 112.8)
- moved C31 174.3 mm to (194.7, 110.8)
- moved C32 174.3 mm to (197.2, 107.0)
- moved C33 174.3 mm to (197.2, 109.0)
- moved R21 174.3 mm to (178.4, 104.7)
- moved R22 174.3 mm to (178.4, 107.2)
- moved U8 174.3 mm to (192.4, 107.1)
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Routing:
- net /MCU/NRST: track 0.00 -> 6.69 mm, vias 0 -> 2
- net GND: track 6.70 -> 9.04 mm, vias 0 -> 1
- net Net-(SW2-B): track 0.00 -> 1.59 mm, vias 0 -> 1

Commit message: address some stuff
Parts:
- removed R10: 0, Resistor_SMD:R_0603_1608Metric_Pad0.98x0.95mm_HandSolder
- removed TP5: 5V, TestPoint:TestPoint_Pad_1.0x1.0mm
- added D11: BUCK, LED_SMD:LED_0805_2012Metric_Pad1.15x1.40mm_HandSolder, F.Cu at (130.0, 143.5)
- added R32: 768, Resistor_SMD:R_0603_1608Metric_Pad0.98x0.95mm_HandSolder, F.Cu at (55.8, 188.5)
- C25, C30, C31, C32, C33, C7, J4, U8: moved to B.Cu
- C9: value 10uF -> 1uF; footprint Capacitor_SMD:C_0805_2012Metric_Pad1.18x1.45mm_HandSolder -> Capacitor_SMD:C_0603_1608Metric_Pad1.08x0.95mm_HandSolder
- D10: footprint Diode_SMD:D_SOD-923 -> Diode_SMD:D_SOD-123F
- D9: value PG -> FLT
- moved J4 145.1 mm to (60.9, 114.6), turned to -90 degrees
- moved MH2 108.6 mm to (80.7, 146.9)
- moved R25 100.9 mm to (58.8, 176.2)
- moved R26 100.9 mm to (58.8, 178.7)
- moved R28 100.9 mm to (58.8, 181.2)
- moved MH3 100.5 mm to (89.2, 146.1)
- moved MH4 100.5 mm to (89.2, 154.0)
- moved TP3 95.4 mm to (149.9, 88.1), turned to 180 degrees
- moved TP7 95.1 mm to (36.2, 110.8)
- moved C32 83.8 mm to (115.2, 89.5), turned to -90 degrees
- moved TP1 82.4 mm to (32.8, 124.2)
- moved C33 82.4 mm to (117.2, 89.3), turned to -90 degrees
- moved TP6 81.0 mm to (107.8, 93.5), turned to 180 degrees
- moved U8 80.4 mm to (115.3, 84.4), turned to 180 degrees
- moved C31 78.8 mm to (120.0, 85.8)
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Connections:
- D9 pad 1: GND -> /PowerDist/FAULT
- J2 pad S1: /USB/SH -> GND
- R28 pad 1: /PowerDist/FAULT -> +24V
- TP1 pad 1: 24V_EXT -> +24V_EXT
- TP2 pad 1: 24V -> +24V
- TP3 pad 1: 5V_BUCK -> +5V_BUCK
- TP4 pad 1: 5V_VBUS -> +5V_VBUS
- TP6 pad 1: 3.3V -> +3.3V
Routing:
- net +3.3V: track 22.6 -> 14.9 mm
- net /USB/CC1: track 0.00 -> 6.10 mm, vias 0 -> 1
- net GND: track 9.04 -> 14.5 mm
- net /USB/CC2: track 0.00 -> 5.33 mm, vias 0 -> 1
- net /USB/VBUS: track 0.00 -> 4.73 mm, vias 0 -> 1
- net /USB/RST: track 0.00 -> 2.94 mm, vias 0 -> 1
- net VDDA: track 5.93 -> 7.68 mm
- net GNDA: track 5.75 -> 7.50 mm
- net /USB/SH: vias 1 -> 0
- added copper zone on F.Cu, net +24V_EXT
- added copper zone on B.Cu, net +3.3V
- added copper zone on In1.Cu, net +3.3V
- added copper zone on F.Cu, net /PowerDist/PowerProtection/RTN
- added copper zone on In2.Cu, net GND
- removed copper zone on F.Cu, net /USB/SH
Other:
- board outline added: 52 x 83.2 mm
- board text added: "BLDR"
- board text added: "FLASH"

Commit message: PP
Parts:
- C1, C2, C20, C23, D2, U7: moved to B.Cu
- C25: moved to F.Cu
- moved R1 153.7 mm to (174.6, 91.7)
- moved R31 152.9 mm to (173.8, 111.8)
- moved R20 141.7 mm to (159.2, 91.2), turned to -90 degrees
- moved D10 141.3 mm to (179.0, 111.8)
- moved R30 140.6 mm to (159.2, 102.5), turned to 90 degrees
- moved R15 139.3 mm to (157.5, 91.2), turned to -90 degrees
- moved R23 138.9 mm to (154.0, 87.5), turned to -90 degrees
- moved R27 138.2 mm to (157.5, 102.5), turned to 90 degrees
- moved R13 136.9 mm to (155.8, 91.2), turned to 90 degrees
- moved R12 134.5 mm to (154.0, 91.2), turned to -90 degrees
- moved D2 129.2 mm to (151.6, 87.8), turned to 0 degrees
- moved C20 126.6 mm to (151.8, 90.1), turned to 180 degrees
- moved C1 124.1 mm to (151.8, 92.1), turned to 180 degrees
- moved U7 121.8 mm to (155.0, 97.1), turned to -90 degrees
- moved C2 113.1 mm to (154.0, 104.0), turned to 0 degrees
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Routing:
- net /PowerDist/PowerProtection/SHDN: track 0.00 -> 7.63 mm, vias 0 -> 2
- net /PowerDist/PowerProtection/OVP: track 0.00 -> 5.99 mm, vias 0 -> 2
- net /PowerDist/PowerProtection/MODE: track 0.00 -> 5.80 mm, vias 0 -> 1
- net /PowerDist/PowerProtection/IMON: track 0.00 -> 5.03 mm, vias 0 -> 1
- net /PowerDist/PowerProtection/ILIM: track 0.00 -> 4.03 mm, vias 0 -> 1
- net Net-(U7-DVDT): track 0.00 -> 4.03 mm, vias 0 -> 1
- net /PowerDist/PowerProtection/UVLO: track 0.00 -> 3.73 mm, vias 0 -> 1
- net +24V_EXT: track 0.00 -> 2.14 mm, vias 0 -> 1
- net +3.3V: track 14.9 -> 16.0 mm, vias 0 -> 1
- net GND: track 14.5 -> 15.5 mm, vias 1 -> 2
- net /PowerDist/PowerProtection/RTN: vias 0 -> 5
- net +24V: vias 0 -> 12
- added copper zone on B.Cu, net +24V
- added copper zone on B.Cu, net +24V_EXT
- added copper zone on B.Cu, net /PowerDist/PowerProtection/RTN
- removed copper zone on F.Cu, net +24V_EXT
- removed copper zone on F.Cu, net /PowerDist/PowerProtection/RTN

Commit message: erm hii
Parts:
- C19, C24, JP1, R7, U4, U5: moved to B.Cu
- TP3: value 5V_BUCK -> 5V_BK
- moved MH2 104.7 mm to (159.2, 77.8)
- moved J4 89.2 mm to (142.0, 77.5), turned to 180 degrees
- moved MH4 80.3 mm to (159.2, 114.8)
- moved D13 79.6 mm to (81.5, 78.5)
- moved D8 79.6 mm to (95.0, 80.2)
- moved D11 79.6 mm to (95.0, 72.0)
- moved D14 79.6 mm to (81.5, 81.5)
- moved D4 79.6 mm to (81.5, 72.4)
- moved D9 79.6 mm to (95.0, 83.2)
- moved D12 79.6 mm to (81.5, 75.4)
- moved D7 79.6 mm to (95.0, 77.2)
- moved C11 71.7 mm to (143.1, 59.2)
- moved R29 71.7 mm to (144.9, 59.2)
- moved SW1 71.7 mm to (144.1, 59.2)
- moved R4 67.6 mm to (132.5, 60.1)
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Connections:
- JP1 pad 1: /CAN_H -> Net-(JP1-A)
- JP1 pad 2: Net-(JP1-B) -> /CAN_L
- R7 pad 1: Net-(JP1-B) -> /CAN_H
- R7 pad 2: /CAN_L -> Net-(JP1-A)
Routing:
- net GND: track 15.5 -> 29.2 mm, vias 2 -> 16
- net /CAN_L: track 9.58 -> 15.4 mm
- net /CAN_H: track 10.6 -> 5.75 mm
- net Net-(JP1-B): track 3.50 -> 0.00 mm
- net Net-(JP1-A): track 0.00 -> 3.28 mm
- net +3.3V: track 16.0 -> 14.3 mm
- added copper zone on B.Cu, net GND
Other:
- board size 52 x 83.2 mm -> 52 x 44 mm

Commit message: smaller
Parts:
- JP1: moved to F.Cu
- moved MH3 5.75 mm to (114.2, 109.0)
- moved MH4 5.75 mm to (159.2, 109.0)
- moved C13 3.95 mm to (126.9, 98.8), turned to 180 degrees
- moved C16 3.30 mm to (137.5, 111.2), turned to 0 degrees
- moved C12 3.26 mm to (131.8, 106.9)
- moved C15 3.26 mm to (130.1, 106.9)
- moved C7 3.26 mm to (133.6, 106.9)
- moved CR1 3.26 mm to (140.2, 108.2)
- moved CR2 3.26 mm to (140.2, 104.2)
- moved FB1 3.26 mm to (130.1, 103.4)
- moved FB4 3.26 mm to (135.3, 106.9)
- moved U1 3.26 mm to (132.2, 105.7)
- moved Y1 3.26 mm to (124.5, 105.2)
- moved C21 3.26 mm to (120.5, 103.2)
- moved C22 3.26 mm to (120.5, 107.2)
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Routing:
- net +3.3V: track 14.3 -> 15.1 mm
Other:
- board size 52 x 44 mm -> 52 x 38.2 mm

Commit message: some lakshay fixes
Parts:
- moved J4 46.7 mm to (101.3, 100.4), turned to -90 degrees
- moved J1 43.6 mm to (189.2, 53.4)
- moved C21 1.09 mm to (121.5, 103.5), turned to -90 degrees
- moved C22 1.05 mm to (121.5, 107.0), turned to 90 degrees

Commit message: move pp and som connector
Parts:
- C1, C2, C20, C23, D2, U7: moved to F.Cu
- C25, R12, R13, R15, R20, R23, R27, R30: moved to B.Cu
- moved J1 81.1 mm to (147.2, 122.8), turned to 0 degrees
- moved D3 59.8 mm to (84.3, 22.6)
- moved R4 59.8 mm to (86.6, 21.7)
- moved R5 59.8 mm to (84.3, 18.6)
- moved C19 59.8 mm to (89.0, 57.9)
- moved C24 59.8 mm to (89.0, 56.1)
- moved JP1 59.8 mm to (86.3, 47.7)
- moved R7 59.8 mm to (89.2, 47.7)
- moved U4 59.8 mm to (89.0, 52.9)
- moved U5 59.8 mm to (92.2, 45.7)
- moved J4 58.3 mm to (159.2, 93.4)
- moved R30 32.6 mm to (139.1, 76.8), turned to 0 degrees
- moved C23 30.5 mm to (135.6, 81.8), turned to 90 degrees
- moved R27 30.1 mm to (139.1, 78.6), turned to 0 degrees
- moved C25 27.7 mm to (139.1, 80.3), turned to 0 degrees
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Routing:
- net /CAN_L: track 15.4 -> 0.00 mm
- net GND: track 29.2 -> 21.3 mm, vias 16 -> 18
- net /CAN_H: track 5.75 -> 0.00 mm
- net +3.3V: track 15.1 -> 11.8 mm, vias 1 -> 0
- net Net-(JP1-A): track 3.28 -> 0.00 mm
- net +24V_EXT: track 2.14 -> 0.00 mm, vias 1 -> 6
- net /PowerDist/PowerProtection/RTN: vias 5 -> 0
- net +24V: vias 12 -> 0
- added copper zone on F.Cu, net +24V_EXT
- added copper zone on F.Cu, net /PowerDist/PowerProtection/RTN
- removed copper zone on B.Cu, net +24V
- removed copper zone on B.Cu, net /PowerDist/PowerProtection/RTN
