File: PeripheralSOM.kicad_pcb (KiCad board)
At the start: 4 copper layers, 52 x 38.2 mm, 114 parts, among them J1 SWD, J2 USB4215-03-A, J4 52465-2470, SW1 RST, SW2 BOOT, U1 STM32L431CBTx, U2 TPS5405DR, U3 LT1963AEST-3.3#TRPBF, U4 TCAN337, U5 CDSOT23-T24CAN, U6 TPS2115ADRBR, U7 LM76202QPWPRQ1, U8 CP2102N-A02-GQFN24, Y1 8M

Commit message: new pwr routing
Routing:
- net +24V: vias 0 -> 13
- added copper zone on In1.Cu, net +24V

Commit message: more stuff
Parts:
- moved U5 100.5 mm to (162.5, 117.5)
- moved C24 86.6 mm to (135.5, 129.1), turned to -90 degrees
- moved C19 84.2 mm to (133.8, 129.1), turned to -90 degrees
- moved U4 82.1 mm to (134.5, 121.2), turned to 0 degrees
- moved R19 74.0 mm to (114.5, 118.5)
- moved SW2 74.0 mm to (115.5, 118.2)
- moved SW1 37.4 mm to (157.2, 94.2)
- moved C11 9.13 mm to (134.0, 59.0)
- moved R29 9.13 mm to (135.8, 59.0)
Routing:
- net /MCU/NRST: track 6.69 -> 0.00 mm
- net GND: track 21.3 -> 18.9 mm, vias 18 -> 26

Commit message: gnd
Parts:
- turned G*** to 0 degrees
Routing:
- net GND: vias 26 -> 27
- net /MCU/NRST: vias 2 -> 0

Commit message: add some lcsc parts
Parts:
- D3: value FAULT -> FLT
- moved SW1 18.6 mm to (174.9, 100.2)

Commit message: more better
Parts:
- moved R11 217.5 mm to (268.1, 162.2)
- moved R17 217.5 mm to (268.1, 164.7)
- moved R18 217.5 mm to (268.1, 167.2)
- moved R25 217.5 mm to (275.8, 162.2)
- moved R26 217.5 mm to (275.8, 164.7)
- moved R28 217.5 mm to (275.8, 167.2)
- moved R32 217.5 mm to (272.8, 174.5)
- moved R6 217.5 mm to (268.1, 159.7)
- moved TP1 213.5 mm to (246.2, 125.8)
- moved TP7 213.5 mm to (249.8, 112.2)
- moved D11 195.8 mm to (278.7, 139.8)
- moved D12 195.8 mm to (265.2, 143.2)
- moved D13 195.8 mm to (265.2, 146.2)
- moved D14 195.8 mm to (265.2, 149.2)
- moved D4 195.8 mm to (265.2, 140.1)
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Routing:
- net +5V_BUCK: track 0.00 -> 18.9 mm, vias 0 -> 2
- net +5V_VBUS: track 0.00 -> 15.3 mm, vias 0 -> 2
- net GND: track 18.9 -> 22.0 mm, vias 27 -> 56
- net /PowerDist/ROSC: track 4.39 -> 4.97 mm
- net +3.3V: vias 0 -> 4
- net +5V: vias 1 -> 0
- net +24V: vias 13 -> 0
- removed copper zone on In1.Cu, net +24V
Other:
- board size 52 x 38.2 mm -> 53.5 x 37.8 mm

Commit message: place mcu/usb-uart
Parts:
- J1: footprint 0022232041:CONN_A-6373-04A_MOL -> Connector_Molex:Molex_Nano-Fit_105309-xx04_1x04_P2.50mm_Vertical
- R21, R22, R24: moved to B.Cu
- moved C12 142.5 mm to (143.7, 97.8)
- moved C13 142.5 mm to (138.7, 89.6)
- moved C14 142.5 mm to (138.8, 91.6)
- moved C15 142.5 mm to (141.9, 97.8)
- moved C16 142.5 mm to (149.3, 102.0)
- moved C17 142.5 mm to (149.4, 91.6)
- moved C21 142.5 mm to (133.3, 94.3)
- moved C22 142.5 mm to (133.3, 97.8)
- moved C7 142.5 mm to (145.4, 97.8)
- moved CR1 142.5 mm to (151.9, 99.0)
- moved CR2 142.5 mm to (151.9, 95.0)
- moved FB1 142.5 mm to (141.9, 94.2)
- moved FB4 142.5 mm to (147.2, 97.8)
- moved U1 142.5 mm to (144.0, 96.5)
- moved Y1 142.5 mm to (136.3, 96.0)
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Routing:
- net GND: track 22.0 -> 12.2 mm, vias 56 -> 54
- net /USB/RST: track 2.94 -> 9.55 mm, vias 1 -> 0
- net /USB/VBUS: track 4.73 -> 7.43 mm, vias 1 -> 0
- net +3.3V: track 11.8 -> 14.0 mm
Other:
- board text added: "label pins!"
